File: atmega module/shm.brd (EAGLE design)
At the start: 53.3 x 51.7 mm, 14 parts, among them IC1 MEGA8-P

Commit message: modify
Parts:
- C1, C2: value (none) -> 22pF
- LED1, SV1, SV2, SV3, SV4: value (none) -> 5v
- Q1: value (none) -> 20Mhz
- R1: value (none) -> 1K
- R2: value (none) -> 330
Connections:
- removed net AVCC: IC1.20
- net GND: now also LED1.K; no longer LED1.A
- net N$22: now also LED1.A; no longer LED1.K
- net VCC: now also IC1.20
Routing:
- net N$13: track 53.1 -> 45.8 mm
- net N$2: track 47.1 -> 41.9 mm
- net VCC: track 37.7 -> 34.0 mm
- net N$1: track 39.8 -> 43.5 mm
- net N$10: track 47.9 -> 50.9 mm
- net N$9: track 42.5 -> 44.8 mm
- net N$14: track 60.0 -> 58.2 mm
- net N$11: vias 0 -> 1

Commit message: smd
Parts:
- C1, C2, C3: device capacitor-wima:C2.5-3 -> SparkFun-Capacitors:0805
- LED1: device led:LED5MM -> SparkFun-Retired:HSMC-C265
- R1, R2: device rcl:0204/7 -> SparkFun-Passives:0805
- moved C3 11.7 mm to (36.8, 5.08)
- moved S1 7.62 mm to (30.5, 5.08)
- moved C2 7.41 mm to (30.5, 29.2)
- moved R1 6.84 mm to (25.8, 19.1)
- moved R2 5.39 mm to (30.5, 19.1), turned to 90 degrees
- moved C1 4.58 mm to (30.5, 24.1), turned to 90 degrees
- moved IC1 4.58 mm to (15.2, 22.9)
- moved Q1 4.58 mm to (25.4, 26.7)
- moved LED1 4.02 mm to (36.8, 24.1)
Connections:
- net GND: now also LED1.C; no longer LED1.K
Routing:
- net VCC: track 34.0 -> 49.9 mm
- net N$13: track 45.8 -> 61.6 mm
- net GND: track 75.2 -> 90.6 mm
- net N$1: track 43.5 -> 32.8 mm
- net N$2: track 41.9 -> 31.7 mm
- net N$9: track 44.8 -> 35.4 mm
- net N$23: track 21.3 -> 13.3 mm
- net N$14: track 58.2 -> 65.9 mm
- net N$5: track 38.7 -> 31.7 mm
- net N$8: track 40.8 -> 36.0 mm
- net N$7: track 40.8 -> 36.0 mm
- net N$6: track 40.8 -> 36.0 mm
- net N$20: track 5.08 -> 9.94 mm
- net N$19: track 5.08 -> 9.94 mm
- net N$18: track 5.08 -> 9.94 mm
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
Commit message: smd2
Parts:
- LED1: device SparkFun-Retired:HSMC-C265 -> led:CHIPLED_0805
- Q1: device crystal:HC49/S -> crystal:SM49
- moved LED1 9.25 mm to (39.4, 33.0), turned to 0 degrees
- moved R2 7.18 mm to (25.4, 14.0), turned to 270 degrees
- moved C1 6.84 mm to (33.0, 30.5), turned to 270 degrees
- moved C2 6.84 mm to (33.0, 35.6)
- moved Q1 5.24 mm to (26.7, 31.8)
- moved S1 1.80 mm to (29.2, 6.35)
- moved C3 1.27 mm to (36.8, 6.35)
Routing:
- net N$22: track 8.68 -> 50.2 mm
- net GND: track 90.6 -> 99.0 mm
- net N$23: track 13.3 -> 17.8 mm
- net N$21: track 20.5 -> 16.9 mm
- net N$24: track 35.7 -> 38.0 mm
- net VCC: track 49.9 -> 48.7 mm
