File: atmega module/shm.sch (EAGLE design)
At the start: 12 parts, among them IC1 MEGA8-P

Commit message: switch m1
Parts:
- added SW2: 430186043916, Eagle_Wuerth_Elektronik_Switch:430186043916
Changed lines of the file:
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@@
 <layer number="48" name="Document" color="7" fill="1" visible="no" active="no"/>
 <layer number="49" name="Reference" color="7" fill="1" visible="no" active="no"/>
+<layer number="50" name="dxf" color="7" fill="1" visible="no" active="no"/>
 <layer number="51" name="tDocu" color="7" fill="1" visible="no" active="no"/>
 <layer number="52" name="bDocu" color="7" fill="1" visible="no" active="no"/>
@@
 <layer number="97" name="Info" color="7" fill="1" visible="yes" active="yes"/>
 <layer number="98" name="Guide" color="6" fill="1" visible="yes" active="yes"/>
+<layer number="250" name="Descript" color="7" fill="1" visible="yes" active="yes"/>
+<layer number="251" name="SMDround" color="7" fill="1" visible="yes" active="yes"/>
 </layers>
 <schematic xreflabel="%F%N/%S.%C%R" xrefpart="/%S.%C%R">
@@
 <part name="SW1" library="special" deviceset="SW_DIP-1" device=""/>
 <part name="R2" library="rcl" deviceset="R-EU_" device="0204/7"/>
+<part name="SW2" library="Eagle_Wuerth_Elektronik_Switch" deviceset="430186043916" device=""/>
 </parts>
 <sheets>
@@
 <instance part="SW1" gate="G$1" x="53.34" y="76.2"/>
 <instance part="R2" gate="G$1" x="48.26" y="66.04" rot="R90"/>
+<instance part="SW2" gate="G$1" x="68.58" y="101.6"/>
 </instances>
 <busses>

Commit message: TACK
Parts:
- removed SW1: (no value), special:SW_DIP-1
- removed SW2: 430186043916, Eagle_Wuerth_Elektronik_Switch:430186043916
- added C3: 10nF, capacitor-wima:C2,5-3
- added LOGO1: OSHW-LOGOL, SparkFun-Aesthetics:OSHW-LOGOL
- added S1: SWITCH-MOMENTARY-2PTH, SparkFun-Electromechanical:SWITCH-MOMENTARY-2PTH
Connections:
- net GND: now also C3.1, S1.2; no longer SW1.1
- net N$24: now also C3.2, S1.1
- net VCC: no longer SW1.2
Other:
- moved on the sheet: LED1, R1, R2, SV1

Commit message: modify
Parts:
- C1, C2: value (none) -> 22pF
- LED1, SV1, SV2, SV3, SV4: value (none) -> 5v
- Q1: value (none) -> 20Mhz
- R1: value (none) -> 1K
- R2: value (none) -> 330
Connections:
- net GND: now also LED1.C; no longer LED1.A
- net N$22: now also LED1.A; no longer LED1.C
- net VCC: now also IC1.AVCC
Other:
- moved on the sheet: LED1, R1
Changed lines of the file:
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@@
 </classes>
 <parts>
-<part name="SV1" library="con-lstb" deviceset="MA04-1" device=""/>
-<part name="SV2" library="con-lstb" deviceset="MA06-1" device=""/>
-<part name="SV4" library="con-lstb" deviceset="MA06-1" device=""/>
-<part name="SV3" library="con-lstb" deviceset="MA08-1" device=""/>
+<part name="SV1" library="con-lstb" deviceset="MA04-1" device="" value="5v"/>
+<part name="SV2" library="con-lstb" deviceset="MA06-1" device="" value="5v"/>
+<part name="SV4" library="con-lstb" deviceset="MA06-1" device="" value="5v"/>
+<part name="SV3" library="con-lstb" deviceset="MA08-1" device="" value="5v"/>
 <part name="IC1" library="atmel" deviceset="MEGA8-P" device=""/>
 <part name="GND1" library="supply1" deviceset="GND" device=""/>
-<part name="Q1" library="crystal" deviceset="CRYSTAL" device="HC49S"/>
-<part name="C1" library="capacitor-wima" deviceset="C" device="2,5-3"/>
-<part name="C2" library="capacitor-wima" deviceset="C" device="2,5-3"/>
+<part name="Q1" library="crystal" deviceset="CRYSTAL" device="HC49S" value="20Mhz"/>
+<part name="C1" library="capacitor-wima" deviceset="C" device="2,5-3" value="22pF"/>
+<part name="C2" library="capacitor-wima" deviceset="C" device="2,5-3" value="22pF"/>
 <part name="P+1" library="supply1" deviceset="VCC" device=""/>
-<part name="LED1" library="led" deviceset="LED" device="5MM"/>
-<part name="R1" library="rcl" deviceset="R-EU_" device="0204/7"/>
-<part name="R2" library="rcl" deviceset="R-EU_" device="0204/7"/>
+<part name="LED1" library="led" deviceset="LED" device="5MM" value="5v"/>
+<part name="R1" library="rcl" deviceset="R-EU_" device="0204/7" value="1K"/>
+<part name="R2" library="rcl" deviceset="R-EU_" device="0204/7" value="330"/>
 <part name="C3" library="capacitor-wima" deviceset="C" device="2,5-3" value="10nF"/>
 <part name="LOGO1" library="SparkFun-Aesthetics" deviceset="OSHW-LOGO" device="L"/>
@@
 <instance part="C2" gate="G$1" x="71.12" y="55.88" rot="R90"/>
 <instance part="P+1" gate="VCC" x="55.88" y="35.56" rot="R180"/>
-<instance part="LED1" gate="G$1" x="63.5" y="71.12" rot="R270"/>
-<instance part="R1" gate="G$1" x="48.26" y="66.04" rot="R90"/>
+<instance part="LED1" gate="G$1" x="60.96" y="71.12" rot="R90"/>
+<instance part="R1" gate="G$1" x="45.72" y="66.04" rot="R90"/>
 <instance part="R2" gate="G$1" x="53.34" y="66.04" rot="R90"/>
 <instance part="C3" gate="G$1" x="81.28" y="81.28" rot="R90"/>
@@
 <wire x1="68.58" y1="60.96" x2="68.58" y2="66.04" width="0.1524" layer="91"/>
 <wire x1="68.58" y1="66.04" x2="68.58" y2="71.12" width="0.1524" layer="91"/>
-<wire x1="68.58" y1="71.12" x2="68.58" y2="76.2" width="0.1524" layer="91"/>
 <pinref part="C1" gate="G$1" pin="1"/>
 <pinref part="C2" gate="G$1" pin="1"/>
-<pinref part="LED1" gate="G$1" pin="A"/>
-<wire x1="66.04" y1="71.12" x2="68.58" y2="71.12" width="0.1524" layer="91"/>
-<junction x="68.58" y="71.12"/>
 <junction x="68.58" y="66.04"/>
 <junction x="68.58" y="60.96"/>
@@
 <junction x="55.88" y="50.8"/>
 <pinref part="IC1" gate="G$1" pin="GND"/>
+<wire x1="68.58" y1="71.12" x2="68.58" y2="76.2" width="0.1524" layer="91"/>
 <wire x1="68.58" y1="76.2" x2="78.74" y2="76.2" width="0.1524" layer="91"/>
 <wire x1="78.74" y1="76.2" x2="91.44" y2="76.2" width="0.1524" layer="91"/>
@@
 <junction x="78.74" y="76.2"/>
 <pinref part="S1" gate="G$1" pin="2"/>
+<pinref part="LED1" gate="G$1" pin="C"/>
+<wire x1="66.04" y1="71.12" x2="68.58" y2="71.12" width="0.1524" layer="91"/>
+<junction x="68.58" y="71.12"/>
 </segment>
 </net>
@@
 <pinref part="SV1" gate="1" pin="1"/>
 <pinref part="IC1" gate="G$1" pin="VCC@1"/>
-<wire x1="55.88" y1="45.72" x2="91.44" y2="45.72" width="0.1524" layer="91"/>
+<wire x1="55.88" y1="45.72" x2="88.9" y2="45.72" width="0.1524" layer="91"/>
 <pinref part="P+1" gate="VCC" pin="VCC"/>
+<wire x1="88.9" y1="45.72" x2="91.44" y2="45.72" width="0.1524" layer="91"/>
 <wire x1="55.88" y1="38.1" x2="55.88" y2="40.64" width="0.1524" layer="91"/>
 <wire x1="55.88" y1="40.64" x2="55.88" y2="45.72" width="0.1524" layer="91"/>
 <wire x1="55.88" y1="40.64" x2="43.18" y2="40.64" width="0.1524" layer="91"/>
 <wire x1="43.18" y1="40.64" x2="43.18" y2="60.96" width="0.1524" layer="91"/>
-<wire x1="43.18" y1="60.96" x2="48.26" y2="60.96" width="0.1524" layer="91"/>
+<wire x1="43.18" y1="60.96" x2="45.72" y2="60.96" width="0.1524" layer="91"/>
 <pinref part="SV1" gate="1" pin="4"/>
-<wire x1="48.26" y1="60.96" x2="53.34" y2="60.96" width="0.1524" layer="91"/>
+<wire x1="45.72" y1="60.96" x2="53.34" y2="60.96" width="0.1524" layer="91"/>
 <wire x1="53.34" y1="60.96" x2="55.88" y2="60.96" width="0.1524" layer="91"/>
 <wire x1="55.88" y1="60.96" x2="55.88" y2="53.34" width="0.1524" layer="91"/>
@@
 <pinref part="R2" gate="G$1" pin="1"/>
 <junction x="53.34" y="60.96"/>
-<junction x="48.26" y="60.96"/>
+<junction x="45.72" y="60.96"/>
 <junction x="55.88" y="40.64"/>
 <junction x="55.88" y="45.72"/>
-</segment>
-</net>
-<net name="N$22" class="0">
-<segment>
-<pinref part="R2" gate="G$1" pin="2"/>
-<pinref part="LED1" gate="G$1" pin="C"/>
-<wire x1="53.34" y1="71.12" x2="58.42" y2="71.12" width="0.1524" layer="91"/>
+<wire x1="88.9" y1="45.72" x2="88.9" y2="71.12" width="0.1524" layer="91"/>
+<pinref part="IC1" gate="G$1" pin="AVCC"/>
+<wire x1="88.9" y1="71.12" x2="91.44" y2="71.12" width="0.1524" layer="91"/>
+<junction x="88.9" y="45.72"/>
 </segment>
 </net>
@@
 <segment>
 <pinref part="R1" gate="G$1" pin="2"/>
-<wire x1="48.26" y1="71.12" x2="48.26" y2="81.28" width="0.1524" layer="91"/>
-<wire x1="48.26" y1="81.28" x2="48.26" y2="91.44" width="0.1524" layer="91"/>
-<wire x1="48.26" y1="91.44" x2="86.36" y2="91.44" width="0.1524" layer="91"/>
+<wire x1="45.72" y1="71.12" x2="45.72" y2="81.28" width="0.1524" layer="91"/>
+<wire x1="45.72" y1="81.28" x2="45.72" y2="91.44" width="0.1524" layer="91"/>
+<wire x1="45.72" y1="91.44" x2="86.36" y2="91.44" width="0.1524" layer="91"/>
 <pinref part="IC1" gate="G$1" pin="PC6(/RESET)"/>
 <wire x1="91.44" y1="81.28" x2="86.36" y2="81.28" width="0.1524" layer="91"/>
@@
 <pinref part="C3" gate="G$1" pin="2"/>
 <junction x="86.36" y="81.28"/>
-<junction x="48.26" y="81.28"/>
-<wire x1="50.8" y1="81.28" x2="48.26" y2="81.28" width="0.1524" layer="91"/>
+<junction x="45.72" y="81.28"/>
+<wire x1="50.8" y1="81.28" x2="45.72" y2="81.28" width="0.1524" layer="91"/>
 <pinref part="S1" gate="G$1" pin="1"/>
 </segment>
 </net>
+<net name="N$22" class="0">
+<segment>
+<pinref part="LED1" gate="G$1" pin="A"/>
+<pinref part="R2" gate="G$1" pin="2"/>
+<wire x1="58.42" y1="71.12" x2="53.34" y2="71.12" width="0.1524" layer="91"/>
+</segment>
+</net>

Commit message: smd
Parts:
- C1, C2, C3: device capacitor-wima:C2,5-3 -> SparkFun-Capacitors:CAP0805
- LED1: device led:LED5MM -> SparkFun-Retired:HSMC-C265
- R1, R2: device rcl:R-EU_0204/7 -> SparkFun-Passives:RESISTOR0805-RES
Other:
- moved on the sheet: C1, C2, C3
Changed lines of the file:
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@@
 <part name="GND1" library="supply1" deviceset="GND" device=""/>
 <part name="Q1" library="crystal" deviceset="CRYSTAL" device="HC49S" value="20Mhz"/>
-<part name="C1" library="capacitor-wima" deviceset="C" device="2,5-3" value="22pF"/>
-<part name="C2" library="capacitor-wima" deviceset="C" device="2,5-3" value="22pF"/>
+<part name="C1" library="SparkFun-Capacitors" deviceset="CAP" device="0805" value="22pF"/>
+<part name="C2" library="SparkFun-Capacitors" deviceset="CAP" device="0805" value="22pF"/>
 <part name="P+1" library="supply1" deviceset="VCC" device=""/>
-<part name="LED1" library="led" deviceset="LED" device="5MM" value="5v"/>
-<part name="R1" library="rcl" deviceset="R-EU_" device="0204/7" value="1K"/>
-<part name="R2" library="rcl" deviceset="R-EU_" device="0204/7" value="330"/>
-<part name="C3" library="capacitor-wima" deviceset="C" device="2,5-3" value="10nF"/>
+<part name="LED1" library="SparkFun-Retired" deviceset="HSMC-C265" device="" value="5v"/>
+<part name="R1" library="SparkFun-Passives" deviceset="RESISTOR" device="0805-RES" value="1K"/>
+<part name="R2" library="SparkFun-Passives" deviceset="RESISTOR" device="0805-RES" value="330"/>
+<part name="C3" library="SparkFun-Capacitors" deviceset="CAP" device="0805" value="10nF"/>
 <part name="LOGO1" library="SparkFun-Aesthetics" deviceset="OSHW-LOGO" device="L"/>
 <part name="S1" library="SparkFun-Electromechanical" deviceset="SWITCH-MOMENTARY-2" device="PTH"/>
@@
 <pinref part="GND1" gate="1" pin="GND"/>
 <wire x1="66.04" y1="60.96" x2="68.58" y2="60.96" width="0.1524" layer="91"/>
-<wire x1="68.58" y1="60.96" x2="68.58" y2="55.88" width="0.1524" layer="91"/>
-<wire x1="68.58" y1="55.88" x2="68.58" y2="50.8" width="0.1524" layer="91"/>
-<wire x1="68.58" y1="60.96" x2="68.58" y2="66.04" width="0.1524" layer="91"/>
-<wire x1="68.58" y1="66.04" x2="68.58" y2="71.12" width="0.1524" layer="91"/>
+<wire x1="68.58" y1="60.96" x2="66.04" y2="55.88" width="0.1524" layer="91"/>
+<wire x1="66.04" y1="55.88" x2="68.58" y2="50.8" width="0.1524" layer="91"/>
+<wire x1="68.58" y1="60.96" x2="66.04" y2="66.04" width="0.1524" layer="91"/>
+<wire x1="66.04" y1="66.04" x2="68.58" y2="71.12" width="0.1524" layer="91"/>
 <pinref part="C1" gate="G$1" pin="1"/>
 <pinref part="C2" gate="G$1" pin="1"/>
-<junction x="68.58" y="66.04"/>
+<junction x="66.04" y="66.04"/>
 <junction x="68.58" y="60.96"/>
-<junction x="68.58" y="55.88"/>
+<junction x="66.04" y="55.88"/>
 <junction x="68.58" y="50.8"/>
 <junction x="55.88" y="50.8"/>
@@
 <wire x1="68.58" y1="76.2" x2="78.74" y2="76.2" width="0.1524" layer="91"/>
 <wire x1="78.74" y1="76.2" x2="91.44" y2="76.2" width="0.1524" layer="91"/>
-<wire x1="60.96" y1="81.28" x2="78.74" y2="81.28" width="0.1524" layer="91"/>
+<wire x1="60.96" y1="81.28" x2="76.2" y2="81.28" width="0.1524" layer="91"/>
 <pinref part="C3" gate="G$1" pin="1"/>
-<wire x1="78.74" y1="81.28" x2="78.74" y2="76.2" width="0.1524" layer="91"/>
-<junction x="78.74" y="81.28"/>
+<wire x1="76.2" y1="81.28" x2="78.74" y2="76.2" width="0.1524" layer="91"/>
+<junction x="76.2" y="81.28"/>
 <junction x="78.74" y="76.2"/>
 <pinref part="S1" gate="G$1" pin="2"/>
@@
 <pinref part="C1" gate="G$1" pin="2"/>
 <wire x1="83.82" y1="63.5" x2="76.2" y2="63.5" width="0.1524" layer="91"/>
-<wire x1="76.2" y1="63.5" x2="76.2" y2="66.04" width="0.1524" layer="91"/>
+<wire x1="76.2" y1="63.5" x2="73.66" y2="66.04" width="0.1524" layer="91"/>
 <junction x="83.82" y="63.5"/>
 </segment>
@@
 <pinref part="C2" gate="G$1" pin="2"/>
 <wire x1="83.82" y1="58.42" x2="76.2" y2="58.42" width="0.1524" layer="91"/>
-<wire x1="76.2" y1="58.42" x2="76.2" y2="55.88" width="0.1524" layer="91"/>
+<wire x1="76.2" y1="58.42" x2="73.66" y2="55.88" width="0.1524" layer="91"/>
 <junction x="83.82" y="58.42"/>
 </segment>
@@
 <wire x1="45.72" y1="91.44" x2="86.36" y2="91.44" width="0.1524" layer="91"/>
 <pinref part="IC1" gate="G$1" pin="PC6(/RESET)"/>
-<wire x1="91.44" y1="81.28" x2="86.36" y2="81.28" width="0.1524" layer="91"/>
-<wire x1="86.36" y1="81.28" x2="86.36" y2="91.44" width="0.1524" layer="91"/>
+<wire x1="91.44" y1="81.28" x2="83.82" y2="81.28" width="0.1524" layer="91"/>
+<wire x1="83.82" y1="81.28" x2="86.36" y2="91.44" width="0.1524" layer="91"/>
 <pinref part="C3" gate="G$1" pin="2"/>
-<junction x="86.36" y="81.28"/>
+<junction x="83.82" y="81.28"/>
 <junction x="45.72" y="81.28"/>
 <wire x1="50.8" y1="81.28" x2="45.72" y2="81.28" width="0.1524" layer="91"/>

Commit message: smd2
Parts:
- LED1: device SparkFun-Retired:HSMC-C265 -> led:LEDCHIPLED_0805
- Q1: device crystal:CRYSTALHC49S -> crystal:CRYSTALSM49
Changed lines of the file:
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@@
 <part name="IC1" library="atmel" deviceset="MEGA8-P" device=""/>
 <part name="GND1" library="supply1" deviceset="GND" device=""/>
-<part name="Q1" library="crystal" deviceset="CRYSTAL" device="HC49S" value="20Mhz"/>
+<part name="Q1" library="crystal" deviceset="CRYSTAL" device="SM49" value="20Mhz"/>
 <part name="C1" library="SparkFun-Capacitors" deviceset="CAP" device="0805" value="22pF"/>
 <part name="C2" library="SparkFun-Capacitors" deviceset="CAP" device="0805" value="22pF"/>
 <part name="P+1" library="supply1" deviceset="VCC" device=""/>
-<part name="LED1" library="SparkFun-Retired" deviceset="HSMC-C265" device="" value="5v"/>
+<part name="LED1" library="led" deviceset="LED" device="CHIPLED_0805" value="5v"/>
 <part name="R1" library="SparkFun-Passives" deviceset="RESISTOR" device="0805-RES" value="1K"/>
 <part name="R2" library="SparkFun-Passives" deviceset="RESISTOR" device="0805-RES" value="330"/>
