File: ARMED BASE/armedbase.brd (EAGLE design)
At the start: 160 x 100 mm, 14 parts, among them K1 CQ1-12V, X1 RJ45-6L2-B, X2 RJ45-6L2-B

Commit message: armed base
Parts:
- added J2, J3, J4, J5: (no value), con-amp:1X2MTA
- added LOGO2: OSHW-LOGOL, SparkFun-Aesthetics:OSHW-LOGO-L
- added OK1: SFH618A-2, optocoupler:DIP4
- added OK2: H11L1M, optocoupler:DIL06
Connections:
- new net GND: OK2.5
- new net VCC: OK2.6
Changed lines of the file:
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@@
 <wire x1="160" y1="100" x2="0" y2="100" width="0" layer="20"/>
 <wire x1="0" y1="100" x2="0" y2="0" width="0" layer="20"/>
+<dimension x1="0" y1="0" x2="160.02" y2="0" x3="80.01" y3="-20.32" textsize="1.778" layer="16"/>
+<dimension x1="0" y1="0" x2="0" y2="100.33" x3="-13.97" y3="50.165" textsize="1.778" layer="16"/>
 </plain>
 <attributes>
@@
 </element>
 <element name="D1" library="diode" package="DO41-10" value="1N4004" x="124.46" y="15.24"/>
+<element name="J2" library="con-amp" package="1X2MTA" value="" x="152.4" y="87.63" rot="R270"/>
+<element name="J3" library="con-amp" package="1X2MTA" value="" x="152.4" y="76.2" rot="R270"/>
+<element name="J4" library="con-amp" package="1X2MTA" value="" x="152.4" y="64.77" rot="R270"/>
+<element name="J5" library="con-amp" package="1X2MTA" value="" x="152.4" y="53.34" rot="R270"/>
+<element name="LOGO2" library="SparkFun-Aesthetics" package="OSHW-LOGO-L" value="OSHW-LOGOL" x="85.09" y="93.98"/>
+<element name="OK1" library="optocoupler" package="DIP4" value="SFH618A-2" x="86.36" y="66.04">
+<attribute name="OC_NEWARK" value="21H7744" x="86.36" y="66.04" size="1.778" layer="27" display="off"/>
+<attribute name="MPN" value="SFH618A-2" x="86.36" y="66.04" size="1.778" layer="27" display="off"/>
+<attribute name="MF" value="VISHAY/TELEFUNKEN" x="86.36" y="66.04" size="1.778" layer="27" display="off"/>
+<attribute name="OC_FARNELL" value="6424855" x="86.36" y="66.04" size="1.778" layer="27" display="off"/>
+</element>
+<element name="OK2" library="optocoupler" package="DIL06" value="H11L1M" x="99.06" y="66.04">
+<attribute name="OC_NEWARK" value="72K8643" x="99.06" y="66.04" size="1.778" layer="27" display="off"/>
+<attribute name="MPN" value="H11L1-M" x="99.06" y="66.04" size="1.778" layer="27" display="off"/>
+<attribute name="MF" value="FAIRCHILD SEMICONDUCTOR" x="99.06" y="66.04" size="1.778" layer="27" display="off"/>
+<attribute name="OC_FARNELL" value="1021127" x="99.06" y="66.04" size="1.778" layer="27" display="off"/>
+</element>
 </elements>
 <signals>
+<signal name="VCC">
+<contactref element="OK2" pad="6"/>
+</signal>
+<signal name="GND">
+<contactref element="OK2" pad="5"/>
+</signal>
 </signals>
 </board>

Commit message: smd
Parts:
- R1: device eagle-ltspice:0204/7 -> SparkFun-Passives:0805
Changed lines of the file:
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@@
 <element name="IC1" library="SparkFun-PowerIC" package="78XXL" value="" x="26.67" y="11.43"/>
 <element name="Q1" library="SparkFun-DiscreteSemi" package="TO-92-AMMO" value="" x="133.35" y="27.94"/>
-<element name="R1" library="eagle-ltspice" package="0204/7" value="" x="43.18" y="21.59">
-<attribute name="SPICEMODEL" value="NONE" x="90.17" y="-39.37" size="1.778" layer="27" display="off"/>
-<attribute name="SPICEPREFIX" value="R" x="90.17" y="-39.37" size="1.778" layer="27" display="off"/>
-</element>
+<element name="R1" library="SparkFun-Passives" package="0805" value="" x="43.18" y="21.59"/>
 <element name="C1" library="capacitor-wima" package="C2.5-3" value="" x="41.91" y="13.97"/>
 <element name="LED1" library="led" package="LED5MM" value="" x="6.35" y="22.86"/>

Commit message: smd2
Parts:
- removed OK1: SFH618A-2, optocoupler:DIP4
- removed OK2: H11L1M, optocoupler:DIL06
- removed Q1: (no value), SparkFun-DiscreteSemi:TO-92-AMMO
- added Q2: (no value), semicon-smd-ipc:SOT23
- added X3: 14867, con-4ucon:14867
- C1: device capacitor-wima:C2.5-3 -> SparkFun-Capacitors:0805
- D1: value 1N4004 -> (none); device diode:DO41-10 -> SparkFun-DiscreteSemi:SMA-DIODE
- IC1: value (none) -> REG1117; device SparkFun-PowerIC:78XXL -> burr-brown:SOT223
- LED1: device led:LED5MM -> led:CHIP-LED0805
- moved LED1 93.4 mm to (99.1, 34.3), turned to 90 degrees
- moved IC1 83.0 mm to (99.1, 52.1)
- moved R1 63.5 mm to (104.1, 39.4)
- moved C1 57.9 mm to (94.0, 39.4)
- moved D1 41.9 mm to (125.7, 57.1)
- moved LOGO2 11.4 mm to (73.7, 94.0)
Connections:
- removed net VCC: OK2.6
- net GND: now also IC1.1; no longer OK2.5
Changed lines of the file:
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@@
 <attribute name="OC_FARNELL" value="unknown" x="1.27" y="66.04" size="1.778" layer="27" rot="R270" display="off"/>
 </element>
-<element name="IC1" library="SparkFun-PowerIC" package="78XXL" value="" x="26.67" y="11.43"/>
-<element name="Q1" library="SparkFun-DiscreteSemi" package="TO-92-AMMO" value="" x="133.35" y="27.94"/>
-<element name="R1" library="SparkFun-Passives" package="0805" value="" x="43.18" y="21.59"/>
-<element name="C1" library="capacitor-wima" package="C2.5-3" value="" x="41.91" y="13.97"/>
-<element name="LED1" library="led" package="LED5MM" value="" x="6.35" y="22.86"/>
+<element name="IC1" library="burr-brown" package="SOT223" value="REG1117" x="99.06" y="52.07">
+<attribute name="OC_NEWARK" value="14P6981" x="99.06" y="52.07" size="1.778" layer="27" display="off"/>
+<attribute name="MPN" value="REG1117" x="99.06" y="52.07" size="1.778" layer="27" display="off"/>
+<attribute name="MF" value="" x="99.06" y="52.07" size="1.778" layer="27" display="off"/>
+<attribute name="OC_FARNELL" value="1097566" x="99.06" y="52.07" size="1.778" layer="27" display="off"/>
+</element>
+<element name="R1" library="SparkFun-Passives" package="0805" value="" x="104.14" y="39.37"/>
+<element name="C1" library="SparkFun-Capacitors" package="0805" value="" x="93.98" y="39.37"/>
+<element name="LED1" library="led" package="CHIP-LED0805" value="" x="99.06" y="34.29" rot="R90"/>
 <element name="K1" library="relay" package="CQ1" value="CQ1-12V" x="147.32" y="11.43">
 <attribute name="OC_NEWARK" value="unknown" x="180.34" y="-17.78" size="1.778" layer="27" display="off"/>
@@
 <attribute name="OC_FARNELL" value="unknown" x="180.34" y="-17.78" size="1.778" layer="27" display="off"/>
 </element>
-<element name="D1" library="diode" package="DO41-10" value="1N4004" x="124.46" y="15.24"/>
+<element name="D1" library="SparkFun-DiscreteSemi" package="SMA-DIODE" value="" x="125.73" y="57.15"/>
 <element name="J2" library="con-amp" package="1X2MTA" value="" x="152.4" y="87.63" rot="R270"/>
 <element name="J3" library="con-amp" package="1X2MTA" value="" x="152.4" y="76.2" rot="R270"/>
 <element name="J4" library="con-amp" package="1X2MTA" value="" x="152.4" y="64.77" rot="R270"/>
 <element name="J5" library="con-amp" package="1X2MTA" value="" x="152.4" y="53.34" rot="R270"/>
-<element name="LOGO2" library="SparkFun-Aesthetics" package="OSHW-LOGO-L" value="OSHW-LOGOL" x="85.09" y="93.98"/>
-<element name="OK1" library="optocoupler" package="DIP4" value="SFH618A-2" x="86.36" y="66.04">
-<attribute name="OC_NEWARK" value="21H7744" x="86.36" y="66.04" size="1.778" layer="27" display="off"/>
-<attribute name="MPN" value="SFH618A-2" x="86.36" y="66.04" size="1.778" layer="27" display="off"/>
-<attribute name="MF" value="VISHAY/TELEFUNKEN" x="86.36" y="66.04" size="1.778" layer="27" display="off"/>
-<attribute name="OC_FARNELL" value="6424855" x="86.36" y="66.04" size="1.778" layer="27" display="off"/>
-</element>
-<element name="OK2" library="optocoupler" package="DIL06" value="H11L1M" x="99.06" y="66.04">
-<attribute name="OC_NEWARK" value="72K8643" x="99.06" y="66.04" size="1.778" layer="27" display="off"/>
-<attribute name="MPN" value="H11L1-M" x="99.06" y="66.04" size="1.778" layer="27" display="off"/>
-<attribute name="MF" value="FAIRCHILD SEMICONDUCTOR" x="99.06" y="66.04" size="1.778" layer="27" display="off"/>
-<attribute name="OC_FARNELL" value="1021127" x="99.06" y="66.04" size="1.778" layer="27" display="off"/>
+<element name="LOGO2" library="SparkFun-Aesthetics" package="OSHW-LOGO-L" value="OSHW-LOGOL" x="73.66" y="93.98"/>
+<element name="Q2" library="semicon-smd-ipc" package="SOT23" value="" x="149.86" y="38.1"/>
+<element name="X3" library="con-4ucon" package="14867" value="14867" x="86.36" y="87.63" rot="R180">
+<attribute name="OC_NEWARK" value="unknown" x="86.36" y="87.63" size="1.778" layer="27" rot="R180" display="off"/>
+<attribute name="MPN" value="" x="86.36" y="87.63" size="1.778" layer="27" rot="R180" display="off"/>
+<attribute name="MF" value="" x="86.36" y="87.63" size="1.778" layer="27" rot="R180" display="off"/>
+<attribute name="OC_FARNELL" value="unknown" x="86.36" y="87.63" size="1.778" layer="27" rot="R180" display="off"/>
 </element>
 </elements>
 <signals>
-<signal name="VCC">
-<contactref element="OK2" pad="6"/>
-</signal>
 <signal name="GND">
-<contactref element="OK2" pad="5"/>
+<contactref element="IC1" pad="1"/>
 </signal>
 </signals>

Commit message: modbus
Parts:
- added C2: 100uf, SparkFun-Capacitors:0805
- added R2: 10k, SparkFun-Passives:0805
- added R3, R4: 680, SparkFun-Passives:0805
- added R5: 120, SparkFun-Passives:0805
- added R6: 2.2k, SparkFun-Passives:0805
- added R7: 1k, SparkFun-Passives:0805
- added R8: 330, SparkFun-Passives:0805
- added S1: (no value), SparkFun-Electromechanical:SWITCH-SPDT-SMD
- added U$1: MAX485DIL, SparkFun-DigitalIC:DIL08
- C1: value (none) -> 10uf
- R1: value (none) -> 10k
- moved D1 116.0 mm to (10.2, 47.0), turned to 270 degrees
- moved IC1 96.5 mm to (6.35, 25.4), turned to 90 degrees
- moved LED1 80.7 mm to (19.1, 24.1), turned to 180 degrees
- moved C1 80.5 mm to (15.2, 22.9)
- moved Q2 65.1 mm to (88.9, 61.0)
- moved R1 30.6 mm to (83.8, 62.2), turned to 180 degrees
- moved J1 30.5 mm to (7.62, 38.1)
Connections:
- new net N$11: LED1.A, R8.1
- new net N$13: D1.A, S1.1
- new net N$14: C2.2, D1.C, IC1.3
- new net N$2: Q2.3, R1.1, U$1.2, U$1.3
- new net N$4: Q2.1, R6.1, R7.2
- new net N$7: R4.2, R5.1, U$1.7, X3.4
- new net N$8: R3.1, R5.2, U$1.6, X3.1
- new net RX: R2.1, U$1.1
- new net TX: R6.2, U$1.4
- new net VCC: J1.3, S1.2
- new net VCC5V: C1.2, IC1.2, R1.2, R2.2, R3.2, R8.2, U$1.8
- net GND: now also C1.1, C2.1, J1.1, LED1.C, Q2.2, R4.1, R7.1, U$1.5
Routing:
- net GND: track 0.00 -> 152.0 mm
- net VCC5V: track 0.00 -> 125.4 mm, vias 0 -> 1
- net N$8: track 0.00 -> 38.3 mm
- net N$7: track 0.00 -> 31.6 mm
- net N$14: track 0.00 -> 22.8 mm
- net RX: track 0.00 -> 21.5 mm
- net VCC: track 0.00 -> 20.9 mm
- net TX: track 0.00 -> 20.5 mm
- net N$4: track 0.00 -> 15.9 mm
- net N$2: track 0.00 -> 10.7 mm
- net N$13: track 0.00 -> 7.80 mm
- net N$11: track 0.00 -> 3.13 mm

Commit message: last
Parts:
- added D10, D11, D12, D13, D14, D15, D16, D17, D2, D3, D4, D5, D6, D7, D8, D9: (no value), SparkFun-DiscreteSemi:SMA-DIODE
- added R10, R11, R12, R13, R14, R15, R16, R17, R18, R19, R20, R21, R22, R23, R24, R9: 10k, SparkFun-Passives:0805
- moved J3 30.6 mm to (154.9, 45.7)
- moved J5 30.6 mm to (154.9, 22.9)
- moved J2 30.6 mm to (154.9, 57.1)
- moved J4 30.6 mm to (154.9, 34.3)
- moved R1 9.16 mm to (76.2, 67.3)
- moved LOGO2 8.98 mm to (64.8, 95.2)
- moved U$1 8.13 mm to (80.0, 74.9)
- moved X3 8.13 mm to (80.0, 92.7)
- moved K1 8.03 mm to (139.7, 8.89)
- moved R6 7.41 mm to (81.3, 67.3)
- moved R2 6.48 mm to (71.1, 74.9)
- moved X1 6.48 mm to (137.2, 88.9)
- moved R5 6.48 mm to (71.1, 67.3)
- moved R3 6.35 mm to (71.1, 71.1)
- moved Q2 5.68 mm to (86.4, 66.0)
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Connections:
- new net INA1: D2.A, R9.2
- new net INA2: D3.A, R10.2
- new net INA3: D4.A, R11.2
- new net INA4: D5.A, R12.2
- new net INA5: D6.A, R13.2
- new net INA6: D7.A, R14.2
- new net INA7: D8.A, R15.2
- new net INA8: D9.A, R16.2
- new net INB1: D10.A, R17.2
- new net INB2: D11.A, R18.2
- new net INB3: D12.A, R19.2
- new net INB4: D13.A, R20.2
- new net INB5: D14.A, R21.2
- new net INB6: D15.A, R22.2
- new net INB7: D16.A, R23.2
- new net INB8: D17.A, R24.2
- new net N$1: D2.C, X1.1
- new net N$10: D13.C, X2.4
- new net N$12: D14.C, X2.5
- new net N$15: D15.C, X2.6
- new net N$16: D16.C, X2.7
- new net N$17: D17.C, X2.8
- new net N$25: D3.C, X1.2
- new net N$26: D4.C, X1.3
- new net N$27: D5.C, X1.4
- new net N$28: D6.C, X1.5
- new net N$29: D7.C, X1.6
- new net N$3: D10.C, X2.1
- new net N$30: D8.C, X1.7
- new net N$31: D9.C, X1.8
- new net N$6: D11.C, X2.2
- new net N$9: D12.C, X2.3
- net VCC5V: now also R10.1, R11.1, R12.1, R13.1, R14.1, R15.1, R16.1, R17.1, R18.1, R19.1, R20.1, R21.1, R22.1, R23.1, R24.1, R9.1
Routing:
- net VCC5V: track 125.4 -> 213.5 mm, vias 1 -> 0
- net N$15: track 0.00 -> 59.6 mm
- net N$27: track 0.00 -> 48.9 mm
- net N$10: track 0.00 -> 45.3 mm, vias 0 -> 1
- net N$12: track 0.00 -> 36.2 mm
- net N$28: track 0.00 -> 35.0 mm
- net N$29: track 0.00 -> 34.7 mm, vias 0 -> 1
- net N$25: track 0.00 -> 32.3 mm, vias 0 -> 1
- net N$6: track 0.00 -> 31.8 mm, vias 0 -> 1
- net N$26: track 0.00 -> 30.4 mm
- net N$9: track 0.00 -> 29.9 mm
- net N$17: track 0.00 -> 29.4 mm
- net N$31: track 0.00 -> 28.8 mm
- net N$16: track 0.00 -> 28.6 mm
- net N$30: track 0.00 -> 28.1 mm
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