File: ARMED BASE/armedbase.sch (EAGLE design)
At the start: 14 parts, among them K1 CQ1-12V, X1 RJ45-6L2-B, X2 RJ45-6L2-B

Commit message: armed base
Parts:
- added J2, J3, J4, J5: (no value), con-amp:MTA02-156
- added LOGO2: OSHW-LOGOL, SparkFun-Aesthetics:OSHW-LOGOL
- added OK1: SFH618A-2, optocoupler:SFH618A-2
- added OK2: H11L1M, optocoupler:H11L1M
Changed lines of the file:
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@@
 <part name="GND1" library="SparkFun-Aesthetics" deviceset="GND" device=""/>
 <part name="SUPPLY1" library="SparkFun-Aesthetics" deviceset="VCC" device=""/>
+<part name="J2" library="con-amp" deviceset="MTA02-156" device=""/>
+<part name="J3" library="con-amp" deviceset="MTA02-156" device=""/>
+<part name="J4" library="con-amp" deviceset="MTA02-156" device=""/>
+<part name="J5" library="con-amp" deviceset="MTA02-156" device=""/>
+<part name="LOGO2" library="SparkFun-Aesthetics" deviceset="OSHW-LOGO" device="L"/>
+<part name="OK1" library="optocoupler" deviceset="SFH618?*" device="A" technology="-2"/>
+<part name="OK2" library="optocoupler" deviceset="H11L*M" device="" technology="1"/>
 </parts>
 <sheets>
@@
 <instance part="GND1" gate="1" x="58.42" y="154.94"/>
 <instance part="SUPPLY1" gate="G$1" x="48.26" y="154.94"/>
+<instance part="J2" gate="G$1" x="66.04" y="93.98"/>
+<instance part="J3" gate="G$1" x="81.28" y="93.98"/>
+<instance part="J4" gate="G$1" x="96.52" y="93.98"/>
+<instance part="J5" gate="G$1" x="111.76" y="93.98"/>
+<instance part="LOGO2" gate="G$1" x="104.14" y="160.02"/>
+<instance part="OK1" gate="G$1" x="152.4" y="160.02"/>
+<instance part="OK2" gate="G$1" x="180.34" y="162.56"/>
 </instances>
 <busses>

Commit message: smd
Parts:
- R1: device eagle-ltspice:R0204/7 -> SparkFun-Passives:RESISTOR0805-RES
Changed lines of the file:
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@@
 <part name="IC1" library="SparkFun-PowerIC" deviceset="V_REG_78XX" device="SIDE"/>
 <part name="Q1" library="SparkFun-DiscreteSemi" deviceset="TRANSISTOR_NPN" device="BC547"/>
-<part name="R1" library="eagle-ltspice" deviceset="R" device="0204/7"/>
+<part name="R1" library="SparkFun-Passives" deviceset="RESISTOR" device="0805-RES"/>
 <part name="C1" library="capacitor-wima" deviceset="C" device="2,5-3"/>
 <part name="LED1" library="led" deviceset="LED" device="5MM"/>

Commit message: smd2
Parts:
- removed OK1: SFH618A-2, optocoupler:SFH618A-2
- removed OK2: H11L1M, optocoupler:H11L1M
- removed Q1: (no value), SparkFun-DiscreteSemi:TRANSISTOR_NPNBC547
- added Q2: (no value), semicon-smd-ipc:NPN-TRANSISTOR_SOT23
- added X3: 14867, con-4ucon:14867
- C1: device capacitor-wima:C2,5-3 -> SparkFun-Capacitors:CAP0805
- D1: value 1N4004 -> (none); device diode:1N4004 -> SparkFun-DiscreteSemi:DIODESMA
- IC1: value (none) -> REG1117; device SparkFun-PowerIC:V_REG_78XXSIDE -> burr-brown:REG1117
- LED1: device led:LED5MM -> led:LEDCHIP-LED0805
Other:
- moved on the sheet: C1
Changed lines of the file:
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@@
 <part name="SV3" library="con-lstb" deviceset="MA08-1" device=""/>
 <part name="SV4" library="con-lstb" deviceset="MA06-1" device=""/>
-<part name="IC1" library="SparkFun-PowerIC" deviceset="V_REG_78XX" device="SIDE"/>
-<part name="Q1" library="SparkFun-DiscreteSemi" deviceset="TRANSISTOR_NPN" device="BC547"/>
+<part name="IC1" library="burr-brown" deviceset="REG1117" device=""/>
 <part name="R1" library="SparkFun-Passives" deviceset="RESISTOR" device="0805-RES"/>
-<part name="C1" library="capacitor-wima" deviceset="C" device="2,5-3"/>
-<part name="LED1" library="led" deviceset="LED" device="5MM"/>
+<part name="C1" library="SparkFun-Capacitors" deviceset="CAP" device="0805"/>
+<part name="LED1" library="led" deviceset="LED" device="CHIP-LED0805"/>
 <part name="K1" library="relay" deviceset="CQ1-12V" device=""/>
-<part name="D1" library="diode" deviceset="1N4004" device=""/>
+<part name="D1" library="SparkFun-DiscreteSemi" deviceset="DIODE" device="SMA"/>
 <part name="GND1" library="SparkFun-Aesthetics" deviceset="GND" device=""/>
 <part name="SUPPLY1" library="SparkFun-Aesthetics" deviceset="VCC" device=""/>
@@
 <part name="J5" library="con-amp" deviceset="MTA02-156" device=""/>
 <part name="LOGO2" library="SparkFun-Aesthetics" deviceset="OSHW-LOGO" device="L"/>
-<part name="OK1" library="optocoupler" deviceset="SFH618?*" device="A" technology="-2"/>
-<part name="OK2" library="optocoupler" deviceset="H11L*M" device="" technology="1"/>
+<part name="Q2" library="semicon-smd-ipc" deviceset="NPN-TRANSISTOR_" device="SOT23"/>
+<part name="X3" library="con-4ucon" deviceset="14867" device=""/>
 </parts>
 <sheets>
@@
 <instance part="SV4" gate="1" x="180.34" y="33.02"/>
 <instance part="IC1" gate="G$1" x="30.48" y="137.16"/>
-<instance part="Q1" gate="G$1" x="167.64" y="114.3"/>
 <instance part="R1" gate="G$1" x="33.02" y="104.14"/>
 <instance part="C1" gate="G$1" x="50.8" y="116.84"/>
@@
 <instance part="K1" gate="1" x="170.18" y="129.54"/>
 <instance part="K1" gate="2" x="187.96" y="129.54"/>
-<instance part="D1" gate="1" x="170.18" y="144.78"/>
+<instance part="D1" gate="G$1" x="170.18" y="144.78"/>
 <instance part="GND1" gate="1" x="58.42" y="154.94"/>
 <instance part="SUPPLY1" gate="G$1" x="48.26" y="154.94"/>
@@
 <instance part="J5" gate="G$1" x="111.76" y="93.98"/>
 <instance part="LOGO2" gate="G$1" x="104.14" y="160.02"/>
-<instance part="OK1" gate="G$1" x="152.4" y="160.02"/>
-<instance part="OK2" gate="G$1" x="180.34" y="162.56"/>
+<instance part="Q2" gate="G$1" x="142.24" y="101.6"/>
+<instance part="X3" gate="G$1" x="144.78" y="157.48"/>
 </instances>
 <busses>

Commit message: modbus
Parts:
- added C2: 100uf, SparkFun-Capacitors:CAP0805
- added R2: 10k, SparkFun-Passives:RESISTOR0805-RES
- added R3, R4: 680, SparkFun-Passives:RESISTOR0805-RES
- added R5: 120, SparkFun-Passives:RESISTOR0805-RES
- added R6: 2.2k, SparkFun-Passives:RESISTOR0805-RES
- added R7: 1k, SparkFun-Passives:RESISTOR0805-RES
- added R8: 330, SparkFun-Passives:RESISTOR0805-RES
- added S1: (no value), SparkFun-Electromechanical:SWITCH-SPDTSMD2
- added U$1: MAX485DIL, SparkFun-DigitalIC:MAX485DIL
- C1: value (none) -> 10uf
- R1: value (none) -> 10k
Connections:
- new net GND: C1.1, C2.1, IC1.GND, J1.1, LED1.C, Q2.E, R4.1, R7.1, U$1.GND
- new net N$11: LED1.A, R8.1
- new net N$13: D1.A, S1.O
- new net N$14: C2.2, D1.C, IC1.VIN
- new net N$2: Q2.C, R1.1, U$1.DE, U$1.RE
- new net N$4: Q2.B, R6.1, R7.2
- new net N$7: R4.2, R5.1, U$1.B, X3.4
- new net N$8: R3.1, R5.2, U$1.A, X3.1
- new net RX: R2.1, U$1.RO
- new net TX: R6.2, U$1.DI
- new net VCC: J1.3, S1.P
- new net VCC5V: C1.2, IC1.VOUT, R1.2, R2.2, R3.2, R8.2, U$1.VCC
Other:
- moved on the sheet: C1, D1, IC1, J1, J2, J3, J4, J5, LED1, Q2, R1, SV1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

Commit message: last
Parts:
- added D10, D11, D12, D13, D14, D15, D16, D17, D2, D3, D4, D5, D6, D7, D8, D9: (no value), SparkFun-DiscreteSemi:DIODESMA
- added R10, R11, R12, R13, R14, R15, R16, R17, R18, R19, R20, R21, R22, R23, R24, R9: 10k, SparkFun-Passives:RESISTOR0805-RES
Connections:
- new net INA1: D2.A, R9.2
- new net INA2: D3.A, R10.2
- new net INA3: D4.A, R11.2
- new net INA4: D5.A, R12.2
- new net INA5: D6.A, R13.2
- new net INA6: D7.A, R14.2
- new net INA7: D8.A, R15.2
- new net INA8: D9.A, R16.2
- new net INB1: D10.A, R17.2
- new net INB2: D11.A, R18.2
- new net INB3: D12.A, R19.2
- new net INB4: D13.A, R20.2
- new net INB5: D14.A, R21.2
- new net INB6: D15.A, R22.2
- new net INB7: D16.A, R23.2
- new net INB8: D17.A, R24.2
- new net N$1: D2.C, X1.1
- new net N$10: D13.C, X2.4
- new net N$12: D14.C, X2.5
- new net N$15: D15.C, X2.6
- new net N$16: D16.C, X2.7
- new net N$17: D17.C, X2.8
- new net N$25: D3.C, X1.2
- new net N$26: D4.C, X1.3
- new net N$27: D5.C, X1.4
- new net N$28: D6.C, X1.5
- new net N$29: D7.C, X1.6
- new net N$3: D10.C, X2.1
- new net N$30: D8.C, X1.7
- new net N$31: D9.C, X1.8
- new net N$6: D11.C, X2.2
- new net N$9: D12.C, X2.3
- net VCC5V: now also R10.1, R11.1, R12.1, R13.1, R14.1, R15.1, R16.1, R17.1, R18.1, R19.1, R20.1, R21.1, R22.1, R23.1, R24.1, R9.1
Other:
- moved on the sheet: Q2, R1, R2, R3, R4, R5, R6, R7, SV1, U$1, X1, X2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
