File: cncWTest/modbus.brd (EAGLE design)
At the start: 39.4 x 34 mm, 10 parts, among them Q2 2N3904

Commit message: WE
Parts:
- added LED1: (no value), led:CHIP-LED0805
- added R8: 10k, SparkFun-Passives:0805
- moved Q2 11.5 mm to (16.5, 16.5), turned to 90 degrees
Connections:
- new net N$1: LED1.A, R8.1
- net GND: now also LED1.C
- net VCC5V: now also R8.2
Routing:
- net GND: track 64.6 -> 12.0 mm, vias 0 -> 2
- net VCC5V: track 107.3 -> 69.0 mm, vias 1 -> 0
- net N$4: track 42.3 -> 36.9 mm
- net N$1: track 0.00 -> 4.40 mm
- net B: track 37.1 -> 33.9 mm
- net TX: track 36.9 -> 38.7 mm
- net RX: track 27.1 -> 28.2 mm, vias 0 -> 1
- net N$2: vias 0 -> 1
- added copper zone on layer 16, net GND
Other:
- board text added: "G 5V T R A B"

Commit message: CNC conf 1
Parts:
- moved R3 10.8 mm to (26.7, 20.3)
- moved R5 9.92 mm to (21.6, 20.3)
- moved R6 7.62 mm to (26.7, 5.08), turned to 90 degrees
- moved R4 7.41 mm to (17.8, 21.6), turned to 270 degrees
- moved R7 6.48 mm to (14.0, 21.6), turned to 270 degrees
- moved U$1 6.35 mm to (22.9, 12.7)
- moved Q2 4.58 mm to (14.0, 12.7)
- moved R1 3.81 mm to (24.1, 5.08), turned to 270 degrees
- moved SV2 3.81 mm to (7.62, 12.7)
- moved LED1 2.54 mm to (12.7, 5.08)
- moved R2 1.27 mm to (20.3, 5.08), turned to 270 degrees
- turned R8 to 90 degrees
Routing:
- net GND: track 12.0 -> 50.5 mm, vias 2 -> 0
- net TX: track 38.7 -> 23.8 mm
- net B: track 33.9 -> 22.3 mm
- net A: track 35.9 -> 24.7 mm
- net VCC5V: track 69.0 -> 59.5 mm
- net N$2: track 24.5 -> 16.6 mm
- net RX: track 28.2 -> 22.0 mm, vias 1 -> 0
- net N$1: track 4.40 -> 3.65 mm
- net N$4: track 36.9 -> 37.0 mm, vias 2 -> 0
- removed copper zone on layer 16, net GND
Other:
- board size 39.4 x 34 mm -> 30.5 x 25.1 mm
