File: cncWTest/modbus.sch (EAGLE design)
At the start: 10 parts, among them Q2 2N3904

Commit message: WE
Parts:
- added LED1: (no value), led:LEDCHIP-LED0805
- added R8: 10k, SparkFun-Passives:RESISTOR0805-RES
Connections:
- new net N$1: LED1.A, R8.1
- net GND: now also LED1.C
- net VCC5V: now also R8.2
Changed lines of the file:
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@@
 <part name="GND2" library="SparkFun-Aesthetics" deviceset="GND" device=""/>
 <part name="SV2" library="con-lsta" deviceset="FE06-1" device=""/>
+<part name="R8" library="SparkFun-Passives" deviceset="RESISTOR" device="0805-RES" value="10k"/>
+<part name="LED1" library="led" deviceset="LED" device="CHIP-LED0805"/>
 </parts>
 <sheets>
@@
 <instance part="GND2" gate="1" x="99.06" y="53.34" rot="R90"/>
 <instance part="SV2" gate="G$1" x="144.78" y="43.18" rot="R180"/>
+<instance part="R8" gate="G$1" x="121.92" y="45.72"/>
+<instance part="LED1" gate="G$1" x="109.22" y="50.8" rot="R180"/>
 </instances>
 <busses>
@@
 <pinref part="SV2" gate="G$1" pin="2"/>
 <wire x1="129.54" y1="45.72" x2="137.16" y2="45.72" width="0.1524" layer="91"/>
+<pinref part="R8" gate="G$1" pin="2"/>
+<wire x1="129.54" y1="45.72" x2="127" y2="45.72" width="0.1524" layer="91"/>
+<junction x="129.54" y="45.72"/>
 </segment>
 </net>
@@
 <pinref part="GND2" gate="1" pin="GND"/>
 <wire x1="96.52" y1="53.34" x2="96.52" y2="58.42" width="0.1524" layer="91"/>
-<wire x1="96.52" y1="58.42" x2="137.16" y2="58.42" width="0.1524" layer="91"/>
+<wire x1="96.52" y1="58.42" x2="109.22" y2="58.42" width="0.1524" layer="91"/>
 <pinref part="SV2" gate="G$1" pin="1"/>
+<wire x1="109.22" y1="58.42" x2="137.16" y2="58.42" width="0.1524" layer="91"/>
 <wire x1="137.16" y1="58.42" x2="137.16" y2="48.26" width="0.1524" layer="91"/>
 <junction x="96.52" y="53.34"/>
+<pinref part="LED1" gate="G$1" pin="C"/>
+<wire x1="109.22" y1="55.88" x2="109.22" y2="58.42" width="0.1524" layer="91"/>
+<junction x="109.22" y="58.42"/>
 </segment>
 </net>
@@
 </segment>
 </net>
+<net name="N$1" class="0">
+<segment>
+<pinref part="R8" gate="G$1" pin="1"/>
+<wire x1="116.84" y1="45.72" x2="109.22" y2="45.72" width="0.1524" layer="91"/>
+<pinref part="LED1" gate="G$1" pin="A"/>
+<wire x1="109.22" y1="45.72" x2="109.22" y2="48.26" width="0.1524" layer="91"/>
+</segment>
+</net>

Commit message: we
Parts:
- R8: value 10k -> 330
Changed lines of the file:
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@@
 <part name="GND2" library="SparkFun-Aesthetics" deviceset="GND" device=""/>
 <part name="SV2" library="con-lsta" deviceset="FE06-1" device=""/>
-<part name="R8" library="SparkFun-Passives" deviceset="RESISTOR" device="0805-RES" value="10k"/>
+<part name="R8" library="SparkFun-Passives" deviceset="RESISTOR" device="0805-RES" value="330"/>
 <part name="LED1" library="led" deviceset="LED" device="CHIP-LED0805"/>
 </parts>
