File: SulaMatik/SulaMatik.brd (EAGLE design)
At the start: 48.3 x 61 mm, 29 parts, among them Q3 2N3904

Commit message: done
Parts:
- added SV1: (no value), con-lstb:MA08-1
Connections:
- net A0: now also SV1.1
- net A1: now also SV1.2
- net A2: now also SV1.3
- net A3: now also SV1.4
- net A4: now also SV1.5
- net A5: now also SV1.6
- net GND: now also SV1.8
- net VCC: now also SV1.7
Routing:
- net A4: track 0.00 -> 23.0 mm
- net A5: track 0.00 -> 11.6 mm
- net VCC: track 105.9 -> 114.4 mm
- net A1: track 0.00 -> 7.40 mm
- net A0: track 0.00 -> 7.39 mm
- net A2: track 0.00 -> 7.39 mm
- net A3: track 0.00 -> 7.39 mm
- net GND: track 162.4 -> 166.7 mm
Other:
- board text added: "Sulamatik"

Commit message: sula
Parts:
- removed IC3: (no value), SparkFun-PowerIC:TO-220-ALT
- removed J1: (no value), con-amp:1X2MTA
- added D3: (no value), SparkFun-DiscreteSemi:SMA-DIODE
- added IC1: REG1117, burr-brown:SOT223
- added LIGHT, MS, PW: (no value), con-amp:1X2MTA
- added PH1: A1050_09, photo-elements:T0-46-A10XX
- added Q1: 2N3904, semicon-smd-ipc:SOT23
- added R14: 1K, SparkFun-Passives:0805
- added R15: THERMISTOR-2,5, varistor:RS-2,5
- added R16, R17, R18: 10K, SparkFun-Passives:0805
- SV1: device con-lstb:MA08-1 -> con-lstb:MA04-1
- moved S2 25.9 mm to (10.2, 30.5), turned to 0 degrees
- moved R12 10.2 mm to (2.54, 27.9)
- moved SV1 3.59 mm to (40.6, 43.2)
- moved C1 2.54 mm to (2.54, 35.6), turned to 270 degrees
- moved JP2 2.54 mm to (31.8, 40.6)
- moved JP6 2.54 mm to (34.3, 52.1)
- moved JP7 2.54 mm to (19.1, 24.1)
- moved R13 2.54 mm to (27.9, 33.0)
- renumbered J2 to PUMP
Connections:
- new net N$19: D3.A, LIGHT.2, Q1.3
- new net N$20: Q1.1, R14.1
- net A0: now also MS.1, R17.1; no longer SV1.1
- net A1: now also R15.1, R18.1; no longer SV1.2
- net A2: now also PH1.1, R16.1; no longer SV1.3
- net A3: now also R14.2; no longer SV1.4
- net A4: now also SV1.1; no longer SV1.5
- net A5: now also SV1.2; no longer SV1.6
- net GND: now also IC1.1, PW.1, Q1.2, R16.2, R17.2, R18.2, SV1.4; no longer IC3.GND, J1.1, SV1.8
- net N$1: now also IC1.3; no longer IC3.IN
- net N$2: now also PW.2; no longer J1.2
- net VCC: now also D3.C, IC1.2, LIGHT.1, MS.2, PH1.2, R15.2, SV1.3; no longer IC3.OUT, SV1.7
Routing:
- net GND: track 166.7 -> 226.1 mm
- net A1: track 7.40 -> 40.2 mm
- net VCC: track 114.4 -> 146.1 mm
- net A0: track 7.39 -> 31.7 mm
- net A2: track 7.39 -> 28.0 mm, vias 0 -> 1
- net N$19: track 0.00 -> 19.5 mm
- net A3: track 7.39 -> 26.4 mm, vias 0 -> 1
- net N$11: track 5.78 -> 15.9 mm
- net N$2: track 22.7 -> 12.6 mm
- net N$20: track 0.00 -> 6.95 mm
- net A5: track 11.6 -> 17.9 mm
- net A4: track 23.0 -> 17.5 mm
- net D10: track 18.2 -> 13.7 mm, vias 0 -> 1
- net MOSI: track 14.8 -> 12.3 mm
- net SCK: track 37.5 -> 35.5 mm
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
Commit message: trimpod
Parts:
- added R19: 10K, pot:CA6V
- moved DZ1 2.54 mm to (15.2, 7.62)
- moved S1 2.54 mm to (7.62, 58.4)
- moved PUMP 2.54 mm to (33.0, 5.08)
Connections:
- new net N$17: MS.2, R19.E
- net VCC: now also R19.S; no longer MS.2
Routing:
- net A0: track 31.7 -> 62.5 mm
- net A1: track 40.2 -> 21.2 mm, vias 0 -> 1
- net N$17: track 0.00 -> 12.1 mm, vias 1 -> 0
- net VCC: track 146.1 -> 151.4 mm
- net N$3: track 3.43 -> 5.97 mm
- net N$4: track 3.48 -> 6.01 mm
- net N$2: track 12.6 -> 10.0 mm
- net N$16: track 3.48 -> 6.00 mm
- net N$7: track 3.48 -> 6.00 mm
- net N$15: track 3.48 -> 6.00 mm
- net N$8: track 3.49 -> 6.00 mm
- net N$14: track 3.49 -> 6.00 mm
- net N$9: track 3.50 -> 6.01 mm
- net N$12: track 3.50 -> 6.02 mm
- net N$10: track 3.53 -> 6.03 mm
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