File: SulaMatik/SulaMatik.sch (EAGLE design)
At the start: 29 parts, among them Q3 2N3904

Commit message: done
Parts:
- added SV1: (no value), con-lstb:MA08-1
Connections:
- net A0: now also SV1.1
- net A1: now also SV1.2
- net A2: now also SV1.3
- net A3: now also SV1.4
- net A4: now also SV1.5
- net A5: now also SV1.6
- net GND: now also SV1.8
- net VCC: now also SV1.7
Changed lines of the file:
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@@
 <part name="R13" library="SparkFun-Passives" deviceset="RESISTOR" device="0805-RES" value="10k"/>
 <part name="GND3" library="supply1" deviceset="GND" device=""/>
+<part name="SV1" library="con-lstb" deviceset="MA08-1" device=""/>
 </parts>
 <sheets>
@@
 <instance part="R13" gate="G$1" x="213.36" y="104.14" rot="R270"/>
 <instance part="GND3" gate="1" x="236.22" y="111.76" rot="R90"/>
+<instance part="SV1" gate="1" x="114.3" y="76.2"/>
 </instances>
 <busses>
@@
 <pinref part="GND3" gate="1" pin="GND"/>
 </segment>
+<segment>
+<pinref part="SV1" gate="1" pin="8"/>
+<label x="124.46" y="86.36" size="1.778" layer="95" xref="yes"/>
+<wire x1="121.92" y1="86.36" x2="124.46" y2="86.36" width="0.1524" layer="91"/>
+</segment>
 </net>
 <net name="RESET" class="0">
@@
 <label x="193.04" y="96.52" size="1.778" layer="95" rot="R180" xref="yes"/>
 </segment>
+<segment>
+<pinref part="SV1" gate="1" pin="7"/>
+<wire x1="121.92" y1="83.82" x2="132.08" y2="83.82" width="0.1524" layer="91"/>
+<label x="132.08" y="83.82" size="1.778" layer="95" xref="yes"/>
+</segment>
 </net>
 <net name="RAW" class="1">
@@
 <pinref part="JP2" gate="G$1" pin="2"/>
 </segment>
+<segment>
+<pinref part="SV1" gate="1" pin="6"/>
+<label x="124.46" y="81.28" size="1.778" layer="95" xref="yes"/>
+<wire x1="121.92" y1="81.28" x2="124.46" y2="81.28" width="0.1524" layer="91"/>
+</segment>
 </net>
 <net name="A4" class="0">
@@
 <pinref part="JP2" gate="G$1" pin="1"/>
 </segment>
+<segment>
+<pinref part="SV1" gate="1" pin="5"/>
+<wire x1="121.92" y1="78.74" x2="129.54" y2="78.74" width="0.1524" layer="91"/>
+<label x="129.54" y="78.74" size="1.778" layer="95" xref="yes"/>
+</segment>
 </net>
 <net name="A3" class="0">
@@
 <pinref part="JP6" gate="G$1" pin="5"/>
 </segment>
+<segment>
+<pinref part="SV1" gate="1" pin="4"/>
+<label x="124.46" y="76.2" size="1.778" layer="95" xref="yes"/>
+<wire x1="121.92" y1="76.2" x2="124.46" y2="76.2" width="0.1524" layer="91"/>
+</segment>
 </net>
 <net name="A2" class="0">
@@
 <pinref part="JP6" gate="G$1" pin="6"/>
 </segment>
+<segment>
+<pinref part="SV1" gate="1" pin="3"/>
+<wire x1="121.92" y1="73.66" x2="129.54" y2="73.66" width="0.1524" layer="91"/>
+<label x="129.54" y="73.66" size="1.778" layer="95" xref="yes"/>
+</segment>
 </net>
 <net name="A1" class="0">
@@
 <pinref part="JP6" gate="G$1" pin="7"/>
 </segment>
+<segment>
+<pinref part="SV1" gate="1" pin="2"/>
+<wire x1="121.92" y1="71.12" x2="124.46" y2="71.12" width="0.1524" layer="91"/>
+<label x="124.46" y="71.12" size="1.778" layer="95" xref="yes"/>
+</segment>
 </net>
 <net name="A0" class="0">
@@
 <pinref part="JP6" gate="G$1" pin="8"/>
 </segment>
-</net>
+<segment>
+<label x="129.54" y="68.58" size="1.778" layer="95" xref="yes"/>
+<wire x1="121.92" y1="68.58" x2="129.54" y2="68.58" width="0.1524" layer="91"/>
+<pinref part="SV1" gate="1" pin="1"/>
+</segment>
+</net>

Commit message: sula
Parts:
- removed IC3: (no value), SparkFun-PowerIC:V_REG_78XX-TO-220
- removed J1: (no value), con-amp:MTA02-156
- added D3: (no value), SparkFun-DiscreteSemi:DIODESMA
- added IC1: REG1117, burr-brown:REG1117
- added LIGHT, MS, PW: (no value), con-amp:MTA02-156
- added PH1: A1050_09, photo-elements:A1050_09
- added Q1: 2N3904, semicon-smd-ipc:NPN-TRANSISTOR_SOT23
- added R14: 1K, SparkFun-Passives:RESISTOR0805-RES
- added R15: THERMISTOR-2,5, varistor:THERMISTOR-2,5
- added R16, R17, R18: 10K, SparkFun-Passives:RESISTOR0805-RES
- SV1: device con-lstb:MA08-1 -> con-lstb:MA04-1
- renumbered J2 to PUMP
Connections:
- new net N$19: D3.A, LIGHT.2, Q1.C
- new net N$20: Q1.B, R14.1
- net A0: now also MS.1, R17.1; no longer SV1.1
- net A1: now also R15.1, R18.1; no longer SV1.2
- net A2: now also PH1.1, R16.1; no longer SV1.3
- net A3: now also R14.2; no longer SV1.4
- net A4: now also SV1.1; no longer SV1.5
- net A5: now also SV1.2; no longer SV1.6
- net GND: now also IC1.GND, PW.1, Q1.E, R16.2, R17.2, R18.2, SV1.4; no longer IC3.GND, J1.1, SV1.8
- net N$1: now also IC1.VIN; no longer IC3.IN
- net N$2: now also PW.2; no longer J1.2
- net VCC: now also D3.C, IC1.VOUT, LIGHT.1, MS.2, PH1.2, R15.2, SV1.3; no longer IC3.OUT, SV1.7
Other:
- note added: "LIGHT"
- note added: "LIGHT SENSOR"
- note added: "MOISTURE SENSOR"
- note added: "THERMO SENSOR"
- moved on the sheet: C2, D1, F1, R13, S1, S2

Commit message: trimpod
Parts:
- added R19: 10K, pot:TRIM_US-CA6V
Connections:
- new net N$17: MS.2, R19.E
- net VCC: now also R19.S; no longer MS.2
Other:
- moved on the sheet: MS, R15, R18
Changed lines of the file:
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@@
 <part name="R18" library="SparkFun-Passives" deviceset="RESISTOR" device="0805-RES" value="10K"/>
 <part name="MS" library="con-amp" deviceset="MTA02-156" device=""/>
+<part name="R19" library="pot" deviceset="TRIM_US-" device="CA6V" value="10K"/>
 </parts>
 <sheets>
@@
 <text x="127" y="119.38" size="1.778" layer="91">LIGHT SENSOR</text>
 <text x="187.96" y="116.84" size="1.778" layer="91">MOISTURE SENSOR</text>
-<text x="190.5" y="96.52" size="1.778" layer="91">THERMO SENSOR</text>
+<text x="187.96" y="88.9" size="1.778" layer="91">THERMO SENSOR</text>
 </plain>
 <instances>
@@
 <instance part="GND4" gate="1" x="172.72" y="121.92" rot="R90"/>
 <instance part="SV1" gate="1" x="86.36" y="58.42"/>
-<instance part="R15" gate="G$1" x="213.36" y="86.36" rot="R90"/>
+<instance part="R15" gate="G$1" x="210.82" y="78.74" rot="R90"/>
 <instance part="PH1" gate="G$1" x="149.86" y="109.22"/>
 <instance part="GND6" gate="1" x="129.54" y="114.3" rot="R270"/>
@@
 <instance part="GND7" gate="1" x="190.5" y="111.76" rot="R270"/>
 <instance part="R17" gate="G$1" x="200.66" y="111.76" rot="R180"/>
-<instance part="GND8" gate="1" x="193.04" y="91.44" rot="R270"/>
-<instance part="R18" gate="G$1" x="203.2" y="91.44" rot="R180"/>
-<instance part="MS" gate="G$1" x="208.28" y="109.22" rot="MR270"/>
+<instance part="GND8" gate="1" x="190.5" y="83.82" rot="R270"/>
+<instance part="R18" gate="G$1" x="200.66" y="83.82" rot="R180"/>
+<instance part="MS" gate="G$1" x="208.28" y="104.14" rot="MR270"/>
+<instance part="R19" gate="G$1" x="220.98" y="99.06" rot="R90"/>
 </instances>
 <busses>
@@
 <pinref part="R18" gate="G$1" pin="2"/>
 <pinref part="GND8" gate="1" pin="GND"/>
-<wire x1="195.58" y1="91.44" x2="198.12" y2="91.44" width="0.1524" layer="91"/>
+<wire x1="193.04" y1="83.82" x2="195.58" y2="83.82" width="0.1524" layer="91"/>
 </segment>
 </net>
@@
 </segment>
 <segment>
-<wire x1="210.82" y1="101.6" x2="220.98" y2="101.6" width="0.1524" layer="91"/>
-<label x="220.98" y="101.6" size="1.778" layer="95" xref="yes"/>
-<pinref part="MS" gate="G$1" pin="2"/>
-<wire x1="210.82" y1="101.6" x2="210.82" y2="106.68" width="0.1524" layer="91"/>
-</segment>
-<segment>
-<wire x1="213.36" y1="81.28" x2="223.52" y2="81.28" width="0.1524" layer="91"/>
-<label x="223.52" y="81.28" size="1.778" layer="95" xref="yes"/>
+<label x="223.52" y="106.68" size="1.778" layer="95" xref="yes"/>
+<pinref part="R19" gate="G$1" pin="S"/>
+<wire x1="220.98" y1="104.14" x2="220.98" y2="106.68" width="0.1524" layer="91"/>
+<wire x1="220.98" y1="106.68" x2="223.52" y2="106.68" width="0.1524" layer="91"/>
+</segment>
+<segment>
+<wire x1="210.82" y1="73.66" x2="220.98" y2="73.66" width="0.1524" layer="91"/>
+<label x="220.98" y="73.66" size="1.778" layer="95" xref="yes"/>
 <pinref part="R15" gate="G$1" pin="2"/>
 </segment>
@@
 </segment>
 <segment>
-<label x="223.52" y="91.44" size="1.778" layer="95" xref="yes"/>
-<wire x1="208.28" y1="91.44" x2="213.36" y2="91.44" width="0.1524" layer="91"/>
+<label x="220.98" y="83.82" size="1.778" layer="95" xref="yes"/>
+<wire x1="205.74" y1="83.82" x2="210.82" y2="83.82" width="0.1524" layer="91"/>
 <pinref part="R18" gate="G$1" pin="1"/>
 <pinref part="R15" gate="G$1" pin="1"/>
-<wire x1="213.36" y1="91.44" x2="223.52" y2="91.44" width="0.1524" layer="91"/>
-<junction x="213.36" y="91.44"/>
+<wire x1="210.82" y1="83.82" x2="220.98" y2="83.82" width="0.1524" layer="91"/>
+<junction x="210.82" y="83.82"/>
 </segment>
 </net>
@@
 <pinref part="MS" gate="G$1" pin="1"/>
 <wire x1="210.82" y1="111.76" x2="220.98" y2="111.76" width="0.1524" layer="91"/>
-<wire x1="210.82" y1="109.22" x2="210.82" y2="111.76" width="0.1524" layer="91"/>
+<wire x1="210.82" y1="104.14" x2="210.82" y2="111.76" width="0.1524" layer="91"/>
 <junction x="210.82" y="111.76"/>
 </segment>
@@
 </segment>
 </net>
+<net name="N$17" class="0">
+<segment>
+<pinref part="MS" gate="G$1" pin="2"/>
+<wire x1="210.82" y1="101.6" x2="210.82" y2="99.06" width="0.1524" layer="91"/>
+<pinref part="R19" gate="G$1" pin="E"/>
+<wire x1="210.82" y1="99.06" x2="213.36" y2="99.06" width="0.1524" layer="91"/>
+</segment>
+</net>
