File: SulaMatikV1/SulaMatikV1.sch (EAGLE design)
At the start: 32 parts, among them IC1 REG1117, Q1 2N3904, Q3 2N3904

Commit message: sula5110
Parts:
- removed SV1: (no value), con-lstb:MA04-1
- added R2: 10k, SparkFun-Passives:RESISTOR0805-RES
- added S3: SWITCH-MOMENTARY-2PTH, SparkFun-Electromechanical:SWITCH-MOMENTARY-2PTH
- added SV3: (no value), con-lsta:FE07-1
Connections:
- net A3: now also SV3.3; no longer R14.2
- net A4: now also SV3.4; no longer SV1.1
- net A5: now also SV3.5; no longer SV1.2
- net D2: now also R2.2, S3.2
- net D3: now also R14.2
- net D4: now also SV3.1
- net D5: now also SV3.2
- net GND: now also R2.1, SV3.7; no longer SV1.4
- net VCC: now also S3.1, SV3.6; no longer SV1.3
Other:
- note added: "GPI1"
- note added: "GPI2"
- note removed: "GPI"
Changed lines of the file:
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@@
 <part name="D3" library="SparkFun-DiscreteSemi" deviceset="DIODE" device="SMA"/>
 <part name="GND4" library="supply1" deviceset="GND" device=""/>
-<part name="SV1" library="con-lstb" deviceset="MA04-1" device=""/>
 <part name="R15" library="varistor" deviceset="THERMISTOR" device="-2,5"/>
 <part name="PH1" library="photo-elements" deviceset="A10" device="" technology="50_09"/>
@@
 <part name="SV2" library="con-lsta" deviceset="FE08-1" device=""/>
 <part name="R1" library="SparkFun-Passives" deviceset="RESISTOR" device="0805-RES" value="330"/>
+<part name="S3" library="SparkFun-Electromechanical" deviceset="SWITCH-MOMENTARY-2" device="PTH"/>
+<part name="R2" library="SparkFun-Passives" deviceset="RESISTOR" device="0805-RES" value="10k"/>
+<part name="GND2" library="supply1" deviceset="GND" device=""/>
+<part name="SV3" library="con-lsta" deviceset="FE07-1" device=""/>
 </parts>
 <sheets>
@@
 <text x="15.24" y="177.8" size="1.778" layer="91">Display</text>
 <text x="157.48" y="180.34" size="1.778" layer="91">POWER</text>
-<text x="127" y="91.44" size="1.778" layer="91">GPI</text>
+<text x="127" y="91.44" size="1.778" layer="91">GPI1</text>
 <text x="127" y="137.16" size="1.778" layer="91">LIGHT</text>
 <text x="127" y="119.38" size="1.778" layer="91">LIGHT SENSOR</text>
 <text x="187.96" y="116.84" size="1.778" layer="91">MOISTURE SENSOR</text>
 <text x="187.96" y="88.9" size="1.778" layer="91">THERMO SENSOR</text>
+<text x="127" y="66.04" size="1.778" layer="91">GPI2</text>
 </plain>
 <instances>
@@
 <instance part="D3" gate="G$1" x="162.56" y="129.54"/>
 <instance part="GND4" gate="1" x="172.72" y="121.92" rot="R90"/>
-<instance part="SV1" gate="1" x="86.36" y="58.42"/>
 <instance part="R15" gate="G$1" x="210.82" y="78.74" rot="R90"/>
 <instance part="PH1" gate="G$1" x="149.86" y="109.22"/>
@@
 <instance part="SV2" gate="G$1" x="15.24" y="160.02"/>
 <instance part="R1" gate="G$1" x="45.72" y="167.64" rot="R180"/>
+<instance part="S3" gate="G$1" x="134.62" y="53.34"/>
+<instance part="R2" gate="G$1" x="144.78" y="60.96" rot="R270"/>
+<instance part="GND2" gate="1" x="167.64" y="68.58" rot="R90"/>
+<instance part="SV3" gate="G$1" x="101.6" y="22.86"/>
 </instances>
 <busses>
@@
 </segment>
 <segment>
-<label x="96.52" y="60.96" size="1.778" layer="95" xref="yes"/>
-<pinref part="SV1" gate="1" pin="4"/>
-<wire x1="93.98" y1="60.96" x2="96.52" y2="60.96" width="0.1524" layer="91"/>
+<label x="114.3" y="30.48" size="1.778" layer="95" xref="yes"/>
+<pinref part="SV3" gate="G$1" pin="7"/>
+<wire x1="114.3" y1="30.48" x2="109.22" y2="30.48" width="0.1524" layer="91"/>
 </segment>
 <segment>
@@
 <wire x1="22.86" y1="170.18" x2="25.4" y2="170.18" width="0.1524" layer="91"/>
 <label x="25.4" y="170.18" size="1.778" layer="95" xref="yes"/>
+</segment>
+<segment>
+<pinref part="R2" gate="G$1" pin="1"/>
+<wire x1="144.78" y1="66.04" x2="144.78" y2="68.58" width="0.1524" layer="91"/>
+<wire x1="144.78" y1="68.58" x2="165.1" y2="68.58" width="0.1524" layer="91"/>
+<pinref part="GND2" gate="1" pin="GND"/>
 </segment>
 </net>
@@
 </segment>
 <segment>
-<wire x1="93.98" y1="58.42" x2="104.14" y2="58.42" width="0.1524" layer="91"/>
-<label x="104.14" y="58.42" size="1.778" layer="95" xref="yes"/>
-<pinref part="SV1" gate="1" pin="3"/>
+<label x="121.92" y="27.94" size="1.778" layer="95" xref="yes"/>
+<pinref part="SV3" gate="G$1" pin="6"/>
+<wire x1="121.92" y1="27.94" x2="109.22" y2="27.94" width="0.1524" layer="91"/>
 </segment>
 <segment>
@@
 <label x="25.4" y="165.1" size="1.778" layer="95" xref="yes"/>
 </segment>
+<segment>
+<wire x1="129.54" y1="53.34" x2="124.46" y2="53.34" width="0.1524" layer="91"/>
+<pinref part="S3" gate="G$1" pin="1"/>
+<label x="124.46" y="53.34" size="1.778" layer="95" rot="R180" xref="yes"/>
+</segment>
 </net>
 <net name="RAW" class="1">
@@
 </segment>
 <segment>
-<label x="96.52" y="55.88" size="1.778" layer="95" xref="yes"/>
-<pinref part="SV1" gate="1" pin="2"/>
-<wire x1="93.98" y1="55.88" x2="96.52" y2="55.88" width="0.1524" layer="91"/>
+<label x="114.3" y="25.4" size="1.778" layer="95" xref="yes"/>
+<pinref part="SV3" gate="G$1" pin="5"/>
+<wire x1="114.3" y1="25.4" x2="109.22" y2="25.4" width="0.1524" layer="91"/>
 </segment>
 </net>
@@
 </segment>
 <segment>
-<wire x1="93.98" y1="53.34" x2="101.6" y2="53.34" width="0.1524" layer="91"/>
-<label x="101.6" y="53.34" size="1.778" layer="95" xref="yes"/>
-<pinref part="SV1" gate="1" pin="1"/>
+<label x="119.38" y="22.86" size="1.778" layer="95" xref="yes"/>
+<pinref part="SV3" gate="G$1" pin="4"/>
+<wire x1="119.38" y1="22.86" x2="109.22" y2="22.86" width="0.1524" layer="91"/>
 </segment>
 </net>
@@
 </segment>
 <segment>
-<label x="129.54" y="129.54" size="1.778" layer="95" rot="R180" xref="yes"/>
-<wire x1="137.16" y1="129.54" x2="129.54" y2="129.54" width="0.1524" layer="91"/>
-<pinref part="R14" gate="G$1" pin="2"/>
+<label x="114.3" y="20.32" size="1.778" layer="95" xref="yes"/>
+<pinref part="SV3" gate="G$1" pin="3"/>
+<wire x1="114.3" y1="20.32" x2="109.22" y2="20.32" width="0.1524" layer="91"/>
 </segment>
 </net>
@@
 <pinref part="JP7" gate="G$1" pin="8"/>
 </segment>
+<segment>
+<pinref part="S3" gate="G$1" pin="2"/>
+<wire x1="139.7" y1="53.34" x2="144.78" y2="53.34" width="0.1524" layer="91"/>
+<pinref part="R2" gate="G$1" pin="2"/>
+<wire x1="144.78" y1="55.88" x2="144.78" y2="53.34" width="0.1524" layer="91"/>
+<wire x1="144.78" y1="53.34" x2="167.64" y2="53.34" width="0.1524" layer="91"/>
+<label x="167.64" y="53.34" size="1.778" layer="95" xref="yes"/>
+<junction x="144.78" y="53.34"/>
+</segment>
 </net>
 <net name="D3" class="0">
@@
 <pinref part="JP7" gate="G$1" pin="7"/>
 </segment>
+<segment>
+<pinref part="R14" gate="G$1" pin="2"/>
+<wire x1="137.16" y1="129.54" x2="129.54" y2="129.54" width="0.1524" layer="91"/>
+<label x="129.54" y="129.54" size="1.778" layer="95" rot="R180" xref="yes"/>
+</segment>
 </net>
 <net name="D4" class="0">
@@
 <pinref part="JP7" gate="G$1" pin="6"/>
 </segment>
+<segment>
+<label x="114.3" y="15.24" size="1.778" layer="95" xref="yes"/>
+<pinref part="SV3" gate="G$1" pin="1"/>
+<wire x1="114.3" y1="15.24" x2="109.22" y2="15.24" width="0.1524" layer="91"/>
+</segment>
 </net>
 <net name="D5" class="0">
@@
 <pinref part="JP7" gate="G$1" pin="5"/>
 </segment>
-</net>
+<segment>
+<label x="119.38" y="17.78" size="1.778" layer="95" xref="yes"/>
+<pinref part="SV3" gate="G$1" pin="2"/>
+<wire x1="119.38" y1="17.78" x2="109.22" y2="17.78" width="0.1524" layer="91"/>
+</segment>
+</net>

Commit message: sula1
Parts:
- removed S2, S3: SWITCH-MOMENTARY-2PTH, SparkFun-Electromechanical:SWITCH-MOMENTARY-2PTH
- removed SV3: (no value), con-lsta:FE07-1
- added D4: (no value), SparkFun-DiscreteSemi:DIODESMA
- added GPI1, GPI2, GPI3, GPI4: SWITCH-MOMENTARY-2PTH, SparkFun-Electromechanical:SWITCH-MOMENTARY-2PTH
- added Q2: 2N5551, semicon-smd-ipc:NPN-TRANSISTOR_SOT23
- added R3: 1K, SparkFun-Passives:RESISTOR0805-RES
- added R4, R5: 10k, SparkFun-Passives:RESISTOR0805-RES
- added SV1: (no value), con-lsta:FE05-1
- Q3: value 2N3904 -> 2N5551
- renumbered S1 to PS
Connections:
- new net N$7: Q2.B, R3.1
- new net N$8: D4.A, Q2.C, SV2.8
- net A3: now also SV1.1; no longer SV3.3
- net A4: now also SV1.2; no longer SV3.4
- net A5: now also SV1.3; no longer SV3.5
- net D10: now also R3.2; no longer R1.1
- net D2: now also GPI2.2; no longer S3.2
- net D4: now also GPI3.2, R4.2; no longer SV3.1
- net D5: now also GPI4.2, R5.2; no longer SV3.2
- net GND: now also Q2.E, R4.1, R5.1, SV1.5; no longer SV2.8, SV3.7
- net SCK: now also GPI1.2; no longer S2.2
- net VCC: now also D4.C, GPI1.1, GPI2.1, GPI3.1, GPI4.1, R1.1, SV1.4; no longer S2.1, S3.1, SV3.6
Other:
- note added: "GPI3"
- note added: "GPI4"
- moved on the sheet: R1, R13, R2, SV2

Commit message: V1
Parts:
- added R6: THERMISTOR-2,5, varistor:THERMISTOR-2,5
- added R7: 10K, SparkFun-Passives:RESISTOR0805-RES
- SV1: device con-lsta:FE05-1 -> con-lstb:MA04-1
Connections:
- removed net N$8: D4.A, Q2.C, SV2.8
- new net N$10: D4.A, Q2.C, R1.1, SV2.8
- net A3: now also R6.1; no longer SV1.1
- net A4: now also SV1.1; no longer SV1.2
- net A5: now also SV1.2; no longer SV1.3
- net GND: now also R7.2, SV1.4; no longer SV1.5
- net VCC: now also R6.2, SV1.3; no longer R1.1, SV1.4
Other:
- note added: "THERMO SENSOR AIR"
- note added: "THERMO SENSOR SOIL"
- note removed: "THERMO SENSOR"
Changed lines of the file:
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@@
 <part name="R5" library="SparkFun-Passives" deviceset="RESISTOR" device="0805-RES" value="10k"/>
 <part name="GND11" library="supply1" deviceset="GND" device=""/>
-<part name="SV1" library="con-lsta" deviceset="FE05-1" device=""/>
+<part name="R6" library="varistor" deviceset="THERMISTOR" device="-2,5"/>
+<part name="GND12" library="supply1" deviceset="GND" device=""/>
+<part name="R7" library="SparkFun-Passives" deviceset="RESISTOR" device="0805-RES" value="10K"/>
+<part name="SV1" library="con-lstb" deviceset="MA04-1" device=""/>
 </parts>
 <sheets>
@@
 <text x="127" y="119.38" size="1.778" layer="91">LIGHT SENSOR</text>
 <text x="187.96" y="116.84" size="1.778" layer="91">MOISTURE SENSOR</text>
-<text x="187.96" y="88.9" size="1.778" layer="91">THERMO SENSOR</text>
+<text x="187.96" y="88.9" size="1.778" layer="91">THERMO SENSOR SOIL</text>
 <text x="22.86" y="114.3" size="1.778" layer="91">GPI2</text>
 <text x="119.38" y="91.44" size="1.778" layer="91">GPI3</text>
 <text x="119.38" y="66.04" size="1.778" layer="91">GPI4</text>
+<text x="187.96" y="63.5" size="1.778" layer="91">THERMO SENSOR AIR</text>
 </plain>
 <instances>
@@
 <instance part="R5" gate="G$1" x="137.16" y="60.96" rot="R270"/>
 <instance part="GND11" gate="1" x="160.02" y="68.58" rot="R90"/>
-<instance part="SV1" gate="G$1" x="96.52" y="25.4"/>
+<instance part="R6" gate="G$1" x="210.82" y="53.34" rot="R90"/>
+<instance part="GND12" gate="1" x="190.5" y="58.42" rot="R270"/>
+<instance part="R7" gate="G$1" x="200.66" y="58.42" rot="R180"/>
+<instance part="SV1" gate="1" x="96.52" y="27.94"/>
 </instances>
 <busses>
@@
 <segment>
 <label x="114.3" y="30.48" size="1.778" layer="95" xref="yes"/>
-<pinref part="SV1" gate="G$1" pin="5"/>
 <wire x1="104.14" y1="30.48" x2="114.3" y2="30.48" width="0.1524" layer="91"/>
+<pinref part="SV1" gate="1" pin="4"/>
 </segment>
 <segment>
@@
 <wire x1="137.16" y1="68.58" x2="157.48" y2="68.58" width="0.1524" layer="91"/>
 <pinref part="GND11" gate="1" pin="GND"/>
+</segment>
+<segment>
+<pinref part="R7" gate="G$1" pin="2"/>
+<pinref part="GND12" gate="1" pin="GND"/>
+<wire x1="193.04" y1="58.42" x2="195.58" y2="58.42" width="0.1524" layer="91"/>
 </segment>
 </net>
@@
 <segment>
 <label x="121.92" y="27.94" size="1.778" layer="95" xref="yes"/>
-<pinref part="SV1" gate="G$1" pin="4"/>
 <wire x1="104.14" y1="27.94" x2="121.92" y2="27.94" width="0.1524" layer="91"/>
+<pinref part="SV1" gate="1" pin="3"/>
 </segment>
 <segment>
@@
 <label x="43.18" y="165.1" size="1.778" layer="95" rot="MR180" xref="yes"/>
 <pinref part="SV2" gate="G$1" pin="6"/>
-<wire x1="17.78" y1="165.1" x2="33.02" y2="165.1" width="0.1524" layer="91"/>
-<pinref part="R1" gate="G$1" pin="1"/>
-<wire x1="33.02" y1="165.1" x2="35.56" y2="165.1" width="0.1524" layer="91"/>
-<wire x1="30.48" y1="167.64" x2="33.02" y2="167.64" width="0.1524" layer="91"/>
-<wire x1="33.02" y1="167.64" x2="33.02" y2="165.1" width="0.1524" layer="91"/>
-<junction x="33.02" y="165.1"/>
+<wire x1="17.78" y1="165.1" x2="35.56" y2="165.1" width="0.1524" layer="91"/>
 <junction x="35.56" y="165.1"/>
 </segment>
@@
 <label x="116.84" y="53.34" size="1.778" layer="95" rot="R180" xref="yes"/>
 </segment>
+<segment>
+<wire x1="210.82" y1="48.26" x2="220.98" y2="48.26" width="0.1524" layer="91"/>
+<label x="220.98" y="48.26" size="1.778" layer="95" xref="yes"/>
+<pinref part="R6" gate="G$1" pin="2"/>
+</segment>
 </net>
 <net name="RAW" class="1">
@@
 <segment>
 <label x="114.3" y="25.4" size="1.778" layer="95" xref="yes"/>
-<pinref part="SV1" gate="G$1" pin="3"/>
 <wire x1="104.14" y1="25.4" x2="114.3" y2="25.4" width="0.1524" layer="91"/>
+<pinref part="SV1" gate="1" pin="2"/>
 </segment>
 </net>
@@
 <segment>
 <label x="119.38" y="22.86" size="1.778" layer="95" xref="yes"/>
-<pinref part="SV1" gate="G$1" pin="2"/>
 <wire x1="104.14" y1="22.86" x2="119.38" y2="22.86" width="0.1524" layer="91"/>
+<pinref part="SV1" gate="1" pin="1"/>
 </segment>
 </net>
@@
 </segment>
 <segment>
-<label x="114.3" y="20.32" size="1.778" layer="95" xref="yes"/>
-<pinref part="SV1" gate="G$1" pin="1"/>
-<wire x1="104.14" y1="20.32" x2="114.3" y2="20.32" width="0.1524" layer="91"/>
+<label x="220.98" y="58.42" size="1.778" layer="95" xref="yes"/>
+<wire x1="205.74" y1="58.42" x2="210.82" y2="58.42" width="0.1524" layer="91"/>
+<pinref part="R6" gate="G$1" pin="1"/>
+<junction x="210.82" y="58.42"/>
+<wire x1="210.82" y1="58.42" x2="220.98" y2="58.42" width="0.1524" layer="91"/>
 </segment>
 </net>
@@
 </segment>
 </net>
-<net name="N$8" class="0">
-<segment>
+<net name="N$10" class="0">
+<segment>
+<pinref part="R1" gate="G$1" pin="1"/>
+<wire x1="30.48" y1="167.64" x2="33.02" y2="167.64" width="0.1524" layer="91"/>
 <pinref part="Q2" gate="G$1" pin="C"/>
 <wire x1="38.1" y1="170.18" x2="35.56" y2="170.18" width="0.1524" layer="91"/>
 <pinref part="SV2" gate="G$1" pin="8"/>
-<wire x1="17.78" y1="170.18" x2="35.56" y2="170.18" width="0.1524" layer="91"/>
+<wire x1="17.78" y1="170.18" x2="33.02" y2="170.18" width="0.1524" layer="91"/>
 <pinref part="D4" gate="G$1" pin="A"/>
 <junction x="35.56" y="170.18"/>
-</segment>
-</net>
+<wire x1="33.02" y1="170.18" x2="35.56" y2="170.18" width="0.1524" layer="91"/>
+<wire x1="33.02" y1="167.64" x2="33.02" y2="170.18" width="0.1524" layer="91"/>
+<junction x="33.02" y="170.18"/>
+</segment>
+</net>

Commit message: v1
Parts:
- removed R15: THERMISTOR-2,5, varistor:THERMISTOR-2,5
- added SOIL: (no value), con-amp:MTA02-100
- LIGHT, MS, PUMP, PW: device con-amp:MTA02-156 -> con-amp:MTA02-100
- renumbered R6 to AIR
Connections:
- net A1: now also SOIL.1; no longer R15.1
- net A3: now also R7.1
- net VCC: now also SOIL.2; no longer R15.2
Other:
- moved on the sheet: R7
Changed lines of the file:
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@@
 <part name="JP7" library="SparkFun" deviceset="M12" device="PTH" value=""/>
 <part name="JP2" library="SparkFun" deviceset="M02" device="PTH"/>
-<part name="PUMP" library="con-amp" deviceset="MTA02-156" device=""/>
+<part name="PUMP" library="con-amp" deviceset="MTA02-100" device=""/>
 <part name="Q3" library="semicon-smd-ipc" deviceset="NPN-TRANSISTOR_" device="SOT23" value="2N5551"/>
 <part name="R11" library="SparkFun-Passives" deviceset="RESISTOR" device="0805-RES" value="1K"/>
@@
 <part name="R12" library="SparkFun-Passives" deviceset="RESISTOR" device="0805-RES" value="330"/>
 <part name="F1" library="_hhn_PtcFuses_Siba_r500_Ozan" deviceset="SIBA194600*" device="" value="1.5A"/>
-<part name="PW" library="con-amp" deviceset="MTA02-156" device=""/>
+<part name="PW" library="con-amp" deviceset="MTA02-100" device=""/>
 <part name="R13" library="SparkFun-Passives" deviceset="RESISTOR" device="0805-RES" value="10k"/>
 <part name="GND3" library="supply1" deviceset="GND" device=""/>
 <part name="IC1" library="burr-brown" deviceset="REG1117" device=""/>
-<part name="LIGHT" library="con-amp" deviceset="MTA02-156" device=""/>
+<part name="LIGHT" library="con-amp" deviceset="MTA02-100" device=""/>
 <part name="Q1" library="semicon-smd-ipc" deviceset="NPN-TRANSISTOR_" device="SOT23" value="2N3904"/>
 <part name="R14" library="SparkFun-Passives" deviceset="RESISTOR" device="0805-RES" value="1K"/>
 <part name="D3" library="SparkFun-DiscreteSemi" deviceset="DIODE" device="SMA"/>
 <part name="GND4" library="supply1" deviceset="GND" device=""/>
-<part name="R15" library="varistor" deviceset="THERMISTOR" device="-2,5"/>
 <part name="PH1" library="photo-elements" deviceset="A10" device="" technology="50_09"/>
 <part name="GND6" library="supply1" deviceset="GND" device=""/>
@@
 <part name="GND8" library="supply1" deviceset="GND" device=""/>
 <part name="R18" library="SparkFun-Passives" deviceset="RESISTOR" device="0805-RES" value="10K"/>
-<part name="MS" library="con-amp" deviceset="MTA02-156" device=""/>
+<part name="MS" library="con-amp" deviceset="MTA02-100" device=""/>
 <part name="R19" library="pot" deviceset="TRIM_US-" device="CA6V" value="10K"/>
 <part name="SV2" library="con-lsta" deviceset="FE08-1" device=""/>
@@
 <part name="R5" library="SparkFun-Passives" deviceset="RESISTOR" device="0805-RES" value="10k"/>
 <part name="GND11" library="supply1" deviceset="GND" device=""/>
-<part name="R6" library="varistor" deviceset="THERMISTOR" device="-2,5"/>
+<part name="AIR" library="varistor" deviceset="THERMISTOR" device="-2,5"/>
 <part name="GND12" library="supply1" deviceset="GND" device=""/>
 <part name="R7" library="SparkFun-Passives" deviceset="RESISTOR" device="0805-RES" value="10K"/>
 <part name="SV1" library="con-lstb" deviceset="MA04-1" device=""/>
+<part name="SOIL" library="con-amp" deviceset="MTA02-100" device=""/>
 </parts>
 <sheets>
@@
 <instance part="D3" gate="G$1" x="162.56" y="129.54"/>
 <instance part="GND4" gate="1" x="172.72" y="121.92" rot="R90"/>
-<instance part="R15" gate="G$1" x="210.82" y="78.74" rot="R90"/>
 <instance part="PH1" gate="G$1" x="149.86" y="109.22"/>
 <instance part="GND6" gate="1" x="129.54" y="114.3" rot="R270"/>
@@
 <instance part="R5" gate="G$1" x="137.16" y="60.96" rot="R270"/>
 <instance part="GND11" gate="1" x="160.02" y="68.58" rot="R90"/>
-<instance part="R6" gate="G$1" x="210.82" y="53.34" rot="R90"/>
+<instance part="AIR" gate="G$1" x="210.82" y="53.34" rot="R90"/>
 <instance part="GND12" gate="1" x="190.5" y="58.42" rot="R270"/>
-<instance part="R7" gate="G$1" x="200.66" y="58.42" rot="R180"/>
+<instance part="R7" gate="G$1" x="198.12" y="58.42" rot="R180"/>
 <instance part="SV1" gate="1" x="96.52" y="27.94"/>
+<instance part="SOIL" gate="G$1" x="208.28" y="78.74" rot="MR270"/>
 </instances>
 <busses>
@@
 <pinref part="R7" gate="G$1" pin="2"/>
 <pinref part="GND12" gate="1" pin="GND"/>
-<wire x1="193.04" y1="58.42" x2="195.58" y2="58.42" width="0.1524" layer="91"/>
 </segment>
 </net>
@@
 <wire x1="210.82" y1="73.66" x2="220.98" y2="73.66" width="0.1524" layer="91"/>
 <label x="220.98" y="73.66" size="1.778" layer="95" xref="yes"/>
-<pinref part="R15" gate="G$1" pin="2"/>
+<pinref part="SOIL" gate="G$1" pin="2"/>
+<wire x1="210.82" y1="73.66" x2="210.82" y2="76.2" width="0.1524" layer="91"/>
 </segment>
 <segment>
@@
 <wire x1="210.82" y1="48.26" x2="220.98" y2="48.26" width="0.1524" layer="91"/>
 <label x="220.98" y="48.26" size="1.778" layer="95" xref="yes"/>
-<pinref part="R6" gate="G$1" pin="2"/>
+<pinref part="AIR" gate="G$1" pin="2"/>
 </segment>
 </net>
@@
 <segment>
 <label x="220.98" y="58.42" size="1.778" layer="95" xref="yes"/>
-<wire x1="205.74" y1="58.42" x2="210.82" y2="58.42" width="0.1524" layer="91"/>
-<pinref part="R6" gate="G$1" pin="1"/>
+<wire x1="203.2" y1="58.42" x2="210.82" y2="58.42" width="0.1524" layer="91"/>
+<pinref part="AIR" gate="G$1" pin="1"/>
 <junction x="210.82" y="58.42"/>
 <wire x1="210.82" y1="58.42" x2="220.98" y2="58.42" width="0.1524" layer="91"/>
+<pinref part="R7" gate="G$1" pin="1"/>
 </segment>
 </net>
@@
 <segment>
 <label x="220.98" y="83.82" size="1.778" layer="95" xref="yes"/>
+<pinref part="R18" gate="G$1" pin="1"/>
 <wire x1="205.74" y1="83.82" x2="210.82" y2="83.82" width="0.1524" layer="91"/>
-<pinref part="R18" gate="G$1" pin="1"/>
-<pinref part="R15" gate="G$1" pin="1"/>
+<pinref part="SOIL" gate="G$1" pin="1"/>
 <wire x1="210.82" y1="83.82" x2="220.98" y2="83.82" width="0.1524" layer="91"/>
+<wire x1="210.82" y1="78.74" x2="210.82" y2="83.82" width="0.1524" layer="91"/>
 <junction x="210.82" y="83.82"/>
 </segment>
