File: SulaMatikV1/SulaMatikV1.brd (EAGLE design)
At the start: 48.3 x 61 mm, 32 parts, among them IC1 REG1117, Q1 2N3904, Q3 2N3904

Commit message: sula5110
Parts:
- removed SV1: (no value), con-lstb:MA04-1
- added R2: 10k, SparkFun-Passives:0805
- added S3: SWITCH-MOMENTARY-2PTH, SparkFun-Electromechanical:TACTILE-PTH
- added SV3: (no value), con-lsta:FE07
- moved R18 44.4 mm to (5.08, 27.9), turned to 180 degrees
- moved R15 42.3 mm to (5.08, 10.2)
- moved R16 33.9 mm to (12.7, 27.9), turned to 180 degrees
- moved PH1 27.0 mm to (22.9, 5.08)
- moved IC1 25.4 mm to (20.3, 35.6), turned to 180 degrees
- moved C1 13.7 mm to (12.7, 35.6), turned to 0 degrees
- moved R12 10.5 mm to (5.08, 33.0), turned to 0 degrees
- moved SV2 10.5 mm to (12.7, 15.2)
- moved C2 10.2 mm to (12.7, 38.1)
- moved F1 10.2 mm to (5.08, 38.1)
- moved Q1 9.16 mm to (33.0, 48.3)
- moved R13 9.16 mm to (33.0, 40.6)
- moved JP7 8.03 mm to (26.7, 21.6)
- moved JP2 8.03 mm to (39.4, 38.1)
- moved JP6 8.03 mm to (41.9, 49.5)
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Connections:
- net A3: now also SV3.3; no longer R14.2
- net A4: now also SV3.4; no longer SV1.1
- net A5: now also SV3.5; no longer SV1.2
- net D2: now also R2.2, S3.3
- net D3: now also R14.2
- net D4: now also SV3.1
- net D5: now also SV3.2
- net GND: now also R2.1, SV3.7; no longer SV1.4
- net VCC: now also S3.1, SV3.6; no longer SV1.3
Routing:
- net A1: track 21.2 -> 81.7 mm, vias 1 -> 0
- net A3: track 25.6 -> 72.9 mm, vias 1 -> 0
- net A2: track 28.0 -> 68.0 mm
- net D5: track 0.00 -> 37.9 mm, vias 0 -> 1
- net A0: track 62.5 -> 26.2 mm
- net A5: track 17.9 -> 53.8 mm, vias 0 -> 1
- net D4: track 0.00 -> 33.0 mm
- net A4: track 17.5 -> 49.9 mm, vias 0 -> 1
- net VCC: track 176.2 -> 205.0 mm
- net D10: track 19.0 -> 43.2 mm, vias 1 -> 0
- net D2: track 0.00 -> 23.9 mm, vias 0 -> 1
- net D3: track 0.00 -> 21.0 mm
- net D9: track 36.3 -> 17.9 mm
- net N$1: track 12.7 -> 29.2 mm, vias 2 -> 0
- net GND: track 215.0 -> 199.0 mm, vias 0 -> 1
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
Commit message: sula1
Parts:
- removed S1: (no value), switch:255SB
- removed S2, S3: SWITCH-MOMENTARY-2PTH, SparkFun-Electromechanical:TACTILE-PTH
- removed SV3: (no value), con-lsta:FE07
- added D4: (no value), SparkFun-DiscreteSemi:SMA-DIODE
- added GPI1, GPI2, GPI3, GPI4: SWITCH-MOMENTARY-2PTH, SparkFun-Electromechanical:TACTILE-PTH
- added PS: (no value), switch:255SB
- added Q2: 2N5551, semicon-smd-ipc:SOT23
- added R3: 1K, SparkFun-Passives:0805
- added R4, R5: 10k, SparkFun-Passives:0805
- added SV1: (no value), con-lsta:FE05-1
- Q3: value 2N3904 -> 2N5551
- moved R15 52.1 mm to (40.6, 48.3), turned to 180 degrees
- moved PH1 50.1 mm to (48.3, 48.3)
- moved MS 46.7 mm to (12.7, 48.3), turned to 0 degrees
- moved PUMP 45.0 mm to (20.3, 48.3), turned to 0 degrees
- moved R19 45.0 mm to (55.9, 48.3), turned to 0 degrees
- moved R18 41.0 mm to (43.2, 43.2)
- moved LED1 33.1 mm to (5.08, 15.2)
- moved R14 29.0 mm to (43.2, 33.0), turned to 270 degrees
- moved D1 26.5 mm to (12.7, 27.9)
- moved JP2 24.0 mm to (59.7, 25.4)
- moved JP6 24.0 mm to (62.2, 36.8)
- moved JP7 24.0 mm to (47.0, 8.89)
- moved C1 23.0 mm to (10.2, 12.7)
- moved R12 23.0 mm to (2.54, 10.2)
- moved R2 20.9 mm to (53.3, 27.9)
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Connections:
- new net N$7: Q2.1, R3.1
- new net N$8: D4.A, Q2.3, SV2.8
- net A3: now also SV1.1; no longer SV3.3
- net A4: now also SV1.2; no longer SV3.4
- net A5: now also SV1.3; no longer SV3.5
- net D10: now also R3.2; no longer R1.1
- net D2: now also GPI2.3; no longer S3.3
- net D4: now also GPI3.3, R4.2; no longer SV3.1
- net D5: now also GPI4.3, R5.2; no longer SV3.2
- net GND: now also Q2.2, R4.1, R5.1, SV1.5; no longer SV2.8, SV3.7
- net N$13: now also PS.1; no longer S1.1
- net N$2: now also PS.2; no longer S1.2
- net SCK: now also GPI1.3; no longer S2.3
- net VCC: now also D4.C, GPI1.1, GPI2.1, GPI3.1, GPI4.1, R1.1, SV1.4; no longer S2.1, S3.1, SV3.6
Routing:
- net GND: track 199.0 -> 250.0 mm
- net A0: track 26.2 -> 76.7 mm, vias 0 -> 2
- net A1: track 81.7 -> 36.5 mm
- net VCC: track 205.0 -> 248.1 mm, vias 0 -> 1
- net A3: track 72.9 -> 30.3 mm, vias 0 -> 1
- net D4: track 33.0 -> 72.4 mm, vias 0 -> 1
- net N$17: track 12.1 -> 51.3 mm
- net N$6: track 7.09 -> 33.2 mm, vias 0 -> 2
- net A5: track 53.8 -> 28.0 mm
- net SCK: track 53.1 -> 77.7 mm, vias 2 -> 1
- net N$1: track 29.2 -> 5.61 mm
- net A4: track 49.9 -> 27.3 mm
- net D5: track 37.9 -> 60.6 mm, vias 1 -> 2
- net N$5: track 17.4 -> 37.9 mm
- net D2: track 23.9 -> 44.3 mm, vias 1 -> 2
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Other:
- board size 48.3 x 61 mm -> 66 x 53.3 mm

Commit message: V1
Parts:
- added R6: THERMISTOR-2,5, varistor:RS-2,5
- added R7: 10K, SparkFun-Passives:0805
- SV1: device con-lsta:FE05-1 -> con-lstb:MA04-1
- moved SV1 2.54 mm to (55.9, 5.08)
Connections:
- removed net N$8: D4.A, Q2.3, SV2.8
- new net N$10: D4.A, Q2.3, R1.1, SV2.8
- net A3: now also R6.1; no longer SV1.1
- net A4: now also SV1.1; no longer SV1.2
- net A5: now also SV1.2; no longer SV1.3
- net GND: now also R7.2, SV1.4; no longer SV1.5
- net VCC: now also R6.2, SV1.3; no longer R1.1, SV1.4
Routing:
- net N$10: track 0.00 -> 29.8 mm
- net N$8: track 19.1 -> 0.00 mm
- net VCC: track 248.1 -> 266.1 mm, vias 1 -> 0
- net MISO: track 24.3 -> 13.1 mm, vias 0 -> 1
- net A3: track 30.3 -> 20.1 mm, vias 1 -> 0
- net D4: track 72.4 -> 62.4 mm
- net D5: track 60.6 -> 51.8 mm, vias 2 -> 3
- net A0: track 76.7 -> 71.1 mm
- net GND: track 250.0 -> 255.6 mm, vias 1 -> 3
- net D6: track 46.4 -> 51.2 mm
- net A4: track 27.3 -> 23.5 mm
- net D3: track 13.1 -> 9.61 mm
- net A5: track 28.0 -> 25.0 mm
- net N$3: track 21.6 -> 18.5 mm, vias 2 -> 1
- net N$6: track 33.2 -> 35.3 mm
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
Commit message: v1
Parts:
- removed R15, R6: THERMISTOR-2,5, varistor:RS-2,5
- added AIR: THERMISTOR-2,5, varistor:RS-2,5
- added SOIL: (no value), con-amp:10X02MTA
- LIGHT, MS, PUMP, PW: device con-amp:1X2MTA -> con-amp:10X02MTA
- moved MS 65.1 mm to (63.5, 7.62), turned to 270 degrees
- moved PW 62.9 mm to (48.3, 2.54), turned to 180 degrees
- moved R12 59.3 mm to (43.2, 53.3), turned to 270 degrees
- moved PS 58.0 mm to (58.4, 2.54), turned to 0 degrees
- moved LED1 57.6 mm to (43.2, 58.4), turned to 90 degrees
- moved PUMP 55.9 mm to (63.5, 12.7), turned to 270 degrees
- moved R4 47.9 mm to (33.0, 45.7), turned to 90 degrees
- moved LIGHT 46.8 mm to (63.5, 17.8), turned to 270 degrees
- moved C1 43.3 mm to (38.1, 45.7)
- moved R11 38.4 mm to (15.2, 25.4)
- moved R17 37.0 mm to (2.54, 12.7)
- moved R19 35.6 mm to (55.9, 12.7)
- moved GPI4 35.3 mm to (5.08, 53.3)
- moved D2 34.2 mm to (5.08, 43.2)
- moved R16 33.0 mm to (2.54, 17.8)
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Connections:
- net A1: now also SOIL.1; no longer R15.1
- net A3: now also AIR.1, R7.1; no longer R6.1
- net VCC: now also AIR.2, SOIL.2; no longer R15.2, R6.2
Routing:
- net N$13: track 8.60 -> 71.6 mm, vias 0 -> 2
- net N$19: track 18.8 -> 71.7 mm, vias 0 -> 3
- net N$5: track 37.9 -> 87.4 mm, vias 0 -> 2
- net A1: track 36.5 -> 83.5 mm, vias 0 -> 1
- net MOSI: track 44.3 -> 90.5 mm, vias 0 -> 1
- net N$17: track 50.6 -> 5.70 mm
- net D4: track 62.4 -> 23.2 mm
- net MISO: track 13.1 -> 49.7 mm, vias 1 -> 2
- net D6: track 51.2 -> 85.5 mm
- net D10: track 31.9 -> 63.6 mm, vias 1 -> 2
- net N$10: track 29.8 -> 60.3 mm
- net GND: track 255.6 -> 226.7 mm, vias 3 -> 1
- net A3: track 20.1 -> 47.0 mm, vias 0 -> 1
- net D3: track 9.61 -> 36.1 mm, vias 0 -> 1
- net N$6: track 35.3 -> 9.33 mm, vias 2 -> 0
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Other:
- board size 66 x 53.3 mm -> 66 x 61 mm

Commit message: v1
Parts:
- moved PUMP 3.59 mm to (66.0, 15.2)
- moved MS 3.59 mm to (66.0, 10.2)
- moved LIGHT 3.59 mm to (66.0, 20.3)
- moved R2 3.59 mm to (53.3, 48.3)
- moved R11 3.59 mm to (17.8, 27.9)
- moved GPI1 3.59 mm to (27.9, 55.9)
- moved Q1 3.59 mm to (27.9, 35.6)
- moved R13 3.59 mm to (27.9, 50.8)
- moved R14 3.59 mm to (25.4, 27.9)
- moved R17 3.59 mm to (5.08, 15.2)
- moved Q2 3.59 mm to (10.2, 10.2)
- moved AIR 3.59 mm to (50.8, 10.2)
- moved D2 3.59 mm to (7.62, 45.7)
- moved D3 3.59 mm to (10.2, 30.5)
- moved F1 3.59 mm to (15.2, 45.7)
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