File: RIO_V0/RIO_V0.brd (EAGLE design)
At the start: 71.1 x 100 mm, 2 parts

Commit message: sulav2
Parts:
- added BTCON: (no value), con-lstb:MA04-1
- added PW: 22-27-2021-02, con-molex:6410-02
- added S1CON, S2CON: (no value), con-lstb:MA03-1
- added SDCON: (no value), con-lstb:MA08-2
- added TMCON: (no value), con-lstb:MA05-1
Changed lines of the file:
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@@
 <element name="JP6" library="SparkFun" package="1X12" value="" x="6.35" y="19.05"/>
 <element name="JP7" library="SparkFun" package="1X12" value="" x="34.29" y="3.81" rot="R180"/>
+<element name="S1CON" library="con-lstb" package="MA03-1" value="" x="11.43" y="67.31">
+<attribute name="OC_NEWARK" value="unknown" x="11.43" y="67.31" size="1.778" layer="27" display="off"/>
+<attribute name="MPN" value="" x="11.43" y="67.31" size="1.778" layer="27" display="off"/>
+<attribute name="MF" value="" x="11.43" y="67.31" size="1.778" layer="27" display="off"/>
+<attribute name="OC_FARNELL" value="unknown" x="11.43" y="67.31" size="1.778" layer="27" display="off"/>
+</element>
+<element name="S2CON" library="con-lstb" package="MA03-1" value="" x="26.67" y="66.04">
+<attribute name="OC_NEWARK" value="unknown" x="26.67" y="66.04" size="1.778" layer="27" display="off"/>
+<attribute name="MPN" value="" x="26.67" y="66.04" size="1.778" layer="27" display="off"/>
+<attribute name="MF" value="" x="26.67" y="66.04" size="1.778" layer="27" display="off"/>
+<attribute name="OC_FARNELL" value="unknown" x="26.67" y="66.04" size="1.778" layer="27" display="off"/>
+</element>
+<element name="TMCON" library="con-lstb" package="MA05-1" value="" x="46.99" y="66.04">
+<attribute name="OC_NEWARK" value="unknown" x="46.99" y="66.04" size="1.778" layer="27" display="off"/>
+<attribute name="MPN" value="" x="46.99" y="66.04" size="1.778" layer="27" display="off"/>
+<attribute name="MF" value="" x="46.99" y="66.04" size="1.778" layer="27" display="off"/>
+<attribute name="OC_FARNELL" value="unknown" x="46.99" y="66.04" size="1.778" layer="27" display="off"/>
+</element>
+<element name="SDCON" library="con-lstb" package="MA08-2" value="" x="20.32" y="41.91">
+<attribute name="OC_NEWARK" value="unknown" x="20.32" y="41.91" size="1.778" layer="27" display="off"/>
+<attribute name="MPN" value="" x="20.32" y="41.91" size="1.778" layer="27" display="off"/>
+<attribute name="MF" value="" x="20.32" y="41.91" size="1.778" layer="27" display="off"/>
+<attribute name="OC_FARNELL" value="unknown" x="20.32" y="41.91" size="1.778" layer="27" display="off"/>
+</element>
+<element name="BTCON" library="con-lstb" package="MA04-1" value="" x="45.72" y="34.29">
+<attribute name="OC_NEWARK" value="unknown" x="45.72" y="34.29" size="1.778" layer="27" display="off"/>
+<attribute name="MPN" value="" x="45.72" y="34.29" size="1.778" layer="27" display="off"/>
+<attribute name="MF" value="" x="45.72" y="34.29" size="1.778" layer="27" display="off"/>
+<attribute name="OC_FARNELL" value="unknown" x="45.72" y="34.29" size="1.778" layer="27" display="off"/>
+</element>
+<element name="PW" library="con-molex" package="6410-02" value="22-27-2021-02" x="59.69" y="7.62">
+<attribute name="OC_NEWARK" value="unknown" x="59.69" y="7.62" size="1.778" layer="27" display="off"/>
+<attribute name="MPN" value="" x="59.69" y="7.62" size="1.778" layer="27" display="off"/>
+<attribute name="MF" value="" x="59.69" y="7.62" size="1.778" layer="27" display="off"/>
+<attribute name="OC_FARNELL" value="unknown" x="59.69" y="7.62" size="1.778" layer="27" display="off"/>
+</element>
 </elements>
 <signals>
