File: RIO_V0/RIO_V0.sch (EAGLE design)
At the start: 2 parts

Commit message: sulav2
Parts:
- added BTCON: (no value), con-lstb:MA04-1
- added PW: 22-27-2021-02, con-molex:22-27-2021-02
- added S1CON, S2CON: (no value), con-lstb:MA03-1
- added SDCON: (no value), con-lstb:MA08-2
- added TMCON: (no value), con-lstb:MA05-1
Changed lines of the file:
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@@
 <part name="JP6" library="SparkFun" deviceset="M12" device="PTH" value=""/>
 <part name="JP7" library="SparkFun" deviceset="M12" device="PTH" value=""/>
+<part name="S1CON" library="con-lstb" deviceset="MA03-1" device=""/>
+<part name="S2CON" library="con-lstb" deviceset="MA03-1" device=""/>
+<part name="TMCON" library="con-lstb" deviceset="MA05-1" device=""/>
+<part name="SDCON" library="con-lstb" deviceset="MA08-2" device=""/>
+<part name="BTCON" library="con-lstb" deviceset="MA04-1" device=""/>
+<part name="PW" library="con-molex" deviceset="22-?-02" device="27-2021"/>
 </parts>
 <sheets>
@@
 <instance part="JP6" gate="G$1" x="55.88" y="33.02" rot="R180"/>
 <instance part="JP7" gate="G$1" x="12.7" y="35.56"/>
+<instance part="S1CON" gate="G$1" x="86.36" y="71.12"/>
+<instance part="S2CON" gate="G$1" x="86.36" y="55.88"/>
+<instance part="TMCON" gate="G$1" x="86.36" y="27.94"/>
+<instance part="SDCON" gate="G$1" x="91.44" y="-5.08"/>
+<instance part="BTCON" gate="1" x="109.22" y="43.18"/>
+<instance part="PW" gate="-1" x="88.9" y="101.6"/>
+<instance part="PW" gate="-2" x="88.9" y="96.52"/>
 </instances>
 <busses>
