File: SulaMatikV2/SulaMatikV2.sch (EAGLE design)
At the start: 39 parts, among them IC1 REG1117, Q1 2N3904, Q2 2N5551, Q3 2N5551

Commit message: v2
Parts:
- removed GPI3, GPI4: SWITCH-MOMENTARY-2PTH, SparkFun-Electromechanical:SWITCH-MOMENTARY-2PTH
- removed R19: 10K, pot:TRIM_US-CA6V
- removed R4, R5: 10k, SparkFun-Passives:RESISTOR0805-RES
- removed SV2: (no value), con-lsta:FE08-1
- added BT: (no value), con-lstb:MA04-1
- added LED2: (no value), led:LEDCHIP-LED0805
- added RTC: (no value), con-lsta:FE05-1
Connections:
- new net N$12: RTC.2
- new net N$14: RTC.1
- new net N$15: BT.4
- new net N$16: BT.3
- new net N$21: BT.1
- new net N$22: LED2.A, R1.1
- new net N$8: RTC.4
- new net SGND: D4.A, LED2.C, Q2.C, R16.2, R17.2, R18.2, R7.2
- net D4: no longer GPI3.2, R4.2
- net D5: no longer GPI4.2, R5.2
- net D6: no longer SV2.1
- net D7: no longer SV2.2
- net D8: no longer SV2.3
- net D9: no longer SV2.4
- net GND: no longer R16.2, R17.2, R18.2, R4.1, R5.1, R7.2
- net MOSI: no longer SV2.5
- net N$10: now also RTC.3; no longer D4.A, Q2.C, R1.1, SV2.8
- net N$17: now also BT.2; no longer MS.2, R19.E
- net N$3: now also RTC.5; no longer R1.2, SV2.7
- net VCC: now also MS.2, R1.2; no longer GPI3.1, GPI4.1, R19.S, SV2.6
Other:
- note added: "Sensor EN (GND for Sensors)"
- note removed: "Display"
- note removed: "GPI3"
- note removed: "GPI4"
- note removed: "Sensor EN"
- moved on the sheet: AIR, D2, D3, D4, JP2, JP6, JP7, LIGHT, MS, PH1, PUMP, Q1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

Commit message: v2
Parts:
- added R2: 1K, SparkFun-Passives:RESISTOR0805-RES
- added R4: 2.2K, SparkFun-Passives:RESISTOR0805-RES
- added R5, R6: 1.8K, SparkFun-Passives:RESISTOR0805-RES
- added R8, R9: 3.3K, SparkFun-Passives:RESISTOR0805-RES
- added SD: (no value), con-lsta:FE08-2
Connections:
- removed net N$10: RTC.3
- removed net N$12: RTC.2
- removed net N$14: RTC.1
- removed net N$15: BT.4
- removed net N$16: BT.3
- removed net N$17: BT.2
- removed net N$21: BT.1
- removed net N$3: RTC.5
- removed net N$8: RTC.4
- new net N$29: SD.3, SD.4
- new net SDCS: R6.2, R8.1, SD.7, SD.8
- new net SDMO: R5.2, R9.1, SD.10, SD.9
- new net SDSCK: R2.2, R4.1, SD.11, SD.12
- net D2: now also BT.1
- net D3: now also BT.2; no longer R14.2
- net D4: now also R6.1
- net D5: now also R14.2
- net D6: now also RTC.3
- net D7: now also RTC.2
- net D8: now also RTC.1
- net D9: now also R11.2
- net GND: now also BT.3, R4.2, R8.2, R9.2, RTC.4, SD.1, SD.15, SD.16, SD.2
- net MISO: now also SD.13, SD.14; no longer R11.2
- net MOSI: now also R5.1
- net SCK: now also R2.1
- net VCC: now also BT.4, RTC.5, SD.5, SD.6
Other:
- note added: "Battery SENSOR(A4)"
- note added: "BlueTooth"
- note added: "CLOCK"
- note added: "SD CARD"
- moved on the sheet: BT, RTC

Commit message: battry buzzer eksik
Parts:
- removed AIR: THERMISTOR-2,5, varistor:THERMISTOR-2,5
- removed LIGHT, PUMP: (no value), con-amp:MTA02-100
- removed R7: 10K, SparkFun-Passives:RESISTOR0805-RES
- removed SV1: (no value), con-lstb:MA04-1
- added DHT, EX, LRV1, PRV, SV2: (no value), con-lstb:MA03-1
- added K1: CQ1-12V, relay:CQ1-12V
- BT: device con-lstb:MA04-1 -> con-lsta:FE06-1
- F1: value 1.5A -> 1A
- MS, PW, SOIL: device con-amp:MTA02-100 -> SparkFun:M02PTH
Connections:
- new net N$10: K12.P, LRV1.2
- new net N$12: K12.O, LRV1.1
- new net N$3: D2.C, PRV.2, PRV.3
- new net N$8: K12.S, LRV1.3
- net A0: now also MS.2; no longer MS.1
- net A1: now also SOIL.2; no longer SOIL.1
- net A3: now also DHT.2; no longer AIR.1, R7.1
- net A4: no longer SV1.1
- net A5: now also EX.1; no longer SV1.2
- net D2: now also BT.2; no longer BT.1
- net D3: now also BT.3; no longer BT.2
- net GND: now also BT.4, EX.3; no longer BT.3, SV1.4
- net N$19: now also K11.1; no longer LIGHT.2
- net N$5: now also PRV.1; no longer PUMP.2
- net SGND: now also DHT.1; no longer R7.2
- net VCC: now also BT.5, DHT.3, EX.2, K11.2, MS.1, SOIL.1; no longer AIR.2, BT.4, D2.C, LIGHT.1, MS.2, PUMP.1, SOIL.2, SV1.3
Other:
- note added: "gnd"
- note added: "vin"
- note added: "vout"
- moved on the sheet: D2, Q3, R11, RTC

Commit message: tamam
Parts:
- removed SV2: (no value), con-lstb:MA03-1
- added R10: 14K, SparkFun-Passives:RESISTOR0805-RES
- added R7: 20K, SparkFun-Passives:RESISTOR0805-RES
- renumbered EX to BZZ
Connections:
- net A4: now also R10.2, R7.1
- net SGND: now also R10.1
- net VCC9V: now also R7.2
Other:
- note added: "BUZZER"
Changed lines of the file:
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@@
 <part name="BT" library="con-lsta" deviceset="FE06-1" device=""/>
 <part name="DHT" library="con-lstb" deviceset="MA03-1" device=""/>
-<part name="SV2" library="con-lstb" deviceset="MA03-1" device=""/>
 <part name="SOIL" library="SparkFun" deviceset="M02" device="PTH"/>
 <part name="PW" library="SparkFun" deviceset="M02" device="PTH"/>
 <part name="MS" library="SparkFun" deviceset="M02" device="PTH"/>
-<part name="EX" library="con-lstb" deviceset="MA03-1" device=""/>
+<part name="BZZ" library="con-lstb" deviceset="MA03-1" device=""/>
 <part name="PRV" library="con-lstb" deviceset="MA03-1" device=""/>
 <part name="K1" library="relay" deviceset="CQ1-12V" device=""/>
 <part name="LRV1" library="con-lstb" deviceset="MA03-1" device=""/>
+<part name="R7" library="SparkFun-Passives" deviceset="RESISTOR" device="0805-RES" value="20K"/>
+<part name="R10" library="SparkFun-Passives" deviceset="RESISTOR" device="0805-RES" value="14K"/>
 </parts>
 <sheets>
@@
 <text x="99.06" y="109.22" size="1.778" layer="91" rot="R90">vout</text>
 <text x="96.52" y="109.22" size="1.778" layer="91" rot="R90">gnd</text>
+<text x="55.88" y="43.18" size="1.778" layer="91">BUZZER</text>
 </plain>
 <instances>
@@
 <instance part="BT" gate="G$1" x="55.88" y="55.88"/>
 <instance part="DHT" gate="G$1" x="7.62" y="60.96"/>
-<instance part="SV2" gate="G$1" x="81.28" y="10.16"/>
 <instance part="SOIL" gate="G$1" x="15.24" y="81.28"/>
 <instance part="PW" gate="G$1" x="144.78" y="154.94"/>
 <instance part="MS" gate="G$1" x="15.24" y="106.68"/>
-<instance part="EX" gate="G$1" x="55.88" y="33.02"/>
+<instance part="BZZ" gate="G$1" x="55.88" y="33.02"/>
 <instance part="PRV" gate="G$1" x="99.06" y="106.68" rot="R270"/>
 <instance part="K1" gate="1" x="91.44" y="152.4" rot="R90"/>
 <instance part="K1" gate="2" x="76.2" y="119.38" rot="R270"/>
 <instance part="LRV1" gate="G$1" x="58.42" y="119.38"/>
+<instance part="R7" gate="G$1" x="139.7" y="127" rot="R180"/>
+<instance part="R10" gate="G$1" x="157.48" y="127" rot="R180"/>
 </instances>
 <busses>
@@
 <label x="73.66" y="35.56" size="1.778" layer="95" xref="yes"/>
 <wire x1="63.5" y1="35.56" x2="73.66" y2="35.56" width="0.1524" layer="91"/>
-<pinref part="EX" gate="G$1" pin="3"/>
+<pinref part="BZZ" gate="G$1" pin="3"/>
 </segment>
 <segment>
@@
 <label x="81.28" y="33.02" size="1.778" layer="95" xref="yes"/>
 <wire x1="63.5" y1="33.02" x2="81.28" y2="33.02" width="0.1524" layer="91"/>
-<pinref part="EX" gate="G$1" pin="2"/>
+<pinref part="BZZ" gate="G$1" pin="2"/>
 </segment>
 <segment>
@@
 <label x="73.66" y="30.48" size="1.778" layer="95" xref="yes"/>
 <wire x1="63.5" y1="30.48" x2="73.66" y2="30.48" width="0.1524" layer="91"/>
-<pinref part="EX" gate="G$1" pin="1"/>
+<pinref part="BZZ" gate="G$1" pin="1"/>
 </segment>
 </net>
@@
 <label x="55.88" y="12.7" size="1.778" layer="95"/>
 <pinref part="JP2" gate="G$1" pin="1"/>
+</segment>
+<segment>
+<pinref part="R7" gate="G$1" pin="1"/>
+<pinref part="R10" gate="G$1" pin="2"/>
+<wire x1="144.78" y1="127" x2="147.32" y2="127" width="0.1524" layer="91"/>
+<wire x1="152.4" y1="127" x2="147.32" y2="127" width="0.1524" layer="91"/>
+<wire x1="147.32" y1="127" x2="147.32" y2="134.62" width="0.1524" layer="91"/>
+<wire x1="147.32" y1="134.62" x2="167.64" y2="134.62" width="0.1524" layer="91"/>
+<label x="167.64" y="134.62" size="1.778" layer="95" xref="yes"/>
 </segment>
 </net>
@@
 <wire x1="175.26" y1="167.64" x2="177.8" y2="167.64" width="0.1524" layer="91"/>
 <pinref part="F1" gate="G$1" pin="1"/>
+</segment>
+<segment>
+<pinref part="R7" gate="G$1" pin="2"/>
+<wire x1="132.08" y1="127" x2="134.62" y2="127" width="0.1524" layer="91"/>
+<label x="132.08" y="127" size="1.778" layer="95" rot="R180" xref="yes"/>
 </segment>
 </net>
@@
 <label x="17.78" y="58.42" size="1.778" layer="95" xref="yes"/>
 </segment>
-</net>
+<segment>
+<pinref part="R10" gate="G$1" pin="1"/>
+<wire x1="162.56" y1="127" x2="167.64" y2="127" width="0.1524" layer="91"/>
+<label x="167.64" y="127" size="1.778" layer="95" xref="yes"/>
+</segment>
+</net>

Commit message: almost v2
Parts:
- removed K1: CQ1-12V, relay:CQ1-12V
- removed LRV1: (no value), con-lstb:MA03-1
- added LRV: (no value), SparkFun:M02PTH
- PRV: device con-lstb:MA03-1 -> con-lsta:FE05-1
- R10: value 14K -> 22K
- R7: value 20K -> 47K
Connections:
- removed net N$10: K12.P, LRV1.2
- removed net N$12: K12.O, LRV1.1
- removed net N$8: K12.S, LRV1.3
- net GND: now also PRV.1
- net N$19: now also LRV.1; no longer K11.1
- net N$3: now also PRV.4; no longer PRV.2
- net N$5: now also PRV.2; no longer PRV.1
- net VCC: now also LRV.2, PRV.5; no longer K11.2
Changed lines of the file:
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@@
 <part name="MS" library="SparkFun" deviceset="M02" device="PTH"/>
 <part name="BZZ" library="con-lstb" deviceset="MA03-1" device=""/>
-<part name="PRV" library="con-lstb" deviceset="MA03-1" device=""/>
-<part name="K1" library="relay" deviceset="CQ1-12V" device=""/>
-<part name="LRV1" library="con-lstb" deviceset="MA03-1" device=""/>
-<part name="R7" library="SparkFun-Passives" deviceset="RESISTOR" device="0805-RES" value="20K"/>
-<part name="R10" library="SparkFun-Passives" deviceset="RESISTOR" device="0805-RES" value="14K"/>
+<part name="R7" library="SparkFun-Passives" deviceset="RESISTOR" device="0805-RES" value="47K"/>
+<part name="R10" library="SparkFun-Passives" deviceset="RESISTOR" device="0805-RES" value="22K"/>
+<part name="PRV" library="con-lsta" deviceset="FE05-1" device=""/>
+<part name="GND3" library="supply1" deviceset="GND" device=""/>
+<part name="LRV" library="SparkFun" deviceset="M02" device="PTH"/>
 </parts>
 <sheets>
@@
 <instance part="MS" gate="G$1" x="15.24" y="106.68"/>
 <instance part="BZZ" gate="G$1" x="55.88" y="33.02"/>
-<instance part="PRV" gate="G$1" x="99.06" y="106.68" rot="R270"/>
-<instance part="K1" gate="1" x="91.44" y="152.4" rot="R90"/>
-<instance part="K1" gate="2" x="76.2" y="119.38" rot="R270"/>
-<instance part="LRV1" gate="G$1" x="58.42" y="119.38"/>
 <instance part="R7" gate="G$1" x="139.7" y="127" rot="R180"/>
 <instance part="R10" gate="G$1" x="157.48" y="127" rot="R180"/>
+<instance part="PRV" gate="G$1" x="99.06" y="106.68" rot="R270"/>
+<instance part="GND3" gate="1" x="86.36" y="99.06" rot="R270"/>
+<instance part="LRV" gate="G$1" x="91.44" y="152.4" rot="R270"/>
 </instances>
 <busses>
@@
 <wire x1="63.5" y1="58.42" x2="81.28" y2="58.42" width="0.1524" layer="91"/>
 </segment>
+<segment>
+<pinref part="PRV" gate="G$1" pin="1"/>
+<wire x1="93.98" y1="99.06" x2="88.9" y2="99.06" width="0.1524" layer="91"/>
+<pinref part="GND3" gate="1" pin="GND"/>
+</segment>
 </net>
 <net name="RESET" class="0">
@@
 <wire x1="96.52" y1="142.24" x2="93.98" y2="142.24" width="0.1524" layer="91"/>
 <junction x="96.52" y="142.24"/>
+<pinref part="LRV" gate="G$1" pin="2"/>
 <wire x1="93.98" y1="142.24" x2="93.98" y2="144.78" width="0.1524" layer="91"/>
-<pinref part="K1" gate="1" pin="2"/>
-<wire x1="93.98" y1="144.78" x2="96.52" y2="144.78" width="0.1524" layer="91"/>
-<wire x1="96.52" y1="144.78" x2="96.52" y2="152.4" width="0.1524" layer="91"/>
 </segment>
 <segment>
@@
 <wire x1="15.24" y1="63.5" x2="17.78" y2="63.5" width="0.1524" layer="91"/>
 <label x="17.78" y="63.5" size="1.778" layer="95" xref="yes"/>
+</segment>
+<segment>
+<pinref part="PRV" gate="G$1" pin="5"/>
+<wire x1="104.14" y1="99.06" x2="104.14" y2="96.52" width="0.1524" layer="91"/>
+<wire x1="104.14" y1="96.52" x2="106.68" y2="96.52" width="0.1524" layer="91"/>
+<label x="106.68" y="96.52" size="1.778" layer="95" xref="yes"/>
 </segment>
 </net>
@@
 <wire x1="91.44" y1="96.52" x2="96.52" y2="96.52" width="0.1524" layer="91"/>
 <junction x="91.44" y="96.52"/>
-<pinref part="PRV" gate="G$1" pin="1"/>
 <wire x1="96.52" y1="96.52" x2="96.52" y2="99.06" width="0.1524" layer="91"/>
+<pinref part="PRV" gate="G$1" pin="2"/>
 </segment>
 </net>
@@
 <wire x1="86.36" y1="142.24" x2="91.44" y2="142.24" width="0.1524" layer="91"/>
 <junction x="86.36" y="142.24"/>
+<pinref part="LRV" gate="G$1" pin="1"/>
 <wire x1="91.44" y1="142.24" x2="91.44" y2="144.78" width="0.1524" layer="91"/>
-<pinref part="K1" gate="1" pin="1"/>
-<wire x1="91.44" y1="144.78" x2="86.36" y2="144.78" width="0.1524" layer="91"/>
-<wire x1="86.36" y1="144.78" x2="86.36" y2="152.4" width="0.1524" layer="91"/>
 </segment>
 </net>
@@
 <pinref part="D2" gate="G$1" pin="C"/>
 <wire x1="99.06" y1="88.9" x2="101.6" y2="88.9" width="0.1524" layer="91"/>
-<pinref part="PRV" gate="G$1" pin="2"/>
 <wire x1="99.06" y1="99.06" x2="99.06" y2="96.52" width="0.1524" layer="91"/>
 <wire x1="99.06" y1="96.52" x2="101.6" y2="96.52" width="0.1524" layer="91"/>
 <wire x1="101.6" y1="96.52" x2="101.6" y2="88.9" width="0.1524" layer="91"/>
+<wire x1="101.6" y1="99.06" x2="101.6" y2="96.52" width="0.1524" layer="91"/>
 <pinref part="PRV" gate="G$1" pin="3"/>
-<wire x1="101.6" y1="99.06" x2="101.6" y2="96.52" width="0.1524" layer="91"/>
-</segment>
-</net>
-<net name="N$8" class="0">
-<segment>
-<pinref part="LRV1" gate="G$1" pin="3"/>
-<wire x1="66.04" y1="121.92" x2="76.2" y2="121.92" width="0.1524" layer="91"/>
-<wire x1="76.2" y1="121.92" x2="76.2" y2="124.46" width="0.1524" layer="91"/>
-<pinref part="K1" gate="2" pin="S"/>
-<wire x1="76.2" y1="124.46" x2="81.28" y2="124.46" width="0.1524" layer="91"/>
-</segment>
-</net>
-<net name="N$10" class="0">
-<segment>
-<pinref part="LRV1" gate="G$1" pin="2"/>
-<pinref part="K1" gate="2" pin="P"/>
-<wire x1="66.04" y1="119.38" x2="73.66" y2="119.38" width="0.1524" layer="91"/>
-</segment>
-</net>
-<net name="N$12" class="0">
-<segment>
-<pinref part="LRV1" gate="G$1" pin="1"/>
-<wire x1="66.04" y1="116.84" x2="76.2" y2="116.84" width="0.1524" layer="91"/>
-<wire x1="76.2" y1="116.84" x2="76.2" y2="111.76" width="0.1524" layer="91"/>
-<pinref part="K1" gate="2" pin="O"/>
-<wire x1="76.2" y1="111.76" x2="81.28" y2="111.76" width="0.1524" layer="91"/>
-<wire x1="81.28" y1="111.76" x2="81.28" y2="114.3" width="0.1524" layer="91"/>
-</segment>
-</net>
+<pinref part="PRV" gate="G$1" pin="4"/>
+</segment>
+</net>

Commit message: sync
Connections:
- net GND: now also R10.1
- net SGND: no longer R10.1
Changed lines of the file:
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@@
 <pinref part="GND3" gate="1" pin="GND"/>
+</segment>
+<segment>
+<pinref part="R10" gate="G$1" pin="1"/>
+<wire x1="162.56" y1="127" x2="167.64" y2="127" width="0.1524" layer="91"/>
+<label x="167.64" y="127" size="1.778" layer="95" xref="yes"/>
 </segment>
 </net>
@@
 <label x="17.78" y="58.42" size="1.778" layer="95" xref="yes"/>
 </segment>
-<segment>
-<pinref part="R10" gate="G$1" pin="1"/>
-<wire x1="162.56" y1="127" x2="167.64" y2="127" width="0.1524" layer="91"/>
-<label x="167.64" y="127" size="1.778" layer="95" xref="yes"/>
-</segment>
-</net>
+</net>

Commit message: sav
Parts:
- added PRV1: (no value), SparkFun-Connectors:M03PTH
- added PRVIN: (no value), SparkFun:M02PTH
- BZZ, DHT: device con-lstb:MA03-1 -> SparkFun-Connectors:M03PTH
- PRV: device con-lsta:FE05-1 -> SparkFun-Connectors:M03PTH
- PS: device switch:255SB -> SparkFun-Connectors:M03PTH
Connections:
- net GND: now also PRV1.3
- net N$13: now also PS.1; no longer PS.O
- net N$2: now also PS.2; no longer PS.P
- net N$3: now also PRVIN.1; no longer PRV.4
- net VCC: now also PRV1.2, PRVIN.2; no longer PRV.5
- net VCC9V: now also PRV1.1
Other:
- moved on the sheet: BZZ, DHT
