File: SulaMatikV3/sulamatikV3.sch (EAGLE design)
At the start: 0 parts

Commit message: v3
Parts:
- added BT: (no value), con-lsta:FE06-1
- added BZZ, PS: (no value), SparkFun-Connectors:M03PTH
- added C1: 10uf, SparkFun-Capacitors:CAP0805
- added C2: 100uf, SparkFun-Capacitors:CAP0805
- added D1, D2: (no value), SparkFun-DiscreteSemi:DIODESMA
- added F1: 1A, _hhn_PtcFuses_Siba_r500_Ozan:SIBA194600
- added GPI3: SWITCH-MOMENTARY-2PTH, SparkFun-Electromechanical:SWITCH-MOMENTARY-2PTH
- added IC1: REG1117, burr-brown:REG1117
- added IC2: 74HC138N, 74xx-eu:74HC138N
- added JP6, JP7: M12PTH, SparkFun:M12PTH
- added LED1: (no value), led:LEDCHIP-LED0805
- added MS, PRVIN, PW: (no value), SparkFun:M02PTH
- added Q3: 2N5551, semicon-smd-ipc:NPN-TRANSISTOR_SOT23
- added R10: 22K, SparkFun-Passives:RESISTOR0805-RES
- added R11, R2: 1K, SparkFun-Passives:RESISTOR0805-RES
- added R12: 220, SparkFun-Passives:RESISTOR0805-RES
- added R17: 10K, SparkFun-Passives:RESISTOR0805-RES
- added R4: 2.2K, SparkFun-Passives:RESISTOR0805-RES
- added R5, R6: 1.8K, SparkFun-Passives:RESISTOR0805-RES
- added R7: 47K, SparkFun-Passives:RESISTOR0805-RES
- added R8, R9: 3.3K, SparkFun-Passives:RESISTOR0805-RES
- added RTC: (no value), con-lsta:FE05-1
- added SD: (no value), con-lsta:FE08-2
Connections:
- new net A0: JP6.8, MS.2, R17.1
- new net A1: JP6.7
- new net A2: JP6.6
- new net A3: JP6.5
- new net A4: R10.2, R7.1
- new net A5: BZZ.1
- new net D10: JP6.12
- new net D2: BT.2, JP7.8
- new net D3: BT.3, JP7.7
- new net D4: JP7.6, R6.1
- new net D5: JP7.5
- new net D6: JP7.4, RTC.3
- new net D7: JP7.3, RTC.2
- new net D8: JP7.2, RTC.1
- new net D9: JP7.1, R11.2
- new net GND: BT.4, BZZ.3, C1.1, C2.1, IC1.GND, JP6.2, JP7.9, LED1.C, PW.1, Q3.E, R10.1, R17.2, R4.2, R8.2, R9.2, RTC.4, SD.1, SD.15, SD.16, SD.2
- new net MISO: JP6.10, SD.13, SD.14
- new net MOSI: JP6.11, R5.1
- new net N$1: F1.2, IC1.VIN
- new net N$11: LED1.A, R12.1
- new net N$13: D1.A, PS.1
- new net N$2: PS.2, PW.2
- new net N$29: SD.3, SD.4
- new net N$5: D2.A, PRVIN.1, Q3.C
- new net N$6: Q3.B, R11.1
- new net RAW: JP6.1
- new net RESET: JP6.3, JP7.10
- new net RXI: JP7.11
- new net SCK: JP6.9, R2.1
- new net SDCS: R6.2, R8.1, SD.7, SD.8
- new net SDMO: R5.2, R9.1, SD.10, SD.9
- new net SDSCK: R2.2, R4.1, SD.11, SD.12
- new net TXO: JP7.12
- new net VCC: BT.5, BZZ.2, C1.2, D2.C, IC1.VOUT, JP6.4, MS.1, PRVIN.2, R12.2, RTC.5, SD.5, SD.6
- new net VCC9V: C2.2, D1.C, F1.1, R7.2
Other:
- note added: "BUZZER"
- note added: "Battery SENSOR(A4)"
- note added: "BlueTooth"
- note added: "CLOCK"
- note added: "MOISTURE SENSOR"
- note added: "POWER"
- note added: "PUMP"
- note added: "Pro Mini Stamp Socket"
- note added: "SD CARD"
