File: SulaMatikV3/sulamatikV3.sch (EAGLE design)
At the start: 31 parts, among them IC1 REG1117, IC2 74HC138N, Q3 2N5551

Commit message: v3
Parts:
- removed BZZ: (no value), SparkFun-Connectors:M03PTH
- removed PRVIN: (no value), SparkFun:M02PTH
- removed R10: 22K, SparkFun-Passives:RESISTOR0805-RES
- removed R7: 47K, SparkFun-Passives:RESISTOR0805-RES
- added PUMP: (no value), SparkFun:M02PTH
- added SRV: (no value), con-lstb:MA03-1
- MS: device SparkFun:M02PTH -> con-lsta:FE08-2
Connections:
- removed net A4: R10.2, R7.1
- removed net A5: BZZ.1
- removed net VCC9V: C2.2, D1.C, F1.1, R7.2
- new net VCCSRV: C1.2, D2.C, IC1.VOUT, PUMP.2, R12.2, SRV.2
- net A0: now also MS.10, MS.12, MS.14, MS.16, MS.4, MS.6, MS.8
- net GND: now also IC2A.G2A, IC2A.G2B, SRV.1; no longer BZZ.3, R10.1
- net N$5: now also PUMP.1; no longer PRVIN.1
- net RAW: now also C2.2, D1.C, F1.1
- net VCC: now also IC2A.G1; no longer BZZ.2, C1.2, D2.C, IC1.VOUT, MS.1, PRVIN.2, R12.2
Other:
- note removed: "BUZZER"
- note removed: "Battery SENSOR(A4)"
- moved on the sheet: D2, GPI3, Q3, R11, R17, R2, R4, R5, R6, R8, R9, SD

Commit message: v3
Connections:
- new net N$10: IC2A.Y3, MS.9
- new net N$12: IC2A.Y4, MS.7
- new net N$14: IC2A.Y5, MS.5
- new net N$15: IC2A.Y6, MS.3
- new net N$16: IC2A.Y7, MS.1
- new net N$3: IC2A.Y0, MS.15
- new net N$7: IC2A.Y1, MS.13
- new net N$8: IC2A.Y2, MS.11
- net A1: now also IC2A.C
- net A2: now also IC2A.B
- net A3: now also IC2A.A
- net D5: now also SRV.3
Changed lines of the file:
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@@
 <pinref part="JP6" gate="G$1" pin="5"/>
+</segment>
+<segment>
+<pinref part="IC2" gate="A" pin="A"/>
+<wire x1="106.68" y1="101.6" x2="104.14" y2="101.6" width="0.1524" layer="91"/>
+<label x="104.14" y="101.6" size="1.778" layer="95" rot="R180" xref="yes"/>
 </segment>
 </net>
@@
 <pinref part="JP6" gate="G$1" pin="6"/>
 </segment>
+<segment>
+<pinref part="IC2" gate="A" pin="B"/>
+<wire x1="106.68" y1="99.06" x2="96.52" y2="99.06" width="0.1524" layer="91"/>
+<label x="96.52" y="99.06" size="1.778" layer="95" rot="R180" xref="yes"/>
+</segment>
 </net>
 <net name="A1" class="0">
@@
 <label x="27.94" y="20.32" size="1.778" layer="95"/>
 <pinref part="JP6" gate="G$1" pin="7"/>
+</segment>
+<segment>
+<pinref part="IC2" gate="A" pin="C"/>
+<wire x1="106.68" y1="96.52" x2="104.14" y2="96.52" width="0.1524" layer="91"/>
+<label x="104.14" y="96.52" size="1.778" layer="95" rot="R180" xref="yes"/>
 </segment>
 </net>
@@
 <pinref part="JP7" gate="G$1" pin="5"/>
 </segment>
+<segment>
+<pinref part="SRV" gate="G$1" pin="3"/>
+<wire x1="17.78" y1="106.68" x2="20.32" y2="106.68" width="0.1524" layer="91"/>
+<label x="20.32" y="106.68" size="1.778" layer="95" xref="yes"/>
+</segment>
 </net>
 <net name="D6" class="0">
@@
 </segment>
 </net>
+<net name="N$3" class="0">
+<segment>
+<pinref part="IC2" gate="A" pin="Y0"/>
+<pinref part="MS" gate="G$1" pin="15"/>
+<wire x1="134.62" y1="101.6" x2="149.86" y2="101.6" width="0.1524" layer="91"/>
+</segment>
+</net>
+<net name="N$7" class="0">
+<segment>
+<pinref part="IC2" gate="A" pin="Y1"/>
+<pinref part="MS" gate="G$1" pin="13"/>
+<wire x1="134.62" y1="99.06" x2="149.86" y2="99.06" width="0.1524" layer="91"/>
+</segment>
+</net>
+<net name="N$8" class="0">
+<segment>
+<pinref part="IC2" gate="A" pin="Y2"/>
+<pinref part="MS" gate="G$1" pin="11"/>
+<wire x1="134.62" y1="96.52" x2="149.86" y2="96.52" width="0.1524" layer="91"/>
+</segment>
+</net>
+<net name="N$10" class="0">
+<segment>
+<pinref part="IC2" gate="A" pin="Y3"/>
+<pinref part="MS" gate="G$1" pin="9"/>
+<wire x1="134.62" y1="93.98" x2="149.86" y2="93.98" width="0.1524" layer="91"/>
+</segment>
+</net>
+<net name="N$12" class="0">
+<segment>
+<pinref part="IC2" gate="A" pin="Y4"/>
+<pinref part="MS" gate="G$1" pin="7"/>
+<wire x1="134.62" y1="91.44" x2="149.86" y2="91.44" width="0.1524" layer="91"/>
+</segment>
+</net>
+<net name="N$14" class="0">
+<segment>
+<pinref part="IC2" gate="A" pin="Y5"/>
+<pinref part="MS" gate="G$1" pin="5"/>
+<wire x1="134.62" y1="88.9" x2="149.86" y2="88.9" width="0.1524" layer="91"/>
+</segment>
+</net>
+<net name="N$15" class="0">
+<segment>
+<pinref part="IC2" gate="A" pin="Y6"/>
+<pinref part="MS" gate="G$1" pin="3"/>
+<wire x1="134.62" y1="86.36" x2="149.86" y2="86.36" width="0.1524" layer="91"/>
+</segment>
+</net>
+<net name="N$16" class="0">
+<segment>
+<pinref part="IC2" gate="A" pin="Y7"/>
+<pinref part="MS" gate="G$1" pin="1"/>
+<wire x1="134.62" y1="83.82" x2="149.86" y2="83.82" width="0.1524" layer="91"/>
+</segment>
+</net>

Commit message: v3
Parts:
- removed GPI3: SWITCH-MOMENTARY-2PTH, SparkFun-Electromechanical:SWITCH-MOMENTARY-2PTH
- added GPI1: SWITCH-MOMENTARY-2PTH, SparkFun-Electromechanical:SWITCH-MOMENTARY-2PTH
- added R1: 10K, SparkFun-Passives:RESISTOR0805-RES
Connections:
- net D10: now also GPI1.2, R1.2
- net GND: now also R1.1
- net VCC: now also GPI1.1
Other:
- note added: "GPI"
- note added: "SERVO"
- moved on the sheet: IC2, MS, R17, SRV
