File: SulaMatikV3/SulaMatikV3.brd (EAGLE design)
At the start: 53.3 x 63.5 mm, 31 parts, among them IC1 REG1117, IC2 74HC138N, Q3 2N5551

Commit message: v3
Parts:
- removed BZZ: (no value), SparkFun-Connectors:1X03
- removed PRVIN: (no value), SparkFun:1X02
- removed R10: 22K, SparkFun-Passives:0805
- removed R7: 47K, SparkFun-Passives:0805
- added PUMP: (no value), SparkFun:1X02
- added SRV: (no value), con-lstb:MA03-1
- MS: device SparkFun:1X02 -> con-lsta:FE08-2
- moved Q3 93.7 mm to (83.8, 71.1)
- moved IC1 83.8 mm to (94.0, 7.62)
- moved R11 81.3 mm to (81.3, 66.0)
- moved IC2 81.0 mm to (-17.8, 76.2)
- moved MS 81.0 mm to (-12.7, 58.4), turned to 270 degrees
- moved F1 76.2 mm to (88.9, 5.08)
- moved R17 75.5 mm to (-7.62, 68.6)
- moved C2 75.4 mm to (88.9, 17.8)
- moved LED1 75.4 mm to (94.0, 17.8)
- moved GPI3 75.0 mm to (86.4, 43.2)
- moved C1 74.1 mm to (94.0, 15.2)
- moved R8 71.1 mm to (5.08, -17.8), flipped to the top
- moved R12 70.3 mm to (88.9, 15.2)
- moved R9 66.2 mm to (10.2, -17.8), flipped to the top
- moved R6 66.1 mm to (20.3, -12.7), flipped to the top
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Connections:
- removed net A4: R10.2, R7.1
- removed net A5: BZZ.1
- removed net VCC9V: C2.2, D1.C, F1.1, R7.2
- new net VCCSRV: C1.2, D2.C, IC1.2, PUMP.2, R12.2, SRV.2
- net A0: now also MS.10, MS.12, MS.14, MS.16, MS.4, MS.6, MS.8
- net GND: now also IC2.4, IC2.5, SRV.1; no longer BZZ.3, R10.1
- net N$5: now also PUMP.1; no longer PRVIN.1
- net RAW: now also C2.2, D1.C, F1.1
- net VCC: now also IC2.6; no longer BZZ.2, C1.2, D2.C, IC1.2, MS.1, PRVIN.2, R12.2
Routing:
- net VCC: track 222.6 -> 0.00 mm
- net GND: track 203.8 -> 0.00 mm, vias 1 -> 0
- net N$5: track 100.1 -> 0.00 mm
- net D3: track 62.6 -> 0.00 mm
- net VCC9V: track 59.0 -> 0.00 mm
- net D2: track 56.7 -> 0.00 mm, vias 1 -> 0
- net MOSI: track 50.7 -> 0.00 mm
- net MISO: track 49.6 -> 0.00 mm, vias 1 -> 0
- net D8: track 48.3 -> 0.00 mm, vias 1 -> 0
- net SCK: track 38.2 -> 0.00 mm
- net D7: track 37.2 -> 0.00 mm, vias 1 -> 0
- net A0: track 36.5 -> 0.00 mm
- net D6: track 35.6 -> 0.00 mm, vias 1 -> 0
- net N$13: track 33.2 -> 0.00 mm
- net D9: track 24.0 -> 0.00 mm, vias 1 -> 0
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
Commit message: v3
Parts:
- moved Q3 93.7 mm to (12.7, 10.2)
- moved PUMP 92.0 mm to (7.62, 10.2)
- moved D2 91.8 mm to (17.8, 7.62)
- moved C1 85.4 mm to (15.2, 48.3), turned to 180 degrees
- moved R12 84.1 mm to (12.7, 50.8), turned to 270 degrees
- moved F1 83.3 mm to (22.9, 55.9), turned to 90 degrees
- moved LED1 83.0 mm to (17.8, 50.8), turned to 180 degrees
- moved R11 82.9 mm to (17.8, 12.7), turned to 90 degrees
- moved PS 81.3 mm to (17.8, 63.5)
- moved D1 78.5 mm to (15.2, 55.9), turned to 270 degrees
- moved IC1 77.8 mm to (33.0, 55.9), turned to 90 degrees
- moved PW 75.5 mm to (30.5, 63.5), turned to 180 degrees
- moved IC2 74.7 mm to (43.2, 33.0)
- moved C2 72.7 mm to (22.9, 48.3), turned to 90 degrees
- moved GPI3 70.6 mm to (25.4, 7.62)
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Connections:
- new net N$10: IC2.12, MS.9
- new net N$12: IC2.11, MS.7
- new net N$14: IC2.10, MS.5
- new net N$15: IC2.9, MS.3
- new net N$16: IC2.7, MS.1
- new net N$3: IC2.15, MS.15
- new net N$7: IC2.14, MS.13
- new net N$8: IC2.13, MS.11
- net A1: now also IC2.3
- net A2: now also IC2.2
- net A3: now also IC2.1
- net D5: now also SRV.3

Commit message: v3
Parts:
- added R1: 10K, SparkFun-Passives:0805
- moved PS 2.54 mm to (15.2, 63.5)
- moved BT 2.54 mm to (7.62, 50.8)
- turned D2 to 270 degrees
- turned GPI1 to 270 degrees
- renumbered GPI3 to GPI1
Connections:
- net D10: now also GPI1.3, R1.2
- net GND: now also R1.1
- net VCC: now also GPI1.1
Routing:
- net GND: track 0.00 -> 229.9 mm
- net VCC: track 0.00 -> 133.5 mm
- net VCCSRV: track 0.00 -> 87.5 mm, vias 0 -> 1
- net N$9: track 0.00 -> 49.7 mm, vias 1 -> 2
- net A0: track 0.00 -> 46.4 mm
- net D4: track 0.00 -> 43.6 mm
- net MOSI: track 0.00 -> 36.1 mm
- net MISO: track 0.00 -> 31.5 mm
- net N$5: track 0.00 -> 26.8 mm
- net SCK: track 0.00 -> 25.4 mm, vias 0 -> 1
- net SDSCK: track 0.00 -> 25.2 mm
- net D3: track 0.00 -> 23.1 mm
- net D2: track 0.00 -> 23.0 mm
- net RAW: track 0.00 -> 21.0 mm
- net N$16: track 0.00 -> 17.4 mm
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