File: KarasolBaxContxxx/KarasolboxCont.brd (EAGLE design)
At the start: 51.7 x 76.2 mm, 26 parts, among them IC1 REG1117

Commit message: karasol rev
Parts:
- removed CCON, ICON, PCON: (no value), con-ptr500:AK300/2
- added CLI, IRR: (no value), SparkFun:1X02
- added J2: (no value), con-jack:SPC4078
- MSENS: device con-amp-mt:S02P -> SparkFun:1X02
- TSENS: device con-amp-mt:S03P -> SparkFun-Connectors:1X03
- moved TSENS 2.54 mm to (47.0, 15.2)
- moved WIFI 1.27 mm to (41.9, 54.6)
- moved F1 1.27 mm to (17.8, 59.7)
- moved IC1 1.27 mm to (30.5, 66.0)
- moved MSENS 1.27 mm to (47.0, 31.8), turned to 270 degrees
- moved S1 1.27 mm to (17.8, 69.8)
- moved PD1 1.27 mm to (11.4, 62.2)
Connections:
- net D11: now also TSENS.1; no longer TSENS.2
- net GND: now also J2.1, TSENS.2; no longer PCON.2, TSENS.3
- net N$2: now also CLI.1; no longer CCON.2
- net N$5: now also IRR.1; no longer ICON.2
- net N$7: now also J2.3; no longer PCON.1
- net RAW: now also CLI.2, IRR.2; no longer CCON.1, ICON.1
- net VCCSRV: now also TSENS.3; no longer TSENS.1
Routing:
- net GND: track 258.2 -> 197.3 mm, vias 5 -> 3
- net D3: track 52.2 -> 80.0 mm
- net VCCSRV: track 108.0 -> 94.4 mm
- net N$3: track 13.6 -> 7.58 mm
- net D2: track 60.6 -> 55.3 mm
- net N$5: track 13.9 -> 11.2 mm
- net N$2: track 13.7 -> 11.5 mm
- net N$7: track 9.85 -> 9.27 mm
