File: KarasolBaxContxxx/KarasolboxCont.sch (EAGLE design)
At the start: 26 parts, among them IC1 REG1117

Commit message: karasol rev
Parts:
- removed CCON, ICON, PCON: (no value), con-ptr500:AK300/2
- added CLI, IRR: (no value), SparkFun:M02PTH
- added J2: (no value), con-jack:JACK-PLUG1
- MSENS: device con-amp-mt:S02P -> SparkFun:M02PTH
- TSENS: device con-amp-mt:S03P -> SparkFun-Connectors:M03PTH
Connections:
- net A0: now also MSENS.1; no longer MSENS-1.S
- net A1: now also MSENS.2; no longer MSENS-2.S
- net D11: now also TSENS.1; no longer TSENS-2.S
- net GND: now also J2.1, TSENS.2; no longer PCON-2.KL, TSENS-3.S
- net N$2: now also CLI.1; no longer CCON-2.KL
- net N$5: now also IRR.1; no longer ICON-2.KL
- net N$7: now also J2.3; no longer PCON-1.KL
- net RAW: now also CLI.2, IRR.2; no longer CCON-1.KL, ICON-1.KL
- net VCCSRV: now also TSENS.3; no longer TSENS-1.S
Other:
- moved on the sheet: CD1, CQ1, CR1, ID1, IQ1, IR1
