File: KarasolBaxCont/KarasolboxCont.sch (EAGLE design)
At the start: 26 parts, among them IC1 REG1117

Commit message: uff
Parts:
- added IC2: 7808DT, linear:7808DT
- added J1: POWER_JACKTOE, SparkFun-Connectors:POWER_JACKTOE
- added J2: 5.5x2.1mm Barrel, SparkFun-Connectors:POWER_JACKSMD
- added Q1: 35A/25V/8.5mΩ, SparkFun-DiscreteSemi:MOSFET-NCH-FDD8780
- added Q2: 100A/100V/6.8mΩ, SparkFun-DiscreteSemi:MOSFET-NCH-PSMN7R0
- added Q3: FDD4141TO252, transistor-fet:FDD4141TO252
- added Q4: IRF3704S, transistor-power:IRF3704S
- added U1: V_REG_317DPACK, SparkFun-IC-Power:V_REG_317DPACK
Other:
- note added: "F12V To 8V"
- note added: "IRF3707 mosfet"
- note added: "Power Jack"
Changed lines of the file:
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@@
 <layer number="56" name="wert" color="7" fill="1" visible="no" active="no"/>
 <layer number="57" name="tCAD" color="7" fill="1" visible="no" active="no"/>
+<layer number="59" name="tCarbon" color="7" fill="1" visible="no" active="no"/>
+<layer number="60" name="bCarbon" color="7" fill="1" visible="no" active="no"/>
 <layer number="90" name="Modules" color="5" fill="1" visible="yes" active="yes"/>
 <layer number="91" name="Nets" color="2" fill="1" visible="yes" active="yes"/>
@@
 <layer number="112" name="tSilk" color="7" fill="1" visible="yes" active="yes"/>
 <layer number="113" name="IDFDebug" color="7" fill="1" visible="yes" active="yes"/>
+<layer number="114" name="Badge_Outline" color="7" fill="1" visible="yes" active="yes"/>
+<layer number="115" name="ReferenceISLANDS" color="7" fill="1" visible="yes" active="yes"/>
 <layer number="116" name="Patch_BOT" color="9" fill="4" visible="yes" active="yes"/>
+<layer number="118" name="Rect_Pads" color="7" fill="1" visible="yes" active="yes"/>
 <layer number="121" name="_tsilk" color="7" fill="1" visible="yes" active="yes"/>
 <layer number="122" name="_bsilk" color="7" fill="1" visible="yes" active="yes"/>
@@
 <layer number="127" name="_tValues" color="7" fill="1" visible="yes" active="yes"/>
 <layer number="128" name="_bValues" color="7" fill="1" visible="yes" active="yes"/>
+<layer number="129" name="Mask" color="7" fill="1" visible="yes" active="yes"/>
 <layer number="131" name="tAdjust" color="7" fill="1" visible="yes" active="yes"/>
 <layer number="132" name="bAdjust" color="7" fill="1" visible="yes" active="yes"/>
@@
 <layer number="223" name="223bmp" color="24" fill="1" visible="no" active="no"/>
 <layer number="224" name="224bmp" color="25" fill="1" visible="no" active="no"/>
+<layer number="225" name="225bmp" color="7" fill="1" visible="yes" active="yes"/>
+<layer number="226" name="226bmp" color="7" fill="1" visible="yes" active="yes"/>
+<layer number="227" name="227bmp" color="7" fill="1" visible="yes" active="yes"/>
+<layer number="228" name="228bmp" color="7" fill="1" visible="yes" active="yes"/>
+<layer number="229" name="229bmp" color="7" fill="1" visible="yes" active="yes"/>
+<layer number="230" name="230bmp" color="7" fill="1" visible="yes" active="yes"/>
+<layer number="231" name="231bmp" color="7" fill="1" visible="yes" active="yes"/>
 <layer number="248" name="Housing" color="7" fill="1" visible="yes" active="yes"/>
 <layer number="249" name="Edge" color="7" fill="1" visible="yes" active="yes"/>
@@
 <layer number="251" name="SMDround" color="12" fill="11" visible="no" active="no"/>
 <layer number="254" name="cooling" color="7" fill="1" visible="yes" active="yes"/>
+<layer number="255" name="routoute" color="7" fill="1" visible="yes" active="yes"/>
 </layers>
 <schematic xreflabel="%F%N/%S.%C%R" xrefpart="/%S.%C%R">
@@
 <part name="ICON" library="con-ptr500" deviceset="AK300/2" device=""/>
 <part name="PCON" library="con-ptr500" deviceset="AK300/2" device=""/>
+<part name="J1" library="SparkFun-Connectors" deviceset="POWER_JACK" device="TOE"/>
+<part name="J2" library="SparkFun-Connectors" deviceset="POWER_JACK" device="SMD" value="5.5x2.1mm Barrel"/>
+<part name="Q1" library="SparkFun-DiscreteSemi" deviceset="MOSFET-NCH" device="-FDD8780" value="35A/25V/8.5mΩ"/>
+<part name="Q2" library="SparkFun-DiscreteSemi" deviceset="MOSFET-NCH" device="-PSMN7R0" value="100A/100V/6.8mΩ"/>
+<part name="Q3" library="transistor-fet" deviceset="FDD4141" device="TO252"/>
+<part name="Q4" library="transistor-power" deviceset="IRF3704" device="S"/>
+<part name="IC2" library="linear" deviceset="78*" device="DT" technology="08"/>
+<part name="U1" library="SparkFun-IC-Power" deviceset="V_REG_317" device="DPACK"/>
 </parts>
 <sheets>
@@
 <text x="137.16" y="132.08" size="1.778" layer="91">TEMPERATURE SENSOR</text>
 <text x="10.16" y="99.06" size="1.778" layer="91">WI-FI</text>
+<text x="76.2" y="175.26" size="1.778" layer="91">IRF3707 mosfet</text>
+<text x="78.74" y="116.84" size="1.778" layer="91">Power Jack</text>
+<text x="134.62" y="99.06" size="1.778" layer="91">F12V To 8V</text>
 </plain>
 <instances>
@@
 <instance part="PCON" gate="-1" x="137.16" y="152.4"/>
 <instance part="PCON" gate="-2" x="137.16" y="147.32"/>
+<instance part="J1" gate="G$1" x="88.9" y="101.6"/>
+<instance part="J2" gate="G$1" x="88.9" y="83.82"/>
+<instance part="Q1" gate="NMOS" x="83.82" y="129.54"/>
+<instance part="Q2" gate="NMOS" x="83.82" y="142.24"/>
+<instance part="Q3" gate="G$1" x="83.82" y="154.94"/>
+<instance part="Q4" gate="G$1" x="83.82" y="167.64"/>
+<instance part="IC2" gate="A1" x="142.24" y="88.9"/>
+<instance part="U1" gate="G$1" x="142.24" y="71.12"/>
 </instances>
 <busses>

Commit message: rev
Parts:
- removed J2: 5.5x2.1mm Barrel, SparkFun-Connectors:POWER_JACKSMD
- removed PCON: (no value), con-ptr500:AK300/2
- removed U1: V_REG_317DPACK, SparkFun-IC-Power:V_REG_317DPACK
- added PC3: 0.33uf, SparkFun-Capacitors:CAP0805
- PC2: value 100uf -> 0.1uf
- PR1: value 220 -> 330
Connections:
- new net N$12: IC1.VIN, IC2.VO, PC2.2
- net GND: now also IC2.GND, J1.GND, PC3.1; no longer PCON-2.KL
- net N$1: now also F1.1, PD1.C; no longer F1.2, IC1.VIN
- net N$7: now also J1.PWR; no longer PCON-1.KL
- net RAW: now also F1.2, IC2.VI, PC3.2; no longer F1.1, PC2.2, PD1.C
Other:
- note removed: "F12V To 8V"
- note removed: "Power Jack"
- moved on the sheet: F1, IC1, IC2, J1, PC2, PD1, Q1, Q2, Q3, Q4, S1

Commit message: ardu bef
Parts:
- removed Q2: 100A/100V/6.8mΩ, SparkFun-DiscreteSemi:MOSFET-NCH-PSMN7R0
- removed Q3: FDD4141TO252, transistor-fet:FDD4141TO252
- Q1: value 35A/25V/8.5mΩ -> IRF3707S; device SparkFun-DiscreteSemi:MOSFET-NCH-FDD8780 -> transistor-power:IRF3704S
- Q4: value IRF3704S -> IRF3707S
Other:
- note removed: "IRF3707 mosfet"
- moved on the sheet: Q4
Changed lines of the file:
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@@
 <part name="ICON" library="con-ptr500" deviceset="AK300/2" device=""/>
 <part name="J1" library="SparkFun-Connectors" deviceset="POWER_JACK" device="TOE"/>
-<part name="Q1" library="SparkFun-DiscreteSemi" deviceset="MOSFET-NCH" device="-FDD8780" value="35A/25V/8.5mΩ"/>
-<part name="Q2" library="SparkFun-DiscreteSemi" deviceset="MOSFET-NCH" device="-PSMN7R0" value="100A/100V/6.8mΩ"/>
-<part name="Q3" library="transistor-fet" deviceset="FDD4141" device="TO252"/>
-<part name="Q4" library="transistor-power" deviceset="IRF3704" device="S"/>
+<part name="Q4" library="transistor-power" deviceset="IRF3704" device="S" value="IRF3707S"/>
 <part name="IC2" library="linear" deviceset="78*" device="DT" technology="08"/>
 <part name="PC3" library="SparkFun-Capacitors" deviceset="CAP" device="0805" value="0.33uf"/>
+<part name="Q1" library="transistor-power" deviceset="IRF3704" device="S" value="IRF3707S"/>
 </parts>
 <sheets>
@@
 <text x="137.16" y="132.08" size="1.778" layer="91">TEMPERATURE SENSOR</text>
 <text x="10.16" y="99.06" size="1.778" layer="91">WI-FI</text>
-<text x="86.36" y="101.6" size="1.778" layer="91">IRF3707 mosfet</text>
 </plain>
 <instances>
@@
 <instance part="ICON" gate="-2" x="38.1" y="172.72" rot="R270"/>
 <instance part="J1" gate="G$1" x="121.92" y="144.78"/>
-<instance part="Q1" gate="NMOS" x="93.98" y="55.88"/>
-<instance part="Q2" gate="NMOS" x="93.98" y="68.58"/>
-<instance part="Q3" gate="G$1" x="93.98" y="81.28"/>
-<instance part="Q4" gate="G$1" x="93.98" y="93.98"/>
+<instance part="Q4" gate="G$1" x="17.78" y="142.24"/>
 <instance part="IC2" gate="A1" x="175.26" y="160.02"/>
 <instance part="PC3" gate="G$1" x="162.56" y="152.4" rot="R180"/>
+<instance part="Q1" gate="G$1" x="17.78" y="106.68"/>
 </instances>
 <busses>

Commit message: mosfet bef
Parts:
- U$1: device Arduino-clone:ABK-PRO-MINI -> Arduino-Clk:ABK-PRO-MINI
Connections:
- removed net A0: MD1.C, MR1.2, MSENS-1.S, U$1.A0
- removed net D12: MD1.A, U$1.D12
- removed net D13: MD2.A, U$1.D13
- new net A0_D: MD2.A, U$1.A0
- new net A2: MD1.C, MR1.2, MSENS-1.S, U$1.A2
- new net A3_D: MD1.A, U$1.A3

Commit message: bef check
Parts:
- removed IQ1: 2N5551, semicon-smd-ipc:NPN-TRANSISTOR_SOT23
- removed Q1: IRF3707S, transistor-power:IRF3704S
- CQ1: value 2N5551 -> IRF3707S; device semicon-smd-ipc:NPN-TRANSISTOR_SOT23 -> transistor-power:IRF3704S
Connections:
- removed net N$10: CQ1.B, CR1.1
- removed net N$6: IQ1.B, IR1.1
- net D10: now also CQ1.G
- net D9: now also Q4.G
- net GND: now also CQ1.S, CR1.1, IR1.1, Q4.S; no longer CQ1.E, IQ1.E
- net N$2: now also CQ1.D; no longer CQ1.C
- net N$5: now also Q4.D; no longer IQ1.C
Other:
- moved on the sheet: CD1, CR1, IR1, Q4
Changed lines of the file:
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@@
 <parts>
 <part name="FRAME1" library="SparkFun" deviceset="FRAME-LETTER" device=""/>
-<part name="IQ1" library="semicon-smd-ipc" deviceset="NPN-TRANSISTOR_" device="SOT23" value="2N5551"/>
 <part name="IR1" library="SparkFun-Passives" deviceset="RESISTOR" device="0805-RES" value="1K"/>
 <part name="ID1" library="SparkFun-DiscreteSemi" deviceset="DIODE" device="SMA"/>
@@
 <part name="F1" library="_hhn_PtcFuses_Siba_r500_Ozan" deviceset="SIBA194600*" device="" value="1A"/>
 <part name="IC1" library="burr-brown" deviceset="REG1117" device=""/>
-<part name="CQ1" library="semicon-smd-ipc" deviceset="NPN-TRANSISTOR_" device="SOT23" value="2N5551"/>
 <part name="CR1" library="SparkFun-Passives" deviceset="RESISTOR" device="0805-RES" value="1K"/>
 <part name="CD1" library="SparkFun-DiscreteSemi" deviceset="DIODE" device="SMA"/>
@@
 <part name="IC2" library="linear" deviceset="78*" device="DT" technology="08"/>
 <part name="PC3" library="SparkFun-Capacitors" deviceset="CAP" device="0805" value="0.33uf"/>
-<part name="Q1" library="transistor-power" deviceset="IRF3704" device="S" value="IRF3707S"/>
+<part name="CQ1" library="transistor-power" deviceset="IRF3704" device="S" value="IRF3707S"/>
 <part name="U$1" library="Arduino-Clk" deviceset="ABK-PRO-MINI" device=""/>
 </parts>
@@
 <instance part="FRAME1" gate="G$1" x="0" y="0"/>
 <instance part="FRAME1" gate="G$2" x="147.32" y="0"/>
-<instance part="IQ1" gate="G$1" x="27.94" y="154.94"/>
-<instance part="IR1" gate="G$1" x="17.78" y="154.94" rot="R180"/>
+<instance part="IR1" gate="G$1" x="17.78" y="152.4" rot="R90"/>
 <instance part="ID1" gate="G$1" x="38.1" y="154.94"/>
 <instance part="GND5" gate="1" x="48.26" y="147.32" rot="R90"/>
@@
 <instance part="F1" gate="G$1" x="154.94" y="170.18"/>
 <instance part="IC1" gate="G$1" x="203.2" y="160.02"/>
-<instance part="CQ1" gate="G$1" x="27.94" y="116.84"/>
-<instance part="CR1" gate="G$1" x="17.78" y="116.84" rot="R180"/>
-<instance part="CD1" gate="G$1" x="38.1" y="116.84"/>
+<instance part="CR1" gate="G$1" x="17.78" y="114.3" rot="R90"/>
+<instance part="CD1" gate="G$1" x="38.1" y="111.76"/>
 <instance part="GND2" gate="1" x="50.8" y="109.22" rot="R90"/>
 <instance part="MR2" gate="G$1" x="226.06" y="114.3" rot="R180"/>
@@
 <instance part="ICON" gate="-2" x="38.1" y="172.72" rot="R270"/>
 <instance part="J1" gate="G$1" x="121.92" y="144.78"/>
-<instance part="Q4" gate="G$1" x="17.78" y="142.24"/>
+<instance part="Q4" gate="G$1" x="27.94" y="154.94"/>
 <instance part="IC2" gate="A1" x="175.26" y="160.02"/>
 <instance part="PC3" gate="G$1" x="162.56" y="152.4" rot="R180"/>
-<instance part="Q1" gate="G$1" x="17.78" y="106.68"/>
+<instance part="CQ1" gate="G$1" x="27.94" y="116.84"/>
 <instance part="U$1" gate="G$1" x="48.26" y="38.1"/>
 </instances>
@@
 <net name="GND" class="0">
 <segment>
-<pinref part="IQ1" gate="G$1" pin="E"/>
 <wire x1="30.48" y1="149.86" x2="30.48" y2="147.32" width="0.1524" layer="91"/>
 <wire x1="30.48" y1="147.32" x2="45.72" y2="147.32" width="0.1524" layer="91"/>
 <pinref part="GND5" gate="1" pin="GND"/>
+<pinref part="Q4" gate="G$1" pin="S"/>
+<pinref part="IR1" gate="G$1" pin="1"/>
+<wire x1="17.78" y1="147.32" x2="30.48" y2="147.32" width="0.1524" layer="91"/>
+<junction x="30.48" y="147.32"/>
 </segment>
 <segment>
@@
 </segment>
 <segment>
-<pinref part="CQ1" gate="G$1" pin="E"/>
 <wire x1="30.48" y1="111.76" x2="30.48" y2="109.22" width="0.1524" layer="91"/>
 <wire x1="30.48" y1="109.22" x2="48.26" y2="109.22" width="0.1524" layer="91"/>
 <pinref part="GND2" gate="1" pin="GND"/>
+<pinref part="CQ1" gate="G$1" pin="S"/>
+<pinref part="CR1" gate="G$1" pin="1"/>
+<wire x1="17.78" y1="109.22" x2="30.48" y2="109.22" width="0.1524" layer="91"/>
+<junction x="30.48" y="109.22"/>
 </segment>
 <segment>
@@
 <label x="50.8" y="162.56" size="1.778" layer="95" xref="yes"/>
 <pinref part="ICON" gate="-1" pin="KL"/>
+<junction x="45.72" y="162.56"/>
 </segment>
 <segment>
 <wire x1="43.18" y1="129.54" x2="43.18" y2="124.46" width="0.1524" layer="91"/>
 <wire x1="43.18" y1="124.46" x2="45.72" y2="124.46" width="0.1524" layer="91"/>
-<wire x1="45.72" y1="124.46" x2="45.72" y2="116.84" width="0.1524" layer="91"/>
+<wire x1="45.72" y1="124.46" x2="45.72" y2="111.76" width="0.1524" layer="91"/>
 <pinref part="CD1" gate="G$1" pin="C"/>
-<wire x1="45.72" y1="116.84" x2="40.64" y2="116.84" width="0.1524" layer="91"/>
+<wire x1="45.72" y1="111.76" x2="40.64" y2="111.76" width="0.1524" layer="91"/>
 <wire x1="45.72" y1="124.46" x2="50.8" y2="124.46" width="0.1524" layer="91"/>
 <label x="50.8" y="124.46" size="1.778" layer="95" xref="yes"/>
 <pinref part="CCON" gate="-1" pin="KL"/>
+<junction x="45.72" y="124.46"/>
 </segment>
 </net>
@@
 <segment>
 <pinref part="IR1" gate="G$1" pin="2"/>
-<wire x1="12.7" y1="154.94" x2="10.16" y2="154.94" width="0.1524" layer="91"/>
-<label x="10.16" y="154.94" size="1.778" layer="95" rot="R180" xref="yes"/>
+<wire x1="17.78" y1="157.48" x2="10.16" y2="157.48" width="0.1524" layer="91"/>
+<label x="10.16" y="157.48" size="1.778" layer="95" rot="R180" xref="yes"/>
+<wire x1="17.78" y1="157.48" x2="22.86" y2="157.48" width="0.1524" layer="91"/>
+<junction x="17.78" y="157.48"/>
+<wire x1="22.86" y1="157.48" x2="22.86" y2="152.4" width="0.1524" layer="91"/>
+<pinref part="Q4" gate="G$1" pin="G"/>
+<wire x1="22.86" y1="152.4" x2="25.4" y2="152.4" width="0.1524" layer="91"/>
 </segment>
 <segment>
@@
 <wire x1="35.56" y1="154.94" x2="33.02" y2="154.94" width="0.1524" layer="91"/>
 <wire x1="33.02" y1="154.94" x2="33.02" y2="162.56" width="0.1524" layer="91"/>
-<pinref part="IQ1" gate="G$1" pin="C"/>
-<wire x1="33.02" y1="162.56" x2="30.48" y2="162.56" width="0.1524" layer="91"/>
-<wire x1="30.48" y1="160.02" x2="30.48" y2="162.56" width="0.1524" layer="91"/>
 <wire x1="33.02" y1="162.56" x2="38.1" y2="162.56" width="0.1524" layer="91"/>
-<junction x="33.02" y="162.56"/>
 <wire x1="38.1" y1="162.56" x2="38.1" y2="167.64" width="0.1524" layer="91"/>
 <pinref part="ICON" gate="-2" pin="KL"/>
-</segment>
-</net>
-<net name="N$6" class="0">
-<segment>
-<pinref part="IQ1" gate="G$1" pin="B"/>
-<wire x1="25.4" y1="154.94" x2="22.86" y2="154.94" width="0.1524" layer="91"/>
-<pinref part="IR1" gate="G$1" pin="1"/>
+<pinref part="Q4" gate="G$1" pin="D"/>
+<wire x1="30.48" y1="160.02" x2="30.48" y2="162.56" width="0.1524" layer="91"/>
+<wire x1="30.48" y1="162.56" x2="33.02" y2="162.56" width="0.1524" layer="91"/>
+<junction x="33.02" y="162.56"/>
 </segment>
 </net>
@@
 <net name="N$2" class="0">
 <segment>
-<pinref part="CD1" gate="G$1" pin="A"/>
-<wire x1="35.56" y1="116.84" x2="33.02" y2="116.84" width="0.1524" layer="91"/>
-<wire x1="33.02" y1="116.84" x2="33.02" y2="124.46" width="0.1524" layer="91"/>
-<pinref part="CQ1" gate="G$1" pin="C"/>
-<wire x1="33.02" y1="124.46" x2="30.48" y2="124.46" width="0.1524" layer="91"/>
-<wire x1="30.48" y1="121.92" x2="30.48" y2="124.46" width="0.1524" layer="91"/>
+<wire x1="30.48" y1="124.46" x2="33.02" y2="124.46" width="0.1524" layer="91"/>
 <wire x1="33.02" y1="124.46" x2="38.1" y2="124.46" width="0.1524" layer="91"/>
-<junction x="33.02" y="124.46"/>
 <wire x1="38.1" y1="124.46" x2="38.1" y2="129.54" width="0.1524" layer="91"/>
 <pinref part="CCON" gate="-2" pin="KL"/>
-</segment>
-</net>
-<net name="N$10" class="0">
-<segment>
-<pinref part="CQ1" gate="G$1" pin="B"/>
-<wire x1="25.4" y1="116.84" x2="22.86" y2="116.84" width="0.1524" layer="91"/>
-<pinref part="CR1" gate="G$1" pin="1"/>
+<pinref part="CQ1" gate="G$1" pin="D"/>
+<wire x1="30.48" y1="121.92" x2="30.48" y2="124.46" width="0.1524" layer="91"/>
+<wire x1="33.02" y1="124.46" x2="33.02" y2="111.76" width="0.1524" layer="91"/>
+<junction x="33.02" y="124.46"/>
+<pinref part="CD1" gate="G$1" pin="A"/>
+<wire x1="33.02" y1="111.76" x2="35.56" y2="111.76" width="0.1524" layer="91"/>
 </segment>
 </net>
@@
 <segment>
 <pinref part="CR1" gate="G$1" pin="2"/>
-<wire x1="12.7" y1="116.84" x2="10.16" y2="116.84" width="0.1524" layer="91"/>
-<label x="10.16" y="116.84" size="1.778" layer="95" rot="R180" xref="yes"/>
-</segment>
-</net>
+<wire x1="17.78" y1="119.38" x2="10.16" y2="119.38" width="0.1524" layer="91"/>
+<label x="10.16" y="119.38" size="1.778" layer="95" rot="R180" xref="yes"/>
+<wire x1="17.78" y1="119.38" x2="22.86" y2="119.38" width="0.1524" layer="91"/>
+<junction x="17.78" y="119.38"/>
+<wire x1="22.86" y1="119.38" x2="22.86" y2="114.3" width="0.1524" layer="91"/>
+<pinref part="CQ1" gate="G$1" pin="G"/>
+<wire x1="22.86" y1="114.3" x2="25.4" y2="114.3" width="0.1524" layer="91"/>
+</segment>
+</net>

Commit message: value changec
Parts:
- PC2: value 0.1uf -> 100nf
- PC3: value 0.33uf -> 1uf
- PR1: value 330 -> 470
Changed lines of the file:
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@@
 <part name="PD1" library="SparkFun-DiscreteSemi" deviceset="DIODE" device="SMA"/>
 <part name="GND1" library="SparkFun-Aesthetics" deviceset="GND" device=""/>
-<part name="PC2" library="SparkFun-Capacitors" deviceset="CAP" device="0805" value="0.1uf"/>
-<part name="PR1" library="SparkFun-Passives" deviceset="RESISTOR" device="0805-RES" value="330"/>
+<part name="PC2" library="SparkFun-Capacitors" deviceset="CAP" device="0805" value="100nf"/>
+<part name="PR1" library="SparkFun-Passives" deviceset="RESISTOR" device="0805-RES" value="470"/>
 <part name="F1" library="_hhn_PtcFuses_Siba_r500_Ozan" deviceset="SIBA194600*" device="" value="1A"/>
 <part name="IC1" library="burr-brown" deviceset="REG1117" device=""/>
@@
 <part name="Q4" library="transistor-power" deviceset="IRF3704" device="S" value="IRF3707S"/>
 <part name="IC2" library="linear" deviceset="78*" device="DT" technology="08"/>
-<part name="PC3" library="SparkFun-Capacitors" deviceset="CAP" device="0805" value="0.33uf"/>
+<part name="PC3" library="SparkFun-Capacitors" deviceset="CAP" device="0805" value="1uf"/>
 <part name="CQ1" library="transistor-power" deviceset="IRF3704" device="S" value="IRF3707S"/>
 <part name="U$1" library="Arduino-Clk" deviceset="ABK-PRO-MINI" device=""/>

Commit message: pto2 v0.1
Connections:
- net GND: now also J1.GNDBREAK; no longer J1.GND
Other:
- moved on the sheet: J1
Changed lines of the file:
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@@
 <?xml version="1.0" encoding="utf-8"?>
 <!DOCTYPE eagle SYSTEM "eagle.dtd">
-<eagle version="8.1.0">
+<eagle version="8.1.1">
 <drawing>
 <settings>
@@
 <instance part="ICON" gate="-1" x="43.18" y="172.72" rot="R270"/>
 <instance part="ICON" gate="-2" x="38.1" y="172.72" rot="R270"/>
-<instance part="J1" gate="G$1" x="121.92" y="144.78"/>
+<instance part="J1" gate="G$1" x="121.92" y="142.24"/>
 <instance part="Q4" gate="G$1" x="27.94" y="154.94"/>
 <instance part="IC2" gate="A1" x="175.26" y="160.02"/>
@@
 <wire x1="218.44" y1="147.32" x2="220.98" y2="147.32" width="0.1524" layer="91"/>
 <pinref part="IC1" gate="G$1" pin="GND"/>
-<pinref part="J1" gate="G$1" pin="GND"/>
+<pinref part="IC2" gate="A1" pin="GND"/>
 <wire x1="124.46" y1="147.32" x2="162.56" y2="147.32" width="0.1524" layer="91"/>
-<pinref part="IC2" gate="A1" pin="GND"/>
 <wire x1="162.56" y1="147.32" x2="175.26" y2="147.32" width="0.1524" layer="91"/>
 <wire x1="175.26" y1="147.32" x2="187.96" y2="147.32" width="0.1524" layer="91"/>
@@
 <pinref part="PC3" gate="G$1" pin="1"/>
 <junction x="162.56" y="147.32"/>
+<pinref part="J1" gate="G$1" pin="GNDBREAK"/>
 </segment>
 <segment>
@@
 <net name="N$7" class="0">
 <segment>
-<wire x1="132.08" y1="152.4" x2="124.46" y2="152.4" width="0.1524" layer="91"/>
+<wire x1="134.62" y1="149.86" x2="124.46" y2="149.86" width="0.1524" layer="91"/>
 <pinref part="S1" gate="1" pin="S"/>
-<wire x1="132.08" y1="152.4" x2="134.62" y2="160.02" width="0.1524" layer="91"/>
+<wire x1="134.62" y1="149.86" x2="134.62" y2="160.02" width="0.1524" layer="91"/>
 <pinref part="J1" gate="G$1" pin="PWR"/>
 </segment>
