File: KarasolBaxCont/KarasolboxCont.sch (EAGLE design)
At the start: 28 parts, among them IC1 REG1117, IC2 7808DT, J1 POWER_JACKTOE, Q4 IRF3707S

Commit message: proto 2 v 0.2 ready
Parts:
- removed S1: 9077-2, switch-misc:9077-2
- added CCON1: (no value), con-ptr500:AK300/2
Connections:
- net N$3: now also CCON1-1.KL; no longer S11.P
- net N$7: now also CCON1-2.KL; no longer S11.S
Changed lines of the file:
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@@
 <part name="GND6" library="supply1" deviceset="GND" device=""/>
 <part name="GND8" library="supply1" deviceset="GND" device=""/>
-<part name="S1" library="switch-misc" deviceset="9077-2" device=""/>
 <part name="MSENS" library="con-amp-mt" deviceset="S02P" device=""/>
 <part name="TSENS" library="con-amp-mt" deviceset="S03P" device=""/>
@@
 <part name="CQ1" library="transistor-power" deviceset="IRF3704" device="S" value="IRF3707S"/>
 <part name="U$1" library="Arduino-Clk" deviceset="ABK-PRO-MINI" device=""/>
+<part name="CCON1" library="con-ptr500" deviceset="AK300/2" device=""/>
 </parts>
 <sheets>
@@
 <text x="10.16" y="167.64" size="1.778" layer="91">IRRIGATION</text>
 <text x="5.08" y="63.5" size="1.778" layer="91">Pro Mini Stamp Socket</text>
-<text x="114.3" y="167.64" size="1.778" layer="91">POWER</text>
+<text x="114.3" y="160.02" size="1.778" layer="91">POWER</text>
 <text x="200.66" y="129.54" size="1.778" layer="91">MOISTURE SENSOR</text>
 <text x="10.16" y="129.54" size="1.778" layer="91">CLIMATE</text>
@@
 <instance part="GND6" gate="1" x="7.62" y="91.44" rot="R270"/>
 <instance part="GND8" gate="1" x="15.24" y="43.18" rot="R270"/>
-<instance part="S1" gate="1" x="137.16" y="165.1" rot="R180"/>
-<instance part="S1" gate="2" x="127" y="165.1" rot="R180"/>
 <instance part="MSENS" gate="-1" x="203.2" y="106.68"/>
 <instance part="MSENS" gate="-2" x="203.2" y="109.22"/>
@@
 <instance part="CQ1" gate="G$1" x="27.94" y="116.84"/>
 <instance part="U$1" gate="G$1" x="48.26" y="38.1"/>
+<instance part="CCON1" gate="-1" x="127" y="170.18"/>
+<instance part="CCON1" gate="-2" x="127" y="165.1"/>
 </instances>
 <busses>
@@
 <segment>
 <pinref part="PD1" gate="G$1" pin="A"/>
-<pinref part="S1" gate="1" pin="P"/>
-<wire x1="137.16" y1="170.18" x2="142.24" y2="170.18" width="0.1524" layer="91"/>
+<pinref part="CCON1" gate="-1" pin="KL"/>
+<wire x1="132.08" y1="170.18" x2="142.24" y2="170.18" width="0.1524" layer="91"/>
 </segment>
 </net>
@@
 <segment>
 <wire x1="134.62" y1="149.86" x2="124.46" y2="149.86" width="0.1524" layer="91"/>
-<pinref part="S1" gate="1" pin="S"/>
-<wire x1="134.62" y1="149.86" x2="134.62" y2="160.02" width="0.1524" layer="91"/>
+<wire x1="134.62" y1="149.86" x2="134.62" y2="165.1" width="0.1524" layer="91"/>
 <pinref part="J1" gate="G$1" pin="PWR"/>
-</segment>
-</net>
+<pinref part="CCON1" gate="-2" pin="KL"/>
+<wire x1="132.08" y1="165.1" x2="134.62" y2="165.1" width="0.1524" layer="91"/>
+</segment>
+</net>
