File: KarasolBaxCont/KarasolboxCont.brd (EAGLE design)
At the start: 44.1 x 76.2 mm, 29 parts, among them IC1 REG1117, IC2 7808DT, J1 POWER_JACKTOE, Q4 IRF3707S

Commit message: pto2 v0.1
Parts:
- U$2: device Logo:IOTECH_COPPER_M -> Logo:IOTECH_COPPER
- moved U$2 59.5 mm to (40.6, 11.4), flipped to the top
Connections:
- net GND: now also J1.GND; no longer J1.P$4
Routing:
- net GND: track 220.7 -> 225.3 mm
- net RAW: track 121.3 -> 120.7 mm, vias 0 -> 1
Changed lines of the file:
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@@
 <autorouter>
 <pass name="Default">
-<param name="RoutingGrid" value="5mm"/>
+<param name="RoutingGrid" value="0.125mm"/>
 <param name="AutoGrid" value="1"/>
 <param name="Efforts" value="2"/>
@@
 <element name="CQ1" library="transistor-power" package="D2PACK" value="IRF3707S" x="30.48" y="7.62" rot="R180"/>
 <element name="U$1" library="Arduino-Clk" package="ABK-PRO-MINI" value="ABK-PRO-MINI" x="12.7" y="40.64"/>
-<element name="U$2" library="Logo" package="IOTECH_COPPER_M" value="" x="29.21" y="69.85" rot="MR0"/>
+<element name="U$2" library="Logo" package="IOTECH_COPPER" value="" x="40.64" y="11.43"/>
 </elements>
 <signals>
@@
 <contactref element="WIFI" pad="GND"/>
 <contactref element="TSENS" pad="3"/>
-<contactref element="J1" pad="P$4"/>
 <contactref element="IC2" pad="3"/>
 <contactref element="PC3" pad="1"/>
@@
 <contactref element="CR1" pad="1"/>
 <contactref element="IR1" pad="1"/>
+<contactref element="J1" pad="GND"/>
 <wire x1="38" y1="60.8" x2="26.8" y2="60.8" width="0.8" layer="1"/>
 <wire x1="26.8" y1="60.8" x2="26.67" y2="60.59" width="0.8" layer="1"/>
@@
 <wire x1="16.8" y1="52.4" x2="16.88" y2="52.07" width="0.8" layer="1"/>
 <wire x1="16.8" y1="56.4" x2="16.7894" y2="56.5404" width="0.8" layer="1"/>
-<wire x1="8" y1="61.2" x2="8" y2="60.4" width="0.8" layer="1"/>
-<wire x1="8" y1="60.4" x2="8" y2="57.2" width="0.8" layer="1"/>
-<wire x1="8.4" y1="61.6" x2="8" y2="61.2" width="0.8" layer="1"/>
-<wire x1="8" y1="57.2" x2="7.84" y2="57.15" width="0.8" layer="1"/>
-<wire x1="8.4" y1="61.6" x2="8.64" y2="61.61" width="0.8" layer="1"/>
+<wire x1="2.8" y1="62" x2="7" y2="57.8" width="0.8" layer="1"/>
+<wire x1="7" y1="57.8" x2="7.6" y2="57.2" width="0.8" layer="1"/>
+<wire x1="7.6" y1="57.2" x2="7.84" y2="57.15" width="0.8" layer="1"/>
+<wire x1="2.8" y1="62" x2="2.54" y2="61.61" width="0.8" layer="1"/>
 <wire x1="8.8" y1="55.2" x2="10" y2="55.2" width="0.8" layer="1"/>
 <wire x1="10" y1="55.2" x2="16.8" y2="55.2" width="0.8" layer="1"/>
@@
 <wire x1="40.4" y1="18.8" x2="40.64" y2="19.09" width="0.8" layer="16"/>
 <wire x1="18" y1="21.2" x2="17.78" y2="21.59" width="0.8" layer="16"/>
-<wire x1="8" y1="60.4" x2="26.4" y2="60.4" width="0.8" layer="1"/>
+<wire x1="12" y1="60.4" x2="26.4" y2="60.4" width="0.8" layer="1"/>
+<wire x1="10.8" y1="59.2" x2="12" y2="60.4" width="0.8" layer="1"/>
+<wire x1="8.4" y1="59.2" x2="10.8" y2="59.2" width="0.8" layer="1"/>
+<wire x1="7" y1="57.8" x2="8.4" y2="59.2" width="0.8" layer="1"/>
 <wire x1="26.4" y1="60.4" x2="26.67" y2="60.59" width="0.8" layer="1"/>
 </signal>
@@
 <contactref element="IC2" pad="1"/>
 <contactref element="PC3" pad="2"/>
-<wire x1="16.73" y1="4" x2="16.73" y2="11.2" width="0.8" layer="1"/>
-<wire x1="16.8" y1="2.8" x2="16.73" y2="4" width="0.8" layer="1"/>
-<wire x1="16.73" y1="11.2" x2="16.9" y2="11.43" width="0.8" layer="1"/>
+<wire x1="16.8" y1="2.8" x2="16.8" y2="11.2" width="0.8" layer="1"/>
+<wire x1="16.8" y1="11.2" x2="16.9" y2="11.43" width="0.8" layer="1"/>
 <wire x1="16.8" y1="2.8" x2="16.5354" y2="2.54" width="0.8" layer="1"/>
 <wire x1="33.2" y1="70" x2="37.2" y2="70" width="0.8" layer="1"/>
@@
 <wire x1="37.2" y1="70" x2="37.2" y2="69.85" width="0.8" layer="1"/>
 <wire x1="32" y1="68.8" x2="31.75" y2="68.63" width="0.8" layer="1"/>
-<wire x1="30.8" y1="67.6" x2="30.8" y2="65.2" width="0.8" layer="1"/>
-<wire x1="30.8" y1="65.2" x2="30.8" y2="63.6" width="0.8" layer="1"/>
+<wire x1="30.8" y1="67.6" x2="30.8" y2="63.6" width="0.8" layer="1"/>
 <wire x1="31.6" y1="68.4" x2="30.8" y2="67.6" width="0.8" layer="1"/>
 <wire x1="30.8" y1="63.6" x2="30.76" y2="63.24" width="0.8" layer="1"/>
@@
 <wire x1="5.2" y1="11.2" x2="5.47" y2="11.43" width="0.8" layer="1"/>
 <wire x1="5.2" y1="2.8" x2="5.1054" y2="2.54" width="0.8" layer="1"/>
-<wire x1="8.4" y1="65.2" x2="30.8" y2="65.2" width="0.8" layer="1"/>
-<wire x1="7.6" y1="64.4" x2="8.4" y2="65.2" width="0.8" layer="1"/>
-<wire x1="6.8" y1="64.4" x2="7.6" y2="64.4" width="0.8" layer="1"/>
-<wire x1="5.2" y1="62.8" x2="6.8" y2="64.4" width="0.8" layer="1"/>
-<wire x1="5.2" y1="11.6" x2="5.2" y2="13.6" width="0.8" layer="1"/>
-<wire x1="5.2" y1="13.6" x2="5.2" y2="62.8" width="0.8" layer="1"/>
-<wire x1="5.2" y1="11.6" x2="5.47" y2="11.43" width="0.8" layer="1"/>
-<wire x1="13.2" y1="11.2" x2="16.33" y2="11.2" width="0.8" layer="1"/>
-<wire x1="16.73" y1="11.2" x2="16.33" y2="11.2" width="0.8" layer="1"/>
+<wire x1="22.8" y1="63.2" x2="30.4" y2="63.2" width="0.8" layer="1"/>
+<wire x1="20.4" y1="63.2" x2="22.8" y2="63.2" width="0.8" layer="16"/>
+<wire x1="5.2" y1="48" x2="20.4" y2="63.2" width="0.8" layer="16"/>
+<wire x1="5.2" y1="2.8" x2="5.2" y2="48" width="0.8" layer="16"/>
+<wire x1="30.4" y1="63.2" x2="30.76" y2="63.24" width="0.8" layer="1"/>
+<wire x1="5.2" y1="2.8" x2="5.1054" y2="2.54" width="0.8" layer="16"/>
+<wire x1="13.2" y1="11.2" x2="16.4" y2="11.2" width="0.8" layer="1"/>
 <wire x1="10.8" y1="13.6" x2="13.2" y2="11.2" width="0.8" layer="1"/>
-<wire x1="5.2" y1="13.6" x2="10.8" y2="13.6" width="0.8" layer="1"/>
-<wire x1="16.33" y1="11.2" x2="16.9" y2="11.43" width="0.8" layer="1"/>
+<wire x1="7.6" y1="13.6" x2="10.8" y2="13.6" width="0.8" layer="1"/>
+<wire x1="5.6" y1="11.6" x2="7.6" y2="13.6" width="0.8" layer="1"/>
+<wire x1="16.4" y1="11.2" x2="16.9" y2="11.43" width="0.8" layer="1"/>
+<wire x1="5.6" y1="11.6" x2="5.47" y2="11.43" width="0.8" layer="1"/>
+<via x="22.8" y="63.2" extent="1-16" drill="0.8"/>
 </signal>
 <signal name="D9">
@@
 <contactref element="CQ1" pad="2"/>
 <contactref element="CD1" pad="A"/>
-<wire x1="21.13" y1="3.6" x2="21.13" y2="5.2" width="0.8" layer="1"/>
-<wire x1="21.13" y1="5.2" x2="21.13" y2="11.2" width="0.8" layer="1"/>
-<wire x1="21.6" y1="2.8" x2="21.13" y2="3.6" width="0.8" layer="1"/>
-<wire x1="21.13" y1="11.2" x2="21.2" y2="11.43" width="0.8" layer="1"/>
-<wire x1="21.6" y1="2.8" x2="21.5392" y2="2.54" width="0.8" layer="1"/>
-<wire x1="30.4" y1="5.2" x2="21.13" y2="5.2" width="0.8" layer="1"/>
+<wire x1="21.2" y1="2.8" x2="21.2" y2="5.2" width="0.8" layer="1"/>
+<wire x1="21.2" y1="5.2" x2="21.2" y2="11.43" width="0.8" layer="1"/>
+<wire x1="21.2" y1="2.8" x2="21.5392" y2="2.54" width="0.8" layer="1"/>
+<wire x1="30.4" y1="5.2" x2="21.2" y2="5.2" width="0.8" layer="1"/>
 <wire x1="30.4" y1="5.2" x2="30.48" y2="5.08" width="0.8" layer="1"/>
 </signal>

Commit message: proto 2 v 0.2 ready
Parts:
- removed S1: 9077-2, switch-misc:9077-2
- added CCON1: (no value), con-ptr500:AK300/2
Connections:
- net N$3: now also CCON1.1; no longer S1.2
- net N$7: now also CCON1.2; no longer S1.1
Routing:
- net N$3: track 10.0 -> 6.71 mm
Changed lines of the file:
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@@
 <element name="PR1" library="SparkFun-Passives" package="0805" value="470" x="12.7" y="57.15"/>
 <element name="WIFI" library="esp8266modules" package="ESP01" value="ESP01" x="35.56" y="57.15"/>
-<element name="S1" library="switch-misc" package="9077-2" value="9077-2" x="19.05" y="71.12"/>
 <element name="MSENS" library="con-amp-mt" package="S02P" value="" x="40.64" y="33.02" rot="R90">
 <attribute name="MF" value="" x="40.64" y="33.02" size="1.778" layer="27" rot="R90" display="off"/>
@@
 <element name="U$1" library="Arduino-Clk" package="ABK-PRO-MINI" value="ABK-PRO-MINI" x="12.7" y="40.64"/>
 <element name="U$2" library="Logo" package="IOTECH_COPPER" value="" x="40.64" y="11.43"/>
+<element name="CCON1" library="con-ptr500" package="AK300/2" value="" x="19.05" y="72.39" rot="R180">
+<attribute name="MF" value="" x="19.05" y="72.39" size="1.778" layer="27" rot="R180" display="off"/>
+<attribute name="MPN" value="" x="19.05" y="72.39" size="1.778" layer="27" rot="R180" display="off"/>
+<attribute name="OC_FARNELL" value="unknown" x="19.05" y="72.39" size="1.778" layer="27" rot="R180" display="off"/>
+<attribute name="OC_NEWARK" value="unknown" x="19.05" y="72.39" size="1.778" layer="27" rot="R180" display="off"/>
+</element>
 </elements>
 <signals>
@@
 <signal name="N$3">
 <contactref element="PD1" pad="A"/>
-<contactref element="S1" pad="2"/>
+<contactref element="CCON1" pad="1"/>
 <wire x1="24.4" y1="69.2" x2="26.4" y2="69.2" width="0.8" layer="1"/>
-<wire x1="22.4" y1="71.2" x2="24.4" y2="69.2" width="0.8" layer="1"/>
-<wire x1="20.8" y1="71.2" x2="22.4" y2="71.2" width="0.8" layer="1"/>
-<wire x1="19.2" y1="72.8" x2="20.8" y2="71.2" width="0.8" layer="1"/>
-<wire x1="19.2" y1="73.6" x2="19.2" y2="72.8" width="0.8" layer="1"/>
+<wire x1="21.6" y1="72" x2="24.4" y2="69.2" width="0.8" layer="1"/>
 <wire x1="26.4" y1="69.2" x2="26.67" y2="68.97" width="0.8" layer="1"/>
-<wire x1="19.2" y1="73.6" x2="19.05" y2="73.66" width="0.8" layer="1"/>
+<wire x1="21.6" y1="72" x2="21.5646" y2="72.39" width="0.8" layer="1"/>
 </signal>
 <signal name="N$7">
-<contactref element="S1" pad="1"/>
 <contactref element="J1" pad="VIN0"/>
+<contactref element="CCON1" pad="2"/>
 <wire x1="4.4" y1="72.8" x2="2.8" y2="72.8" width="0.8" layer="1"/>
 <wire x1="6.8" y1="70.4" x2="4.4" y2="72.8" width="0.8" layer="1"/>
-<wire x1="13.2" y1="70.4" x2="6.8" y2="70.4" width="0.8" layer="1"/>
-<wire x1="16.4" y1="73.6" x2="13.2" y2="70.4" width="0.8" layer="1"/>
+<wire x1="14.8" y1="70.4" x2="6.8" y2="70.4" width="0.8" layer="1"/>
+<wire x1="16.4" y1="72" x2="14.8" y2="70.4" width="0.8" layer="1"/>
 <wire x1="2.8" y1="72.8" x2="2.54" y2="73.01" width="0.8" layer="1"/>
-<wire x1="16.4" y1="73.6" x2="16.51" y2="73.66" width="0.8" layer="1"/>
+<wire x1="16.4" y1="72" x2="16.5608" y2="72.39" width="0.8" layer="1"/>
 </signal>
 <signal name="N$2">

Commit message: gcode
Parts:
- added U$3: (no value), Logo:IOTECH_COPPER_M
Other:
- board size 44.1 x 76.2 mm -> 45.4 x 77.5 mm
Changed lines of the file:
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@@
 <board>
 <plain>
-<wire x1="0" y1="0" x2="44.12" y2="0" width="0" layer="20"/>
-<wire x1="44.12" y1="0" x2="44.12" y2="76.19" width="0" layer="20"/>
-<wire x1="44.12" y1="76.19" x2="0" y2="76.19" width="0" layer="20"/>
-<wire x1="0" y1="76.19" x2="0" y2="0" width="0" layer="20"/>
+<wire x1="0" y1="0" x2="45.39" y2="0" width="0" layer="20"/>
+<wire x1="45.39" y1="0" x2="45.39" y2="77.46" width="0" layer="20"/>
+<wire x1="45.39" y1="77.46" x2="0" y2="77.46" width="0" layer="20"/>
+<wire x1="0" y1="77.46" x2="0" y2="0" width="0" layer="20"/>
 </plain>
 <attributes>
@@
 <attribute name="OC_NEWARK" value="unknown" x="19.05" y="72.39" size="1.778" layer="27" rot="R180" display="off"/>
 </element>
+<element name="U$3" library="Logo" package="IOTECH_COPPER_M" value="" x="34.29" y="66.04" rot="MR0"/>
 </elements>
 <signals>

Commit message: proto 2 in action
Parts:
- added U$4: (no value), Logo:IOTECH_COPPER_M
- moved U$2 28.4 mm to (15.2, 24.1)
- moved U$3 2.54 mm to (34.3, 63.5)
Changed lines of the file:
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@@
 <?xml version="1.0" encoding="utf-8"?>
 <!DOCTYPE eagle SYSTEM "eagle.dtd">
-<eagle version="8.1.1">
+<eagle version="8.0.2">
 <drawing>
 <settings>
@@
 <element name="CQ1" library="transistor-power" package="D2PACK" value="IRF3707S" x="30.48" y="7.62" rot="R180"/>
 <element name="U$1" library="Arduino-Clk" package="ABK-PRO-MINI" value="ABK-PRO-MINI" x="12.7" y="40.64"/>
-<element name="U$2" library="Logo" package="IOTECH_COPPER" value="" x="40.64" y="11.43"/>
+<element name="U$2" library="Logo" package="IOTECH_COPPER" value="" x="15.24" y="24.13"/>
 <element name="CCON1" library="con-ptr500" package="AK300/2" value="" x="19.05" y="72.39" rot="R180">
 <attribute name="MF" value="" x="19.05" y="72.39" size="1.778" layer="27" rot="R180" display="off"/>
@@
 <attribute name="OC_NEWARK" value="unknown" x="19.05" y="72.39" size="1.778" layer="27" rot="R180" display="off"/>
 </element>
-<element name="U$3" library="Logo" package="IOTECH_COPPER_M" value="" x="34.29" y="66.04" rot="MR0"/>
+<element name="U$3" library="Logo" package="IOTECH_COPPER_M" value="" x="34.29" y="63.5" rot="MR0"/>
+<element name="U$4" library="Logo" package="IOTECH_COPPER_M" value="" x="40.64" y="11.43"/>
 </elements>
 <signals>
