File: KMO_IO_M/KMO_IO_M.sch (EAGLE design)
At the start: 8 parts, among them IC1 LM317MBSTT3

Commit message: update
Parts:
- removed C1: 0.1uF, rcl:C-EU075-052X106
- removed C2: 1uF, resistor:CPOL-US085CS-1AR
- removed C3: 10uF, resistor:CPOL-US085CS-1AR
- removed D1, D2: 1N4002, diode:1N4004
- removed R1: 240Ω, resistor:R-US_M0805
- removed R2: 394Ω, resistor:R-US_M0805
- added F1: 1A, _hhn_PtcFuses_Siba_r500_Ozan:SIBA194600
- added IC2: 7808DT, linear:7808DT
- added ICON, ICON1: (no value), con-ptr500:AK300/2
- added ID1, ID2, PD1: (no value), SparkFun-DiscreteSemi:DIODESMA
- added IR1, IR2: 1K, SparkFun-Passives:RESISTOR0805-RES
- added J1: POWER_JACKTOE, SparkFun-Connectors:POWER_JACKTOE
- added JP1: (no value), jumper:JP1E
- added MC: ARDUINO_PRO_MINI, srg:ARDUINO_PRO_MINI
- added PC1: 10uf, SparkFun-Capacitors:CAP0805
- added PC2: 100nf, SparkFun-Capacitors:CAP0805
- added PC3: 1uf, SparkFun-Capacitors:CAP0805
- added PLED1: (no value), led:LEDCHIP-LED0805
- added PR1: 470, SparkFun-Passives:RESISTOR0805-RES
- added Q1, Q4: IRF3707S, transistor-power:IRF3704S
- added TR1, TR2: 4700, SparkFun-Passives:RESISTOR0805-RES
- added TSENS, TSENS1: (no value), con-amp-mt:S03P
- IC1: value LM317MBSTT3 -> REG1117; device v-reg:LM317MBSTT3 -> burr-brown:REG1117; PARTNUMBER LM317M -> (none)
Connections:
- removed net VIN: C1.1, D1.C, IC1.IN
- removed net VO: C2.+, D1.A, D2.C, IC1.OUT, R1.2
- new net A1: TR2.1, TSENS1-2.S
- new net D11: TR1.1, TSENS-2.S
- new net N$11: PLED1.A, PR1.1
- new net N$12: IC1.VIN, IC2.VO, PC2.2
- new net N$2: F1.1, JP1.1, PD1.C
- new net N$3: ICON-2.KL, ID1.A, Q4.D
- new net N$4: ICON1-2.KL, ID2.A, Q1.D
- new net N$7: J1.PWR, PD1.A
- new net OUT1: IR1.2, Q4.G
- new net OUT2: IR2.2, Q1.G
- new net RAW_IV: F1.2, IC2.VI, ICON-1.KL, ICON1-1.KL, ID1.C, ID2.C, JP1.2, PC3.2
- new net VCC3.3: IC1.VOUT, PC1.2, PR1.2, TR1.2, TR2.2, TSENS-1.S, TSENS1-1.S
- new net VCCSRV: MC.VCC$1
- net GND: now also IC1.GND, IC2.GND, IR1.1, IR2.1, J1.GNDBREAK, MC.GND$4, PC1.1, PC2.1, PC3.1, PLED1.C, Q1.S, Q4.S, TSENS-3.S, TSENS1-3.S; no longer C1.2, C2.-, C3.-, R2.1
- net N$1: now also MC.RAW; no longer C3.+, D2.A, IC1.ADJ, R1.1, R2.2
Other:
- note added: "IN1"
- note added: "NATIVE ANALOG-DIGITAL SENSOR"
- note added: "NATIVE DIGITAL SENSOR"
- note added: "OUT1"
- note added: "OUT2"
- note added: "POWER"
- note removed: "3.3V Voltage Regulator"
- note removed: "3.3V, 500mA"
- note removed: "3V to 40V DC"
- note removed: "C2 of 1 µF tantalum capacitor on the output helps to improve transient response"
- note removed: "C3 helps in ripple rejection upto 15dB"
- note removed: "D1 protect the device against input short circuit"
- note removed: "D2 protect against output short circuit for capacitance discharging"
- note removed: "Useful Notes"
- note removed: "Vref = 1.25V"

Commit message: lib
Connections:
- removed net VCCSRV: MC.VCC$1
- net VCC3.3: now also MC.VCC$1
Changed lines of the file:
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@@
-</segment>
-</net>
-<net name="VCCSRV" class="0">
-<segment>
-<pinref part="MC" gate="G$1" pin="VCC$1"/>
-<wire x1="66.04" y1="68.58" x2="73.66" y2="68.58" width="0.1524" layer="91"/>
-<label x="73.66" y="68.58" size="1.778" layer="95" xref="yes"/>
 </segment>
 </net>
@@
 <wire x1="190.5" y1="195.58" x2="193.04" y2="195.58" width="0.1524" layer="91"/>
 </segment>
+<segment>
+<pinref part="MC" gate="G$1" pin="VCC$1"/>
+<wire x1="66.04" y1="68.58" x2="73.66" y2="68.58" width="0.1524" layer="91"/>
+<label x="73.66" y="68.58" size="1.778" layer="95" xref="yes"/>
+</segment>
 </net>

Commit message: rj45
Parts:
- added M1: ETHERNET-ENC28J60, diy-modules:ETHERNET-ENC28J60
Changed lines of the file:
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@@
 <part name="ICON1" library="con-ptr500" deviceset="AK300/2" device=""/>
 <part name="Q1" library="transistor-power" deviceset="IRF3704" device="S" value="IRF3707S"/>
+<part name="M1" library="diy-modules" deviceset="ETHERNET-ENC28J60" device=""/>
 </parts>
 <sheets>
@@
 <instance part="ICON1" gate="-2" x="127" y="180.34" rot="R270"/>
 <instance part="Q1" gate="G$1" x="116.84" y="162.56"/>
+<instance part="M1" gate="G$1" x="116.84" y="109.22"/>
 </instances>
 <busses>

Commit message: input haric
Parts:
- removed ICON: (no value), con-ptr500:AK300/2
- removed M1: ETHERNET-ENC28J60, diy-modules:ETHERNET-ENC28J60
- removed Q4: IRF3707S, transistor-power:IRF3704S
- added ETH: ETHERNET-ENC28J60, diy-modules:ETHERNET-ENC28J60
- added ICON2: (no value), con-ptr500:AK300/2
- added Q2: IRF3707S, transistor-power:IRF3704S
- added WIFI: ESP01, esp8266modules:ESP01
- renumbered ID1 to OD1, ID2 to OD2, IR1 to OR1, IR2 to OR2, J1 to PJ1, JP1 to JPF1
Connections:
- removed net OUT1: OR1.2, Q4.G
- removed net OUT2: OR2.2, Q1.G
- new net A0: MC.A0, TR1.1, TSENS-2.S
- new net A2: MC.A2
- new net A3: MC.A3
- new net A4: MC.A4
- new net A5: MC.A5
- new net A6: MC.A6
- new net A7: MC.A7
- new net D10: ETH.CS, MC.D10
- new net D12: ETH.SO, MC.D12
- new net D13: ETH.SCK, MC.D13
- new net D2: ETH.INT, MC.D2
- new net D3: MC.D3, OR1.2, Q1.G
- new net D4: MC.D4, OR2.2, Q2.G
- new net D5: MC.D5, WIFI.RXD
- new net D6: MC.D6, WIFI.TXD
- new net D7: MC.D7
- new net D8: MC.D8
- new net D9: MC.D9
- new net N$5: ETH.5V
- net A1: now also MC.A1
- net D11: now also ETH.SI, MC.D11; no longer TR1.1, TSENS-2.S
- net GND: now also ETH.GND.1, Q2.S, WIFI.GND; no longer Q4.S
- net N$3: now also ICON1-2.KL, Q1.D; no longer ICON-2.KL, Q4.D
- net N$4: now also ICON2-2.KL, Q2.D; no longer ICON1-2.KL, Q1.D
- net RAW_IV: now also ICON2-1.KL; no longer ICON-1.KL
- net VCC3.3: now also ETH.3V3, WIFI.CH_PD, WIFI.VCC
Other:
- note added: "A0 NATIVE ANALOG-DIGITAL SENSOR 1"
- note added: "A1 NATIVE ANALOG-DIGITAL SENSOR 2"
- note added: "D10 ETH CS"
- note added: "D11 ETH SI"
- note added: "D12 ETH SO"
- note added: "D13 ETH SCK"
- note added: "D2 ETH INT"
- note added: "D3 OUT1"
- note added: "D4 OUT2"
- note added: "D5 WIFI RXD"
- note added: "D6 WIFI TXD"
- note added: "EMPTY"
- note added: "ETHERNET"
- note added: "NATIVE ANALOG-DIGITAL SENSOR 1"
- note added: "NATIVE ANALOG-DIGITAL SENSOR 2"
- note added: "WI-FI"
- note removed: "NATIVE ANALOG-DIGITAL SENSOR"
- note removed: "NATIVE DIGITAL SENSOR"
- moved on the sheet: ICON1-1, ICON1-2, MC, Q1

Commit message: isimlendirme std
Parts:
- renumbered F1 to PF1, IC1 to PIC1, IC2 to PIC2, ICON1 to OT1, ICON2 to OT2, JPF1 to PFJ1, Q1 to OQ1, Q2 to OQ2, TR1 to NIR1, TR2 to NIR2, TSENS to NIT1, TSENS1 to NIT2

Commit message: lib modified
Parts:
- ETH: value ETHERNET-ENC28J60 -> ETHERNET-ENC28J60_PER; device diy-modules:ETHERNET-ENC28J60 -> personal_diy-modules:ETHERNET-ENC28J60_PER
- MC: value ARDUINO_PRO_MINI -> ARDUINO_PRO_MINI2; device srg:ARDUINO_PRO_MINI -> personal_srgPersonal:ARDUINO_PRO_MINI2; SPICEPREFIX X -> (none)
Connections:
- removed net A4: MC.A4
- removed net A5: MC.A5
- removed net A6: MC.A6
- removed net A7: MC.A7
- removed net N$5: ETH.5V

Commit message: yerlestir
Parts:
- removed OT1, OT2: (no value), con-ptr500:AK300/2
- added OD3: (no value), SparkFun-DiscreteSemi:DIODESMA
- added OQ3: IRF3707S, transistor-power:IRF3704S
- added OR3: 1K, SparkFun-Passives:RESISTOR0805-RES
- added XI, XO: MSTBA6, con-phoenix-508:MSTBA6
Connections:
- net A0: no longer NIR1.1, NIT1-2.S
- net A1: no longer NIR2.1, NIT2-2.S
- net D3: now also WIFI.TXD; no longer OQ1.G, OR1.2
- net D4: now also WIFI.RXD; no longer OQ2.G, OR2.2
- net D5: now also OQ3.G, OR3.2; no longer WIFI.RXD
- net D6: now also OQ2.G, OR2.2; no longer WIFI.TXD
- net D7: now also OQ1.G, OR1.2
- net D8: now also NIR1.1, NIT1-2.S
- net D9: now also NIR2.1, NIT2-2.S
- net GND: now also OQ3.S, OR3.1
- net N$1: now also OD3.A, OQ3.D, XO-6.1; no longer MC.RAW
- net N$3: now also XO-2.1; no longer OT1-2.KL
- net N$4: now also XO-4.1; no longer OT2-2.KL
- net RAW_IV: now also OD3.C, XO-1.1, XO-3.1, XO-5.1; no longer OT1-1.KL, OT2-1.KL
Other:
- note added: "D3 WIFI TXD"
- note added: "D4 WIFI RXD"
- note added: "D5 OUT3"
- note added: "D6 OUT2"
- note added: "D7 OUT1"
- note added: "D8 NATIVE DIGITAL SENSOR 1"
- note added: "D9 NATIVE DIGITAL SENSOR 2"
- note added: "OUT3"
- note removed: "A0 NATIVE ANALOG-DIGITAL SENSOR 1"
- note removed: "A1 NATIVE ANALOG-DIGITAL SENSOR 2"
- note removed: "D3 OUT1"
- note removed: "D4 OUT2"
- note removed: "D5 WIFI RXD"
- note removed: "D6 WIFI TXD"

Commit message: input eksik
Parts:
- added MCA45J: (no value), jumper:JP1E
- added NIR3: 4700, SparkFun-Passives:RESISTOR0805-RES
- added NIT3: (no value), con-amp-mt:S03P
Connections:
- new net A4: MCA45J.1, NIR3.1, NIT3-2.S
- new net A5: MCA45J.2
- net GND: now also NIT3-3.S
- net VCC3.3: now also NIR3.2, NIT3-1.S
Other:
- note added: "NATIVE ANALOG-DIGITAL SENSOR 3"
- note added: "NATIVE DIGITAL SENSOR 1"
- note added: "NATIVE DIGITAL SENSOR 2"
- note removed: "NATIVE ANALOG-DIGITAL SENSOR 1"
- note removed: "NATIVE ANALOG-DIGITAL SENSOR 2"
Changed lines of the file:
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@@
 <part name="GND8" library="supply1" deviceset="GND" device=""/>
 <part name="OQ3" library="transistor-power" deviceset="IRF3704" device="S" value="IRF3707S"/>
+<part name="GND9" library="SparkFun-Aesthetics" deviceset="GND" device=""/>
+<part name="NIR3" library="SparkFun-Passives" deviceset="RESISTOR" device="0805-RES" value="4700"/>
+<part name="NIT3" library="con-amp-mt" deviceset="S03P" device=""/>
+<part name="MCA45J" library="jumper" library_urn="urn:adsk.eagle:library:252" deviceset="JP1E" device="" package3d_urn="urn:adsk.eagle:package:15455/1"/>
 </parts>
 <sheets>
@@
 <text x="27.94" y="175.26" size="1.778" layer="91">OUT1</text>
 <frame x1="0" y1="0" x2="381" y2="254" columns="8" rows="5" layer="91"/>
-<text x="180.34" y="236.22" size="1.778" layer="91">NATIVE ANALOG-DIGITAL SENSOR 1</text>
+<text x="180.34" y="236.22" size="1.778" layer="91">NATIVE DIGITAL SENSOR 1</text>
 <text x="27.94" y="144.78" size="1.778" layer="91">IN1</text>
-<text x="180.34" y="208.28" size="1.778" layer="91">NATIVE ANALOG-DIGITAL SENSOR 2</text>
+<text x="180.34" y="208.28" size="1.778" layer="91">NATIVE DIGITAL SENSOR 2</text>
 <text x="99.06" y="175.26" size="1.778" layer="91">OUT2</text>
 <text x="182.88" y="177.8" size="1.778" layer="91">WI-FI</text>
@@
 <text x="30.48" y="50.8" size="1.778" layer="97">D6 OUT2</text>
 <text x="30.48" y="53.34" size="1.778" layer="97">D5 OUT3</text>
+<text x="243.84" y="236.22" size="1.778" layer="91">NATIVE ANALOG-DIGITAL SENSOR 3</text>
 </plain>
 <instances>
@@
 <instance part="GND8" gate="1" x="66.04" y="101.6" rot="R90"/>
 <instance part="OQ3" gate="G$1" x="45.72" y="109.22"/>
+<instance part="GND9" gate="1" x="266.7" y="226.06" rot="R90"/>
+<instance part="NIR3" gate="G$1" x="276.86" y="226.06" rot="R270"/>
+<instance part="NIT3" gate="-1" x="248.92" y="223.52"/>
+<instance part="NIT3" gate="-2" x="248.92" y="228.6"/>
+<instance part="NIT3" gate="-3" x="248.92" y="226.06"/>
+<instance part="MCA45J" gate="A" x="58.42" y="38.1" rot="R270"/>
 </instances>
 <busses>
@@
 <junction x="48.26" y="101.6"/>
 </segment>
+<segment>
+<pinref part="GND9" gate="1" pin="GND"/>
+<pinref part="NIT3" gate="-3" pin="S"/>
+<wire x1="254" y1="226.06" x2="264.16" y2="226.06" width="0.1524" layer="91"/>
+</segment>
 </net>
 <net name="RAW_IV" class="1">
@@
 <junction x="226.06" y="162.56"/>
 </segment>
+<segment>
+<wire x1="256.54" y1="223.52" x2="256.54" y2="218.44" width="0.1524" layer="91"/>
+<wire x1="256.54" y1="218.44" x2="276.86" y2="218.44" width="0.1524" layer="91"/>
+<label x="284.48" y="218.44" size="1.778" layer="95" xref="yes"/>
+<pinref part="NIR3" gate="G$1" pin="2"/>
+<wire x1="276.86" y1="218.44" x2="284.48" y2="218.44" width="0.1524" layer="91"/>
+<wire x1="276.86" y1="220.98" x2="276.86" y2="218.44" width="0.1524" layer="91"/>
+<junction x="276.86" y="218.44"/>
+<pinref part="NIT3" gate="-1" pin="S"/>
+<wire x1="254" y1="223.52" x2="256.54" y2="223.52" width="0.1524" layer="91"/>
+</segment>
 </net>
 <net name="N$4" class="0">
@@
 </segment>
 </net>
+<net name="A4" class="0">
+<segment>
+<pinref part="MCA45J" gate="A" pin="1"/>
+<wire x1="55.88" y1="38.1" x2="53.34" y2="38.1" width="0.1524" layer="91"/>
+<label x="53.34" y="38.1" size="1.778" layer="95" rot="R180" xref="yes"/>
+</segment>
+<segment>
+<wire x1="256.54" y1="228.6" x2="256.54" y2="233.68" width="0.1524" layer="91"/>
+<wire x1="256.54" y1="233.68" x2="276.86" y2="233.68" width="0.1524" layer="91"/>
+<label x="284.48" y="233.68" size="1.778" layer="95" xref="yes"/>
+<pinref part="NIR3" gate="G$1" pin="1"/>
+<wire x1="276.86" y1="233.68" x2="284.48" y2="233.68" width="0.1524" layer="91"/>
+<wire x1="276.86" y1="231.14" x2="276.86" y2="233.68" width="0.1524" layer="91"/>
+<junction x="276.86" y="233.68"/>
+<pinref part="NIT3" gate="-2" pin="S"/>
+<wire x1="254" y1="228.6" x2="256.54" y2="228.6" width="0.1524" layer="91"/>
+</segment>
+</net>
+<net name="A5" class="0">
+<segment>
+<pinref part="MCA45J" gate="A" pin="2"/>
+<wire x1="55.88" y1="35.56" x2="48.26" y2="35.56" width="0.1524" layer="91"/>
+<label x="48.26" y="35.56" size="1.778" layer="95" rot="R180" xref="yes"/>
+</segment>
+</net>
