File: KMO_IO_M/KMO_IO_MV3.brd (EAGLE design)
At the start: 84.5 x 96.5 mm, 63 parts, among them IC1 ENC28J60SO, Q1 25MHz, U1 ENC28J60-SSOP, U2 Tyco 5-6605758-1

Commit message: evde
Parts:
- added EC3: 10u, rcl:E2,5-5
Connections:
- net GND: now also EC3.-
Changed lines of the file:
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@@
 <element name="R22" library="SparkFun-Passives" package="0805" value="100R" x="20" y="40.25"/>
 <element name="U1" library="microchip-enc28j60" package="SSOP28" value="ENC28J60-SSOP" x="7.25" y="42.5" rot="R270"/>
+<element name="EC3" library="rcl" package="E2,5-5" value="10u" x="-0.5" y="-3.25"/>
 </elements>
 <signals>
@@
 <contactref element="C13" pad="2"/>
 <contactref element="R19" pad="2"/>
+<contactref element="EC3" pad="-"/>
 <wire x1="78" y1="76.25" x2="78" y2="90.5" width="0" layer="19" extent="1-1"/>
 <wire x1="78" y1="62" x2="78" y2="76.25" width="0" layer="19" extent="1-1"/>
@@
 <wire x1="27.22" y1="35.17" x2="36.78" y2="35.17" width="0" layer="19" extent="1-1"/>
 <wire x1="30.6" y1="26.25" x2="27.22" y2="35.17" width="0" layer="19" extent="1-1"/>
-<wire x1="40.15" y1="25.5" x2="36.78" y2="35.17" width="0" layer="19" extent="1-1"/>
+<wire x1="40.15" y1="25.5" x2="30.6" y2="26.25" width="0" layer="19" extent="1-1"/>
 <wire x1="40.15" y1="21.25" x2="40.15" y2="25.5" width="0" layer="19" extent="1-1"/>
 <wire x1="44.25" y1="17.85" x2="40.15" y2="21.25" width="0" layer="19" extent="1-1"/>
@@
 <wire x1="79.8069" y1="23.2769" x2="72.1413" y2="22.647" width="0" layer="19" extent="1-1"/>
 <wire x1="81" y1="15.7" x2="79.8069" y2="23.2769" width="0" layer="19" extent="1-1"/>
-<wire x1="11.5" y1="55.02" x2="24.85" y2="53.25" width="0" layer="19" extent="1-1"/>
 <wire x1="37.14" y1="78.04" x2="37.39" y2="65.04" width="0" layer="19" extent="1-1"/>
 <wire x1="41.5" y1="78.4" x2="37.14" y2="78.04" width="0" layer="19" extent="1-1"/>
@@
 <wire x1="72.1413" y1="37.9325" x2="66.46" y2="34.695" width="0" layer="19" extent="1-1"/>
 <wire x1="80.1244" y1="37.2231" x2="72.1413" y2="37.9325" width="0" layer="19" extent="1-1"/>
+<wire x1="11.5" y1="55.02" x2="24.85" y2="53.25" width="0" layer="19" extent="1-1"/>
 <wire x1="13.25" y1="18.4" x2="30.6" y2="26.25" width="0" layer="19" extent="1-1"/>
 <wire x1="13.25" y1="13.4" x2="13.25" y2="18.4" width="0" layer="19" extent="1-1"/>
 <wire x1="13.25" y1="8.4" x2="13.25" y2="13.4" width="0" layer="19" extent="1-1"/>
 <wire x1="7.08" y1="26.87" x2="13.25" y2="18.4" width="0" layer="19" extent="1-1"/>
+<wire x1="0.77" y1="-3.25" x2="13.25" y2="8.4" width="0" layer="19" extent="1-1"/>
 </signal>
 <signal name="N$11">
@@
 <wire x1="27.22" y1="38.98" x2="19.1" y2="40.25" width="0" layer="19" extent="1-1"/>
 </signal>
+<signal name="VSS">
+<contactref element="U1" pad="2"/>
+</signal>
+<signal name="VSSRX">
+<contactref element="U1" pad="11"/>
+</signal>
+<signal name="VDDTX">
+<contactref element="U1" pad="15"/>
+</signal>
+<signal name="VSSTX">
+<contactref element="U1" pad="18"/>
+</signal>
+<signal name="VDDPLL">
+<contactref element="U1" pad="20"/>
+</signal>
+<signal name="VDDRX">
+<contactref element="U1" pad="19"/>
+</signal>
+<signal name="VSSPLL">
+<contactref element="U1" pad="21"/>
+</signal>
+<signal name="VSSOSC">
+<contactref element="U1" pad="22"/>
+</signal>
+<signal name="VDDOSC">
+<contactref element="U1" pad="25"/>
+</signal>
+<signal name="VDD">
+<contactref element="U1" pad="28"/>
+</signal>
 <signal name="VCAP">
 <contactref element="U1" pad="1"/>
 </signal>
-<signal name="VSS">
-<contactref element="U1" pad="2"/>
-</signal>
-<signal name="VSSRX">
-<contactref element="U1" pad="11"/>
-</signal>
-<signal name="VDDTX">
-<contactref element="U1" pad="15"/>
-</signal>
-<signal name="VSSTX">
-<contactref element="U1" pad="18"/>
-</signal>
-<signal name="VDDPLL">
-<contactref element="U1" pad="20"/>
-</signal>
-<signal name="VDDRX">
-<contactref element="U1" pad="19"/>
-</signal>
-<signal name="VSSPLL">
-<contactref element="U1" pad="21"/>
-</signal>
-<signal name="VSSOSC">
-<contactref element="U1" pad="22"/>
-</signal>
-<signal name="VDDOSC">
-<contactref element="U1" pad="25"/>
-</signal>
-<signal name="VDD">
-<contactref element="U1" pad="28"/>
-</signal>
 </signals>

Commit message: eth
Parts:
- removed C1, C2: 22p, SparkFun-Passives:0805
- removed C11, C12, C15, C5, C6, C8: 100n, SparkFun-Passives:0805
- removed C13: 10n, SparkFun-Passives:0805
- removed C3: 10u, rcl:E2,5-5
- removed IC1: ENC28J60SO, microchip-6:SO28W
- removed L2: 3.3µH/±20%/450mA, SparkFun-Coils:0805
- removed Q1: 25MHz, crystal:HC49/S
- removed R1: 2k7, SparkFun-Passives:0805
- removed R10, R11, R13, R14, R15, R16, R17, R18, R20, R21, R22: 100R, SparkFun-Passives:0805
- removed R19: 15k, SparkFun-Passives:0805
- removed R2, R6: 10k, SparkFun-Passives:0805
- removed U1: ENC28J60-SSOP, microchip-enc28j60:SSOP28
- removed U2: Tyco 5-6605758-1, con-tycoelectronics-1:5-6605758-1
- added EC1, EC2: 100n, SparkFun-Passives:0805
- added EC4, EC5: 22p, SparkFun-Passives:0805
- added EL1: 3.3µH/±20%/450mA, SparkFun-Coils:0805
- added ENC: ENC28J60-SSOP, microchip-enc28j60:SSOP28
- added ER1, ER2, ER3, ER4: 50R, SparkFun-Passives:0805
- added ER10, ER8, ER9: 100R, SparkFun-Passives:0805
- added ER5: 2.3K, SparkFun-Passives:0805
- added ER6, ER7: 10k, SparkFun-Passives:0805
- added EU: Tyco 5-6605758-1, con-tycoelectronics-1:5-6605758-1
- added Q2: 25MHz, crystal:HC49/S
- moved EC3 65.6 mm to (37.5, 50.2), turned to 180 degrees
Connections:
- removed net N$10: C13.1, R15.1, R16.1, R17.1, R18.1
- removed net N$16: C15.1, L2.1, R10.2, R11.2, R13.2, R14.2, U2.4
- removed net N$23: IC1.8, R22.1
- removed net N$9: IC1.14, R1.1, R19.1
- removed net RST: IC1.10, R2.1
- removed net TPIN+: IC1.13, R17.2, R18.2, U2.1
- removed net TPIN-: IC1.12, R15.2, R16.2, U2.2
- removed net TPOUT+: IC1.17, R10.1, R11.1, U2.5
- removed net TPOUT-: IC1.16, R13.1, R14.1, U2.6
- removed net VCAP: U1.1
- removed net VDD: U1.28
- removed net VDDOSC: U1.25
- removed net VDDPLL: U1.20
- removed net VDDRX: U1.19
- removed net VDDTX: U1.15
- removed net VSS: U1.2
- removed net VSSOSC: U1.22
- removed net VSSPLL: U1.21
- removed net VSSRX: U1.11
- removed net VSSTX: U1.18
- new net N$13: EC3.+, ENC.1
- new net N$14: ENC.9, ER10.1, ER7.1
- new net N$15: ENC.7, ER8.1
- new net N$17: ENC.10, ER6.1
- new net N$18: ENC.8, ER9.1
- new net N$19: ENC.14, ER5.1
- new net N$22: EC5.1, ENC.24, Q2.1
- new net N$24: EC4.1, ENC.23, Q2.2
- new net N$26: ENC.13, ER4.2, EU.1
- net +3V3: now also EL1.1, ENC.15, ENC.19, ENC.20, ENC.25, ENC.28, ER6.2, ER7.2; no longer C11.1, C12.1, C5.1, C6.1, C8.1, IC1.15, IC1.19, IC1.20, IC1.25, IC1.28, L2.2, R2.2, R6.2
- net D10: now also ER10.2; no longer R21.2
- net D11: now also ER8.2; no longer R20.2
- net D12: now also ENC.6; no longer IC1.6
- net D13: now also ER9.2; no longer R22.2
- net D2: now also ENC.4; no longer IC1.4
- net GND: now also EC1.2, EC2.2, EC4.2, EC5.2, ENC.11, ENC.18, ENC.2, ENC.21, ENC.22, ER5.2, EU.8, EU.D2, EU.D4, EU.M1, EU.M2; no longer C1.2, C11.2, C12.2, C13.2, C15.2, C2.2, C3.-, C5.2, C6.2, C8.2, IC1.11, IC1.18, IC1.2, IC1.21, IC1.22, R1.2, R19.2, U2.8, U2.D2, U2.D4, U2.M1, U2.M2
- net LEDA: now also ENC.27, EU.D3; no longer IC1.27, U2.D3
- net LEDB: now also ENC.26, EU.D1; no longer IC1.26, U2.D1
- net N$20: now also ENC.16, ER1.1, EU.6; no longer IC1.7, R20.1
- net N$21: now also ENC.12, ER3.2, EU.2; no longer IC1.9, R21.1, R6.1
- net N$5: now also EC1.1, EL1.2, ER1.2, ER2.2, EU.4; no longer C1.1, IC1.23, Q1.1
- net N$6: now also EC2.1, ER3.1, ER4.1; no longer C2.1, IC1.24, Q1.2
- net N$8: now also ENC.17, ER2.1, EU.5; no longer C3.+, IC1.1
Routing:
- net GND: track 0.00 -> 441.4 mm, vias 0 -> 1
- net +3V3: track 0.00 -> 281.5 mm, vias 0 -> 5
- net RAW_IV: track 0.00 -> 174.4 mm
- net A2: track 0.00 -> 99.8 mm, vias 0 -> 2
- net A3: track 0.00 -> 95.8 mm, vias 0 -> 2
- net A1: track 0.00 -> 95.7 mm
- net D4: track 0.00 -> 84.8 mm
- net D3: track 0.00 -> 74.5 mm
- net D10: track 0.00 -> 64.5 mm
- net D13: track 0.00 -> 59.6 mm
- net D12: track 0.00 -> 58.2 mm, vias 0 -> 2
- net D11: track 0.00 -> 55.2 mm, vias 0 -> 1
- net LEDA: track 0.00 -> 53.0 mm
- net N$26: track 0.00 -> 48.6 mm, vias 0 -> 1
- net D2: track 0.00 -> 48.4 mm
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
Commit message: route
Parts:
- added C2: (no value), rcl:SANYO-OSCON_SMD_B6
Routing:
- net LEDB: track 0.00 -> 50.9 mm, vias 0 -> 3
Changed lines of the file:
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@@
 <element name="EU" library="con-tycoelectronics-1" package="5-6605758-1" value="Tyco 5-6605758-1" x="69" y="35.25" rot="R90"/>
 <element name="EC2" library="SparkFun-Passives" package="0805" value="100n" x="51.25" y="28.75" rot="R180"/>
+<element name="C2" library="rcl" library_urn="urn:adsk.eagle:library:334" package="SANYO-OSCON_SMD_B6" package3d_urn="urn:adsk.eagle:package:23461/1" value="" x="23.5" y="24">
+<attribute name="SPICEPREFIX" value="C" x="23.5" y="24" size="1.778" layer="27" display="off"/>
+</element>
 </elements>
 <signals>
@@
 <contactref element="EU" pad="D1"/>
 <contactref element="ENC" pad="26"/>
-<wire x1="44.125" y1="36.925" x2="77.9018" y2="28.2768" width="0" layer="19" extent="1-1"/>
+<wire x1="47.20281875" y1="39" x2="48.25" y2="39" width="0.3" layer="1"/>
+<wire x1="44.125" y1="36.925" x2="44.274978125" y2="36.975" width="0.3" layer="1"/>
+<wire x1="44.274978125" y1="36.975" x2="45.17781875" y2="36.975" width="0.3" layer="1"/>
+<wire x1="45.17781875" y1="36.975" x2="47.20281875" y2="39" width="0.3" layer="1"/>
+<via x="48.25" y="39" extent="1-16" drill="0.5"/>
+<wire x1="48.25" y1="39" x2="58" y2="48.75" width="0.3" layer="16"/>
+<via x="58" y="48.75" extent="1-16" drill="0.5"/>
+<wire x1="58" y1="48.75" x2="62.2" y2="44.55" width="0.3" layer="1"/>
+<wire x1="62.2" y1="44.55" x2="62.37781875" y2="44.55" width="0.3" layer="1"/>
+<wire x1="62.37781875" y1="44.55" x2="62.42781875" y2="44.5" width="0.3" layer="1"/>
+<wire x1="62.42781875" y1="44.5" x2="67.75" y2="44.5" width="0.3" layer="1"/>
+<via x="67.75" y="44.5" extent="1-16" drill="0.5"/>
+<wire x1="78.1162" y1="28.3892" x2="77.9528" y2="28.2258" width="0.3" layer="16"/>
+<wire x1="67.75" y1="44.5" x2="78.1162" y2="34.1338" width="0.3" layer="16"/>
+<wire x1="78.1162" y1="34.1338" x2="78.1162" y2="28.3892" width="0.3" layer="16"/>
+<wire x1="77.9528" y1="28.2258" x2="77.9018" y2="28.2768" width="0" layer="19" extent="16-16"/>
 </signal>
 <signal name="N$13">

Commit message: KMOV3 cam
Parts:
- removed C2: (no value), rcl:SANYO-OSCON_SMD_B6
- EC3: value 10u -> (none); device rcl:E2,5-5 -> rcl:SANYO-OSCON_SMD_B6
- moved Q2 11.5 mm to (53.0, 42.0)
- moved EC3 6.41 mm to (39.8, 44.2), turned to 0 degrees
- moved ER10 4.50 mm to (28.0, 35.0), flipped to the top
- moved EL1 1.25 mm to (60.2, 42.2)
Routing:
- net RAW_IV: track 174.4 -> 192.0 mm
- net D7: track 31.5 -> 44.6 mm
- net N$24: track 28.5 -> 16.8 mm
- net N$22: track 23.8 -> 12.1 mm
- net N$26: track 48.6 -> 36.9 mm, vias 1 -> 2
- net GND: track 441.4 -> 451.3 mm, vias 1 -> 0
- net LEDB: track 50.9 -> 60.6 mm, vias 3 -> 0
- net A2: track 99.8 -> 90.3 mm
- net A1: track 95.7 -> 86.9 mm, vias 0 -> 1
- net LEDA: track 53.0 -> 48.3 mm
- net N$13: track 12.9 -> 8.45 mm
- net N$14: track 6.36 -> 10.8 mm, vias 1 -> 2
- net D12: track 58.2 -> 61.7 mm
- net D13: track 59.6 -> 56.2 mm
- net A3: track 95.8 -> 92.7 mm
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
Commit message: v03
Parts:
- removed ER10: 100R, SparkFun-Passives:0805
- removed EU: Tyco 5-6605758-1, con-tycoelectronics-1:5-6605758-1
- added U$1: (no value), Logo:IOTECH_COPPER_W_TEXT
- added U$2: HR911105A, HR911105A:RJ45
- EC3: value (none) -> 10u
- ER8, ER9: value 100R -> 250R
- moved ER9 47.7 mm to (77.2, 49.8)
- moved ER8 46.4 mm to (77.2, 46.8), turned to 180 degrees
- moved WIFI 11.3 mm to (29.0, 16.8), turned to 90 degrees
- moved EC3 9.33 mm to (31.0, 41.0), turned to 90 degrees
- moved ER5 1.25 mm to (33.0, 28.5), turned to 180 degrees
- moved ER6 0.50 mm to (31.5, 31.2)
Connections:
- removed net N$15: ENC.7, ER8.1
- removed net N$18: ENC.8, ER9.1
- removed net N$20: ENC.16, ER1.1, EU.6
- removed net N$21: ENC.12, ER3.2, EU.2
- removed net N$26: ENC.13, ER4.2, EU.1
- removed net N$5: EC1.1, EL1.2, ER1.2, ER2.2, EU.4
- removed net N$8: ENC.17, ER2.1, EU.5
- new net EP4: EC1.1, EL1.2, ER1.2, ER2.2, U$2.P4
- new net N$9: ENC.27, ER8.2
- new net RD+: ENC.13, ER4.2, U$2.RD+
- new net RD-: ENC.12, ER3.2, U$2.RD-
- new net TD+: ENC.17, ER2.1, U$2.TD+
- new net TD-: ENC.16, ER1.1, U$2.TD-
- net D10: now also ENC.9, ER7.1; no longer ER10.2
- net D11: now also ENC.7; no longer ER8.2
- net D13: now also ENC.8; no longer ER9.2
- net GND: now also U$2.G-, U$2.GND, U$2.SHIELD1, U$2.SHIELD2, U$2.Y-; no longer EU.8, EU.D2, EU.D4, EU.M1, EU.M2
- net LEDA: now also ER8.1, U$2.Y+; no longer ENC.27, EU.D3
- net LEDB: now also ER9.1, U$2.G+; no longer ENC.26, EU.D1
- net N$14: now also ENC.26, ER9.2; no longer ENC.9, ER10.1, ER7.1
Routing:
- net RD+: track 0.00 -> 47.3 mm, vias 0 -> 2
- net TD+: track 0.00 -> 46.5 mm
- net LEDA: track 48.3 -> 5.97 mm
- net N$20: track 42.1 -> 0.00 mm
- net N$9: track 0.00 -> 39.0 mm
- net N$21: track 37.0 -> 0.00 mm
- net N$26: track 36.9 -> 0.00 mm, vias 2 -> 0
- net LEDB: track 60.6 -> 24.6 mm
- net RD-: track 0.00 -> 35.5 mm, vias 0 -> 3
- net N$8: track 33.6 -> 0.00 mm, vias 1 -> 0
- net N$14: track 10.8 -> 39.0 mm
- net TD-: track 0.00 -> 27.7 mm
- net +3V3: track 279.0 -> 251.8 mm, vias 4 -> 6
- net N$5: track 24.8 -> 0.00 mm
- net EP4: track 0.00 -> 23.2 mm
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Other:
- outline, holes or cut-outs redrawn
- board text added: "IOTB v0.3 TOP"
- board text added: "IOTECH © 2018"
- board text removed: "IOTB v0.1 TOP"
- board text removed: "IOTECH 2018"
