File: KMO_IO_M/KMO_IO_MV3.sch (EAGLE design)
At the start: 63 parts, among them IC1 ENC28J60SO, Q1 25MHz, U1 ENC28J60-SSOP, U2 Tyco 5-6605758-1

Commit message: evde
Parts:
- added EC3: 10u, rcl:CPOL-EUE2.5-5
Connections:
- net GND: now also EC3.-
Other:
- moved on the sheet: U1
Changed lines of the file:
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@@
 <part name="FRAME2" library="frames" library_urn="urn:adsk.eagle:library:229" deviceset="LETTER_L" device=""/>
 <part name="U1" library="microchip-enc28j60" deviceset="ENC28J60-*" device="SSOP"/>
+<part name="GND14" library="supply1" deviceset="GND" device=""/>
+<part name="EC3" library="rcl" deviceset="CPOL-EU" device="E2.5-5" value="10u"/>
 </parts>
 <sheets>
@@
 </instance>
 <instance part="FRAME2" gate="G$2" x="274.32" y="5.08"/>
-<instance part="U1" gate="G$1" x="43.18" y="132.08"/>
+<instance part="U1" gate="G$1" x="83.9" y="107.68"/>
+<instance part="GND14" gate="1" x="48.45" y="84.55"/>
+<instance part="EC3" gate="G$1" x="48.45" y="97.25"/>
 </instances>
 <busses>
@@
 <pinref part="R19" gate="G$1" pin="2"/>
 </segment>
-</net>
+<segment>
+<wire x1="48.45" y1="87.09" x2="48.45" y2="89.63" width="0.1524" layer="91"/>
+<wire x1="48.45" y1="89.63" x2="58.61" y2="89.63" width="0.1524" layer="91"/>
+<wire x1="48.45" y1="89.63" x2="48.45" y2="92.17" width="0.1524" layer="91"/>
+<junction x="48.45" y="89.63"/>
+<pinref part="GND14" gate="1" pin="GND"/>
+<pinref part="EC3" gate="G$1" pin="-"/>
+</segment>
+</net>

Commit message: eth
Parts:
- removed C1, C2: 22p, SparkFun-Passives:CAP0805
- removed C11, C12, C15, C5, C6, C8: 100n, SparkFun-Passives:CAP0805
- removed C13: 10n, SparkFun-Passives:CAP0805
- removed C3: 10u, rcl:CPOL-EUE2.5-5
- removed IC1: ENC28J60SO, microchip-6:ENC28J60SO
- removed L2: 3.3µH/±20%/450mA, SparkFun-Coils:INDUCTOR-0805-3.3UH
- removed Q1: 25MHz, crystal:CRYSTALHC49S
- removed R1: 2k7, SparkFun-Passives:RESISTOR0805-RES
- removed R10, R11, R13, R14, R15, R16, R17, R18, R20, R21, R22: 100R, SparkFun-Passives:RESISTOR0805-RES
- removed R19: 15k, SparkFun-Passives:RESISTOR0805-RES
- removed R2, R6: 10k, SparkFun-Passives:RESISTOR0805-RES
- removed U1: ENC28J60-SSOP, microchip-enc28j60:ENC28J60-SSOP
- removed U2: Tyco 5-6605758-1, con-tycoelectronics-1:5-6605758-1
- added EC1, EC2: 100n, SparkFun-Passives:CAP0805
- added EC4, EC5: 22p, SparkFun-Passives:CAP0805
- added EL1: 3.3µH/±20%/450mA, SparkFun-Coils:INDUCTOR-0805-3.3UH
- added ENC: ENC28J60-SSOP, microchip-enc28j60:ENC28J60-SSOP
- added ER1, ER2, ER3, ER4: 50R, SparkFun-Passives:RESISTOR0805-RES
- added ER10, ER8, ER9: 100R, SparkFun-Passives:RESISTOR0805-RES
- added ER5: 2.3K, SparkFun-Passives:RESISTOR0805-RES
- added ER6, ER7: 10k, SparkFun-Passives:RESISTOR0805-RES
- added EU: Tyco 5-6605758-1, con-tycoelectronics-1:5-6605758-1
- added Q2: 25MHz, crystal:CRYSTALHC49S
Connections:
- removed net N$10: C13.1, R15.1, R16.1, R17.1, R18.1
- removed net N$16: C15.1, L2.1, R10.2, R11.2, R13.2, R14.2, U2.CT1
- removed net N$23: IC1.SCK, R22.1
- removed net N$9: IC1.RBIAS, R1.1, R19.1
- removed net RST: IC1.!RESET, R2.1
- removed net TPIN+: IC1.TPIN+, R17.2, R18.2, U2.RD+1
- removed net TPIN-: IC1.TPIN-, R15.2, R16.2, U2.RD-1
- removed net TPOUT+: IC1.TPOUT+, R10.1, R11.1, U2.TD+1
- removed net TPOUT-: IC1.TPOUT-, R13.1, R14.1, U2.TD-1
- new net N$13: EC3.+, ENC.VCAP
- new net N$14: ENC.CS, ER10.1, ER7.1
- new net N$15: ENC.SI, ER8.1
- new net N$17: ENC.RESET, ER6.1
- new net N$18: ENC.SCK, ER9.1
- new net N$19: ENC.RBIAS, ER5.1
- new net N$22: EC5.1, ENC.OSC2, Q2.1
- new net N$24: EC4.1, ENC.OSC1, Q2.2
- new net N$26: ENC.TPIN+, ER4.2, EU.RD+1
- net +3V3: now also EL1.1, ENC.VDD, ENC.VDDOSC, ENC.VDDPLL, ENC.VDDRX, ENC.VDDTX, ER6.2, ER7.2; no longer C11.1, C12.1, C5.1, C6.1, C8.1, IC1.VDD, IC1.VDDOSC, IC1.VDDPLL, IC1.VDDRX, IC1.VDDTX, L2.2, R2.2, R6.2
- net D10: now also ER10.2; no longer R21.2
- net D11: now also ER8.2; no longer R20.2
- net D12: now also ENC.SO; no longer IC1.SO
- net D13: now also ER9.2; no longer R22.2
- net D2: now also ENC.INT; no longer IC1.!INT
- net GND: now also EC1.2, EC2.2, EC4.2, EC5.2, ENC.VSS, ENC.VSSOSC, ENC.VSSPLL, ENC.VSSRX, ENC.VSSTX, ER5.2, EU.D2, EU.D4, EU.SH@1, EU.SH@2, EU.SH@3; no longer C1.2, C11.2, C12.2, C13.2, C15.2, C2.2, C3.-, C5.2, C6.2, C8.2, IC1.VSS, IC1.VSSOSC, IC1.VSSPLL, IC1.VSSRX, IC1.VSSTX, R1.2, R19.2, U2.D2, U2.D4, U2.SH@1, U2.SH@2, U2.SH@3
- net LEDA: now also ENC.LEDA, EU.D3; no longer IC1.LEDA, U2.D3
- net LEDB: now also ENC.LEDB, EU.D1; no longer IC1.LEDB, U2.D1
- net N$20: now also ENC.TPOUT-, ER1.1, EU.TD-1; no longer IC1.SI, R20.1
- net N$21: now also ENC.TPIN-, ER3.2, EU.RD-1; no longer IC1.!CS, R21.1, R6.1
- net N$5: now also EC1.1, EL1.2, ER1.2, ER2.2, EU.CT1; no longer C1.1, IC1.OSC1, Q1.1
- net N$6: now also EC2.1, ER3.1, ER4.1; no longer C2.1, IC1.OSC2, Q1.2
- net N$8: now also ENC.TPOUT+, ER2.1, EU.TD+1; no longer C3.+, IC1.VCAP
Other:
- note removed: "For new Revs RBAIS needs to be 2.32k, achived via 2k7 parallel to 15k."
- note removed: "NOTE: R12 is NOT required for Rev1 and Rev4 of ENC28J60."

Commit message: route
Parts:
- added C2: (no value), rcl:CPOL-EUSANYO_SMD_B6
Changed lines of the file:
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@@
 <part name="EC2" library="SparkFun-Passives" deviceset="CAP" device="0805" value="100n"/>
 <part name="GND15" library="supply1" deviceset="GND" device=""/>
+<part name="C2" library="rcl" library_urn="urn:adsk.eagle:library:334" deviceset="CPOL-EU" device="SANYO_SMD_B6" package3d_urn="urn:adsk.eagle:package:23461/1"/>
 </parts>
 <sheets>
@@
 <instance part="EC2" gate="G$1" x="139.7" y="144.78"/>
 <instance part="GND15" gate="1" x="147.32" y="132.08"/>
+<instance part="C2" gate="G$1" x="25.4" y="116.84"/>
 </instances>
 <busses>
@@
 packages will not be understood (or retained) with this version.
 </note>
+<note version="8.4" severity="warning">
+Since Version 8.4, EAGLE supports properties for SPICE simulation.
+Probes in schematics and SPICE mapping objects found in parts and library devices
+will not be understood with this version. Update EAGLE to the latest version
+for full support of SPICE simulation.
+</note>
 </compatibility>

Commit message: KMOV3 cam
Parts:
- removed C2: (no value), rcl:CPOL-EUSANYO_SMD_B6
- EC3: value 10u -> (none); device rcl:CPOL-EUE2.5-5 -> rcl:CPOL-EUSANYO_SMD_B6
Changed lines of the file:
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@@
 <part name="FRAME2" library="frames" library_urn="urn:adsk.eagle:library:229" deviceset="LETTER_L" device=""/>
 <part name="ENC" library="microchip-enc28j60" deviceset="ENC28J60-*" device="SSOP"/>
-<part name="EC3" library="rcl" deviceset="CPOL-EU" device="E2.5-5" value="10u"/>
 <part name="ER6" library="SparkFun-Passives" deviceset="RESISTOR" device="0805-RES" value="10k"/>
 <part name="ER7" library="SparkFun-Passives" deviceset="RESISTOR" device="0805-RES" value="10k"/>
@@
 <part name="EC2" library="SparkFun-Passives" deviceset="CAP" device="0805" value="100n"/>
 <part name="GND15" library="supply1" deviceset="GND" device=""/>
-<part name="C2" library="rcl" library_urn="urn:adsk.eagle:library:334" deviceset="CPOL-EU" device="SANYO_SMD_B6" package3d_urn="urn:adsk.eagle:package:23461/1"/>
+<part name="EC3" library="rcl" library_urn="urn:adsk.eagle:library:334" deviceset="CPOL-EU" device="SANYO_SMD_B6" package3d_urn="urn:adsk.eagle:package:23461/1"/>
 </parts>
 <sheets>
@@
 <instance part="FRAME2" gate="G$2" x="274.32" y="5.08"/>
 <instance part="ENC" gate="G$1" x="83.82" y="190.5"/>
-<instance part="EC3" gate="G$1" x="45.72" y="177.8"/>
 <instance part="ER6" gate="G$1" x="43.18" y="218.44" rot="R90"/>
 <instance part="ER7" gate="G$1" x="20.32" y="218.44" rot="R90"/>
@@
 <instance part="EC2" gate="G$1" x="139.7" y="144.78"/>
 <instance part="GND15" gate="1" x="147.32" y="132.08"/>
-<instance part="C2" gate="G$1" x="25.4" y="116.84"/>
+<instance part="EC3" gate="G$1" x="45.72" y="177.8"/>
 </instances>
 <busses>
@@
 <pinref part="GND16" gate="1" pin="GND"/>
 <wire x1="81.28" y1="165.1" x2="81.28" y2="162.56" width="0.1524" layer="91"/>
-<pinref part="EC3" gate="G$1" pin="-"/>
 <wire x1="45.72" y1="172.72" x2="45.72" y2="165.1" width="0.1524" layer="91"/>
 <wire x1="45.72" y1="165.1" x2="55.88" y2="165.1" width="0.1524" layer="91"/>
@@
 <junction x="111.76" y="165.1"/>
 <junction x="86.36" y="165.1"/>
+<pinref part="EC3" gate="G$1" pin="-"/>
 </segment>
 <segment>
@@
 <segment>
 <pinref part="ENC" gate="G$1" pin="VCAP"/>
-<pinref part="EC3" gate="G$1" pin="+"/>
 <wire x1="58.42" y1="182.88" x2="45.72" y2="182.88" width="0.1524" layer="91"/>
 <wire x1="45.72" y1="182.88" x2="45.72" y2="180.34" width="0.1524" layer="91"/>
-</segment>
-</net>
+<pinref part="EC3" gate="G$1" pin="+"/>
+</segment>
+</net>

Commit message: v03
Parts:
- removed ER10: 100R, SparkFun-Passives:RESISTOR0805-RES
- removed EU: Tyco 5-6605758-1, con-tycoelectronics-1:5-6605758-1
- added U$2: HR911105A, HR911105A:HR911105A
- EC3: value (none) -> 10u
- ER8, ER9: value 100R -> 250R
Connections:
- removed net N$15: ENC.SI, ER8.1
- removed net N$18: ENC.SCK, ER9.1
- removed net N$20: ENC.TPOUT-, ER1.1, EU.TD-1
- removed net N$21: ENC.TPIN-, ER3.2, EU.RD-1
- removed net N$26: ENC.TPIN+, ER4.2, EU.RD+1
- removed net N$5: EC1.1, EL1.2, ER1.2, ER2.2, EU.CT1
- removed net N$8: ENC.TPOUT+, ER2.1, EU.TD+1
- new net EP4: EC1.1, EL1.2, ER1.2, ER2.2, U$2.P4
- new net N$9: ENC.LEDA, ER8.2
- new net RD+: ENC.TPIN+, ER4.2, U$2.RD+
- new net RD-: ENC.TPIN-, ER3.2, U$2.RD-
- new net TD+: ENC.TPOUT+, ER2.1, U$2.TD+
- new net TD-: ENC.TPOUT-, ER1.1, U$2.TD-
- net D10: now also ENC.CS, ER7.1; no longer ER10.2
- net D11: now also ENC.SI; no longer ER8.2
- net D13: now also ENC.SCK; no longer ER9.2
- net GND: now also U$2.G-, U$2.GND, U$2.SHIELD0, U$2.SHIELD1, U$2.Y-; no longer EU.D2, EU.D4, EU.SH@1, EU.SH@2, EU.SH@3
- net LEDA: now also ER8.1, U$2.Y+; no longer ENC.LEDA, EU.D3
- net LEDB: now also ER9.1, U$2.G+; no longer ENC.LEDB, EU.D1
- net N$14: now also ENC.LEDB, ER9.2; no longer ENC.CS, ER10.1, ER7.1
