File: KMO_IO_M/KMO_IO_MV4.sch (EAGLE design)
At the start: 51 parts, among them Q2 25MHz

Commit message: ttl v4
Parts:
- added PP: 22-05-7048-04, con-molex:22-05-7048-04
- added X1: SSW-101-02-G-S, con-samtec:SSW-101-02-G-S
Connections:
- new net BLK: PP-1.S, X1.1
- new net RX: MC.RX1$1, PP-4.S
- new net TX: MC.TX0$1, PP-3.S
- net GND: now also MC.GND$1, PP-2.S
Other:
- note added: "0.4"
- note added: "MC"
- note added: "TTL"
- note removed: "0.3"
Changed lines of the file:
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@@
 <part name="ER6" library="SparkFun-Passives" deviceset="RESISTOR" device="0805-RES" value="10k"/>
 <part name="ER7" library="SparkFun-Passives" deviceset="RESISTOR" device="0805-RES" value="10k"/>
-<part name="+3V5" library="supply1" deviceset="+3V3" device=""/>
 <part name="ER5" library="SparkFun-Passives" deviceset="RESISTOR" device="0805-RES" value="2.3K"/>
 <part name="Q2" library="crystal" deviceset="CRYSTAL" device="HC49S" value="25MHz"/>
@@
 <part name="EC1" library="SparkFun-Passives" deviceset="CAP" device="0805" value="100n"/>
 <part name="EL1" library="SparkFun-Coils" deviceset="INDUCTOR" device="-0805-3.3UH" value="3.3µH/±20%/450mA"/>
-<part name="+3V1" library="supply1" deviceset="+3V3" device=""/>
-<part name="GND7" library="supply1" deviceset="GND" device=""/>
 <part name="EC2" library="SparkFun-Passives" deviceset="CAP" device="0805" value="100n"/>
 <part name="EC3" library="rcl" library_urn="urn:adsk.eagle:library:334" deviceset="CPOL-EU" device="SANYO_SMD_B6" package3d_urn="urn:adsk.eagle:package:23461/1" value="10u"/>
@@
 <part name="U$2" library="HR911105A" deviceset="HR911105A" device=""/>
 <part name="GND14" library="supply1" deviceset="GND" device=""/>
+<part name="PP" library="con-molex" library_urn="urn:adsk.eagle:library:165" deviceset="22-?-04" device="05-7048"/>
+<part name="X1" library="con-samtec" library_urn="urn:adsk.eagle:library:184" deviceset="SSW-101-02-G-S" device=""/>
+<part name="+3V2" library="supply1" deviceset="+3V3" device=""/>
 </parts>
 <sheets>
@@
 <text x="96.52" y="99.06" size="1.778" layer="91">IN3</text>
 <text x="309.88" y="15.24" size="2.54" layer="94">IOTB by Team IOTECH</text>
-<text x="365.76" y="12.7" size="2.54" layer="94">0.3</text>
+<text x="365.76" y="12.7" size="2.54" layer="94">0.4</text>
 <text x="170.18" y="170.18" size="1.778" layer="91">ETHERNET</text>
 <text x="175.26" y="109.22" size="1.778" layer="97">D2  -&gt;INT
@@
 D12-&gt;SO
 D13-&gt;SCK</text>
+<text x="132.08" y="81.28" size="1.778" layer="91">TTL</text>
+<text x="50.8" y="81.28" size="1.778" layer="91">MC</text>
 </plain>
 <instances>
@@
 <instance part="ER6" gate="G$1" x="185.42" y="157.48" rot="R90"/>
 <instance part="ER7" gate="G$1" x="177.8" y="157.48" rot="R90"/>
-<instance part="+3V5" gate="G$1" x="223.52" y="172.72" rot="MR0"/>
 <instance part="ER5" gate="G$1" x="198.12" y="111.76" smashed="yes" rot="R270">
 <attribute name="NAME" x="196.6214" y="107.95" size="1.778" layer="95" rot="R90"/>
@@
 <instance part="EC1" gate="G$1" x="314.96" y="162.56" rot="R90"/>
 <instance part="EL1" gate="G$1" x="304.8" y="170.18" rot="MR0"/>
-<instance part="+3V1" gate="G$1" x="322.58" y="177.8" rot="R270"/>
-<instance part="GND7" gate="1" x="322.58" y="162.56" rot="R90"/>
 <instance part="EC2" gate="G$1" x="287.02" y="99.06"/>
 <instance part="EC3" gate="G$1" x="187.96" y="116.84"/>
@@
 <instance part="U$2" gate="G$1" x="325.12" y="124.46"/>
 <instance part="GND14" gate="1" x="287.02" y="88.9"/>
+<instance part="PP" gate="-1" x="165.1" y="73.66"/>
+<instance part="PP" gate="-2" x="165.1" y="71.12"/>
+<instance part="PP" gate="-3" x="165.1" y="68.58"/>
+<instance part="PP" gate="-4" x="165.1" y="66.04"/>
+<instance part="X1" gate="-1" x="137.16" y="73.66"/>
+<instance part="+3V2" gate="G$1" x="261.62" y="170.18" rot="R180"/>
 </instances>
 <busses>
@@
 <segment>
 <pinref part="EC1" gate="G$1" pin="2"/>
-<pinref part="GND7" gate="1" pin="GND"/>
 <wire x1="317.5" y1="162.56" x2="320.04" y2="162.56" width="0.1524" layer="91"/>
-</segment>
-<segment>
 <pinref part="U$2" gate="G$1" pin="G-"/>
 <wire x1="342.9" y1="111.76" x2="355.6" y2="111.76" width="0.1524" layer="91"/>
@@
 <wire x1="287.02" y1="93.98" x2="287.02" y2="91.44" width="0.1524" layer="91"/>
 <pinref part="GND14" gate="1" pin="GND"/>
+<wire x1="320.04" y1="162.56" x2="355.6" y2="162.56" width="0.1524" layer="91"/>
+<wire x1="355.6" y1="162.56" x2="355.6" y2="139.7" width="0.1524" layer="91"/>
+<junction x="355.6" y="139.7"/>
+</segment>
+<segment>
+<pinref part="MC" gate="G$1" pin="GND$1"/>
+<wire x1="93.98" y1="68.58" x2="96.52" y2="68.58" width="0.1524" layer="91"/>
+<label x="96.52" y="68.58" size="1.778" layer="95" xref="yes"/>
+</segment>
+<segment>
+<pinref part="PP" gate="-2" pin="S"/>
+<wire x1="162.56" y1="71.12" x2="160.02" y2="71.12" width="0.1524" layer="91"/>
+<label x="160.02" y="71.12" size="1.778" layer="95" rot="R180" xref="yes"/>
 </segment>
 </net>
@@
 <wire x1="228.6" y1="154.94" x2="228.6" y2="165.1" width="0.1524" layer="91"/>
 <wire x1="218.44" y1="165.1" x2="220.98" y2="165.1" width="0.1524" layer="91"/>
-<pinref part="+3V5" gate="G$1" pin="+3V3"/>
 <wire x1="220.98" y1="165.1" x2="223.52" y2="165.1" width="0.1524" layer="91"/>
 <wire x1="223.52" y1="165.1" x2="226.06" y2="165.1" width="0.1524" layer="91"/>
@@
 <junction x="185.42" y="165.1"/>
 <junction x="218.44" y="165.1"/>
-</segment>
-<segment>
+<wire x1="223.52" y1="170.18" x2="223.52" y2="177.8" width="0.1524" layer="91"/>
 <pinref part="EL1" gate="G$1" pin="1"/>
 <wire x1="304.8" y1="175.26" x2="304.8" y2="177.8" width="0.1524" layer="91"/>
-<wire x1="304.8" y1="177.8" x2="320.04" y2="177.8" width="0.1524" layer="91"/>
-<pinref part="+3V1" gate="G$1" pin="+3V3"/>
+<wire x1="304.8" y1="177.8" x2="261.62" y2="177.8" width="0.1524" layer="91"/>
+<wire x1="223.52" y1="177.8" x2="261.62" y2="177.8" width="0.1524" layer="91"/>
+<wire x1="261.62" y1="177.8" x2="261.62" y2="172.72" width="0.1524" layer="91"/>
+<pinref part="+3V2" gate="G$1" pin="+3V3"/>
 </segment>
 </net>
@@
 </segment>
 </net>
+<net name="RX" class="0">
+<segment>
+<pinref part="MC" gate="G$1" pin="RX1$1"/>
+<wire x1="68.58" y1="68.58" x2="66.04" y2="68.58" width="0.1524" layer="91"/>
+<label x="66.04" y="68.58" size="1.778" layer="95" rot="R180" xref="yes"/>
+</segment>
+<segment>
+<pinref part="PP" gate="-4" pin="S"/>
+<wire x1="162.56" y1="66.04" x2="160.02" y2="66.04" width="0.1524" layer="91"/>
+<label x="160.02" y="66.04" size="1.778" layer="95" rot="R180" xref="yes"/>
+</segment>
+</net>
+<net name="TX" class="0">
+<segment>
+<pinref part="MC" gate="G$1" pin="TX0$1"/>
+<wire x1="68.58" y1="71.12" x2="60.96" y2="71.12" width="0.1524" layer="91"/>
+<label x="60.96" y="71.12" size="1.778" layer="95" rot="R180" xref="yes"/>
+</segment>
+<segment>
+<pinref part="PP" gate="-3" pin="S"/>
+<wire x1="162.56" y1="68.58" x2="152.4" y2="68.58" width="0.1524" layer="91"/>
+<label x="152.4" y="68.58" size="1.778" layer="95" rot="R180" xref="yes"/>
+</segment>
+</net>
+<net name="BLK" class="0">
+<segment>
+<pinref part="PP" gate="-1" pin="S"/>
+<wire x1="162.56" y1="73.66" x2="160.02" y2="73.66" width="0.1524" layer="91"/>
+<label x="160.02" y="73.66" size="1.778" layer="95" rot="R90" xref="yes"/>
+<pinref part="X1" gate="-1" pin="1"/>
+<wire x1="139.7" y1="73.66" x2="160.02" y2="73.66" width="0.1524" layer="91"/>
+</segment>
+</net>
