File: KMO_IO_M/KMO_IO_MV5.brd (EAGLE design)
At the start: 84.5 x 96.5 mm, 63 parts, among them Q1 8/16/20MHz, Q2 25MHz, U1 ATMEGA328

Commit message: v5rev
Parts:
- C1, C2, C3: device SparkFun:0603-CAP -> SparkFun-Passives:0805
- D3: device Testing:0603-LED-ALT1 -> led:CHIP-LED0805
- EC3: device rcl:SANYO-OSCON_SMD_B6 -> SparkFun-Passives:EIA3216-KIT
- PLED1: value (none) -> Green
- Q1: value 8/16/20MHz -> 16MHz
- Q2: device crystal:HC49/S -> crystal-geyer_V1_0:5.0X3.2_2
- R1, R2, R3, R6: device SparkFun:0603-RES -> SparkFun-Passives:0805
- moved EC3 1.00 mm to (32.0, 41.0)
Connections:
- removed net VCC: C3.2, R1.2, R2.2, R3.2, U1.18, U1.4, U1.6
- net +3V3: now also C3.2, R1.2, R2.2, R3.2, U1.18, U1.4, U1.6
- net GND: now also EC3.C; no longer EC3.-
- net N$13: now also EC3.A; no longer EC3.+
Routing:
- net +3V3: track 212.0 -> 298.4 mm, vias 4 -> 7
- net VCC: track 59.4 -> 0.00 mm, vias 4 -> 0
- net N$14: track 0.00 -> 40.3 mm, vias 0 -> 2
- net D10: track 57.7 -> 97.8 mm, vias 2 -> 0
- net A2: track 89.3 -> 111.5 mm, vias 2 -> 1
- net GND: track 564.0 -> 543.8 mm, vias 0 -> 3
- net RESET: track 69.9 -> 52.6 mm
- net A3: track 87.9 -> 96.6 mm, vias 2 -> 1
- net D7: track 40.1 -> 32.8 mm
- net RAW_IV: track 182.8 -> 187.3 mm
- net A0: track 31.2 -> 34.0 mm
- net D4: track 66.7 -> 64.5 mm
- net DTR: track 95.2 -> 93.0 mm
- net RD+: track 35.7 -> 37.2 mm
- net N$13: track 7.94 -> 6.73 mm
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
Commit message: kmoV5rev
Parts:
- moved R2 16.5 mm to (46.5, 91.5)
- moved S1 3.26 mm to (53.0, 90.2)
- moved D3 1.58 mm to (57.5, 83.5), turned to 0 degrees
- moved C2 1.00 mm to (59.5, 91.5)
Connections:
- removed net MISO: U1.16
- removed net MOSI: U1.15
- removed net SCK: R6.1, U1.17
- net D11: now also U1.16
- net D12: now also U1.15
- net D13: now also R6.1, U1.17
Routing:
- net D13: track 0.00 -> 105.7 mm
- net D11: track 0.00 -> 68.2 mm, vias 0 -> 2
- net D12: track 0.00 -> 67.2 mm, vias 0 -> 2
- net GND: track 543.8 -> 480.2 mm, vias 3 -> 4
- net A3: track 96.6 -> 121.3 mm, vias 1 -> 2
- net D10: track 97.8 -> 76.6 mm, vias 0 -> 2
- net DTR: track 93.0 -> 74.4 mm, vias 0 -> 1
- net D7: track 32.8 -> 49.4 mm, vias 3 -> 0
- net RESET: track 52.6 -> 39.2 mm, vias 0 -> 2
- net D2: track 40.0 -> 52.6 mm
- net A2: track 111.5 -> 102.2 mm, vias 1 -> 2
- net D3: track 73.1 -> 64.5 mm, vias 0 -> 2
- net A1: track 97.5 -> 105.7 mm
- net SCK: track 5.94 -> 0.00 mm
- net A0: track 34.0 -> 38.0 mm, vias 0 -> 1
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
Commit message: kmoV5befTest
Parts:
- added OP: (no value), con-lstb:MA03-2
Connections:
- net +3V3: now also OP.1
- net A4: now also OP.3
- net A5: now also OP.4
- net A6: now also OP.5
- net A7: now also OP.6
- net GND: now also OP.2
Routing:
- net GND: track 480.2 -> 544.7 mm, vias 4 -> 1
- net D13: track 105.7 -> 67.6 mm, vias 0 -> 3
- net A0: track 38.0 -> 74.5 mm, vias 1 -> 0
- net A3: track 121.3 -> 91.9 mm, vias 2 -> 0
- net A4: track 5.87 -> 34.4 mm
- net +3V3: track 295.4 -> 323.0 mm, vias 8 -> 10
- net D11: track 68.2 -> 94.1 mm, vias 2 -> 0
- net D5: track 31.4 -> 56.0 mm
- net A6: track 0.00 -> 24.5 mm
- net A7: track 0.00 -> 23.6 mm
- net A2: track 102.2 -> 83.3 mm
- net A5: track 8.66 -> 26.8 mm
- net D7: track 49.4 -> 32.2 mm, vias 0 -> 2
- net D10: track 76.6 -> 60.2 mm
- net D2: track 52.6 -> 40.0 mm
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