File: KMO_IO_M/KMO_IO_MV5.sch (EAGLE design)
At the start: 62 parts, among them Q1 8/16/20MHz, Q2 25MHz, U1 ATMEGA328

Commit message: v5rev
Parts:
- C1, C2, C3: device SparkFun:CAP0603-CAP -> SparkFun-Passives:CAP0805
- D3: device Testing:LED -> led:LEDCHIP-LED0805
- EC3: device rcl:CPOL-EUSANYO_SMD_B6 -> SparkFun-Passives:CAP_POL1206-KIT
- PLED1: value (none) -> Green
- Q1: value 8/16/20MHz -> 16MHz
- Q2: device crystal:CRYSTALHC49S -> crystal-geyer_V1_0:KX-9B
- R1, R2, R3, R6: device SparkFun:RESISTOR0603-RES -> SparkFun-Passives:RESISTOR0805-RES
Connections:
- removed net VCC: C3.2, R1.2, R2.2, R3.2, U1.AVCC, U1.VCC@1, U1.VCC@2
- net +3V3: now also C3.2, R1.2, R2.2, R3.2, U1.AVCC, U1.VCC@1, U1.VCC@2
Other:
- moved on the sheet: C3

Commit message: kmoV5rev
Connections:
- removed net MISO: U1.PB4(MISO)
- removed net MOSI: U1.PB3(MOSI/OC2)
- removed net SCK: R6.1, U1.PB5(SCK)
- net D11: now also U1.PB4(MISO)
- net D12: now also U1.PB3(MOSI/OC2)
- net D13: now also R6.1, U1.PB5(SCK)
Changed lines of the file:
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@@
 <grid distance="0.1" unitdist="inch" unit="inch" style="lines" multiple="1" display="no" altdistance="0.01" altunitdist="inch" altunit="inch"/>
 <layers>
-<layer number="1" name="Top" color="4" fill="1" visible="yes" active="no"/>
-<layer number="16" name="Bottom" color="1" fill="1" visible="yes" active="no"/>
-<layer number="17" name="Pads" color="2" fill="1" visible="yes" active="no"/>
-<layer number="18" name="Vias" color="2" fill="1" visible="yes" active="no"/>
-<layer number="19" name="Unrouted" color="6" fill="1" visible="yes" active="no"/>
-<layer number="20" name="Dimension" color="24" fill="1" visible="yes" active="no"/>
-<layer number="21" name="tPlace" color="7" fill="1" visible="yes" active="no"/>
-<layer number="22" name="bPlace" color="7" fill="1" visible="yes" active="no"/>
-<layer number="23" name="tOrigins" color="15" fill="1" visible="yes" active="no"/>
-<layer number="24" name="bOrigins" color="15" fill="1" visible="yes" active="no"/>
-<layer number="25" name="tNames" color="7" fill="1" visible="yes" active="no"/>
-<layer number="26" name="bNames" color="7" fill="1" visible="yes" active="no"/>
-<layer number="27" name="tValues" color="7" fill="1" visible="yes" active="no"/>
-<layer number="28" name="bValues" color="7" fill="1" visible="yes" active="no"/>
+<layer number="1" name="Top" color="4" fill="1" visible="no" active="no"/>
+<layer number="16" name="Bottom" color="1" fill="1" visible="no" active="no"/>
+<layer number="17" name="Pads" color="2" fill="1" visible="no" active="no"/>
+<layer number="18" name="Vias" color="2" fill="1" visible="no" active="no"/>
+<layer number="19" name="Unrouted" color="6" fill="1" visible="no" active="no"/>
+<layer number="20" name="Dimension" color="24" fill="1" visible="no" active="no"/>
+<layer number="21" name="tPlace" color="7" fill="1" visible="no" active="no"/>
+<layer number="22" name="bPlace" color="7" fill="1" visible="no" active="no"/>
+<layer number="23" name="tOrigins" color="15" fill="1" visible="no" active="no"/>
+<layer number="24" name="bOrigins" color="15" fill="1" visible="no" active="no"/>
+<layer number="25" name="tNames" color="7" fill="1" visible="no" active="no"/>
+<layer number="26" name="bNames" color="7" fill="1" visible="no" active="no"/>
+<layer number="27" name="tValues" color="7" fill="1" visible="no" active="no"/>
+<layer number="28" name="bValues" color="7" fill="1" visible="no" active="no"/>
 <layer number="29" name="tStop" color="7" fill="3" visible="no" active="no"/>
 <layer number="30" name="bStop" color="7" fill="6" visible="no" active="no"/>
@@
 <layer number="35" name="tGlue" color="7" fill="4" visible="no" active="no"/>
 <layer number="36" name="bGlue" color="7" fill="5" visible="no" active="no"/>
-<layer number="37" name="tTest" color="7" fill="1" visible="yes" active="no"/>
-<layer number="38" name="bTest" color="7" fill="1" visible="yes" active="no"/>
+<layer number="37" name="tTest" color="7" fill="1" visible="no" active="no"/>
+<layer number="38" name="bTest" color="7" fill="1" visible="no" active="no"/>
 <layer number="39" name="tKeepout" color="4" fill="11" visible="no" active="no"/>
 <layer number="40" name="bKeepout" color="1" fill="11" visible="no" active="no"/>
@@
 <layer number="44" name="Drills" color="7" fill="1" visible="no" active="no"/>
 <layer number="45" name="Holes" color="7" fill="1" visible="no" active="no"/>
-<layer number="46" name="Milling" color="3" fill="1" visible="yes" active="no"/>
-<layer number="47" name="Measures" color="7" fill="1" visible="yes" active="no"/>
-<layer number="48" name="Document" color="7" fill="1" visible="yes" active="no"/>
-<layer number="49" name="Reference" color="7" fill="1" visible="yes" active="no"/>
-<layer number="50" name="dxf" color="7" fill="1" visible="yes" active="no"/>
-<layer number="51" name="tDocu" color="7" fill="1" visible="yes" active="no"/>
-<layer number="52" name="bDocu" color="7" fill="1" visible="yes" active="no"/>
-<layer number="53" name="tGND_GNDA" color="7" fill="9" visible="yes" active="no"/>
-<layer number="54" name="bGND_GNDA" color="1" fill="9" visible="yes" active="no"/>
-<layer number="56" name="wert" color="7" fill="1" visible="yes" active="no"/>
-<layer number="57" name="tCAD" color="7" fill="1" visible="yes" active="no"/>
-<layer number="58" name="tCAD" color="7" fill="1" visible="yes" active="no"/>
-<layer number="59" name="tCarbon" color="7" fill="1" visible="yes" active="no"/>
-<layer number="60" name="bCarbon" color="7" fill="1" visible="yes" active="no"/>
+<layer number="46" name="Milling" color="3" fill="1" visible="no" active="no"/>
+<layer number="47" name="Measures" color="7" fill="1" visible="no" active="no"/>
+<layer number="48" name="Document" color="7" fill="1" visible="no" active="no"/>
+<layer number="49" name="Reference" color="7" fill="1" visible="no" active="no"/>
+<layer number="50" name="dxf" color="7" fill="1" visible="no" active="no"/>
+<layer number="51" name="tDocu" color="7" fill="1" visible="no" active="no"/>
+<layer number="52" name="bDocu" color="7" fill="1" visible="no" active="no"/>
+<layer number="53" name="tGND_GNDA" color="7" fill="9" visible="no" active="no"/>
+<layer number="54" name="bGND_GNDA" color="1" fill="9" visible="no" active="no"/>
+<layer number="56" name="wert" color="7" fill="1" visible="no" active="no"/>
+<layer number="57" name="tCAD" color="7" fill="1" visible="no" active="no"/>
+<layer number="58" name="tCAD" color="7" fill="1" visible="no" active="no"/>
+<layer number="59" name="tCarbon" color="7" fill="1" visible="no" active="no"/>
+<layer number="60" name="bCarbon" color="7" fill="1" visible="no" active="no"/>
 <layer number="88" name="SimResults" color="9" fill="1" visible="yes" active="yes"/>
 <layer number="89" name="SimProbes" color="9" fill="1" visible="yes" active="yes"/>
@@
 </variantdefs>
 <classes>
-<class number="0" name="default" width="0.2032" drill="0">
+<class number="0" name="default" width="0.2032" drill="0.3">
+<clearance class="0" value="0.16"/>
 </class>
-<class number="1" name="vcc" width="0.254" drill="0">
+<class number="1" name="vcc" width="0.254" drill="0.3">
+<clearance class="1" value="0.16"/>
 </class>
 </classes>
@@
 <wire x1="223.52" y1="165.1" x2="226.06" y2="165.1" width="0.1524" layer="91"/>
 <wire x1="226.06" y1="165.1" x2="228.6" y2="165.1" width="0.1524" layer="91"/>
-<wire x1="223.52" y1="165.1" x2="223.52" y2="170.18" width="0.1524" layer="91"/>
 <pinref part="ENC" gate="G$1" pin="VDDPLL"/>
 <wire x1="220.98" y1="154.94" x2="220.98" y2="165.1" width="0.1524" layer="91"/>
@@
 <junction x="185.42" y="165.1"/>
 <junction x="218.44" y="165.1"/>
-<wire x1="223.52" y1="170.18" x2="223.52" y2="177.8" width="0.1524" layer="91"/>
+<wire x1="223.52" y1="165.1" x2="223.52" y2="177.8" width="0.1524" layer="91"/>
 <pinref part="EL1" gate="G$1" pin="1"/>
 <wire x1="304.8" y1="175.26" x2="304.8" y2="177.8" width="0.1524" layer="91"/>
-<wire x1="304.8" y1="177.8" x2="261.62" y2="177.8" width="0.1524" layer="91"/>
-<wire x1="223.52" y1="177.8" x2="261.62" y2="177.8" width="0.1524" layer="91"/>
-<wire x1="261.62" y1="177.8" x2="307.34" y2="193.04" width="0.1524" layer="91"/>
+<wire x1="304.8" y1="177.8" x2="223.52" y2="177.8" width="0.1524" layer="91"/>
 </segment>
 </net>
@@
 </segment>
 </net>
-<net name="SCK" class="0">
+<net name="D13" class="0">
 <segment>
 <wire x1="114.3" y1="160.02" x2="114.3" y2="152.4" width="0.1524" layer="91"/>
@@
 </segment>
 </net>
-<net name="MISO" class="0">
+<net name="D11" class="0">
 <segment>
 <wire x1="111.76" y1="162.56" x2="114.3" y2="162.56" width="0.1524" layer="91"/>
@@
 </segment>
 </net>
-<net name="MOSI" class="0">
+<net name="D12" class="0">
 <segment>
 <wire x1="111.76" y1="165.1" x2="114.3" y2="165.1" width="0.1524" layer="91"/>
@@
 <pinref part="R3" gate="G$1" pin="1"/>
 <wire x1="147.32" y1="205.74" x2="147.32" y2="210.82" width="0.1524" layer="91"/>
+<label x="147.32" y="205.74" size="1.778" layer="95" xref="yes"/>
 </segment>
 </net>
@@
 <pinref part="U1" gate="G$1" pin="PC4(ADC4/SDA)"/>
 <pinref part="R1" gate="G$1" pin="1"/>
-</segment>
-</net>
+<label x="139.7" y="208.28" size="1.778" layer="95" xref="yes"/>
+</segment>
+</net>

Commit message: kmoV5befTest
Parts:
- added OP: (no value), con-lstb:MA03-2
Connections:
- net +3V3: now also OP.1
- net A4: now also OP.3
- net A5: now also OP.4
- net A6: now also OP.5
- net A7: now also OP.6
- net GND: now also OP.2
Changed lines of the file:
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@@
 <part name="Q1" library="Testing" deviceset="RESONATOR" device="1:1" value="16MHz"/>
 <part name="R3" library="SparkFun-Passives" deviceset="RESISTOR" device="0805-RES"/>
+<part name="OP" library="con-lstb" library_urn="urn:adsk.eagle:library:162" deviceset="MA03-2" device="" package3d_urn="urn:adsk.eagle:package:8334/1"/>
+<part name="GND20" library="SparkFun" deviceset="GND" device=""/>
+<part name="+3V1" library="supply1" deviceset="+3V3" device=""/>
 </parts>
 <sheets>
@@
 <instance part="R3" gate="G$1" x="147.32" y="215.9" rot="R90"/>
 <instance part="+3V2" gate="G$1" x="83.82" y="238.76"/>
+<instance part="OP" gate="1" x="30.48" y="139.7"/>
+<instance part="GND20" gate="1" x="20.32" y="132.08"/>
+<instance part="+3V1" gate="G$1" x="40.64" y="132.08" rot="R180"/>
 </instances>
 <busses>
@@
 <pinref part="GND19" gate="1" pin="GND"/>
 </segment>
+<segment>
+<pinref part="OP" gate="1" pin="2"/>
+<wire x1="22.86" y1="137.16" x2="20.32" y2="137.16" width="0.1524" layer="91"/>
+<pinref part="GND20" gate="1" pin="GND"/>
+<wire x1="20.32" y1="137.16" x2="20.32" y2="134.62" width="0.1524" layer="91"/>
+</segment>
 </net>
 <net name="AREF" class="0">
@@
 <label x="147.32" y="205.74" size="1.778" layer="95" xref="yes"/>
 </segment>
+<segment>
+<pinref part="OP" gate="1" pin="4"/>
+<wire x1="22.86" y1="139.7" x2="20.32" y2="139.7" width="0.1524" layer="91"/>
+<label x="20.32" y="139.7" size="1.778" layer="95" rot="R180" xref="yes"/>
+</segment>
 </net>
 <net name="A4" class="0">
@@
 <label x="139.7" y="208.28" size="1.778" layer="95" xref="yes"/>
 </segment>
+<segment>
+<pinref part="OP" gate="1" pin="3"/>
+<wire x1="38.1" y1="139.7" x2="40.64" y2="139.7" width="0.1524" layer="91"/>
+<label x="40.64" y="139.7" size="1.778" layer="95" xref="yes"/>
+</segment>
 </net>
 <net name="A3" class="0">
@@
 <label x="114.3" y="203.2" size="1.27" layer="95" xref="yes"/>
 </segment>
+<segment>
+<pinref part="OP" gate="1" pin="5"/>
+<wire x1="38.1" y1="142.24" x2="45.72" y2="142.24" width="0.1524" layer="91"/>
+<label x="45.72" y="142.24" size="1.778" layer="95" xref="yes"/>
+</segment>
 </net>
 <net name="A7" class="0">
@@
 <pinref part="U1" gate="G$1" pin="ADC7"/>
 <label x="114.3" y="200.66" size="1.27" layer="95" xref="yes"/>
+</segment>
+<segment>
+<pinref part="OP" gate="1" pin="6"/>
+<wire x1="22.86" y1="142.24" x2="15.24" y2="142.24" width="0.1524" layer="91"/>
+<label x="15.24" y="142.24" size="1.778" layer="95" rot="R180" xref="yes"/>
 </segment>
 </net>
@@
 <junction x="96.52" y="233.68"/>
 </segment>
-</net>
+<segment>
+<pinref part="OP" gate="1" pin="1"/>
+<wire x1="38.1" y1="137.16" x2="40.64" y2="137.16" width="0.1524" layer="91"/>
+<pinref part="+3V1" gate="G$1" pin="+3V3"/>
+<wire x1="40.64" y1="137.16" x2="40.64" y2="134.62" width="0.1524" layer="91"/>
+</segment>
+</net>
