File: KMO_IO_M/KMO_IO_MV7.brd (EAGLE design)
At the start: 84.5 x 96.5 mm, 67 parts, among them IC1 LM2596S, Q1 16MHz, Q2 25MHz, U1 ATMEGA328

Commit message: v7
Parts:
- removed PC1: 22uf, rcl:CT3216
- removed PC2: 10uf, rcl:CT3216
- removed PIC1: REG1117, burr-brown:SOT223
- moved C4 25.2 mm to (42.2, 23.5)
- moved PR1 20.1 mm to (57.5, 9.75), turned to 180 degrees
- moved C5 17.5 mm to (59.8, 19.8)
- moved D1 1.25 mm to (28.2, 4.50)
- moved IC1 1.25 mm to (26.8, 16.5)
- moved U$3 0.35 mm to (43.0, 8.25)
Connections:
- removed net +5V: C5.+, IC1.4, PC2.+, PIC1.3, U$3.P$1
- net +3V3: now also C5.+, IC1.4, U$3.P$1; no longer PC1.+, PIC1.2
- net GND: no longer PC1.-, PC2.-, PIC1.1
Routing:
- net +5V: track 52.3 -> 0.00 mm
- net GND: track 583.4 -> 537.6 mm, vias 2 -> 3
- net RAW_IV: track 178.2 -> 213.8 mm, vias 3 -> 1
- net TXO: track 77.9 -> 55.5 mm
- net D6: track 69.8 -> 49.2 mm
- net +3V3: track 354.5 -> 336.5 mm, vias 3 -> 8
- net A6: track 50.6 -> 33.2 mm, vias 0 -> 1
- net N$11: track 17.4 -> 2.33 mm
- net A3: track 92.0 -> 105.3 mm
- net D13: track 57.0 -> 69.7 mm
- net D3: track 37.5 -> 27.0 mm, vias 0 -> 1
- net D7: track 34.2 -> 43.7 mm
- net RXI: track 55.4 -> 64.2 mm, vias 2 -> 1
- net A2: track 102.1 -> 93.4 mm, vias 1 -> 3
- net A7: track 33.7 -> 26.2 mm, vias 3 -> 2
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Other:
- board text added: "IOTB v0.7 TOP"
- board text removed: "IOTB v0.6 TOP"

Commit message: 7rev
Parts:
- PCO: value (none) -> 33 uh
- PD2: value (none) -> SS54
- S1: value Reset -> (none); device Testing:TACTILE-SWITCH-SMD-ALT01 -> switch-omron:B3F-31XX
- moved S1 60.3 mm to (3.50, 55.8), turned to 270 degrees
- moved WIFI 26.1 mm to (30.8, 38.0), turned to 270 degrees
- moved C2 9.50 mm to (51.8, 86.0)
- moved R2 5.77 mm to (48.2, 86.0)
- moved PP 4.50 mm to (11.5, 44.2)
- moved D3 2.51 mm to (60.0, 83.2), turned to 180 degrees
- moved R6 1.77 mm to (55.5, 83.2)
- moved ER5 0.79 mm to (33.2, 32.2)
- renumbered C4 to PC1, C5 to PC2, D1 to PD2, IC1 to PIC1, U$3 to PCO
Connections:
- net GND: no longer S1.1
- net RESET: now also S1.1; no longer S1.3, S1.4
Routing:
- net RESET: track 37.2 -> 83.8 mm
- net D12: track 48.7 -> 89.6 mm
- net D4: track 19.3 -> 52.1 mm, vias 0 -> 2
- net GND: track 537.6 -> 512.4 mm, vias 3 -> 4
- net D10: track 61.4 -> 86.5 mm, vias 2 -> 4
- net D3: track 27.0 -> 50.4 mm
- net D5: track 33.9 -> 56.0 mm, vias 5 -> 0
- net A0: track 52.2 -> 72.8 mm
- net D6: track 49.2 -> 31.1 mm, vias 2 -> 0
- net D11: track 61.9 -> 77.9 mm
- net RAW_IV: track 213.8 -> 199.4 mm, vias 1 -> 3
- net RXI: track 64.2 -> 52.5 mm, vias 1 -> 3
- net RD-: track 33.8 -> 44.2 mm
- net A5: track 36.4 -> 26.8 mm
- net A6: track 33.2 -> 24.5 mm, vias 1 -> 0
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
Commit message: rev7 out
Parts:
- D3: value Green -> BLUE
- PLED1: value Blue -> RED
- moved D3 40.9 mm to (81.2, 48.2), turned to 0 degrees
- moved R6 40.9 mm to (76.8, 48.2), turned to 270 degrees
- moved OP 34.3 mm to (59.8, 89.8), turned to 180 degrees
- moved ER9 32.1 mm to (45.2, 47.2)
- moved ER8 27.8 mm to (49.5, 47.2)
- moved PLED1 23.2 mm to (81.2, 22.2), turned to 0 degrees
- moved PR1 21.6 mm to (75.8, 21.2)
- moved U1 4.42 mm to (60.5, 76.0)
- moved Q1 2.69 mm to (66.0, 66.0)
- moved PC2 2.46 mm to (58.8, 17.5)
- moved PF1 1.00 mm to (56.8, 5.50)
- moved PD1 0.75 mm to (66.2, 5.50)
- renumbered PIC1 to PIC33, S1 to SR
Routing:
- net +3V3: track 335.4 -> 387.0 mm
- net A0: track 72.8 -> 26.7 mm
- net D13: track 69.1 -> 109.5 mm, vias 3 -> 2
- net D12: track 89.6 -> 54.0 mm
- net N$14: track 35.8 -> 7.95 mm, vias 2 -> 0
- net LEDB: track 22.8 -> 50.5 mm, vias 0 -> 1
- net A5: track 26.8 -> 53.7 mm
- net LEDA: track 5.92 -> 32.7 mm
- net D10: track 86.5 -> 59.9 mm, vias 4 -> 3
- net N$9: track 34.2 -> 8.17 mm
- net RAW_IV: track 199.4 -> 175.7 mm, vias 3 -> 2
- net D5: track 56.0 -> 35.3 mm, vias 0 -> 2
- net D6: track 31.1 -> 49.7 mm
- net GND: track 512.4 -> 525.4 mm
- net D11: track 77.9 -> 90.6 mm, vias 4 -> 0
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