File: KMO_IO_M/KMO_IO_MV7.sch (EAGLE design)
At the start: 62 parts, among them IC1 LM2596S, Q1 16MHz, Q2 25MHz, U1 ATMEGA328

Commit message: 7rev
Parts:
- PCO: value (none) -> 33 uh
- PD2: value (none) -> SS54
- S1: value Reset -> (none); device Testing:SWITCH-MOMENTARY-2SMD-ALT01 -> switch-omron:31-XX
- renumbered C4 to PC1, C5 to PC2, D1 to PD2, IC1 to PIC1, U$3 to PCO
Connections:
- net GND: now also S1.S; no longer S1.1
- net RESET: now also S1.P; no longer S1.2
Changed lines of the file:
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@@
 <part name="C2" library="SparkFun-Passives" deviceset="CAP" device="0805" value="0.1uF"/>
 <part name="R1" library="SparkFun-Passives" deviceset="RESISTOR" device="0805-RES"/>
-<part name="S1" library="Testing" deviceset="SWITCH-MOMENTARY-2" device="SMD-ALT01" value="Reset"/>
 <part name="Q1" library="Testing" deviceset="RESONATOR" device="1:1" value="16MHz"/>
 <part name="R3" library="SparkFun-Passives" deviceset="RESISTOR" device="0805-RES"/>
@@
 <part name="GND20" library="SparkFun" deviceset="GND" device=""/>
 <part name="+3V1" library="supply1" deviceset="+3V3" device=""/>
-<part name="C4" library="rcl" library_urn="urn:adsk.eagle:library:334" deviceset="CPOL-EU" device="140CLH-1010" package3d_urn="urn:adsk.eagle:package:23391/1" value="680uf"/>
-<part name="C5" library="rcl" library_urn="urn:adsk.eagle:library:334" deviceset="CPOL-EU" device="140CLH-1010" package3d_urn="urn:adsk.eagle:package:23391/1" value="220uf"/>
-<part name="U$3" library="inductor-coilcraft" deviceset="MSS1260" device=""/>
-<part name="IC1" library="national-semiconductor" library_urn="urn:adsk.eagle:library:307" deviceset="LM2596" device="S" package3d_urn="urn:adsk.eagle:package:21218/1"/>
-<part name="D1" library="diode" library_urn="urn:adsk.eagle:library:210" deviceset="SCHOTTKY-DIODE" device="SMD" package3d_urn="urn:adsk.eagle:package:43404/2"/>
+<part name="PC1" library="rcl" library_urn="urn:adsk.eagle:library:334" deviceset="CPOL-EU" device="140CLH-1010" package3d_urn="urn:adsk.eagle:package:23391/1" value="680uf"/>
+<part name="PC2" library="rcl" library_urn="urn:adsk.eagle:library:334" deviceset="CPOL-EU" device="140CLH-1010" package3d_urn="urn:adsk.eagle:package:23391/1" value="220uf"/>
+<part name="PCO" library="inductor-coilcraft" deviceset="MSS1260" device="" value="33 uh"/>
+<part name="PIC1" library="national-semiconductor" library_urn="urn:adsk.eagle:library:307" deviceset="LM2596" device="S" package3d_urn="urn:adsk.eagle:package:21218/1"/>
+<part name="PD2" library="diode" library_urn="urn:adsk.eagle:library:210" deviceset="SCHOTTKY-DIODE" device="SMD" package3d_urn="urn:adsk.eagle:package:43404/2" value="SS54"/>
+<part name="S1" library="switch-omron" library_urn="urn:adsk.eagle:library:377" deviceset="31-XX" device="" package3d_urn="urn:adsk.eagle:package:27487/1"/>
 </parts>
 <sheets>
@@
 <instance part="PP" gate="-3" x="205.74" y="190.5"/>
 <instance part="PP" gate="-4" x="205.74" y="187.96"/>
-<instance part="C4" gate="G$1" x="45.72" y="223.52"/>
-<instance part="C5" gate="G$1" x="116.84" y="223.52"/>
-<instance part="U$3" gate="G$1" x="106.68" y="231.14" rot="R270"/>
-<instance part="IC1" gate="G$1" x="68.58" y="228.6"/>
-<instance part="D1" gate="G$1" x="96.52" y="223.52" rot="R90"/>
+<instance part="PC1" gate="G$1" x="45.72" y="223.52"/>
+<instance part="PC2" gate="G$1" x="116.84" y="223.52"/>
+<instance part="PCO" gate="G$1" x="106.68" y="231.14" rot="R270"/>
+<instance part="PIC1" gate="G$1" x="68.58" y="228.6"/>
+<instance part="PD2" gate="G$1" x="96.52" y="223.52" rot="R90"/>
 <instance part="OP" gate="1" x="134.62" y="129.54"/>
 <instance part="GND20" gate="1" x="124.46" y="121.92"/>
@@
 </instance>
 <instance part="R1" gate="G$1" x="142.24" y="76.2" rot="R90"/>
-<instance part="S1" gate="G$1" x="40.64" y="71.12" rot="R90"/>
 <instance part="Q1" gate="G$1" x="63.5" y="50.8" smashed="yes" rot="R270">
 <attribute name="NAME" x="59.944" y="54.61" size="1.778" layer="95"/>
@@
 <instance part="R3" gate="G$1" x="149.86" y="76.2" rot="R90"/>
 <instance part="+3V2" gate="G$1" x="86.36" y="99.06"/>
+<instance part="S1" gate="1" x="40.64" y="71.12" rot="R180"/>
 </instances>
 <busses>
@@
 <wire x1="109.22" y1="215.9" x2="116.84" y2="215.9" width="0.1524" layer="91"/>
 <pinref part="PJ1" gate="G$1" pin="GNDBREAK"/>
-<pinref part="IC1" gate="G$1" pin="!ON!/OFF"/>
+<pinref part="PIC1" gate="G$1" pin="!ON!/OFF"/>
 <wire x1="55.88" y1="228.6" x2="53.34" y2="228.6" width="0.1524" layer="91"/>
 <wire x1="53.34" y1="228.6" x2="53.34" y2="223.52" width="0.1524" layer="91"/>
-<pinref part="IC1" gate="G$1" pin="GND"/>
+<pinref part="PIC1" gate="G$1" pin="GND"/>
 <wire x1="53.34" y1="223.52" x2="53.34" y2="215.9" width="0.1524" layer="91"/>
 <wire x1="55.88" y1="223.52" x2="53.34" y2="223.52" width="0.1524" layer="91"/>
 <junction x="53.34" y="223.52"/>
 <junction x="53.34" y="215.9"/>
-<pinref part="C4" gate="G$1" pin="-"/>
+<pinref part="PC1" gate="G$1" pin="-"/>
 <wire x1="45.72" y1="218.44" x2="45.72" y2="215.9" width="0.1524" layer="91"/>
 <junction x="45.72" y="215.9"/>
-<pinref part="D1" gate="G$1" pin="A"/>
+<pinref part="PD2" gate="G$1" pin="A"/>
 <wire x1="96.52" y1="220.98" x2="96.52" y2="215.9" width="0.1524" layer="91"/>
 <junction x="96.52" y="215.9"/>
-<pinref part="C5" gate="G$1" pin="-"/>
+<pinref part="PC2" gate="G$1" pin="-"/>
 <wire x1="116.84" y1="218.44" x2="116.84" y2="215.9" width="0.1524" layer="91"/>
 <junction x="116.84" y="215.9"/>
@@
 <wire x1="40.64" y1="66.04" x2="40.64" y2="63.5" width="0.1524" layer="91"/>
 <pinref part="GND7" gate="1" pin="GND"/>
-<pinref part="S1" gate="G$1" pin="1"/>
+<pinref part="S1" gate="1" pin="S"/>
 </segment>
 <segment>
@@
 <pinref part="PF1" gate="G$1" pin="2"/>
 <wire x1="40.64" y1="241.3" x2="45.72" y2="241.3" width="0.1524" layer="91"/>
-<pinref part="C4" gate="G$1" pin="+"/>
+<pinref part="PC1" gate="G$1" pin="+"/>
 <wire x1="45.72" y1="241.3" x2="45.72" y2="233.68" width="0.1524" layer="91"/>
 <junction x="45.72" y="241.3"/>
 <wire x1="45.72" y1="233.68" x2="45.72" y2="226.06" width="0.1524" layer="91"/>
 <wire x1="45.72" y1="241.3" x2="124.46" y2="241.3" width="0.1524" layer="91"/>
-<pinref part="IC1" gate="G$1" pin="VIN"/>
+<pinref part="PIC1" gate="G$1" pin="VIN"/>
 <wire x1="55.88" y1="233.68" x2="45.72" y2="233.68" width="0.1524" layer="91"/>
 <junction x="45.72" y="233.68"/>
@@
 <wire x1="134.62" y1="231.14" x2="137.16" y2="231.14" width="0.1524" layer="91"/>
 <junction x="134.62" y="231.14"/>
-<pinref part="C5" gate="G$1" pin="+"/>
-<pinref part="U$3" gate="G$1" pin="P$1"/>
+<pinref part="PC2" gate="G$1" pin="+"/>
+<pinref part="PCO" gate="G$1" pin="P$1"/>
 <wire x1="114.3" y1="231.14" x2="116.84" y2="231.14" width="0.1524" layer="91"/>
 <wire x1="116.84" y1="231.14" x2="116.84" y2="226.06" width="0.1524" layer="91"/>
@@
 </segment>
 <segment>
-<pinref part="IC1" gate="G$1" pin="FB"/>
+<pinref part="PIC1" gate="G$1" pin="FB"/>
 <wire x1="81.28" y1="226.06" x2="83.82" y2="226.06" width="0.1524" layer="91"/>
 <label x="83.82" y="226.06" size="1.778" layer="95" xref="yes"/>
@@
 <net name="N$16" class="0">
 <segment>
-<pinref part="IC1" gate="G$1" pin="OUT"/>
+<pinref part="PIC1" gate="G$1" pin="OUT"/>
 <wire x1="81.28" y1="231.14" x2="96.52" y2="231.14" width="0.1524" layer="91"/>
-<pinref part="D1" gate="G$1" pin="C"/>
+<pinref part="PD2" gate="G$1" pin="C"/>
 <wire x1="96.52" y1="231.14" x2="96.52" y2="226.06" width="0.1524" layer="91"/>
 <junction x="96.52" y="231.14"/>
-<pinref part="U$3" gate="G$1" pin="P$2"/>
+<pinref part="PCO" gate="G$1" pin="P$2"/>
 <wire x1="96.52" y1="231.14" x2="99.06" y2="231.14" width="0.1524" layer="91"/>
 </segment>
@@
 <pinref part="R2" gate="G$1" pin="1"/>
 <pinref part="C2" gate="G$1" pin="1"/>
-<pinref part="S1" gate="G$1" pin="2"/>
-</segment>
-</net>
+<pinref part="S1" gate="1" pin="P"/>
+</segment>
+</net>

Commit message: rev7 out
Parts:
- D3: value Green -> BLUE
- PLED1: value Blue -> RED
- renumbered PIC1 to PIC33, S1 to SR
Changed lines of the file:
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@@
 </classes>
 <parts>
-<part name="PLED1" library="led" library_urn="urn:adsk.eagle:library:259" deviceset="LED" device="CHIP-LED0805" package3d_urn="urn:adsk.eagle:package:15818/2" value="Blue"/>
+<part name="PLED1" library="led" library_urn="urn:adsk.eagle:library:259" deviceset="LED" device="CHIP-LED0805" package3d_urn="urn:adsk.eagle:package:15818/2" value="RED"/>
 <part name="PD1" library="SparkFun-DiscreteSemi" deviceset="DIODE" device="SMA" value="M7"/>
 <part name="GND1" library="SparkFun-Aesthetics" deviceset="GND" device=""/>
@@
 <part name="GND16" library="SparkFun" deviceset="GND" device=""/>
 <part name="R6" library="SparkFun-Passives" deviceset="RESISTOR" device="0805-RES" value="330"/>
-<part name="D3" library="led" library_urn="urn:adsk.eagle:library:259" deviceset="LED" device="CHIP-LED0805" package3d_urn="urn:adsk.eagle:package:15818/2" value="Green"/>
+<part name="D3" library="led" library_urn="urn:adsk.eagle:library:259" deviceset="LED" device="CHIP-LED0805" package3d_urn="urn:adsk.eagle:package:15818/2" value="BLUE"/>
 <part name="GND17" library="SparkFun" deviceset="GND" device=""/>
 <part name="GND18" library="SparkFun" deviceset="GND" device=""/>
@@
 <part name="PC2" library="rcl" library_urn="urn:adsk.eagle:library:334" deviceset="CPOL-EU" device="140CLH-1010" package3d_urn="urn:adsk.eagle:package:23391/1" value="220uf"/>
 <part name="PCO" library="inductor-coilcraft" deviceset="MSS1260" device="" value="33 uh"/>
-<part name="PIC1" library="national-semiconductor" library_urn="urn:adsk.eagle:library:307" deviceset="LM2596" device="S" package3d_urn="urn:adsk.eagle:package:21218/1"/>
+<part name="PIC33" library="national-semiconductor" library_urn="urn:adsk.eagle:library:307" deviceset="LM2596" device="S" package3d_urn="urn:adsk.eagle:package:21218/1"/>
 <part name="PD2" library="diode" library_urn="urn:adsk.eagle:library:210" deviceset="SCHOTTKY-DIODE" device="SMD" package3d_urn="urn:adsk.eagle:package:43404/2" value="SS54"/>
-<part name="S1" library="switch-omron" library_urn="urn:adsk.eagle:library:377" deviceset="31-XX" device="" package3d_urn="urn:adsk.eagle:package:27487/1"/>
+<part name="SR" library="switch-omron" library_urn="urn:adsk.eagle:library:377" deviceset="31-XX" device="" package3d_urn="urn:adsk.eagle:package:27487/1"/>
 </parts>
 <sheets>
@@
 <instance part="PC2" gate="G$1" x="116.84" y="223.52"/>
 <instance part="PCO" gate="G$1" x="106.68" y="231.14" rot="R270"/>
-<instance part="PIC1" gate="G$1" x="68.58" y="228.6"/>
+<instance part="PIC33" gate="G$1" x="68.58" y="228.6"/>
 <instance part="PD2" gate="G$1" x="96.52" y="223.52" rot="R90"/>
 <instance part="OP" gate="1" x="134.62" y="129.54"/>
@@
 <instance part="R3" gate="G$1" x="149.86" y="76.2" rot="R90"/>
 <instance part="+3V2" gate="G$1" x="86.36" y="99.06"/>
-<instance part="S1" gate="1" x="40.64" y="71.12" rot="R180"/>
+<instance part="SR" gate="1" x="40.64" y="71.12" rot="R180"/>
 </instances>
 <busses>
@@
 <wire x1="109.22" y1="215.9" x2="116.84" y2="215.9" width="0.1524" layer="91"/>
 <pinref part="PJ1" gate="G$1" pin="GNDBREAK"/>
-<pinref part="PIC1" gate="G$1" pin="!ON!/OFF"/>
+<pinref part="PIC33" gate="G$1" pin="!ON!/OFF"/>
 <wire x1="55.88" y1="228.6" x2="53.34" y2="228.6" width="0.1524" layer="91"/>
 <wire x1="53.34" y1="228.6" x2="53.34" y2="223.52" width="0.1524" layer="91"/>
-<pinref part="PIC1" gate="G$1" pin="GND"/>
+<pinref part="PIC33" gate="G$1" pin="GND"/>
 <wire x1="53.34" y1="223.52" x2="53.34" y2="215.9" width="0.1524" layer="91"/>
 <wire x1="55.88" y1="223.52" x2="53.34" y2="223.52" width="0.1524" layer="91"/>
@@
 <wire x1="40.64" y1="66.04" x2="40.64" y2="63.5" width="0.1524" layer="91"/>
 <pinref part="GND7" gate="1" pin="GND"/>
-<pinref part="S1" gate="1" pin="S"/>
+<pinref part="SR" gate="1" pin="S"/>
 </segment>
 <segment>
@@
 <wire x1="45.72" y1="233.68" x2="45.72" y2="226.06" width="0.1524" layer="91"/>
 <wire x1="45.72" y1="241.3" x2="124.46" y2="241.3" width="0.1524" layer="91"/>
-<pinref part="PIC1" gate="G$1" pin="VIN"/>
+<pinref part="PIC33" gate="G$1" pin="VIN"/>
 <wire x1="55.88" y1="233.68" x2="45.72" y2="233.68" width="0.1524" layer="91"/>
 <junction x="45.72" y="233.68"/>
@@
 </segment>
 <segment>
-<pinref part="PIC1" gate="G$1" pin="FB"/>
+<pinref part="PIC33" gate="G$1" pin="FB"/>
 <wire x1="81.28" y1="226.06" x2="83.82" y2="226.06" width="0.1524" layer="91"/>
 <label x="83.82" y="226.06" size="1.778" layer="95" xref="yes"/>
@@
 <net name="N$16" class="0">
 <segment>
-<pinref part="PIC1" gate="G$1" pin="OUT"/>
+<pinref part="PIC33" gate="G$1" pin="OUT"/>
 <wire x1="81.28" y1="231.14" x2="96.52" y2="231.14" width="0.1524" layer="91"/>
 <pinref part="PD2" gate="G$1" pin="C"/>
@@
 <pinref part="R2" gate="G$1" pin="1"/>
 <pinref part="C2" gate="G$1" pin="1"/>
-<pinref part="S1" gate="1" pin="P"/>
-</segment>
-</net>
+<pinref part="SR" gate="1" pin="P"/>
+</segment>
+</net>
