File: KMO_IO_M/KMO_IO_MV8.brd (EAGLE design)
At the start: 84.5 x 96.5 mm, 64 parts, among them Q1 16MHz, Q2 25MHz, U1 ATMEGA328

Commit message: v8
Parts:
- moved PD2 25.6 mm to (47.0, 22.0), turned to 180 degrees
- moved PIC33 21.3 mm to (47.2, 10.8), turned to 180 degrees
- moved PCO 9.80 mm to (33.2, 9.25)
- moved PC1 9.50 mm to (32.8, 23.5), turned to 270 degrees
- moved PF1 2.25 mm to (59.0, 5.50)
- moved PC2 2.24 mm to (59.8, 15.5), turned to 270 degrees
- moved PD1 0.25 mm to (66.5, 5.50)
Routing:
- net +3V3: track 356.0 -> 383.1 mm, vias 6 -> 4
- net A0: track 55.4 -> 79.5 mm, vias 0 -> 1
- net D11: track 88.6 -> 66.4 mm
- net D13: track 111.8 -> 95.8 mm, vias 2 -> 3
- net RESET: track 91.9 -> 106.2 mm, vias 3 -> 2
- net RD+: track 42.8 -> 54.2 mm, vias 2 -> 1
- net A2: track 103.5 -> 114.1 mm
- net A3: track 100.4 -> 109.9 mm
- net D4: track 59.3 -> 68.3 mm, vias 1 -> 3
- net D9: track 19.7 -> 28.2 mm, vias 0 -> 1
- net RD-: track 49.5 -> 42.1 mm
- net GND: track 470.8 -> 465.2 mm
- net D3: track 62.4 -> 57.5 mm
- net D8: track 59.3 -> 54.8 mm, vias 2 -> 1
- net D7: track 39.4 -> 43.7 mm
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
Commit message: v8out
Parts:
- renumbered D3 to INDL, PLED1 to PL
Other:
- board text added: "IOTB v0.8 TOP"
- board text removed: "IOTB v0.7 TOP"
Changed lines of the file:
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@@
 <drawing>
 <settings>
-<setting alwaysvectorfont="no"/>
+<setting alwaysvectorfont="yes"/>
 <setting verticaltext="up"/>
 </settings>
@@
 <wire x1="84.5" y1="96.5" x2="84.5" y2="0" width="0.1524" layer="20" locked="yes"/>
 <wire x1="84.5" y1="0" x2="0" y2="0" width="0.1524" layer="20" locked="yes"/>
-<text x="44.75" y="52.5" size="1.6764" layer="21">IOTB v0.7 TOP</text>
+<text x="44.75" y="52.5" size="1.6764" layer="21">IOTB v0.8 TOP</text>
 <text x="46.25" y="56.25" size="1.6764" layer="21">IOTECH © 2018</text>
 <wire x1="44" y1="57.25" x2="43.25" y2="58" width="0.1524" layer="21"/>
@@
 </autorouter>
 <elements>
-<element name="PLED1" library="led" library_urn="urn:adsk.eagle:library:259" package="CHIP-LED0805" package3d_urn="urn:adsk.eagle:package:15818/2" value="RED" x="81.25" y="22.25"/>
+<element name="PL" library="led" library_urn="urn:adsk.eagle:library:259" package="CHIP-LED0805" package3d_urn="urn:adsk.eagle:package:15818/2" value="RED" x="81.25" y="22.25"/>
 <element name="PD1" library="SparkFun-DiscreteSemi" package="SMA-DIODE" value="M7" x="66.5" y="5.5" rot="R180"/>
 <element name="PR1" library="SparkFun-Passives" package="0805" value="470" x="75.75" y="21.25" rot="R180"/>
@@
 <element name="C1" library="SparkFun-Passives" package="0805" value="0.1uF" x="47.5" y="76.5"/>
 <element name="R6" library="SparkFun-Passives" package="0805" value="330" x="76.75" y="48.25" rot="R270"/>
-<element name="D3" library="led" library_urn="urn:adsk.eagle:library:259" package="CHIP-LED0805" package3d_urn="urn:adsk.eagle:package:15818/2" value="BLUE" x="81.25" y="48.25"/>
+<element name="INDL" library="led" library_urn="urn:adsk.eagle:library:259" package="CHIP-LED0805" package3d_urn="urn:adsk.eagle:package:15818/2" value="BLUE" x="81.25" y="48.25"/>
 <element name="U1" library="SparkFun" package="TQFP32-08" value="ATMEGA328" x="60.5" y="76" rot="R135"/>
 <element name="C2" library="SparkFun-Passives" package="0805" value="0.1uF" x="51.75" y="86" rot="R270"/>
@@
 </signal>
 <signal name="GND">
-<contactref element="PLED1" pad="C"/>
+<contactref element="PL" pad="C"/>
 <contactref element="PJ1" pad="GND"/>
 <contactref element="OQ1" pad="3"/>
@@
 <contactref element="C3" pad="1"/>
 <contactref element="C1" pad="1"/>
-<contactref element="D3" pad="C"/>
+<contactref element="INDL" pad="C"/>
 <contactref element="Q1" pad="2"/>
 <contactref element="U1" pad="5"/>
@@
 <signal name="N$11">
 <contactref element="PR1" pad="1"/>
-<contactref element="PLED1" pad="A"/>
+<contactref element="PL" pad="A"/>
 <wire x1="76.7416" y1="21.2264" x2="81.2318" y2="21.2264" width="0.2032" layer="1"/>
 <wire x1="81.2318" y1="21.2264" x2="81.25" y2="21.2" width="0.2032" layer="1"/>
@@
 <signal name="N$5">
 <contactref element="R6" pad="2"/>
-<contactref element="D3" pad="A"/>
+<contactref element="INDL" pad="A"/>
 <wire x1="76.84365" y1="47.24915" x2="81.2318" y2="47.24915" width="0.2032" layer="1"/>
 <wire x1="81.2318" y1="47.24915" x2="81.25" y2="47.2" width="0.2032" layer="1"/>
