File: KMO_IO_M/KMO_IO_MV8.sch (EAGLE design)
At the start: 62 parts, among them Q1 16MHz, Q2 25MHz, U1 ATMEGA328

Commit message: v8out
Parts:
- renumbered D3 to INDL, PLED1 to PL
Other:
- note added: "0.8"
- note added: "IOTECH Yazılım Sanayi ve Ticaret A.Ş. TESA IO Board Design."
- note removed: "0.7"
- note removed: "IOTECH Yazılım Sanayi ve Ticaret A.Ş. TESA IO Kart Tasarımı."
Changed lines of the file:
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@@
 </classes>
 <parts>
-<part name="PLED1" library="led" library_urn="urn:adsk.eagle:library:259" deviceset="LED" device="CHIP-LED0805" package3d_urn="urn:adsk.eagle:package:15818/2" value="RED"/>
+<part name="PL" library="led" library_urn="urn:adsk.eagle:library:259" deviceset="LED" device="CHIP-LED0805" package3d_urn="urn:adsk.eagle:package:15818/2" value="RED"/>
 <part name="PD1" library="SparkFun-DiscreteSemi" deviceset="DIODE" device="SMA" value="M7"/>
 <part name="GND1" library="SparkFun-Aesthetics" deviceset="GND" device=""/>
@@
 <part name="GND16" library="SparkFun" deviceset="GND" device=""/>
 <part name="R6" library="SparkFun-Passives" deviceset="RESISTOR" device="0805-RES" value="330"/>
-<part name="D3" library="led" library_urn="urn:adsk.eagle:library:259" deviceset="LED" device="CHIP-LED0805" package3d_urn="urn:adsk.eagle:package:15818/2" value="BLUE"/>
+<part name="INDL" library="led" library_urn="urn:adsk.eagle:library:259" deviceset="LED" device="CHIP-LED0805" package3d_urn="urn:adsk.eagle:package:15818/2" value="BLUE"/>
 <part name="GND17" library="SparkFun" deviceset="GND" device=""/>
 <part name="GND18" library="SparkFun" deviceset="GND" device=""/>
@@
 <text x="193.04" y="30.48" size="1.778" layer="91">IN3</text>
 <text x="309.88" y="15.24" size="2.54" layer="94">IOTB by Team IOTECH</text>
-<text x="365.76" y="12.7" size="2.54" layer="94">0.7</text>
+<text x="365.76" y="12.7" size="2.54" layer="94">0.8</text>
 <text x="170.18" y="170.18" size="1.778" layer="91">ETHERNET</text>
 <text x="175.26" y="109.22" size="1.778" layer="97">D2  -&gt;INT
@@
 <text x="172.72" y="203.2" size="1.778" layer="91">TTL</text>
 <text x="294.64" y="30.48" size="2.54" layer="94">IOTECH Yazılım Sanayi ve Ticaret A.Ş.
-TESA IO Kart Tasarımı.</text>
+TESA IO Board Design.</text>
 <wire x1="129.54" y1="101.6" x2="164.592" y2="101.6" width="0.2032" layer="97" style="shortdash"/>
 <wire x1="164.592" y1="61.468" x2="129.54" y2="61.468" width="0.2032" layer="97" style="shortdash"/>
@@
 </plain>
 <instances>
-<instance part="PLED1" gate="G$1" x="129.54" y="215.9" rot="R270"/>
+<instance part="PL" gate="G$1" x="129.54" y="215.9" rot="R270"/>
 <instance part="PD1" gate="G$1" x="40.64" y="223.52" rot="R90"/>
 <instance part="GND1" gate="1" x="76.2" y="210.82"/>
@@
 <instance part="GND16" gate="1" x="48.26" y="48.26"/>
 <instance part="R6" gate="G$1" x="121.92" y="12.7"/>
-<instance part="D3" gate="G$1" x="132.08" y="12.7" smashed="yes" rot="R90">
+<instance part="INDL" gate="G$1" x="132.08" y="12.7" smashed="yes" rot="R90">
 <attribute name="NAME" x="132.334" y="6.858" size="1.778" layer="95"/>
 <attribute name="VALUE" x="134.366" y="16.383" size="1.778" layer="96" rot="R180"/>
@@
 <segment>
 <pinref part="GND1" gate="1" pin="GND"/>
-<pinref part="PLED1" gate="G$1" pin="C"/>
+<pinref part="PL" gate="G$1" pin="C"/>
 <wire x1="30.48" y1="215.9" x2="45.72" y2="215.9" width="0.1524" layer="91"/>
 <wire x1="45.72" y1="215.9" x2="53.34" y2="215.9" width="0.1524" layer="91"/>
@@
 <segment>
 <wire x1="139.7" y1="12.7" x2="137.16" y2="12.7" width="0.1524" layer="91"/>
-<pinref part="D3" gate="G$1" pin="C"/>
+<pinref part="INDL" gate="G$1" pin="C"/>
 <pinref part="GND17" gate="1" pin="GND"/>
 </segment>
@@
 <segment>
 <pinref part="PR1" gate="G$1" pin="1"/>
-<pinref part="PLED1" gate="G$1" pin="A"/>
+<pinref part="PL" gate="G$1" pin="A"/>
 <wire x1="132.08" y1="215.9" x2="134.62" y2="215.9" width="0.1524" layer="91"/>
 </segment>
@@
 <wire x1="127" y1="12.7" x2="129.54" y2="12.7" width="0.1524" layer="91"/>
 <pinref part="R6" gate="G$1" pin="2"/>
-<pinref part="D3" gate="G$1" pin="A"/>
-</segment>
-</net>
+<pinref part="INDL" gate="G$1" pin="A"/>
+</segment>
+</net>
