File: KMO_IO_M/KMO_IO_MV1_0.brd (EAGLE design)
At the start: 84.5 x 96.5 mm, 67 parts, among them Q1 8MHz, Q2 25MHz, U1 ATMEGA328

Commit message: V1
Parts:
- added BL: (no value), con_io_sxp:S06P
Connections:
- net +3V3: now also BL.2
- net D11: now also BL.5
- net D12: now also BL.6
- net D13: now also BL.4
- net GND: now also BL.1
- net RESET: now also BL.3
Routing:
- net D13: track 107.6 -> 181.8 mm, vias 4 -> 1
- net +3V3: track 308.9 -> 372.6 mm, vias 9 -> 6
- net D3: track 114.5 -> 51.1 mm, vias 0 -> 1
- net D11: track 139.0 -> 98.8 mm
- net DTR: track 42.1 -> 78.0 mm, vias 1 -> 0
- net A6: track 154.2 -> 120.9 mm
- net A5: track 113.8 -> 86.0 mm, vias 2 -> 3
- net A1: track 90.0 -> 65.2 mm, vias 1 -> 2
- net A2: track 96.6 -> 73.7 mm, vias 3 -> 0
- net A4: track 108.4 -> 85.8 mm
- net D5: track 55.1 -> 37.4 mm, vias 2 -> 3
- net GND: track 517.9 -> 501.5 mm, vias 3 -> 1
- net RD+: track 51.7 -> 36.6 mm, vias 1 -> 2
- net TD-: track 38.2 -> 51.8 mm, vias 0 -> 1
- net RAW_IV: track 168.1 -> 156.2 mm, vias 0 -> 3
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
Commit message: v1
Parts:
- BL: value (none) -> 057-006-1; device con_io_sxp:S06P -> con-panduit:057-006-1
- moved BL 4.60 mm to (62.5, 90.0), turned to 0 degrees
- moved U1 3.76 mm to (60.2, 72.2)
- moved Q1 1.58 mm to (67.5, 65.5), turned to 45 degrees
- moved NIR1 1.50 mm to (73.2, 61.2)
- moved NIR2 1.50 mm to (73.2, 73.8)
- moved NIR3 1.50 mm to (73.2, 86.2)
- moved C1 0.25 mm to (47.8, 76.5)
- moved C3 0.25 mm to (47.8, 81.2)
- moved R1 0.25 mm to (47.8, 69.2)
- moved R3 0.25 mm to (47.8, 63.8)
Connections:
- net D11: now also BL.1; no longer BL.5
- net D12: now also BL.4; no longer BL.6
- net D13: now also BL.3; no longer BL.4
- net GND: now also BL.6; no longer BL.1
- net RESET: now also BL.5; no longer BL.3
Routing:
- net D13: track 181.8 -> 127.7 mm, vias 1 -> 4
- net +3V3: track 372.6 -> 338.9 mm, vias 6 -> 9
- net RAW_IV: track 156.2 -> 187.8 mm, vias 3 -> 0
- net D10: track 91.9 -> 65.2 mm, vias 4 -> 6
- net D7: track 41.8 -> 63.0 mm
- net D11: track 98.8 -> 79.1 mm, vias 2 -> 3
- net TD-: track 51.8 -> 33.0 mm, vias 1 -> 2
- net A7: track 117.4 -> 98.8 mm, vias 1 -> 3
- net A0: track 31.2 -> 49.6 mm, vias 0 -> 1
- net D12: track 71.6 -> 89.3 mm, vias 4 -> 2
- net RESET: track 95.3 -> 110.4 mm, vias 2 -> 3
- net A1: track 65.2 -> 79.8 mm, vias 2 -> 1
- net A4: track 85.8 -> 98.1 mm
- net GND: track 501.5 -> 489.6 mm, vias 1 -> 2
- net TD+: track 46.5 -> 35.2 mm, vias 1 -> 2
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