File: KMO_IO_M/KMO_IO_MV1_0.sch (EAGLE design)
At the start: 65 parts, among them Q1 8MHz, Q2 25MHz, U1 ATMEGA328

Commit message: V1
Parts:
- added BL: (no value), con_io_sxp:S06P
Connections:
- net +3V3: now also BL-2.S
- net D11: now also BL-5.S
- net D12: now also BL-6.S
- net D13: now also BL-4.S
- net GND: now also BL-1.S
- net RESET: now also BL-3.S
Other:
- note added: "-> D10"
- note added: "-> D11"
- note added: "-> D12"
- note added: "-> D13"
- note added: "-> GND"
- note added: "-> V3.3"
- note added: "BOOTLOADER"
Changed lines of the file:
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@@
 <part name="GND24" library="supply1" deviceset="GND" device=""/>
 <part name="+3V1" library="supply1" deviceset="+3V3" device=""/>
+<part name="BL" library="con_io_sxp" deviceset="S06P" device=""/>
+<part name="+3V3" library="supply1" deviceset="+3V3" device=""/>
+<part name="GND20" library="SparkFun" deviceset="GND" device=""/>
 </parts>
 <sheets>
@@
 <text x="307.34" y="76.2" size="1.778" layer="91">IN6</text>
 <text x="307.34" y="63.5" size="1.778" layer="91">IN7</text>
+<text x="144.78" y="55.88" size="1.778" layer="91">BOOTLOADER</text>
+<text x="165.1" y="50.8" size="1.778" layer="97">-&gt; D11</text>
+<text x="165.1" y="45.72" size="1.778" layer="97">-&gt; D12</text>
+<text x="165.1" y="40.64" size="1.778" layer="97">-&gt; D13</text>
+<text x="165.1" y="35.56" size="1.778" layer="97">-&gt; D10</text>
+<text x="165.1" y="30.48" size="1.778" layer="97">-&gt; V3.3</text>
+<text x="165.1" y="25.4" size="1.778" layer="97">-&gt; GND</text>
 </plain>
 <instances>
@@
 <instance part="+3V1" gate="G$1" x="264.16" y="182.88" smashed="yes">
 <attribute name="VALUE" x="261.62" y="177.8" size="1.778" layer="96" rot="R90"/>
+</instance>
+<instance part="BL" gate="-1" x="154.94" y="25.4" smashed="yes" rot="R180">
+<attribute name="NAME" x="155.448" y="24.384" size="1.778" layer="95"/>
+<attribute name="VALUE" x="154.686" y="27.813" size="1.778" layer="96" rot="R180"/>
+</instance>
+<instance part="BL" gate="-2" x="154.94" y="30.48" smashed="yes" rot="R180">
+<attribute name="NAME" x="155.448" y="29.464" size="1.778" layer="95"/>
+<attribute name="VALUE" x="154.686" y="32.893" size="1.778" layer="96" rot="R180"/>
+</instance>
+<instance part="BL" gate="-3" x="154.94" y="35.56" smashed="yes" rot="R180">
+<attribute name="NAME" x="155.448" y="34.544" size="1.778" layer="95"/>
+<attribute name="VALUE" x="154.686" y="37.973" size="1.778" layer="96" rot="R180"/>
+</instance>
+<instance part="BL" gate="-4" x="154.94" y="40.64" smashed="yes" rot="R180">
+<attribute name="NAME" x="155.448" y="39.624" size="1.778" layer="95"/>
+<attribute name="VALUE" x="154.686" y="43.053" size="1.778" layer="96" rot="R180"/>
+</instance>
+<instance part="BL" gate="-5" x="154.94" y="45.72" smashed="yes" rot="R180">
+<attribute name="NAME" x="155.448" y="44.704" size="1.778" layer="95"/>
+<attribute name="VALUE" x="154.686" y="48.133" size="1.778" layer="96" rot="R180"/>
+</instance>
+<instance part="BL" gate="-6" x="154.94" y="50.8" smashed="yes" rot="R180">
+<attribute name="NAME" x="155.448" y="49.784" size="1.778" layer="95"/>
+<attribute name="VALUE" x="154.686" y="53.213" size="1.778" layer="96" rot="R180"/>
+</instance>
+<instance part="+3V3" gate="G$1" x="144.78" y="30.48" smashed="yes" rot="R90">
+<attribute name="VALUE" x="149.86" y="27.94" size="1.778" layer="96" rot="R180"/>
+</instance>
+<instance part="GND20" gate="1" x="142.24" y="25.4" smashed="yes" rot="R270">
+<attribute name="VALUE" x="139.7" y="27.94" size="1.778" layer="96" rot="R270"/>
 </instance>
 </instances>
@@
 <pinref part="GND24" gate="1" pin="GND"/>
 </segment>
+<segment>
+<pinref part="BL" gate="-1" pin="S"/>
+<pinref part="GND20" gate="1" pin="GND"/>
+<wire x1="144.78" y1="25.4" x2="149.86" y2="25.4" width="0.1524" layer="91"/>
+</segment>
 </net>
 <net name="RAW_IV" class="1">
@@
 <pinref part="U1" gate="G$1" pin="PB4(MISO)"/>
 <label x="116.84" y="22.86" size="1.27" layer="95" xref="yes"/>
+</segment>
+<segment>
+<pinref part="BL" gate="-5" pin="S"/>
+<wire x1="149.86" y1="45.72" x2="147.32" y2="45.72" width="0.1524" layer="91"/>
+<label x="147.32" y="45.72" size="1.778" layer="95" rot="R180" xref="yes"/>
 </segment>
 </net>
@@
 <label x="83.82" y="226.06" size="1.778" layer="95" xref="yes"/>
 </segment>
+<segment>
+<pinref part="BL" gate="-2" pin="S"/>
+<pinref part="+3V3" gate="G$1" pin="+3V3"/>
+<wire x1="149.86" y1="30.48" x2="147.32" y2="30.48" width="0.1524" layer="91"/>
+</segment>
 </net>
 <net name="N$4" class="0">
@@
 <label x="119.38" y="20.32" size="1.27" layer="95" xref="yes"/>
 </segment>
+<segment>
+<pinref part="BL" gate="-4" pin="S"/>
+<wire x1="149.86" y1="40.64" x2="147.32" y2="40.64" width="0.1524" layer="91"/>
+<label x="147.32" y="40.64" size="1.778" layer="95" rot="R180" xref="yes"/>
+</segment>
 </net>
 <net name="D12" class="0">
@@
 <pinref part="U1" gate="G$1" pin="PB3(MOSI/OC2)"/>
 <label x="116.84" y="25.4" size="1.27" layer="95" xref="yes"/>
+</segment>
+<segment>
+<pinref part="BL" gate="-6" pin="S"/>
+<wire x1="149.86" y1="50.8" x2="147.32" y2="50.8" width="0.1524" layer="91"/>
+<label x="147.32" y="50.8" size="1.778" layer="95" rot="R180" xref="yes"/>
 </segment>
 </net>
@@
 <pinref part="SR" gate="1" pin="P"/>
 </segment>
-</net>
+<segment>
+<pinref part="BL" gate="-3" pin="S"/>
+<wire x1="149.86" y1="35.56" x2="147.32" y2="35.56" width="0.1524" layer="91"/>
+<label x="147.32" y="35.56" size="1.778" layer="95" rot="R180" xref="yes"/>
+</segment>
+</net>

Commit message: v1
Parts:
- BL: value (none) -> 057-006-1; device con_io_sxp:S06P -> con-panduit:057-006-1
Connections:
- net D11: now also BL-1.S; no longer BL-5.S
- net D12: now also BL-4.S; no longer BL-6.S
- net D13: now also BL-3.S; no longer BL-4.S
- net GND: now also BL-6.S; no longer BL-1.S
- net RESET: now also BL-5.S; no longer BL-3.S
Other:
- moved on the sheet: BL-1, BL-2, BL-3, BL-4, BL-5, BL-6
Changed lines of the file:
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@@
 <part name="GND24" library="supply1" deviceset="GND" device=""/>
 <part name="+3V1" library="supply1" deviceset="+3V3" device=""/>
-<part name="BL" library="con_io_sxp" deviceset="S06P" device=""/>
 <part name="+3V3" library="supply1" deviceset="+3V3" device=""/>
 <part name="GND20" library="SparkFun" deviceset="GND" device=""/>
+<part name="BL" library="con-panduit" library_urn="urn:adsk.eagle:library:169" deviceset="057-006-" device="1" package3d_urn="urn:adsk.eagle:package:9198/1"/>
 </parts>
 <sheets>
@@
 <attribute name="VALUE" x="261.62" y="177.8" size="1.778" layer="96" rot="R90"/>
 </instance>
-<instance part="BL" gate="-1" x="154.94" y="25.4" smashed="yes" rot="R180">
-<attribute name="NAME" x="155.448" y="24.384" size="1.778" layer="95"/>
-<attribute name="VALUE" x="154.686" y="27.813" size="1.778" layer="96" rot="R180"/>
-</instance>
-<instance part="BL" gate="-2" x="154.94" y="30.48" smashed="yes" rot="R180">
-<attribute name="NAME" x="155.448" y="29.464" size="1.778" layer="95"/>
-<attribute name="VALUE" x="154.686" y="32.893" size="1.778" layer="96" rot="R180"/>
-</instance>
-<instance part="BL" gate="-3" x="154.94" y="35.56" smashed="yes" rot="R180">
-<attribute name="NAME" x="155.448" y="34.544" size="1.778" layer="95"/>
-<attribute name="VALUE" x="154.686" y="37.973" size="1.778" layer="96" rot="R180"/>
-</instance>
-<instance part="BL" gate="-4" x="154.94" y="40.64" smashed="yes" rot="R180">
-<attribute name="NAME" x="155.448" y="39.624" size="1.778" layer="95"/>
-<attribute name="VALUE" x="154.686" y="43.053" size="1.778" layer="96" rot="R180"/>
-</instance>
-<instance part="BL" gate="-5" x="154.94" y="45.72" smashed="yes" rot="R180">
-<attribute name="NAME" x="155.448" y="44.704" size="1.778" layer="95"/>
-<attribute name="VALUE" x="154.686" y="48.133" size="1.778" layer="96" rot="R180"/>
-</instance>
-<instance part="BL" gate="-6" x="154.94" y="50.8" smashed="yes" rot="R180">
-<attribute name="NAME" x="155.448" y="49.784" size="1.778" layer="95"/>
-<attribute name="VALUE" x="154.686" y="53.213" size="1.778" layer="96" rot="R180"/>
-</instance>
 <instance part="+3V3" gate="G$1" x="144.78" y="30.48" smashed="yes" rot="R90">
 <attribute name="VALUE" x="149.86" y="27.94" size="1.778" layer="96" rot="R180"/>
@@
 <instance part="GND20" gate="1" x="142.24" y="25.4" smashed="yes" rot="R270">
 <attribute name="VALUE" x="139.7" y="27.94" size="1.778" layer="96" rot="R270"/>
+</instance>
+<instance part="BL" gate="-1" x="154.94" y="45.72" smashed="yes">
+<attribute name="NAME" x="155.956" y="44.958" size="1.524" layer="95"/>
+<attribute name="VALUE" x="152.4" y="47.625" size="1.778" layer="96"/>
+</instance>
+<instance part="BL" gate="-2" x="154.94" y="30.48" smashed="yes">
+<attribute name="NAME" x="155.956" y="29.718" size="1.524" layer="95"/>
+</instance>
+<instance part="BL" gate="-3" x="154.94" y="40.64" smashed="yes">
+<attribute name="NAME" x="155.956" y="39.878" size="1.524" layer="95"/>
+</instance>
+<instance part="BL" gate="-4" x="154.94" y="50.8" smashed="yes">
+<attribute name="NAME" x="155.956" y="50.038" size="1.524" layer="95"/>
+</instance>
+<instance part="BL" gate="-5" x="154.94" y="35.56" smashed="yes">
+<attribute name="NAME" x="155.956" y="34.798" size="1.524" layer="95"/>
+</instance>
+<instance part="BL" gate="-6" x="154.94" y="25.4" smashed="yes">
+<attribute name="NAME" x="155.956" y="24.638" size="1.524" layer="95"/>
 </instance>
 </instances>
@@
 </segment>
 <segment>
-<pinref part="BL" gate="-1" pin="S"/>
 <pinref part="GND20" gate="1" pin="GND"/>
 <wire x1="144.78" y1="25.4" x2="149.86" y2="25.4" width="0.1524" layer="91"/>
+<pinref part="BL" gate="-6" pin="S"/>
 </segment>
 </net>
@@
 </segment>
 <segment>
-<pinref part="BL" gate="-5" pin="S"/>
 <wire x1="149.86" y1="45.72" x2="147.32" y2="45.72" width="0.1524" layer="91"/>
 <label x="147.32" y="45.72" size="1.778" layer="95" rot="R180" xref="yes"/>
+<pinref part="BL" gate="-1" pin="S"/>
 </segment>
 </net>
@@
 </segment>
 <segment>
-<pinref part="BL" gate="-2" pin="S"/>
 <pinref part="+3V3" gate="G$1" pin="+3V3"/>
 <wire x1="149.86" y1="30.48" x2="147.32" y2="30.48" width="0.1524" layer="91"/>
+<pinref part="BL" gate="-2" pin="S"/>
 </segment>
 </net>
@@
 </segment>
 <segment>
-<pinref part="BL" gate="-4" pin="S"/>
 <wire x1="149.86" y1="40.64" x2="147.32" y2="40.64" width="0.1524" layer="91"/>
 <label x="147.32" y="40.64" size="1.778" layer="95" rot="R180" xref="yes"/>
+<pinref part="BL" gate="-3" pin="S"/>
 </segment>
 </net>
@@
 </segment>
 <segment>
-<pinref part="BL" gate="-6" pin="S"/>
 <wire x1="149.86" y1="50.8" x2="147.32" y2="50.8" width="0.1524" layer="91"/>
 <label x="147.32" y="50.8" size="1.778" layer="95" rot="R180" xref="yes"/>
+<pinref part="BL" gate="-4" pin="S"/>
 </segment>
 </net>
@@
 </segment>
 <segment>
-<pinref part="BL" gate="-3" pin="S"/>
 <wire x1="149.86" y1="35.56" x2="147.32" y2="35.56" width="0.1524" layer="91"/>
 <label x="147.32" y="35.56" size="1.778" layer="95" rot="R180" xref="yes"/>
-</segment>
-</net>
+<pinref part="BL" gate="-5" pin="S"/>
+</segment>
+</net>
