File: KMO_IO_M/KMO_IO_MV1_2.brd (EAGLE design)
At the start: 84.5 x 96.5 mm, 93 parts, among them IC1 100p, IC2 100p, IC3 100p, IC4 100p, IC5 100p, IC6 100p, IC7 100p, Q1 8MHz, Q2 25MHz, U1 ATMEGA328

Commit message: 12
Parts:
- IR1: value 10M -> 10K
Changed lines of the file:
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@@
 <?xml version="1.0" encoding="utf-8"?>
 <!DOCTYPE eagle SYSTEM "eagle.dtd">
-<eagle version="9.3.1">
+<eagle version="9.3.0">
 <drawing>
 <settings>
@@
 <attribute name="VALUE" x="71.853" y="87.266" size="0.4064" layer="27" rot="R270"/>
 </element>
-<element name="IR1" library="SparkFun-Passives" package="0805" value="10M" x="11.5" y="37" smashed="yes" rot="R90">
+<element name="IR1" library="SparkFun-Passives" package="0805" value="10K" x="11.5" y="37" smashed="yes" rot="R90">
 <attribute name="NAME" x="10.6745" y="36.238" size="0.4064" layer="25" rot="R90"/>
 <attribute name="VALUE" x="12.897" y="35.984" size="0.4064" layer="27" rot="R90"/>

Commit message: 12 inductor rev
Parts:
- PCO: value 33 uh -> 220 uh
Changed lines of the file:
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@@
 <?xml version="1.0" encoding="utf-8"?>
 <!DOCTYPE eagle SYSTEM "eagle.dtd">
-<eagle version="9.3.0">
+<eagle version="9.3.1">
 <drawing>
 <settings>
@@
 <attribute name="VALUE" x="56.865" y="18.875" size="1.27" layer="27" rot="R270"/>
 </element>
-<element name="PCO" library="inductor-coilcraft" package="MSS1260" value="33 uh" x="33.25" y="9.25" smashed="yes">
+<element name="PCO" library="inductor-coilcraft" package="MSS1260" value="220 uh" x="33.25" y="9.25" smashed="yes">
 <attribute name="NAME" x="30.25" y="9.75" size="1.27" layer="25"/>
 <attribute name="VALUE" x="30.25" y="7.25" size="1.27" layer="27"/>

Commit message: kapasitör value
Parts:
- C1, C2, C3: value 0.1uF -> 100nF
Changed lines of the file:
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@@
 <attribute name="VALUE" x="52.897" y="82.984" size="0.4064" layer="27" rot="R90"/>
 </element>
-<element name="C3" library="SparkFun-Passives" package="0805" value="0.1uF" x="48.25" y="79.5" smashed="yes">
+<element name="C3" library="SparkFun-Passives" package="0805" value="100nF" x="48.25" y="79.5" smashed="yes">
 <attribute name="NAME" x="47.488" y="80.3255" size="0.4064" layer="25"/>
 <attribute name="VALUE" x="47.234" y="78.103" size="0.4064" layer="27"/>
 </element>
-<element name="C1" library="SparkFun-Passives" package="0805" value="0.1uF" x="48.25" y="75.25" smashed="yes">
+<element name="C1" library="SparkFun-Passives" package="0805" value="100nF" x="48.25" y="75.25" smashed="yes">
 <attribute name="NAME" x="47.488" y="76.0755" size="0.4064" layer="25"/>
 <attribute name="VALUE" x="47.234" y="73.853" size="0.4064" layer="27"/>
@@
 <attribute name="VALUE" x="66.536178125" y="74.944075" size="0.4064" layer="27" rot="R135"/>
 </element>
-<element name="C2" library="SparkFun-Passives" package="0805" value="0.1uF" x="55" y="80.5" smashed="yes" rot="R180">
+<element name="C2" library="SparkFun-Passives" package="0805" value="100nF" x="55" y="80.5" smashed="yes" rot="R180">
 <attribute name="NAME" x="55.762" y="79.6745" size="0.4064" layer="25" rot="R180"/>
 <attribute name="VALUE" x="56.016" y="81.897" size="0.4064" layer="27" rot="R180"/>
