File: KMO_IO_M/KMO_IO_MV1_2.sch (EAGLE design)
At the start: 92 parts, among them IC1 100p, IC2 100p, IC3 100p, IC4 100p, IC5 100p, IC6 100p, IC7 100p, Q1 8MHz, Q2 25MHz, U1 ATMEGA328

Commit message: v12 bl rev
Parts:
- removed D1, D2: M7, SparkFun-DiscreteSemi:DIODESMA
- added BLS: (no value), special:SW_DIP-1
- IIR1: value 22 -> 10K
- IIR2: value 22 -> 22K
- IR1, IR2: value 10K -> 10M
Connections:
- removed net A10: IC4.1, ID4.C, IIR4.1
- removed net A11: IC5.1, ID5.C, IIR5.1
- removed net A12: IC6.1, ID6.C, IIR6.1
- removed net A13: IC7.1, ID7.C, IIR7.1
- removed net A8: IC2.1, ID2.C, IIR2.1
- removed net A9: IC3.1, ID3.C, IIR3.1
- net +3V3: now also BLS.1; no longer D1.A
- net A2: now also IC2.1, ID2.C, IIR2.1
- net A3: now also IC3.1, ID3.C, IIR3.1
- net A4: now also IC4.1, ID4.C, IIR4.1
- net A5: now also IC5.1, ID5.C, IIR5.1
- net A6: now also IC6.1, ID6.C, IIR6.1
- net A7: now also IC7.1, ID7.C, IIR7.1
- net BLG: no longer C1.1, C3.2, D2.A, INDL.C, Q1.2, SR.S, U1.AGND, U1.GND@1, U1.GND@2
- net BLV: now also BLS.2; no longer D1.C
- net GND: now also C1.1, C3.2, INDL.C, Q1.2, SR.S, U1.AGND, U1.GND@1, U1.GND@2; no longer D2.C

Commit message: 12
Parts:
- IR1: value 10M -> 10K
Changed lines of the file:
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@@
 <part name="NIR3" library="SparkFun-Passives" deviceset="RESISTOR" device="0805-RES" value="4700"/>
 <part name="GND10" library="supply1" deviceset="GND" device=""/>
-<part name="IR1" library="SparkFun-Passives" deviceset="RESISTOR" device="0805-RES" value="10M"/>
+<part name="IR1" library="SparkFun-Passives" deviceset="RESISTOR" device="0805-RES" value="10K"/>
 <part name="GND11" library="supply1" deviceset="GND" device=""/>
 <part name="IR2" library="SparkFun-Passives" deviceset="RESISTOR" device="0805-RES" value="10M"/>

Commit message: 12 inductor rev
Parts:
- PCO: value 33 uh -> 220 uh
Changed lines of the file:
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@@
 <?xml version="1.0" encoding="utf-8"?>
 <!DOCTYPE eagle SYSTEM "eagle.dtd">
-<eagle version="9.3.0">
+<eagle version="9.3.1">
 <drawing>
 <settings>
@@
 <part name="PC1" library="rcl" library_urn="urn:adsk.eagle:library:334" deviceset="CPOL-EU" device="140CLH-1010" package3d_urn="urn:adsk.eagle:package:23391/1" value="470uf 25v"/>
 <part name="PC2" library="rcl" library_urn="urn:adsk.eagle:library:334" deviceset="CPOL-EU" device="140CLH-1010" package3d_urn="urn:adsk.eagle:package:23391/1" value="220uf 50v"/>
-<part name="PCO" library="inductor-coilcraft" deviceset="MSS1260" device="" value="33 uh"/>
+<part name="PCO" library="inductor-coilcraft" deviceset="MSS1260" device="" value="220 uh"/>
 <part name="PIC33" library="national-semiconductor" library_urn="urn:adsk.eagle:library:307" deviceset="LM2596" device="S" package3d_urn="urn:adsk.eagle:package:21218/1"/>
 <part name="PD2" library="diode" library_urn="urn:adsk.eagle:library:210" deviceset="SCHOTTKY-DIODE" device="SMD" package3d_urn="urn:adsk.eagle:package:43404/2" value="SS54"/>

Commit message: kapasitör value
Parts:
- C1, C2, C3: value 0.1uF -> 100nF
Changed lines of the file:
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@@
 <part name="+3V2" library="supply1" deviceset="+3V3" device=""/>
 <part name="R2" library="SparkFun-Passives" deviceset="RESISTOR" device="0805-RES" value="10K"/>
-<part name="C3" library="SparkFun-Passives" deviceset="CAP" device="0805" value="0.1uF"/>
-<part name="C1" library="SparkFun-Passives" deviceset="CAP" device="0805" value="0.1uF"/>
+<part name="C3" library="SparkFun-Passives" deviceset="CAP" device="0805" value="100nF"/>
+<part name="C1" library="SparkFun-Passives" deviceset="CAP" device="0805" value="100nF"/>
 <part name="R6" library="SparkFun-Passives" deviceset="RESISTOR" device="0805-RES" value="1k"/>
 <part name="INDL" library="led" library_urn="urn:adsk.eagle:library:259" deviceset="LED" device="CHIP-LED0805" package3d_urn="urn:adsk.eagle:package:15818/2" value="BLU"/>
 <part name="U1" library="SparkFun" deviceset="ATMEGA168" device="" value="ATMEGA328"/>
-<part name="C2" library="SparkFun-Passives" deviceset="CAP" device="0805" value="0.1uF"/>
+<part name="C2" library="SparkFun-Passives" deviceset="CAP" device="0805" value="100nF"/>
 <part name="R1" library="SparkFun-Passives" deviceset="RESISTOR" device="0805-RES"/>
 <part name="Q1" library="Testing" deviceset="RESONATOR" device="1:1" value="8MHz"/>
