File: KMO_IO_M/KMO_IO_MV1_3.sch (EAGLE design)
At the start: 79 parts, among them Q1 8MHz, Q2 25MHz, U1 ATMEGA328

Commit message: connector rew 3,81
Parts:
- added X1: MC10, con-phoenix-381_l:MC10
- added X2: MC6, con-phoenix-381_l:MC6
- added X3: MC2, con-phoenix-381_l:MC2
Changed lines of the file:
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@@
 <part name="IR7" library="SparkFun-Passives" deviceset="RESISTOR" device="0805-RES" value="1K"/>
 <part name="IL7" library="led" library_urn="urn:adsk.eagle:library:259" deviceset="LED" device="CHIP-LED0805" package3d_urn="urn:adsk.eagle:package:15818/2" value="BLU"/>
+<part name="X1" library="con-phoenix-381_l" deviceset="MC10" device=""/>
+<part name="X2" library="con-phoenix-381_l" deviceset="MC6" device=""/>
+<part name="X3" library="con-phoenix-381_l" deviceset="MC2" device=""/>
 </parts>
 <sheets>
@@
 <attribute name="VALUE" x="344.932" y="53.975" size="1.778" layer="96" rot="R180"/>
 </instance>
+<instance part="X1" gate=".1" x="-33.02" y="68.58" smashed="yes">
+<attribute name="NAME" x="-40.64" y="70.485" size="1.524" layer="95"/>
+</instance>
+<instance part="X1" gate=".2" x="-33.02" y="63.5" smashed="yes">
+<attribute name="NAME" x="-40.64" y="65.405" size="1.524" layer="95"/>
+</instance>
+<instance part="X1" gate=".3" x="-33.02" y="58.42" smashed="yes">
+<attribute name="NAME" x="-40.64" y="60.325" size="1.524" layer="95"/>
+</instance>
+<instance part="X1" gate=".4" x="-33.02" y="53.34" smashed="yes">
+<attribute name="NAME" x="-40.64" y="55.245" size="1.524" layer="95"/>
+</instance>
+<instance part="X1" gate=".5" x="-33.02" y="48.26" smashed="yes">
+<attribute name="NAME" x="-40.64" y="50.165" size="1.524" layer="95"/>
+</instance>
+<instance part="X1" gate=".6" x="-33.02" y="43.18" smashed="yes">
+<attribute name="NAME" x="-40.64" y="45.085" size="1.524" layer="95"/>
+</instance>
+<instance part="X1" gate=".7" x="-33.02" y="38.1" smashed="yes">
+<attribute name="NAME" x="-40.64" y="40.005" size="1.524" layer="95"/>
+</instance>
+<instance part="X1" gate=".8" x="-33.02" y="33.02" smashed="yes">
+<attribute name="NAME" x="-40.64" y="34.925" size="1.524" layer="95"/>
+</instance>
+<instance part="X1" gate=".9" x="-33.02" y="27.94" smashed="yes">
+<attribute name="NAME" x="-40.64" y="29.845" size="1.524" layer="95"/>
+</instance>
+<instance part="X1" gate=".10" x="-33.02" y="22.86" smashed="yes">
+<attribute name="NAME" x="-40.64" y="24.765" size="1.524" layer="95"/>
+</instance>
+<instance part="X2" gate=".1" x="-33.02" y="127" smashed="yes">
+<attribute name="NAME" x="-40.64" y="128.905" size="1.524" layer="95"/>
+</instance>
+<instance part="X2" gate=".2" x="-33.02" y="121.92" smashed="yes">
+<attribute name="NAME" x="-40.64" y="123.825" size="1.524" layer="95"/>
+</instance>
+<instance part="X2" gate=".3" x="-33.02" y="116.84" smashed="yes">
+<attribute name="NAME" x="-40.64" y="118.745" size="1.524" layer="95"/>
+</instance>
+<instance part="X2" gate=".4" x="-33.02" y="111.76" smashed="yes">
+<attribute name="NAME" x="-40.64" y="113.665" size="1.524" layer="95"/>
+</instance>
+<instance part="X2" gate=".5" x="-33.02" y="106.68" smashed="yes">
+<attribute name="NAME" x="-40.64" y="108.585" size="1.524" layer="95"/>
+</instance>
+<instance part="X2" gate=".6" x="-33.02" y="101.6" smashed="yes">
+<attribute name="NAME" x="-40.64" y="103.505" size="1.524" layer="95"/>
+</instance>
+<instance part="X3" gate=".1" x="-35.56" y="88.9" smashed="yes">
+<attribute name="NAME" x="-43.18" y="90.805" size="1.524" layer="95"/>
+</instance>
+<instance part="X3" gate=".2" x="-35.56" y="83.82" smashed="yes">
+<attribute name="NAME" x="-43.18" y="85.725" size="1.524" layer="95"/>
+</instance>
 </instances>

Commit message: v13
Parts:
- removed X2: MC6, con-phoenix-381_l:MC6
- removed X3: MC2, con-phoenix-381_l:MC2
- X1: value MC10 -> MC3; device con-phoenix-381_l:MC10 -> con-phoenix-381_l:MC3
- XI: value MSTBA10 -> MC10; device con-phoenix-508:MSTBA10 -> con-phoenix-381_l:MC10
- XO: value MSTBA6 -> MC6; device con-phoenix-508:MSTBA6 -> con-phoenix-381_l:MC6
Connections:
- removed net N$18: PD1.A, PJ1.PWR
- new net VIN: PD1.A, PJ1.PWR, X1.3.SK
- new net WFGPIO2: WIFI.GPIO2
- net GND: now also X1.2.SK; no longer XI-2.1
- net N$1: now also XO.6.SK; no longer XO-6.1
- net N$12: now also XI.4.SK; no longer XI-4.1
- net N$20: now also XI.5.SK; no longer XI-5.1
- net N$21: now also XI.6.SK; no longer XI-6.1
- net N$23: now also XI.7.SK; no longer XI-7.1
- net N$25: now also XI.8.SK; no longer XI-8.1
- net N$26: now also XI.9.SK; no longer XI-9.1
- net N$27: now also XI.10.SK; no longer XI-10.1
- net N$28: now also XI.2.SK; no longer XI-3.1
- net N$3: now also XO.2.SK; no longer XO-2.1
- net N$4: now also XO.4.SK; no longer XO-4.1
- net RAW_IV: now also X1.1.SK, XO.1.SK, XO.3.SK, XO.5.SK; no longer XI-1.1, XO-1.1, XO-3.1, XO-5.1
Other:
- note added: "COM"
- note added: "V OUT-IN"
- note added: "WIN2"
- moved on the sheet: IL0, IR0, PC1, X1.1, X1.2, X1.3

Commit message: 13
Parts:
- removed IL0: BLU, led:LEDCHIP-LED0805
- removed IR0: 1K, SparkFun-Passives:RESISTOR0805-RES
- added WIL0, WIL2: BLU, led:LEDCHIP-LED0805
- added WIR0, WIR2: 1K, SparkFun-Passives:RESISTOR0805-RES
Connections:
- new net N$18: WIL2.C, XI.3.SK
- net +3V3: now also WIR0.1, WIR2.1; no longer IR0.1
- net N$28: now also WIL0.C; no longer IL0.C
- net WFGPIO0: now also WIL0.A, WIR0.2; no longer IL0.A, IR0.2
- net WFGPIO2: now also WIL2.A, WIR2.2
Other:
- moved on the sheet: IL1, IL2, IL3, IR1, IR2, IR3, XI.2, XI.3, XI.4, XI.5, XI.6

Commit message: 13
Parts:
- added IR: 10K, SparkFun-Passives:RESISTOR0805-RES
Connections:
- new net N$29: IR.1, XI.1.SK
- net GND: now also IR.2
Other:
- moved on the sheet: XI.1
Changed lines of the file:
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@@
 <?xml version="1.0" encoding="utf-8"?>
 <!DOCTYPE eagle SYSTEM "eagle.dtd">
-<eagle version="9.3.1">
+<eagle version="9.3.2">
 <drawing>
 <settings>
@@
 <part name="+3V11" library="supply1" deviceset="+3V3" device=""/>
 <part name="WIL2" library="led" library_urn="urn:adsk.eagle:library:259" deviceset="LED" device="CHIP-LED0805" package3d_urn="urn:adsk.eagle:package:15818/2" value="BLU"/>
+<part name="IR" library="SparkFun-Passives" deviceset="RESISTOR" device="0805-RES" value="10K"/>
+<part name="GND11" library="supply1" deviceset="GND" device=""/>
 </parts>
 <sheets>
@@
 <attribute name="VALUE" x="344.932" y="53.975" size="1.778" layer="96" rot="R180"/>
 </instance>
-<instance part="XI" gate=".1" x="190.5" y="91.44" smashed="yes">
-<attribute name="NAME" x="182.88" y="93.345" size="1.524" layer="95"/>
+<instance part="XI" gate=".1" x="193.04" y="91.44" smashed="yes">
+<attribute name="NAME" x="185.42" y="93.345" size="1.524" layer="95"/>
 </instance>
 <instance part="XI" gate=".2" x="228.6" y="68.58" smashed="yes" rot="R180">
@@
 <attribute name="NAME" x="217.932" y="56.896" size="1.778" layer="95" rot="R180"/>
 <attribute name="VALUE" x="217.932" y="59.055" size="1.778" layer="96" rot="R180"/>
+</instance>
+<instance part="IR" gate="G$1" x="203.2" y="91.44" smashed="yes">
+<attribute name="NAME" x="199.39" y="92.9386" size="1.778" layer="95"/>
+<attribute name="VALUE" x="199.39" y="88.138" size="1.778" layer="96"/>
+</instance>
+<instance part="GND11" gate="1" x="213.36" y="91.44" smashed="yes" rot="R90">
+<attribute name="VALUE" x="215.9" y="88.9" size="1.778" layer="96" rot="R90"/>
 </instance>
 </instances>
@@
 <junction x="63.5" y="10.16"/>
 </segment>
+<segment>
+<pinref part="IR" gate="G$1" pin="2"/>
+<pinref part="GND11" gate="1" pin="GND"/>
+<wire x1="208.28" y1="91.44" x2="210.82" y2="91.44" width="0.1524" layer="91"/>
+</segment>
 </net>
 <net name="RAW_IV" class="1">
@@
 </segment>
 </net>
+<net name="N$29" class="0">
+<segment>
+<pinref part="XI" gate=".1" pin="SK"/>
+<pinref part="IR" gate="G$1" pin="1"/>
+<wire x1="193.04" y1="91.44" x2="198.12" y2="91.44" width="0.1524" layer="91"/>
+</segment>
+</net>
