File: KMO_IO_M/KMO_IO_MV1_3.brd (EAGLE design)
At the start: 84.5 x 96.5 mm, 81 parts, among them Q1 8MHz, Q2 25MHz, U1 ATMEGA328

Commit message: connector rew 3,81
Parts:
- added X1: MC10, con-phoenix-381_l:MC10
- added X2: MC6, con-phoenix-381_l:MC6
- added X3: MC2, con-phoenix-381_l:MC2
Changed lines of the file:
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@@
 <attribute name="VALUE" x="14.52" y="8.79" size="1.27" layer="27" rot="R180"/>
+</element>
+<element name="X1" library="con-phoenix-381_l" package="MC10" value="MC10" x="5" y="22.5" smashed="yes" rot="R270">
+<attribute name="NAME" x="7.54" y="40.915" size="1.27" layer="21" rot="R270"/>
+<attribute name="VALUE" x="0.555" y="40.915" size="1.27" layer="21" rot="R270"/>
+</element>
+<element name="X2" library="con-phoenix-381_l" package="MC6" value="MC6" x="5" y="82" smashed="yes" rot="R270">
+<attribute name="NAME" x="7.54" y="92.795" size="1.27" layer="21" rot="R270"/>
+<attribute name="VALUE" x="0.555" y="92.795" size="1.27" layer="21" rot="R270"/>
+</element>
+<element name="X3" library="con-phoenix-381_l" package="MC2" value="MC2" x="5" y="51.25" smashed="yes" rot="R270">
+<attribute name="NAME" x="7.54" y="54.425" size="1.27" layer="21" rot="R270"/>
+<attribute name="VALUE" x="0.555" y="54.425" size="1.27" layer="21" rot="R270"/>
 </element>
 </elements>

Commit message: v13
Parts:
- removed X2: MC6, con-phoenix-381_l:MC6
- removed X3: MC2, con-phoenix-381_l:MC2
- X1: value MC10 -> MC3; device con-phoenix-381_l:MC10 -> con-phoenix-381_l:MC3
- XI: value MSTBA10 -> MC10; device con-phoenix-508:MSTBA10 -> con-phoenix-381_l:MC10
- XO: value MSTBA6 -> MC6; device con-phoenix-508:MSTBA6 -> con-phoenix-381_l:MC6
- moved X1 33.5 mm to (5.00, 56.0)
- moved IL1 8.53 mm to (12.5, 28.2)
- moved IL2 7.54 mm to (12.5, 24.2)
- moved XI 7.39 mm to (5.00, 22.5)
- moved OL3 6.75 mm to (12.0, 74.2)
- moved IL0 6.29 mm to (12.5, 35.8)
- moved IL3 6.29 mm to (12.5, 20.5)
- moved XO 5.20 mm to (5.00, 82.0)
- moved IL4 5.06 mm to (12.5, 16.8)
- moved OL2 4.51 mm to (12.0, 82.0)
- moved IL5 3.58 mm to (12.5, 13.0)
- moved IL6 2.37 mm to (12.5, 9.25)
- moved OL1 2.02 mm to (12.0, 89.8)
- moved IL7 1.06 mm to (12.5, 5.50)
- moved OD3 0.50 mm to (17.0, 63.8)
Connections:
- removed net N$18: PD1.A, PJ1.VIN0
- new net VIN: PD1.A, PJ1.VIN0, X1.3
- new net WFGPIO2: WIFI.GPIO2
- net GND: now also X1.2; no longer XI.2
- net N$28: now also XI.2; no longer XI.3
- net RAW_IV: now also X1.1; no longer XI.1
Routing:
- net GND: track 469.5 -> 0.00 mm, vias 3 -> 0
- net +3V3: track 355.8 -> 0.00 mm, vias 2 -> 0
- net RAW_IV: track 177.7 -> 0.00 mm, vias 1 -> 0
- net D13: track 117.7 -> 0.00 mm, vias 1 -> 0
- net A7: track 111.2 -> 0.00 mm, vias 2 -> 0
- net A6: track 108.5 -> 0.00 mm, vias 2 -> 0
- net RESET: track 98.9 -> 0.00 mm, vias 3 -> 0
- net BLV: track 87.0 -> 0.00 mm, vias 2 -> 0
- net A5: track 83.0 -> 0.00 mm, vias 4 -> 0
- net A4: track 75.7 -> 0.00 mm, vias 4 -> 0
- net DTR: track 73.0 -> 0.00 mm
- net D11: track 70.1 -> 0.00 mm, vias 3 -> 0
- net A3: track 67.1 -> 0.00 mm
- net D12: track 64.9 -> 0.00 mm, vias 3 -> 0
- net D4: track 63.5 -> 0.00 mm, vias 1 -> 0
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
Commit message: 13
Parts:
- removed IR0: 1K, SparkFun-Passives:0805
- added WIL2: BLU, led:CHIP-LED0805
- added WIR0, WIR2: 1K, SparkFun-Passives:0805
- moved IR1 8.50 mm to (17.5, 28.2)
- moved IR2 7.50 mm to (17.2, 24.2)
- moved IR3 6.25 mm to (17.2, 20.5)
- moved IR5 5.67 mm to (21.5, 13.2)
- moved IR4 5.00 mm to (17.2, 16.8)
- moved IR7 0.75 mm to (17.2, 5.50)
- moved IR6 0.25 mm to (17.2, 9.25)
- renumbered IL0 to WIL0
Connections:
- new net N$18: WIL2.C, XI.3
- net +3V3: now also WIR0.1, WIR2.1; no longer IR0.1
- net WFGPIO0: now also WIR0.2; no longer IR0.2
- net WFGPIO2: now also WIL2.A, WIR2.2

Commit message: 13
Parts:
- added IR: 10K, SparkFun-Passives:0805
Connections:
- new net N$29: IR.1, XI.1
- net GND: now also IR.2
Changed lines of the file:
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@@
 <?xml version="1.0" encoding="utf-8"?>
 <!DOCTYPE eagle SYSTEM "eagle.dtd">
-<eagle version="9.3.1">
+<eagle version="9.3.2">
 <drawing>
 <settings>
@@
 <attribute name="VALUE" x="10.77" y="32.54" size="1.27" layer="27" rot="R180"/>
 </element>
+<element name="IR" library="SparkFun-Passives" package="0805" value="10K" x="12.5" y="39.5" smashed="yes">
+<attribute name="NAME" x="11.738" y="40.3255" size="0.4064" layer="25"/>
+<attribute name="VALUE" x="11.484" y="38.103" size="0.4064" layer="27"/>
+</element>
 </elements>
 <signals>
@@
 <contactref element="C3" pad="2"/>
 <contactref element="X1" pad="2"/>
+<contactref element="IR" pad="2"/>
 <wire x1="79.75" y1="77.75" x2="79.75" y2="90.25" width="0" layer="19" extent="1-1"/>
 <wire x1="79.75" y1="65.25" x2="79.75" y2="77.75" width="0" layer="19" extent="1-1"/>
@@
 <wire x1="12" y1="83.05" x2="12" y2="75.3" width="0" layer="19" extent="1-1"/>
 <wire x1="12" y1="90.8" x2="12" y2="83.05" width="0" layer="19" extent="1-1"/>
+<wire x1="13.4" y1="39.5" x2="32.75" y2="27.65" width="0" layer="19" extent="1-1"/>
 </signal>
 <signal name="N$11">
@@
 <wire x1="11.45" y1="32" x2="5" y2="32.025" width="0" layer="19" extent="1-1"/>
 </signal>
+<signal name="N$29">
+<contactref element="XI" pad="1"/>
+<contactref element="IR" pad="1"/>
+<wire x1="11.6" y1="39.5" x2="5" y2="39.645" width="0" layer="19" extent="1-1"/>
+</signal>
 </signals>

Commit message: bom
Routing:
- net GND: track 0.00 -> 503.8 mm, vias 0 -> 3
- net +3V3: track 0.00 -> 306.9 mm, vias 0 -> 4
- net RAW_IV: track 0.00 -> 181.2 mm, vias 0 -> 1
- net VIN: track 0.00 -> 131.4 mm
- net A7: track 0.00 -> 116.2 mm, vias 0 -> 2
- net D13: track 0.00 -> 115.3 mm, vias 0 -> 1
- net RESET: track 0.00 -> 104.2 mm, vias 0 -> 2
- net A6: track 0.00 -> 91.1 mm, vias 0 -> 4
- net A5: track 0.00 -> 86.3 mm, vias 0 -> 3
- net BLV: track 0.00 -> 86.1 mm, vias 0 -> 2
- net A4: track 0.00 -> 78.5 mm, vias 0 -> 3
- net A3: track 0.00 -> 77.8 mm, vias 0 -> 2
- net A1: track 0.00 -> 73.6 mm, vias 0 -> 2
- net A2: track 0.00 -> 73.3 mm
- net D11: track 0.00 -> 68.1 mm, vias 0 -> 3
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