File: KMO_IO_M/KMO_IO_MV2_0.brd (EAGLE design)
At the start: 84.5 x 96.5 mm, 85 parts, among them Q1 8MHz, Q2 25MHz, U1 ATMEGA328, X1 MC3

Commit message: v2
Parts:
- removed IR: 10K, SparkFun-Passives:0805
- removed WIL0, WIL2: BLU, led:CHIP-LED0805
- removed WIR0, WIR2: 1K, SparkFun-Passives:0805
- added IL8: BLU, led:CHIP-LED0805
- added IR8: 1K, SparkFun-Passives:0805
- added ITR1, ITR2, ITR3, ITR4, ITR5, ITR6, ITR7, ITR8: 6.8K, SparkFun-Passives:0805
- added OK1, OK2: TLP283-4, optocoupler:MINI-FLAT-16
- added X2, X4: MC5, con-phoenix-381_l:MC5
- added X3: MC2, con-phoenix-381_l:MC2
- moved WIFI 45.7 mm to (64.5, 68.8), turned to 0 degrees
- moved U$1 44.6 mm to (19.5, 8.00)
- moved IL2 20.0 mm to (30.8, 32.5), turned to 270 degrees
- moved IL3 20.0 mm to (30.8, 28.8), turned to 270 degrees
- moved IL1 19.9 mm to (30.8, 36.2), turned to 270 degrees
- moved IL4 19.9 mm to (30.8, 24.8), turned to 270 degrees
- moved EC3 19.7 mm to (51.2, 47.0), turned to 0 degrees
- moved ER10 19.0 mm to (52.2, 31.0), turned to 0 degrees
- moved IL5 18.7 mm to (30.8, 17.2), turned to 270 degrees
- moved IL6 18.7 mm to (30.8, 13.5), turned to 270 degrees
- moved IL7 18.7 mm to (30.8, 9.75), turned to 270 degrees
- moved ER1 18.4 mm to (48.8, 31.0)
- moved IR7 16.7 mm to (25.0, 20.2)
- moved ER2 16.3 mm to (45.8, 31.8), turned to 270 degrees
- moved IR4 15.6 mm to (25.0, 30.2)
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Connections:
- new net COM1: OK1.2, OK1.4, OK1.6, OK1.8, XI.1
- new net N$30: ITR2.2, OK1.3
- new net N$31: ITR3.2, OK1.5
- new net N$32: ITR4.2, OK1.7
- new net N$33: ITR3.1, XI.4
- new net N$34: ITR4.1, XI.5
- new net N$35: OK2.2, OK2.4, OK2.6, OK2.8, XI.6
- new net N$36: ITR5.1, XI.7
- new net N$37: ITR5.2, OK2.1
- new net N$38: ITR6.1, XI.8
- new net N$39: ITR6.2, OK2.3
- new net N$40: ITR7.1, XI.9
- new net N$41: ITR7.2, OK2.5
- new net N$42: ITR8.1, XI.10
- new net N$43: ITR8.2, OK2.7
- new net N$44: IL8.A, OK2.9
- net +3V3: now also IR8.1; no longer WIR0.1, WIR2.1
- net A1: now also OK1.16; no longer IL1.A
- net A2: now also OK1.14; no longer IL2.A
- net A3: now also OK1.12; no longer IL3.A
- net A4: now also OK1.10; no longer IL4.A
- net A5: now also OK2.16; no longer IL5.A
- net A6: now also OK2.14; no longer IL6.A
- net A7: now also OK2.12; no longer IL7.A
- net GND: now also IL1.C, IL2.C, IL3.C, IL4.C, IL5.C, IL6.C, IL7.C, IL8.C; no longer IR.2
- net N$12: now also IL1.A, OK1.15; no longer IL1.C, XI.4
- net N$18: now also ITR1.1, XI.2; no longer WIL2.C, XI.3
- net N$20: now also IL2.A, OK1.13; no longer IL2.C, XI.5
- net N$21: now also IL3.A, OK1.11; no longer IL3.C, XI.6
- net N$23: now also IL4.A, OK1.9; no longer IL4.C, XI.7
- net N$25: now also IL5.A, OK2.15; no longer IL5.C, XI.8
- net N$26: now also IL6.A, OK2.13; no longer IL6.C, XI.9
- net N$27: now also IL7.A, OK2.11; no longer IL7.C, XI.10
- net N$28: now also ITR2.1, XI.3; no longer WIL0.C, XI.2
- net N$29: now also ITR1.2, OK1.1; no longer IR.1, XI.1
- net WFGPIO0: now also IR8.2, OK2.10; no longer WIL0.A, WIR0.2
- net WFGPIO2: no longer WIL2.A, WIR2.2
Routing:
- net GND: track 503.8 -> 0.00 mm, vias 3 -> 0
- net +3V3: track 306.9 -> 0.00 mm, vias 4 -> 0
- net RAW_IV: track 181.2 -> 0.00 mm, vias 1 -> 0
- net VIN: track 131.4 -> 0.00 mm
- net A7: track 116.2 -> 0.00 mm, vias 2 -> 0
- net D13: track 115.3 -> 0.00 mm, vias 1 -> 0
- net RESET: track 104.2 -> 0.00 mm, vias 2 -> 0
- net A6: track 91.1 -> 0.00 mm, vias 4 -> 0
- net A5: track 86.3 -> 0.00 mm, vias 3 -> 0
- net BLV: track 86.1 -> 0.00 mm, vias 2 -> 0
- net A4: track 78.5 -> 0.00 mm, vias 3 -> 0
- net A3: track 77.8 -> 0.00 mm, vias 2 -> 0
- net A1: track 73.6 -> 0.00 mm, vias 2 -> 0
- net A2: track 73.3 -> 0.00 mm
- net D11: track 68.1 -> 0.00 mm, vias 3 -> 0
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Other:
- board text added: "IOTB v2.0 TOP"
- board text removed: "IOTB v1.3 TOP"

Commit message: v2
Parts:
- removed X2, X4: MC5, con-phoenix-381_l:MC5
- removed X3: MC2, con-phoenix-381_l:MC2
- added XI1: MC10, con-phoenix-381_l:MC10
- moved X1 14.5 mm to (5.00, 48.2)
- moved OK1 1.75 mm to (17.8, 35.2)
- moved XI 0.25 mm to (5.00, 22.2)
