File: KMO_IO_M/KMO_IO_MV2_0.sch (EAGLE design)
At the start: 83 parts, among them Q1 8MHz, Q2 25MHz, U1 ATMEGA328, X1 MC3

Commit message: v2
Parts:
- removed IR: 10K, SparkFun-Passives:RESISTOR0805-RES
- removed WIL0, WIL2: BLU, led:LEDCHIP-LED0805
- removed WIR0, WIR2: 1K, SparkFun-Passives:RESISTOR0805-RES
- added IL8: BLU, led:LEDCHIP-LED0805
- added IR8: 1K, SparkFun-Passives:RESISTOR0805-RES
- added ITR1, ITR2, ITR3, ITR4, ITR5, ITR6, ITR7, ITR8: 6.8K, SparkFun-Passives:RESISTOR0805-RES
- added OK1, OK2: TLP283-4, optocoupler:TLP283-4
- added X2, X4: MC5, con-phoenix-381_l:MC5
- added X3: MC2, con-phoenix-381_l:MC2
Connections:
- new net COM1: OK1A.C, OK1B.C, OK1C.C, OK1D.C, XI.1.SK
- new net N$30: ITR2.2, OK1B.A
- new net N$31: ITR3.2, OK1C.A
- new net N$32: ITR4.2, OK1D.A
- new net N$33: ITR3.1, XI.4.SK
- new net N$34: ITR4.1, XI.5.SK
- new net N$35: OK2A.C, OK2B.C, OK2C.C, OK2D.C, XI.6.SK
- new net N$36: ITR5.1, XI.7.SK
- new net N$37: ITR5.2, OK2A.A
- new net N$38: ITR6.1, XI.8.SK
- new net N$39: ITR6.2, OK2B.A
- new net N$40: ITR7.1, XI.9.SK
- new net N$41: ITR7.2, OK2C.A
- new net N$42: ITR8.1, XI.10.SK
- new net N$43: ITR8.2, OK2D.A
- new net N$44: IL8.A, OK2D.EMIT
- net +3V3: now also IR8.1; no longer WIR0.1, WIR2.1
- net A1: now also OK1A.COL; no longer IL1.A
- net A2: now also OK1B.COL; no longer IL2.A
- net A3: now also OK1C.COL; no longer IL3.A
- net A4: now also OK1D.COL; no longer IL4.A
- net A5: now also OK2A.COL; no longer IL5.A
- net A6: now also OK2B.COL; no longer IL6.A
- net A7: now also OK2C.COL; no longer IL7.A
- net GND: now also IL1.C, IL2.C, IL3.C, IL4.C, IL5.C, IL6.C, IL7.C, IL8.C; no longer IR.2
- net N$12: now also IL1.A, OK1A.EMIT; no longer IL1.C, XI.4.SK
- net N$18: now also ITR1.1, XI.2.SK; no longer WIL2.C, XI.3.SK
- net N$20: now also IL2.A, OK1B.EMIT; no longer IL2.C, XI.5.SK
- net N$21: now also IL3.A, OK1C.EMIT; no longer IL3.C, XI.6.SK
- net N$23: now also IL4.A, OK1D.EMIT; no longer IL4.C, XI.7.SK
- net N$25: now also IL5.A, OK2A.EMIT; no longer IL5.C, XI.8.SK
- net N$26: now also IL6.A, OK2B.EMIT; no longer IL6.C, XI.9.SK
- net N$27: now also IL7.A, OK2C.EMIT; no longer IL7.C, XI.10.SK
- net N$28: now also ITR2.1, XI.3.SK; no longer WIL0.C, XI.2.SK
- net N$29: now also ITR1.2, OK1A.A; no longer IR.1, XI.1.SK
- net WFGPIO0: now also IR8.2, OK2D.COL; no longer WIL0.A, WIR0.2
- net WFGPIO2: no longer WIL2.A, WIR2.2
Other:
- note added: "2.0"
- note removed: "1.3"
- note removed: "WIN2"

Commit message: v2
Parts:
- removed X2, X4: MC5, con-phoenix-381_l:MC5
- removed X3: MC2, con-phoenix-381_l:MC2
- added XI1: MC10, con-phoenix-381_l:MC10
Changed lines of the file:
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@@
 <?xml version="1.0" encoding="utf-8"?>
 <!DOCTYPE eagle SYSTEM "eagle.dtd">
-<eagle version="9.3.2">
+<eagle version="9.4.0">
 <drawing>
 <settings>
@@
 <part name="IL8" library="led" library_urn="urn:adsk.eagle:library:259" deviceset="LED" device="CHIP-LED0805" package3d_urn="urn:adsk.eagle:package:15818/2" value="BLU"/>
 <part name="GND19" library="supply1" deviceset="GND" device=""/>
-<part name="X2" library="con-phoenix-381_l" deviceset="MC5" device=""/>
-<part name="X3" library="con-phoenix-381_l" deviceset="MC2" device=""/>
-<part name="X4" library="con-phoenix-381_l" deviceset="MC5" device=""/>
+<part name="XI1" library="con-phoenix-381_l" deviceset="MC10" device=""/>
 </parts>
 <sheets>
@@
 <attribute name="NAME" x="111.76" y="131.445" size="1.524" layer="95"/>
 </instance>
-<instance part="X2" gate=".1" x="218.44" y="71.12" smashed="yes">
-<attribute name="NAME" x="210.82" y="73.025" size="1.524" layer="95"/>
-</instance>
-<instance part="X2" gate=".2" x="218.44" y="66.04" smashed="yes">
-<attribute name="NAME" x="210.82" y="67.945" size="1.524" layer="95"/>
-</instance>
-<instance part="X2" gate=".3" x="218.44" y="60.96" smashed="yes">
-<attribute name="NAME" x="210.82" y="62.865" size="1.524" layer="95"/>
-</instance>
-<instance part="X2" gate=".4" x="218.44" y="55.88" smashed="yes">
-<attribute name="NAME" x="210.82" y="57.785" size="1.524" layer="95"/>
-</instance>
-<instance part="X2" gate=".5" x="218.44" y="50.8" smashed="yes">
-<attribute name="NAME" x="210.82" y="52.705" size="1.524" layer="95"/>
-</instance>
-<instance part="X3" gate=".1" x="218.44" y="33.02" smashed="yes">
-<attribute name="NAME" x="210.82" y="34.925" size="1.524" layer="95"/>
-</instance>
-<instance part="X3" gate=".2" x="218.44" y="27.94" smashed="yes">
-<attribute name="NAME" x="210.82" y="29.845" size="1.524" layer="95"/>
-</instance>
-<instance part="X4" gate=".1" x="248.92" y="76.2" smashed="yes">
-<attribute name="NAME" x="241.3" y="78.105" size="1.524" layer="95"/>
-</instance>
-<instance part="X4" gate=".2" x="248.92" y="71.12" smashed="yes">
-<attribute name="NAME" x="241.3" y="73.025" size="1.524" layer="95"/>
-</instance>
-<instance part="X4" gate=".3" x="248.92" y="66.04" smashed="yes">
-<attribute name="NAME" x="241.3" y="67.945" size="1.524" layer="95"/>
-</instance>
-<instance part="X4" gate=".4" x="248.92" y="60.96" smashed="yes">
-<attribute name="NAME" x="241.3" y="62.865" size="1.524" layer="95"/>
-</instance>
-<instance part="X4" gate=".5" x="248.92" y="55.88" smashed="yes">
-<attribute name="NAME" x="241.3" y="57.785" size="1.524" layer="95"/>
+<instance part="XI1" gate=".1" x="248.92" y="78.74" smashed="yes">
+<attribute name="NAME" x="241.3" y="80.645" size="1.524" layer="95"/>
+</instance>
+<instance part="XI1" gate=".2" x="248.92" y="73.66" smashed="yes">
+<attribute name="NAME" x="241.3" y="75.565" size="1.524" layer="95"/>
+</instance>
+<instance part="XI1" gate=".3" x="248.92" y="68.58" smashed="yes">
+<attribute name="NAME" x="241.3" y="70.485" size="1.524" layer="95"/>
+</instance>
+<instance part="XI1" gate=".4" x="248.92" y="63.5" smashed="yes">
+<attribute name="NAME" x="241.3" y="65.405" size="1.524" layer="95"/>
+</instance>
+<instance part="XI1" gate=".5" x="248.92" y="58.42" smashed="yes">
+<attribute name="NAME" x="241.3" y="60.325" size="1.524" layer="95"/>
+</instance>
+<instance part="XI1" gate=".6" x="248.92" y="53.34" smashed="yes">
+<attribute name="NAME" x="241.3" y="55.245" size="1.524" layer="95"/>
+</instance>
+<instance part="XI1" gate=".7" x="248.92" y="48.26" smashed="yes">
+<attribute name="NAME" x="241.3" y="50.165" size="1.524" layer="95"/>
+</instance>
+<instance part="XI1" gate=".8" x="248.92" y="43.18" smashed="yes">
+<attribute name="NAME" x="241.3" y="45.085" size="1.524" layer="95"/>
+</instance>
+<instance part="XI1" gate=".9" x="248.92" y="38.1" smashed="yes">
+<attribute name="NAME" x="241.3" y="40.005" size="1.524" layer="95"/>
+</instance>
+<instance part="XI1" gate=".10" x="248.92" y="33.02" smashed="yes">
+<attribute name="NAME" x="241.3" y="34.925" size="1.524" layer="95"/>
 </instance>
 </instances>
