File: KMO_IO_M/KMO_IO_MV2_1.sch (EAGLE design)
At the start: 91 parts, among them IC1 MCP23017SS, Q1 8MHz, Q2 25MHz, U1 ATMEGA328

Commit message: 2.1
Parts:
- added XNO: MC2, con-phoenix-381_l:MC2
Connections:
- net A4: no longer IR4.2, OK1D.COL
- net A5: no longer IR5.2, OK2A.COL
Other:
- note added: "2.1"
- note removed: "2.0"
Changed lines of the file:
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@@
 <part name="GND19" library="supply1" deviceset="GND" device=""/>
 <part name="IC1" library="microchip" library_urn="urn:adsk.eagle:library:294" deviceset="MCP23017" device="SS" package3d_urn="urn:adsk.eagle:package:20800/2"/>
+<part name="XNO" library="con-phoenix-381_l" deviceset="MC2" device=""/>
 </parts>
 <sheets>
@@
 <text x="299.72" y="238.76" size="1.778" layer="91">NATIVE ANALOG-DIGITAL SENSOR 3</text>
 <text x="309.88" y="15.24" size="2.54" layer="94">IOTB by Team IOTECH</text>
-<text x="365.76" y="12.7" size="2.54" layer="94">2.0</text>
+<text x="365.76" y="12.7" size="2.54" layer="94">2.1</text>
 <text x="170.18" y="170.18" size="1.778" layer="91">ETHERNET</text>
 <text x="175.26" y="109.22" size="1.778" layer="97">D2  -&gt;INT
@@
 <instance part="XV" gate=".3" x="215.9" y="58.42" smashed="yes">
 <attribute name="NAME" x="208.28" y="60.325" size="1.524" layer="95"/>
+</instance>
+<instance part="XNO" gate=".1" x="261.62" y="68.58" smashed="yes">
+<attribute name="NAME" x="254" y="70.485" size="1.524" layer="95"/>
+</instance>
+<instance part="XNO" gate=".2" x="261.62" y="63.5" smashed="yes">
+<attribute name="NAME" x="254" y="65.405" size="1.524" layer="95"/>
 </instance>
 </instances>
@@
 <net name="A5" class="0">
 <segment>
-<label x="218.44" y="233.68" size="1.778" layer="95" xref="yes"/>
-<pinref part="IR5" gate="G$1" pin="2"/>
-<wire x1="198.12" y1="233.68" x2="200.66" y2="233.68" width="0.1524" layer="91"/>
-<wire x1="200.66" y1="233.68" x2="218.44" y2="233.68" width="0.1524" layer="91"/>
-<wire x1="200.66" y1="233.68" x2="200.66" y2="220.98" width="0.1524" layer="91"/>
-<pinref part="OK2" gate="A" pin="COL"/>
-<wire x1="200.66" y1="220.98" x2="195.58" y2="220.98" width="0.1524" layer="91"/>
-<junction x="200.66" y="233.68"/>
+<label x="335.28" y="210.82" size="1.778" layer="95" xref="yes"/>
+<wire x1="317.5" y1="210.82" x2="335.28" y2="210.82" width="0.1524" layer="91"/>
 </segment>
 </net>
 <net name="A4" class="0">
 <segment>
-<label x="96.52" y="142.24" size="1.778" layer="95" xref="yes"/>
-<pinref part="IR4" gate="G$1" pin="2"/>
-<wire x1="76.2" y1="142.24" x2="78.74" y2="142.24" width="0.1524" layer="91"/>
-<wire x1="78.74" y1="142.24" x2="96.52" y2="142.24" width="0.1524" layer="91"/>
-<wire x1="78.74" y1="142.24" x2="78.74" y2="129.54" width="0.1524" layer="91"/>
-<pinref part="OK1" gate="D" pin="COL"/>
-<wire x1="78.74" y1="129.54" x2="73.66" y2="129.54" width="0.1524" layer="91"/>
-<junction x="78.74" y="142.24"/>
-</segment>
-</net>
+<label x="335.28" y="218.44" size="1.778" layer="95" xref="yes"/>
+<wire x1="317.5" y1="218.44" x2="335.28" y2="218.44" width="0.1524" layer="91"/>
+</segment>
+</net>

Commit message: 21
Parts:
- removed OD2, OD3: M7, SparkFun-DiscreteSemi:DIODESMA
- removed OL2, OL3: YLW, led:LEDCHIP-LED0805
- removed OQ2, OQ3: IRF3707S, transistor-power:IRF3704S
- removed OR2, OR3: 1K, SparkFun-Passives:RESISTOR0805-RES
- added OK3: TLP283-4, optocoupler:TLP283-4
- PC1: value 470uf 25v -> 220uf 50v
Connections:
- removed net N$3: OD1.A, OQ1.D
- removed net N$4: OD2.A, OQ2.D
- removed net N$6 (its old number): OL3.A, OR3.1
- removed net N$7: OL2.A, OR2.1
- net D5: now also OQ1.G, OR1.2; no longer OQ3.G, OR3.2
- net D6: no longer OQ2.G, OR2.2
- net D7: no longer OQ1.G, OR1.2
- net GND: no longer OL2.C, OL3.C, OQ2.S, OQ3.S
- net N$1: now also OD1.A, OQ1.D, XNO.2.SK; no longer OD3.A, OQ3.D
- net RAW_IV: now also XNO.1.SK; no longer OD2.C, OD3.C
Other:
- note removed: "OUT2"
- note removed: "OUT3"
- moved on the sheet: OD1, OL1, OQ1, OR1, XNO.1, XNO.2, XO.3, XO.4, XO.5, XO.6, XV.1, XV.2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

Commit message: v2
Parts:
- removed ER6, ER7, ER8, ER9: 50R, SparkFun-Passives:RESISTOR0805-RES
- removed IR3, IR4, IR5, IR6, IR7, IR8, OR1: 1K, SparkFun-Passives:RESISTOR0805-RES
- removed ITR1, ITR2, ITR3, ITR4, ITR5, ITR6, ITR7, ITR8: 6.8K, SparkFun-Passives:RESISTOR0805-RES
- removed OQ1: IRF3707S, transistor-power:IRF3704S
- removed XI: MC10, con-phoenix-381_l:MC10
- added ERN1: 49.9R, resistor-dil:4R-N0603-ARV
- added IIR1, IIR2: 6.8K, resistor-dil:4R-N0603-ARV
- added MR1, MR2: 1.5K, SparkFun-Passives:RESISTOR0805-RES
- added MR3: 10K, SparkFun-Passives:RESISTOR0805-RES
- added OD2: (no value), diode:ZENER-DIODESMB
- added OF1: 750mA, _hhn_PtcFuses_Siba_r500_Ozan:SIBA194600
- added OL2, OL3, OL4: BLU, led:LEDCHIP-LED0805
- added ORN1: 1K, resistor-dil:4R-N0603-ARV
- added ORN2, ORN3: 10K, resistor-dil:4R-N0603-ARV
- added XI1, XI2: MC5, con-phoenix-381_l:MC5
- IR1, IR2: device SparkFun-Passives:RESISTOR0805-RES -> resistor-dil:4R-N0603-ARV
- OD1: value M7 -> SS54; device SparkFun-DiscreteSemi:DIODESMA -> diode:SCHOTTKY-DIODESMD
- OL1: value YLW -> BLU
Connections:
- removed net N$6: OL1.A, OR1.1
- new net COM2: OK2A.C, OK2B.C, OK2C.C, OK2D.C, XI2.1.SK
- new net GNDO: OD2.A, ORN2A.2, ORN2B.2, ORN2C.2, ORN2D.2, XO.2.SK
- new net GPA0: IC1.GPA0, IR1A.2, OK1A.COL
- new net GPA1: IC1.GPA1, IR1B.2, OK1B.COL
- new net GPA2: IC1.GPA2, IR1C.2, OK1C.COL
- new net GPA3: IC1.GPA3, IR1D.2, OK1D.COL
- new net GPA4: IC1.GPA4, IR2A.2, OK2A.COL
- new net GPA5: IC1.GPA5, IR2B.2, OK2B.COL
- new net GPA6: IC1.GPA6, IR2C.2, OK2C.COL
- new net GPA7: IC1.GPA7, IR2D.2, OK2D.COL
- new net GPB0: IC1.GPB0, ORN1A.2
- new net GPB1: IC1.GPB1, ORN1B.2
- new net GPB2: IC1.GPB2, ORN1C.2
- new net GPB3: IC1.GPB3, ORN1D.2
- new net GPB4: IC1.GPB4
- new net GPB5: IC1.GPB5
- new net GPB6: IC1.GPB6
- new net GPB7: IC1.GPB7
- new net N$3: IC1.A0, MR3.1
- new net N$4: OD1.C, OF1.2
- new net N$45: OK3C.A, ORN1C.1
- new net N$46: OK3D.A, ORN1D.1
- new net N$47: OK3A.EMIT, ORN2A.1, XO.3.SK
- new net N$48: OK3A.COL, ORN3A.1
- new net N$53: OK3B.COL, ORN3B.1
- new net N$54: OK3B.EMIT, ORN2B.1, XO.4.SK
- new net N$56: OK3C.COL, ORN3C.1
- new net N$57: OK3C.EMIT, ORN2C.1, XO.5.SK
- new net N$58: OK3D.COL, ORN3D.1
- new net N$59: OK3D.EMIT, ORN2D.1, XO.6.SK
- new net N$60: OK3A.C, OL1.A
- new net N$61: OK3B.C, OL2.A
- new net N$62: OK3C.C, OL3.A
- new net N$63: OK3D.C, OL4.A
- new net N$8: OK3A.A, ORN1A.1
- new net VDDO: OD2.C, OF1.1, ORN3A.2, ORN3B.2, ORN3C.2, ORN3D.2
- net +3V3: now also IC1.!RESET, IC1.VDD, IR1A.1, IR1B.1, IR1C.1, IR1D.1, IR2A.1, IR2B.1, IR2C.1, IR2D.1, MR1.2, MR2.2, MR3.2; no longer IR1.1, IR2.1, IR3.1, IR4.1, IR5.1, IR6.1, IR7.1, IR8.1
- net A1: no longer IR1.2, OK1A.COL
- net A2: no longer IR2.2, OK1B.COL
- net A3: no longer IR3.2, OK1C.COL
- net A4: now also IC1.SDA, MR1.1
- net A5: now also IC1.SCL, MR2.1
- net A6: no longer IR6.2, OK2B.COL
- net A7: no longer IR7.2, OK2C.COL
- net COM1: now also XI1.1.SK; no longer XI.1.SK
- net D5: no longer OQ1.G, OR1.2
- net EP4: now also ERN1A.2, ERN1B.2; no longer ER6.2, ER7.2
- net EP5: now also ERN1C.1, ERN1D.1; no longer ER8.1, ER9.1
- net GND: now also IC1.A1, IC1.A2, IC1.VSS, OL2.C, OL3.C, OL4.C; no longer OQ1.S
- net N$1: now also XO.1.SK; no longer OQ1.D, XNO.2.SK
- net N$18: now also IIR1A.1, XI1.2.SK; no longer ITR1.1, XI.2.SK
- net N$28: now also IIR1B.1, XI1.3.SK; no longer ITR2.1, XI.3.SK
- net N$29: now also IIR1A.2; no longer ITR1.2
- net N$30: now also IIR1B.2; no longer ITR2.2
- net N$31: now also IIR1C.2; no longer ITR3.2
- net N$32: now also IIR1D.2; no longer ITR4.2
- net N$33: now also IIR1C.1, XI1.4.SK; no longer ITR3.1, XI.4.SK
- net N$34: now also IIR1D.1, XI1.5.SK; no longer ITR4.1, XI.5.SK
- net N$35: now also OK3B.A, ORN1B.1; no longer OK2A.C, OK2B.C, OK2C.C, OK2D.C, XI.6.SK
- net N$36: now also IIR2A.1, XI2.2.SK; no longer ITR5.1, XI.7.SK
- net N$37: now also IIR2A.2; no longer ITR5.2
- net N$38: now also IIR2B.1, XI2.3.SK; no longer ITR6.1, XI.8.SK
- net N$39: now also IIR2B.2; no longer ITR6.2
- net N$40: now also IIR2C.1, XI2.4.SK; no longer ITR7.1, XI.9.SK
- net N$41: now also IIR2C.2; no longer ITR7.2
- net N$42: now also IIR2D.1, XI2.5.SK; no longer ITR8.1, XI.10.SK
- net N$43: now also IIR2D.2; no longer ITR8.2
- net RAW_IV: no longer OD1.C, XNO.1.SK
- net RD+: now also ERN1C.2; no longer ER8.2
- net RD-: now also ERN1D.2; no longer ER9.2
- net TD+: now also ERN1A.1; no longer ER6.1
- net TD-: now also ERN1B.1; no longer ER7.1
- net WFGPIO0: no longer IR8.2, OK2D.COL

Commit message: v2
Parts:
- removed XNO: MC2, con-phoenix-381_l:MC2
- added EC6: 10u, rcl:CPOL-EUCT3216
- added GPIO: 057-014-1, con-panduit:057-014-1
- added OF2, OF3, OF4, OF5, OF6, OF7, OF8, OF9: 100mA, _hhn_PtcFuses_Siba_r500_Ozan:SIBA194600
- added OK4: TLP283-4, optocoupler:TLP283-4
- added OL5, OL6, OL7, OL8: BLU, led:LEDCHIP-LED0805
- added ORN4: 1K, resistor-dil:4R-N0603-ARV
- added ORN5, ORN6: 10K, resistor-dil:4R-N0603-ARV
- added U2: ULN2803ADW, ULN2803ADW:ULN2803ADW
- XO: value MC6 -> MC10; device con-phoenix-381_l:MC6 -> con-phoenix-381_l:MC10
- XV: value MC3 -> MC2; device con-phoenix-381_l:MC3 -> con-phoenix-381_l:MC2
Connections:
- new net IO5: OK4A.EMIT, ORN6A.2, U2.4B
- new net IO6: OK4B.EMIT, ORN6B.1, U2.3B
- new net IO7: OK4C.EMIT, ORN6C.1, U2.2B
- new net IO8: OK4D.EMIT, ORN6D.1, U2.1B
- new net N$49: OF4.2, U2.3C
- new net N$50: OF5.2, U2.4C
- new net N$51: OF3.1, XO.9.SK
- new net N$52: OF4.1, XO.8.SK
- new net N$55: OF6.1, XO.6.SK
- new net N$6: OF2.1, XO.10.SK
- new net N$64: OF9.2, U2.8C
- new net N$65: OF6.2, U2.5C
- new net N$66: OF7.1, XO.5.SK
- new net N$67: OF8.1, XO.4.SK
- new net N$68: OF9.1, XO.3.SK
- new net N$69: OK4A.A, ORN4D.1
- new net N$7: OF3.2, U2.2C
- new net N$70: OK4B.A, ORN4C.1
- new net N$71: OK4C.A, ORN4B.1
- new net N$72: OK4D.A, ORN4A.1
- new net N$73: OK4A.COL, ORN5A.1
- new net N$74: OK4B.COL, ORN5B.1
- new net N$75: OK4C.COL, ORN5C.1
- new net N$76: OK4D.COL, ORN5D.1
- new net N$77: OK4A.C, OL5.A
- new net N$78: OK4B.C, OL6.A
- new net N$79: OK4C.C, OL7.A
- new net N$80: OK4D.C, OL8.A
- new net OI1: OK3A.EMIT, ORN2A.1, U2.8B
- new net OI2: OK3B.EMIT, ORN2B.1, U2.7B
- new net OI3: OK3C.EMIT, ORN2C.1, U2.6B
- new net OI4: OK3D.EMIT, ORN2D.1, U2.5B
- net +3V3: now also GPIO-2.S
- net A1: now also GPIO-8.S
- net A2: now also GPIO-9.S
- net A3: now also GPIO-10.S
- net A6: now also GPIO-11.S
- net A7: now also GPIO-12.S
- net D5: now also GPIO-5.S
- net D6: now also GPIO-6.S
- net D7: now also GPIO-7.S
- net GND: now also GPIO-3.S, GPIO-4.S, OL5.C, OL6.C, OL7.C, OL8.C, XV.1.SK; no longer XV.2.SK
- net GNDO: now also EC6.-, ORN6A.1, ORN6B.2, ORN6C.2, ORN6D.2, U2.GND
- net GPB0: now also ORN4A.2; no longer ORN1A.2
- net GPB1: now also ORN4B.2; no longer ORN1B.2
- net GPB2: now also ORN4C.2; no longer ORN1C.2
- net GPB3: now also ORN4D.2; no longer ORN1D.2
- net GPB4: now also ORN1A.2
- net GPB5: now also ORN1B.2
- net GPB6: now also ORN1C.2
- net GPB7: now also ORN1D.2
- net N$35: now also ORN1C.1; no longer ORN1B.1
- net N$45: now also ORN1B.1; no longer ORN1C.1
- net N$46: now also ORN1A.1; no longer ORN1D.1
- net N$47: now also OF2.2, U2.1C; no longer OK3A.EMIT, ORN2A.1, XO.3.SK
- net N$54: now also OF5.1, XO.7.SK; no longer OK3B.EMIT, ORN2B.1, XO.4.SK
- net N$57: now also OF7.2, U2.6C; no longer OK3C.EMIT, ORN2C.1, XO.5.SK
- net N$59: now also OF8.2, U2.7C; no longer OK3D.EMIT, ORN2D.1, XO.6.SK
- net N$8: now also ORN1D.1; no longer ORN1A.1
- net RAW_IV: now also GPIO-1.S; no longer XV.1.SK
- net VDDO: now also EC6.+, ORN5A.2, ORN5B.2, ORN5C.2, ORN5D.2, U2.COM
- net VIN: now also XV.2.SK; no longer XV.3.SK
- net WFGPIO0: now also GPIO-13.S
- net WFGPIO2: now also GPIO-14.S
Other:
- note added: "GPIO"
- moved on the sheet: IC1, IIR1A, IIR1B, IIR1C, IIR1D, IIR2A, IIR2B, IIR2C, IIR2D, IL1, IL2, IL3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

Commit message: v2
Parts:
- OF2, OF3, OF4, OF5, OF6, OF7, OF8, OF9: value 100mA -> 6V/0.75A; device _hhn_PtcFuses_Siba_r500_Ozan:SIBA194600 -> SparkFun-Fuses:PPTC_0.75A
Other:
- note added: "IO EXTENDER"
- note added: "OUT"
- note removed: "OUT1"
- moved on the sheet: EC6, OD1, OD2, OF1, OK3A, OK3B, OK3C, OK3D, OK4A, OK4B, OK4C, OK4D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

Commit message: v2
Parts:
- removed U2: ULN2803ADW, ULN2803ADW:ULN2803ADW
- added D1, D2, D3, D4: BAV70, BAV70:BAV70
- added MC: ATMEGA328, SparkFun:ATMEGA168
- U1: value ATMEGA328 -> ULN2803ADW; device SparkFun:ATMEGA168 -> ULN2803ADW:ULN2803ADW
Connections:
- net A0: now also MC.PC0(ADC0); no longer U1.PC0(ADC0)
- net A1: now also MC.PC1(ADC1); no longer U1.PC1(ADC1)
- net A2: now also MC.PC2(ADC2); no longer U1.PC2(ADC2)
- net A3: now also MC.PC3(ADC3); no longer U1.PC3(ADC3)
- net A4: now also MC.PC4(ADC4/SDA); no longer U1.PC4(ADC4/SDA)
- net A5: now also MC.PC5(ADC5/SCL); no longer U1.PC5(ADC5/SCL)
- net A6: now also MC.ADC6; no longer U1.ADC6
- net A7: now also MC.ADC7; no longer U1.ADC7
- net AREF: now also MC.AREF; no longer U1.AREF
- net BLV: now also MC.AVCC, MC.VCC@1, MC.VCC@2; no longer U1.AVCC, U1.VCC@1, U1.VCC@2
- net D10: now also MC.PB2(SS/OC1B); no longer U1.PB2(SS/OC1B)
- net D11: now also MC.PB3(MOSI/OC2); no longer U1.PB3(MOSI/OC2)
- net D12: now also MC.PB4(MISO); no longer U1.PB4(MISO)
- net D13: now also MC.PB5(SCK); no longer U1.PB5(SCK)
- net D2: now also MC.PD2(INT0); no longer U1.PD2(INT0)
- net D3: now also MC.PD3(INT1); no longer U1.PD3(INT1)
- net D4: now also MC.PD4(XCK/T0); no longer U1.PD4(XCK/T0)
- net D5: now also MC.PD5(T1); no longer U1.PD5(T1)
- net D6: now also MC.PD6(AIN0); no longer U1.PD6(AIN0)
- net D7: now also MC.PD7(AIN1); no longer U1.PD7(AIN1)
- net D8: now also MC.PB0(ICP); no longer U1.PB0(ICP)
- net D9: now also MC.PB1(OC1A); no longer U1.PB1(OC1A)
- net GND: now also MC.AGND, MC.GND@1, MC.GND@2; no longer U1.AGND, U1.GND@1, U1.GND@2
- net GNDO: now also U1.GND; no longer U2.GND
- net IO5: now also U1.4B; no longer U2.4B
- net IO6: now also U1.3B; no longer U2.3B
- net IO7: now also U1.2B; no longer U2.2B
- net IO8: now also U1.1B; no longer U2.1B
- net N$10: now also MC.PB7(XTAL2/TOSC2); no longer U1.PB7(XTAL2/TOSC2)
- net N$15: now also MC.PB6(XTAL1/TOSC1); no longer U1.PB6(XTAL1/TOSC1)
- net N$47: now also D1.2, U1.1C; no longer U2.1C
- net N$49: now also D2.2, U1.3C; no longer U2.3C
- net N$50: now also D2.1, U1.4C; no longer U2.4C
- net N$57: now also D3.1, U1.6C; no longer U2.6C
- net N$59: now also D4.2, U1.7C; no longer U2.7C
- net N$64: now also D4.1, U1.8C; no longer U2.8C
- net N$65: now also D3.2, U1.5C; no longer U2.5C
- net N$7: now also D1.1, U1.2C; no longer U2.2C
- net OI1: now also U1.8B; no longer U2.8B
- net OI2: now also U1.7B; no longer U2.7B
- net OI3: now also U1.6B; no longer U2.6B
- net OI4: now also U1.5B; no longer U2.5B
- net RESET: now also MC.PC6(/RESET); no longer U1.PC6(/RESET)
- net RXI: now also MC.PD0(RXD); no longer U1.PD0(RXD)
- net TXO: now also MC.PD1(TXD); no longer U1.PD1(TXD)
- net VDDO: now also D1.3, D2.3, D3.3, D4.3, U1.COM; no longer U2.COM
Other:
- moved on the sheet: EC6

Commit message: 3d some
Parts:
- BLS: value (none) -> on-off
- OD2: value (none) -> 28V
- OK1, OK2: SPICEPREFIX (none) -> O
- SR: value (none) -> gnd
- SV1, SV2, SV3: value (none) -> 3.3V
Connections:
- removed net BLG: BL-6.S
- net GND: now also BL-6.S
- net N$47: now also OF3.2; no longer OF2.2
- net N$51: now also OF2.1; no longer OF3.1
- net N$6: now also OF3.1; no longer OF2.1
- net N$7: now also OF2.2; no longer OF3.2
Other:
- moved on the sheet: OF2, OF3
