File: KMO_IO_M/KMO_IO_MV2_2.sch (EAGLE design)
At the start: 102 parts, among them IC1 MCP23017SS, Q1 8MHz, Q2 25MHz, U1 ULN2803ADW

Commit message: v2.2
Parts:
- removed MR1, MR2: 1.5K, SparkFun-Passives:RESISTOR0805-RES
- OF1: device _hhn_PtcFuses_Siba_r500_Ozan:SIBA194600 -> SparkFun-Fuses:PPTC_0.75A
- OF2, OF3, OF4, OF5, OF6, OF7, OF8, OF9: value 6V/0.75A -> 100mA
- R1, R3: value (none) -> 1.5K
Connections:
- net +3V3: no longer MR1.2, MR2.2
- net A4: now also GPIO-4.S; no longer MR1.1
- net A5: now also GPIO-5.S; no longer MR2.1
- net D5: now also IC1.INTB; no longer GPIO-5.S
- net GND: no longer GPIO-4.S
Other:
- note added: "500ma çıkış"
- moved on the sheet: IC1, MR3, R3, XO.10, XO.4, XO.5, XO.6, XO.7, XO.8, XO.9
