File: KMO_IO_M/KMO_IO_MV2_3.brd (EAGLE design)
At the start: 84.5 x 96.5 mm, 104 parts, among them IC1 MCP23017SS, Q1 8MHz, Q2 25MHz, U1 ULN2803ADW

Commit message: 2.3
Parts:
- renumbered ORN1 to OR1, ORN2 to OR2, ORN3 to OR3, ORN4 to OR4, ORN5 to OR5, ORN6 to OR6

Commit message: 2.3Cam
Parts:
- moved IIR1 0.75 mm to (10.2, 26.5)
- moved IR2 0.75 mm to (10.2, 14.8), turned to 90 degrees
- turned IR1 to 90 degrees
Connections:
- net +3V3: now also OK1.10, OK1.12, OK1.14, OK2.10, OK2.12, OK2.14, OK2.16; no longer IR1.2, IR1.3, IR1.4, IR2.1, IR2.2, IR2.3, IR2.4
- net GND: now also IR1.5, IR1.6, IR1.7, IR2.5, IR2.6, IR2.7, IR2.8; no longer OK1.11, OK1.13, OK1.9, OK2.11, OK2.13, OK2.15, OK2.9
- net GPA0: now also IR1.4; no longer IR1.1
- net GPA1: now also IR1.3, OK1.13; no longer IR1.7, OK1.14
- net GPA2: now also IR1.2, OK1.11; no longer IR1.6, OK1.12
- net GPA3: now also IR1.1, OK1.9; no longer IR1.5, OK1.10
- net GPA4: now also IR2.4, OK2.15; no longer IR2.8, OK2.16
- net GPA5: now also IR2.3, OK2.13; no longer IR2.7, OK2.14
- net GPA6: now also IR2.2, OK2.11; no longer IR2.6, OK2.12
- net GPA7: now also IR2.1, OK2.9; no longer IR2.5, OK2.10
Routing:
- net GND: track 0.00 -> 626.7 mm, vias 0 -> 11
- net +3V3: track 0.00 -> 336.2 mm, vias 0 -> 5
- net D13: track 0.00 -> 124.8 mm, vias 0 -> 1
- net A4: track 0.00 -> 122.4 mm, vias 0 -> 2
- net VIN: track 0.00 -> 113.9 mm
- net RESET: track 0.00 -> 106.5 mm, vias 0 -> 2
- net D5: track 0.00 -> 105.1 mm, vias 0 -> 4
- net D6: track 0.00 -> 98.4 mm, vias 0 -> 1
- net VDDO: track 0.00 -> 95.6 mm, vias 0 -> 5
- net GNDO: track 0.00 -> 88.1 mm, vias 0 -> 3
- net D11: track 0.00 -> 79.8 mm, vias 0 -> 4
- net A5: track 0.00 -> 76.5 mm, vias 0 -> 3
- net D10: track 0.00 -> 76.3 mm, vias 0 -> 4
- net D12: track 0.00 -> 71.7 mm, vias 0 -> 4
- net GPA5: track 0.00 -> 68.3 mm, vias 0 -> 3
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- added copper zone on layer 1, net GND
- added copper zone on layer 16, net GND
