File: KMO_IO_M/KMO_IO_MV2_3.sch (EAGLE design)
At the start: 102 parts, among them IC1 MCP23017SS, Q1 8MHz, Q2 25MHz, U1 ULN2803ADW

Commit message: 2.3
Parts:
- renumbered ORN1 to OR1, ORN2 to OR2, ORN3 to OR3, ORN4 to OR4, ORN5 to OR5, ORN6 to OR6
Other:
- moved on the sheet: IIR2A, IIR2B, IIR2C, IIR2D, IL5, IL6, IL7, IL8, IR2A, IR2B, IR2C, IR2D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

Commit message: 2.3Cam
Connections:
- net +3V3: now also OK1B.COL, OK1C.COL, OK1D.COL, OK2A.COL, OK2B.COL, OK2C.COL, OK2D.COL; no longer IR1B.1, IR1C.1, IR1D.1, IR2A.1, IR2B.1, IR2C.1, IR2D.1
- net GND: now also IR1B.2, IR1C.2, IR1D.2, IR2A.2, IR2B.2, IR2C.2, IR2D.2; no longer OK1B.EMIT, OK1C.EMIT, OK1D.EMIT, OK2A.EMIT, OK2B.EMIT, OK2C.EMIT, OK2D.EMIT
- net GPA0: now also IR1D.1; no longer IR1A.1
- net GPA1: now also IR1C.1, OK1B.EMIT; no longer IR1B.2, OK1B.COL
- net GPA2: now also IR1B.1, OK1C.EMIT; no longer IR1C.2, OK1C.COL
- net GPA3: now also IR1A.1, OK1D.EMIT; no longer IR1D.2, OK1D.COL
- net GPA4: now also IR2D.1, OK2A.EMIT; no longer IR2A.2, OK2A.COL
- net GPA5: now also IR2C.1, OK2B.EMIT; no longer IR2B.2, OK2B.COL
- net GPA6: now also IR2B.1, OK2C.EMIT; no longer IR2C.2, OK2C.COL
- net GPA7: now also IR2A.1, OK2D.EMIT; no longer IR2D.2, OK2D.COL
Other:
- moved on the sheet: IL2, IL3, IL4, IL5, IL6, IL7, IL8, IR1A, IR1B, IR1C, IR1D, IR2A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
