File: KMO_IO_M/KMO_IO_MV2_4.brd (EAGLE design)
At the start: 84.5 x 96.5 mm, 104 parts, among them IC1 MCP23017SS, Q1 8MHz, Q2 25MHz, U1 ULN2803ADW

Commit message: end of end
Routing:
- net N$10: track 2.95 -> 4.09 mm
- net IO7: track 25.2 -> 25.9 mm
Changed lines of the file:
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@@
 <setting verticaltext="up"/>
 </settings>
-<grid distance="0.16" unitdist="mm" unit="mm" style="lines" multiple="1" display="yes" altdistance="5" altunitdist="mil" altunit="mm"/>
+<grid distance="0.127" unitdist="mm" unit="mm" style="lines" multiple="1" display="yes" altdistance="0.127" altunitdist="mm" altunit="mm"/>
 <layers>
 <layer number="1" name="Top" color="4" fill="1" visible="yes" active="yes"/>
@@
 </layers>
 <board>
-<fusionsync huburn="a.cGVyc29uYWw6dWUyYzc1ODdm" projecturn="a.cGVyc29uYWw6dWUyYzc1ODdmIzIwMTkwNDI1MTkwMzAwMTgx" f3durn="urn:adsk.wipprod:dm.lineage:NyGoLFpNTXyJCtd3-WzVqQ" pcbguid="dda2ae1a-66fa-46dd-96ea-e6794cc07e63" lastpulledtime="" lastsyncedchangeguid="26bf622e-7293-418d-f36e-aa942b9fc4ce"/>
+<fusionsync huburn="a.cGVyc29uYWw6dWUyYzc1ODdm" projecturn="a.cGVyc29uYWw6dWUyYzc1ODdmIzIwMTkwNDI1MTkwMzAwMTgx" f3durn="urn:adsk.wipprod:dm.lineage:NyGoLFpNTXyJCtd3-WzVqQ" pcbguid="dda2ae1a-66fa-46dd-96ea-e6794cc07e63" lastpulledtime="" lastsyncedchangeguid="6025e090-d2eb-548c-78ae-7d63f40098b2"/>
 <plain>
 <hole x="17.25" y="83.25" drill="3" locked="yes"/>
@@
 </element>
 <element name="EC1" library="SparkFun-Passives" package="0805" override_package3d_urn="urn:adsk.eagle:package:10708048/2" override_package_urn="urn:adsk.eagle:footprint:10708050/1" value="18p" x="58.25" y="37" smashed="yes">
-<attribute name="NAME" x="56.988" y="35.0755" size="1.016" layer="25"/>
+<attribute name="NAME" x="57.623" y="34.9485" size="1.016" layer="25"/>
 <attribute name="VALUE" x="57.734" y="36.853" size="0.4064" layer="27"/>
 </element>
@@
 </element>
 <element name="ER4" library="SparkFun-Passives" package="0805" override_package3d_urn="urn:adsk.eagle:package:10707864/2" override_package_urn="urn:adsk.eagle:footprint:10707865/1" value="1k" x="56.25" y="45.25" smashed="yes" rot="R180">
-<attribute name="NAME" x="57.512" y="44.4245" size="1.016" layer="25" rot="R180"/>
+<attribute name="NAME" x="53.8735" y="46.717" size="1.016" layer="25" rot="R270"/>
 <attribute name="VALUE" x="56.516" y="45.397" size="0.4064" layer="27" rot="R180"/>
 </element>
@@
 <attribute name="MF" value="" x="17.5" y="26" size="1.778" layer="27" display="off"/>
 <attribute name="MPN" value="" x="17.5" y="26" size="1.778" layer="27" display="off"/>
-<attribute name="NAME" x="15.595" y="31.715" size="1.016" layer="25"/>
+<attribute name="NAME" x="16.23" y="19.269" size="1.016" layer="25"/>
 <attribute name="OC_FARNELL" value="unknown" x="17.5" y="26" size="1.778" layer="27" display="off"/>
 <attribute name="OC_NEWARK" value="unknown" x="17.5" y="26" size="1.778" layer="27" display="off"/>
@@
 <attribute name="MF" value="" x="5.5" y="26.25" size="1.778" layer="27" display="off"/>
 <attribute name="MPN" value="" x="5.5" y="26.25" size="1.778" layer="27" display="off"/>
-<attribute name="NAME" x="22.095" y="16.715" size="1.016" layer="25"/>
+<attribute name="NAME" x="22.603" y="4.269" size="1.016" layer="25"/>
 <attribute name="OC_FARNELL" value="unknown" x="5.5" y="26.25" size="1.778" layer="27" display="off"/>
 <attribute name="OC_NEWARK" value="unknown" x="5.5" y="26.25" size="1.778" layer="27" display="off"/>
@@
 <attribute name="MF" value="" x="60.5" y="32.75" size="1.778" layer="27" rot="R270" display="off"/>
 <attribute name="MPN" value="" x="60.5" y="32.75" size="1.778" layer="27" rot="R270" display="off"/>
-<attribute name="NAME" x="57.96" y="34.655" size="1.016" layer="25" ratio="10" rot="R270"/>
+<attribute name="NAME" x="58.69" y="29.639" size="1.016" layer="25" ratio="10"/>
 <attribute name="OC_FARNELL" value="unknown" x="60.5" y="32.75" size="1.778" layer="27" rot="R270" display="off"/>
 <attribute name="OC_NEWARK" value="unknown" x="60.5" y="32.75" size="1.778" layer="27" rot="R270" display="off"/>
@@
 <wire x1="70.31245" y1="71.94525" x2="70.31245" y2="72.14935" width="0.2032" layer="1"/>
 <wire x1="71.53705" y1="70.72065" x2="70.31245" y2="71.94525" width="0.2032" layer="1"/>
-<wire x1="71.53705" y1="69.90425" x2="71.53705" y2="70.72065" width="0.2032" layer="1"/>
+<wire x1="71.53705" y1="70.72065" x2="71.53705" y2="69.90425" width="0.2032" layer="1"/>
 <wire x1="70.31245" y1="72.14935" x2="70.265225" y2="72.202571875" width="0.2032" layer="1"/>
 <wire x1="71.53705" y1="69.90425" x2="71.63010625" y2="69.824946875" width="0.2032" layer="1"/>
-<wire x1="71.63010625" y1="69.824946875" x2="72.348528125" y2="69.106528125" width="0" layer="19" extent="1-1"/>
+<wire x1="71.53705" y1="69.90425" x2="72.334771875" y2="69.106528125" width="0.2032" layer="1"/>
+<wire x1="72.334771875" y1="69.106528125" x2="72.348528125" y2="69.106528125" width="0.2032" layer="1"/>
 </signal>
 <signal name="N$15">
@@
 <contactref element="OR6" pad="3"/>
 <wire x1="47.5553" y1="66.3325" x2="47.86145" y2="66.3325" width="0.2032" layer="1"/>
-<wire x1="46.943" y1="65.7202" x2="47.5553" y2="66.3325" width="0.2032" layer="1"/>
-<wire x1="46.943" y1="65.41405" x2="46.943" y2="65.7202" width="0.2032" layer="1"/>
-<wire x1="44.0856" y1="65.41405" x2="46.943" y2="65.41405" width="0.2032" layer="16"/>
+<wire x1="46.054" y1="64.8312" x2="47.5553" y2="66.3325" width="0.2032" layer="1"/>
+<wire x1="46.054" y1="64.52505" x2="46.054" y2="64.8312" width="0.2032" layer="1"/>
+<wire x1="46.054" y1="64.52505" x2="44.9746" y2="64.52505" width="0.2032" layer="16"/>
+<wire x1="44.0856" y1="65.41405" x2="44.9746" y2="64.52505" width="0.2032" layer="16"/>
 <wire x1="43.8815" y1="65.41405" x2="44.0856" y2="65.41405" width="0.2032" layer="1"/>
 <wire x1="43.0651" y1="64.59765" x2="43.8815" y2="65.41405" width="0.2032" layer="1"/>
@@
 <wire x1="44.0856" y1="65.41405" x2="39.69745" y2="69.8022" width="0.2032" layer="16"/>
 <wire x1="26.7371" y1="70.10835" x2="26.6736" y2="70.19" width="0.2032" layer="1"/>
-<via x="46.943" y="65.41405" extent="1-16" drill="0.35"/>
+<via x="46.054" y="64.52505" extent="1-16" drill="0.35"/>
 <via x="44.0856" y="65.41405" extent="1-16" drill="0.35"/>
 <via x="33.6765" y="69.8022" extent="1-16" drill="0.35"/>
