File: KMO_IO_M/KMO_IO_MV2_5.brd (EAGLE design)
At the start: 84.5 x 96.5 mm, 106 parts, among them IC1 MCP23017SS, Q1 8MHz, Q2 25MHz, U1 ULN2803ADW

Commit message: 2.5 silk scr
Routing:
- net N$57: track 18.0 -> 21.9 mm
- net +3V3: track 335.8 -> 337.7 mm
- net OI1: track 28.0 -> 29.6 mm
- net N$10: track 2.95 -> 4.09 mm
- net GND: track 609.5 -> 610.3 mm
- net D13: vias 2 -> 4
