File: KMO_IO_M/KMO_IO_MV2_9_mout.brd (EAGLE design)
At the start: 84.5 x 96.5 mm, 86 parts, among them Q1 8MHz, Q2 25MHz, U1 ULN2803ADW

Commit message: 29mout
Parts:
- moved GPIO 24.8 mm to (19.3, 27.8)
- moved THM 9.44 mm to (12.3, 13.0)
Routing:
- net GND: track 0.00 -> 526.2 mm, vias 0 -> 13
- net +3V3: track 0.00 -> 253.8 mm, vias 0 -> 4
- net D8: track 0.00 -> 168.1 mm, vias 0 -> 3
- net A7: track 0.00 -> 140.5 mm, vias 0 -> 3
- net RESET: track 0.00 -> 124.6 mm, vias 0 -> 2
- net VIN: track 0.00 -> 119.8 mm
- net VDDO: track 0.00 -> 118.5 mm, vias 0 -> 4
- net D6: track 0.00 -> 109.3 mm, vias 0 -> 5
- net D13: track 0.00 -> 108.5 mm, vias 0 -> 6
- net A6: track 0.00 -> 103.4 mm, vias 0 -> 2
- net GNDO: track 0.00 -> 101.5 mm, vias 0 -> 1
- net D12: track 0.00 -> 93.2 mm, vias 0 -> 4
- net D7: track 0.00 -> 82.1 mm, vias 0 -> 7
- net WFGPIO0: track 0.00 -> 80.7 mm
- net D11: track 0.00 -> 80.1 mm, vias 0 -> 5
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- added copper zone on layer 1, net GND
- added copper zone on layer 16, net GND
Other:
- board text added: "MOUT"
