File: KMO_IO_M/KMO_IO_MV2_9.brd (EAGLE design)
At the start: 84.5 x 96.5 mm, 107 parts, among them IC1 MCP23017SS, Q1 8MHz, Q2 25MHz, U1 ULN2803ADW

Commit message: sht30 check
Parts:
- moved NIR2 0.52 mm to (75.1, 86.7)
- moved NIR1 0.52 mm to (75.1, 82.8)
- moved NIR3 0.25 mm to (75.1, 90.6)
Routing:
- net D10: track 127.3 -> 57.1 mm, vias 0 -> 4
- net D5: track 124.1 -> 73.6 mm, vias 4 -> 2
- net D7: track 68.8 -> 103.9 mm, vias 1 -> 0
- net N$64: track 22.5 -> 49.2 mm, vias 2 -> 0
- net GND: track 666.7 -> 640.9 mm
- net N$27: track 0.00 -> 23.8 mm, vias 0 -> 2
- net RESET: track 102.2 -> 122.1 mm
- net VDDO: track 116.9 -> 134.9 mm
- net D6: track 54.2 -> 68.7 mm
- net RXI: track 33.2 -> 45.9 mm, vias 2 -> 0
- net GPA5: track 62.9 -> 51.5 mm
- net A4: track 160.7 -> 150.7 mm, vias 3 -> 4
- net N$46: track 37.4 -> 46.5 mm
- net N$16: track 24.6 -> 32.2 mm
- net N$61: track 48.1 -> 53.3 mm
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
Commit message: sht
Parts:
- added SC1: 100nF, SparkFun-Passives:0805
- added SR1, SR2: 10K, SparkFun-Passives:0805
- moved SHT 3.43 mm to (41.8, 91.9)
- moved TR 0.13 mm to (55.0, 84.8)
Connections:
- net +3V3: now also SC1.1, SR1.2, SR2.2
- net A4: now also SR1.1
- net A5: now also SR2.1
- net GND: now also SC1.2
Routing:
- net A4: track 150.7 -> 104.6 mm, vias 4 -> 3
- net D11: track 69.3 -> 110.6 mm
- net D7: track 103.9 -> 64.3 mm
- net D5: track 73.6 -> 106.6 mm
- net N$64: track 49.2 -> 22.3 mm, vias 0 -> 2
- net +3V3: track 381.2 -> 406.1 mm, vias 7 -> 8
- net D12: track 62.8 -> 87.6 mm, vias 3 -> 4
- net N$59: track 20.8 -> 39.6 mm, vias 2 -> 0
- net RD-: track 35.9 -> 53.0 mm, vias 2 -> 1
- net RXI: track 45.9 -> 29.5 mm, vias 0 -> 2
- net VDDO: track 134.9 -> 118.6 mm, vias 6 -> 7
- net D10: track 57.1 -> 70.9 mm, vias 4 -> 2
- net N$62: track 41.0 -> 52.9 mm
- net GND: track 640.9 -> 629.2 mm, vias 14 -> 10
- net N$63: track 40.7 -> 51.3 mm
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