File: KMO_IO_M/KMO_IO_MV2_91.brd (EAGLE design)
At the start: 84.5 x 96.5 mm, 110 parts, among them IC1 MCP23017SS, Q1 8MHz, Q2 25MHz, U1 ULN2803ADW

Commit message: 91
Parts:
- moved EC6 4.32 mm to (24.5, 87.1)
- moved OMF 3.05 mm to (17.8, 87.5)
- moved SR1 2.09 mm to (31.4, 90.2)
- moved SR2 2.05 mm to (31.4, 93.1)
Routing:
- net GND: track 0.00 -> 643.1 mm, vias 0 -> 14
- net +3V3: track 0.00 -> 428.0 mm, vias 0 -> 8
- net A4: track 0.00 -> 155.1 mm, vias 0 -> 6
- net A5: track 0.00 -> 149.8 mm, vias 0 -> 6
- net D13: track 0.00 -> 133.6 mm, vias 0 -> 4
- net RESET: track 0.00 -> 118.9 mm, vias 0 -> 2
- net D5: track 0.00 -> 110.3 mm, vias 0 -> 2
- net VIN: track 0.00 -> 108.1 mm
- net D7: track 0.00 -> 103.6 mm
- net VDDO: track 0.00 -> 101.3 mm, vias 0 -> 4
- net D11: track 0.00 -> 99.1 mm, vias 0 -> 2
- net D12: track 0.00 -> 91.6 mm, vias 0 -> 4
- net GNDO: track 0.00 -> 89.8 mm, vias 0 -> 2
- net GPA5: track 0.00 -> 78.1 mm, vias 0 -> 3
- net D10: track 0.00 -> 72.6 mm, vias 0 -> 2
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Other:
- outline, holes or cut-outs redrawn
- board text added: "IOTB v2.91 TOP"
- board text added: "IOTECH © 2020"
- board text removed: "IOTB v2.9 TOP"
- board text removed: "IOTECH © 2019"

Commit message: 91
Other:
- outline, holes or cut-outs redrawn
Changed lines of the file:
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@@
 <drawing>
 <settings>
-<setting alwaysvectorfont="yes"/>
+<setting alwaysvectorfont="no"/>
 <setting verticaltext="up"/>
 </settings>
@@
 <rectangle x1="11.44" y1="93.52" x2="11.92" y2="93.68" layer="26"/>
 <text x="0" y="-0.8" size="0.32" layer="26" font="vector" rot="MR0">C:/Users/celikada/Downloads/5.bmp</text>
-<wire x1="38.481" y1="94.742" x2="36.195" y2="94.742" width="0.1524" layer="20"/>
-<wire x1="36.195" y1="94.742" x2="36.195" y2="86.868" width="0.1524" layer="20"/>
-<wire x1="36.195" y1="86.868" x2="36.322" y2="86.741" width="0.1524" layer="20"/>
-<wire x1="36.322" y1="86.741" x2="44.958" y2="86.741" width="0.1524" layer="20"/>
-<wire x1="44.958" y1="86.741" x2="44.958" y2="88.9" width="0.1524" layer="20"/>
-<wire x1="44.958" y1="88.9" x2="38.481" y2="88.9" width="0.1524" layer="20"/>
-<wire x1="38.481" y1="88.9" x2="38.481" y2="94.742" width="0.1524" layer="20"/>
+<wire x1="36.195" y1="94.742" x2="36.195" y2="87.884" width="0.1524" layer="20"/>
+<wire x1="37.211" y1="86.868" x2="44.704" y2="86.868" width="0.1524" layer="20"/>
+<wire x1="44.704" y1="89.154" x2="38.481" y2="89.154" width="0.1524" layer="20"/>
+<wire x1="38.481" y1="89.154" x2="38.481" y2="94.742" width="0.1524" layer="20"/>
+<wire x1="37.211" y1="86.868" x2="36.195" y2="87.884" width="0.1524" layer="20" curve="-106.260205"/>
+<wire x1="36.195" y1="94.742" x2="38.481" y2="94.742" width="0.1524" layer="20" curve="-180"/>
+<wire x1="44.704" y1="89.154" x2="44.704" y2="86.868" width="0.1524" layer="20" curve="-180"/>
 </plain>
 <attributes>
