File: KMO_IO_M/KMO_IO_MV2_91.sch (EAGLE design)
At the start: 108 parts, among them IC1 MCP23017SS, Q1 8MHz, Q2 25MHz, U1 ULN2803ADW

Commit message: 91
Other:
- note added: "2.91"
- note removed: "2.9"
Changed lines of the file:
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@@
 <text x="299.72" y="241.3" size="1.778" layer="91">NATIVE ANALOG-DIGITAL SENSOR 3</text>
 <text x="309.88" y="15.24" size="2.54" layer="94">IOTB by Team IOTECH</text>
-<text x="365.76" y="12.7" size="2.54" layer="94">2.9</text>
+<text x="365.76" y="12.7" size="2.54" layer="94">2.91</text>
 <text x="187.96" y="170.18" size="1.778" layer="91">ETHERNET</text>
 <text x="193.04" y="109.22" size="1.778" layer="97">D2  -&gt;INT
